File: USB_PD_Boost_TestBoard/USB_PD.kicad_sch (KiCad schematic)
At the start: 30 parts, among them IC1 CYPD3177-24LQXQ, Q1 SI7997DP-T1-GE3, Q2 SI7997DP-T1-GE3

Commit message: some stuff
Parts:
- added TP11: PD_VBUS_OUT, TestPoint:TestPoint_Pad_1.0x1.0mm, symbol Connector:TestPoint
- added TP13: VBUS_MAX, TestPoint:TestPoint_Pad_1.0x1.0mm, symbol Connector:TestPoint
- added TP14: VBUS_MIN, TestPoint:TestPoint_Pad_1.0x1.0mm, symbol Connector:TestPoint
- added TP15: ISINK_COARSE, TestPoint:TestPoint_Pad_1.0x1.0mm, symbol Connector:TestPoint
- added TP16: ISINK_FINE, TestPoint:TestPoint_Pad_1.0x1.0mm, symbol Connector:TestPoint
- added TP17: VBUS_FET_EN, TestPoint:TestPoint_Pad_1.0x1.0mm, symbol Connector:TestPoint
- added TP18: PD_3V3, TestPoint:TestPoint_Pad_1.0x1.0mm, symbol Connector:TestPoint
- added TP19: SAFE_PWR_EN, TestPoint:TestPoint_Pad_1.0x1.0mm, symbol Connector:TestPoint
- added TP20: VBUS_FET_GATE, TestPoint:TestPoint_Pad_1.0x1.0mm, symbol Connector:TestPoint
- added TP21: SAFE_PWR_GATE, TestPoint:TestPoint_Pad_1.0x1.0mm, symbol Connector:TestPoint
- added TP22: PD_5V_OUT, TestPoint:TestPoint_Pad_1.0x1.0mm, symbol Connector:TestPoint
- added TP23: VBUS_IN, TestPoint:TestPoint_Pad_1.0x1.0mm, symbol Connector:TestPoint
- added TP24: PD_FAULT, TestPoint:TestPoint_Pad_1.0x1.0mm, symbol Connector:TestPoint
- renumbered D1 to D3, D5 to D4, D6 to D5, D2 to D6, R7 to R10, R8 to R11, R9 to R12, R10 to R13, R11 to R14, R13 to R16, R14 to R17, R1 to R4, R2 to R5, R3 to R6, R4 to R7, R5 to R8, R6 to R9
Connections:
- net GND: now also TP16.1
- net ISINK_COARSE: now also TP15.1
- net PD_3V3: now also TP13.1, TP18.1
- net PD_5V_OUT: now also TP22.1
- net PD_FAULT: now also TP24.1
- net PD_VBUS_OUT: now also TP11.1
- net SAFE_PWR_EN: now also TP19.1
- net VBUS_FET_EN: now also TP17.1
- net VBUS_IN: now also TP23.1
- net VBUS_MIN: now also TP14.1
- net SAFE_PWR_GATE: now reaches C3.2, C5.2, D5.2 (A), Q2.2 (G1), Q2.4 (G2), R7.1, R9.1
- net SAFE_PWR_GATE: now also TP21.1
- net VBUS_FET_GATE: now reaches C2.2, C4.2, D6.2 (A), Q1.2 (G1), Q1.4 (G2), R14.1, R6.1, R8.1
- net VBUS_FET_GATE: now also TP20.1
Other:
- note added: "Testpoints"

Commit message: idk
Parts:
- renumbered R9 to R10, R10 to R11, R11 to R12, R12 to R13, R13 to R14, R14 to R15, R15 to R16, R16 to R17, R17 to R18, R4 to R5, R5 to R6, R6 to R7, R7 to R8, R8 to R9, TP21 to TP10, TP24 to TP11, TP11 to TP12, TP22 to TP13, TP23 to TP14, TP18 to TP15, TP13 to TP3, TP14 to TP4, TP15 to TP5, TP16 to TP6, TP17 to TP7, TP20 to TP8, TP19 to TP9

Commit message: schematic
Parts:
- removed D3: TPD2EUSB30DRTR, UTSVT_ICs:TPD2EUSB30DRTR, symbol USB_PD_Symbols:TPD2EUSB30DRTR
- removed D4: SMBJ24A-E3_52, Diode_SMD:D_SMB, symbol USB_PD_Symbols:SMBJ24A-E3_52
- removed D5, D6: SMBJ10A-E3_52, Diode_SMD:D_SMB, symbol USB_PD_Symbols:SMBJ10A-E3_52
- removed IC1: CYPD3177-24LQXQ, UTSVT_ICs:CYPD3177-24LQXQ, symbol USB_PD_Symbols:CYPD3177-24LQXQ
- removed Q1, Q2: SI7997DP-T1-GE3, UTSVT_ICs:SI7997DP-T1-GE3, symbol USB_PD_Symbols:SI7997DP-T1-GE3
- removed TP10: SAFE_PWR_GATE, TestPoint:TestPoint_Pad_1.0x1.0mm, symbol Connector:TestPoint
- removed TP3: VBUS_MAX, TestPoint:TestPoint_Pad_1.0x1.0mm, symbol Connector:TestPoint
- removed TP4: VBUS_MIN, TestPoint:TestPoint_Pad_1.0x1.0mm, symbol Connector:TestPoint
- removed TP6: ISINK_FINE, TestPoint:TestPoint_Pad_1.0x1.0mm, symbol Connector:TestPoint
- added D3: TPD2EUSB30DRTR, UTSVT_ICs:TPD2EUSB30DRTR, symbol UTSVT_ICs:TPD2EUSB30DRTR
- added D4: SMBJ24A-E3_52, Diode_SMD:D_SMB, symbol UTSVT_Power:SMBJ24A-E3_52
- added D5, D6: SMBJ10A-E3_52, Diode_SMD:D_SMB, symbol UTSVT_Power:SMBJ10A-E3_52
- added D7: FAULT, LED_SMD:LED_0603_1608Metric_Pad1.05x0.95mm_HandSolder, symbol Device:LED
- added IC1: CYPD3177-24LQXQ, UTSVT_ICs:CYPD3177-24LQXQ, symbol UTSVT_ICs:CYPD3177-24LQXQ
- added Q1, Q2: SI7997DP-T1-GE3, UTSVT_ICs:SI7997DP-T1-GE3, symbol UTSVT_ICs:SI7997DP-T1-GE3
- added Q3: IRLML0030, Package_TO_SOT_SMD:SOT-23, symbol Transistor_FET:IRLML0030
- added R19: 10k, Resistor_SMD:R_0603_1608Metric_Pad0.98x0.95mm_HandSolder, symbol Device:R_Small
- added TP7: VBUS_MIN, TestPoint:TestPoint_Pad_1.0x1.0mm, symbol Connector:TestPoint
- added TP9: ISINK_FINE, TestPoint:TestPoint_Pad_1.0x1.0mm, symbol Connector:TestPoint
- TP10: renamed from TP12; footprint TestPoint:TestPoint_Pad_1.0x1.0mm -> Connector_PinHeader_2.54mm:PinHeader_1x01_P2.54mm_Vertical
- TP11: renamed from TP13; footprint TestPoint:TestPoint_Pad_1.0x1.0mm -> Connector_PinHeader_2.54mm:PinHeader_1x01_P2.54mm_Vertical
- TP12: renamed from TP15; footprint TestPoint:TestPoint_Pad_1.0x1.0mm -> Connector_PinHeader_2.54mm:PinHeader_1x01_P2.54mm_Vertical
- TP5: value ISINK_COARSE -> VBUS_IN; footprint TestPoint:TestPoint_Pad_1.0x1.0mm -> Connector_PinHeader_2.54mm:PinHeader_1x01_P2.54mm_Vertical
- TP6: renamed from TP14; value VBUS_IN -> VBUS_MAX
- TP8: value VBUS_FET_GATE -> ISINK_COARSE
- renumbered TP11 to TP13, TP7 to TP3, TP9 to TP4
Connections:
- net CC1: now also IC1.15 (CC1)
- net CC2: now also IC1.14 (CC2)
- net D+: now also D3.1 (D+)
- net D-: now also D3.2 (D-)
- net ISINK_COARSE: now also TP8.1, IC1.5 (ISNK_COARSE); no longer TP5.1
- net PD_3V3: now also TP6.1, IC1.2 (VBUS_MAX), IC1.23 (VDDD), R19.2
- net PD_5V_OUT: now also Q2.10 (D2), Q2.12 (D2), Q2.5 (D2), Q2.6 (D2)
- net PD_FAULT: now also IC1.9 (FAULT), Q3.1 (G)
- net PD_GPIO_1: now also IC1.8 (GPIO_1)
- net PD_HPI_INT: now also IC1.7 (HPI_INT)
- net PD_VBUS_OUT: now also IC1.11 (VDC_OUT), Q1.10 (D2), Q1.12 (D2), Q1.5 (D2), Q1.6 (D2)
- net SAFE_PWR_EN: now also IC1.4 (SAFE_PWR_EN)
- net SCL: now also IC1.13 (HPI_SCL)
- net SDA: now also IC1.12 (HPI_SDA)
- net VBUS_FET_EN: now also IC1.3 (VBUS_FET_EN)
- net VBUS_IN: now also TP5.1, D4.1 (K), IC1.18 (VBUS_IN), Q1.11 (D1), Q1.7 (D1), Q1.8 (D1), Q1.9 (D1), Q2.11 (D1), Q2.7 (D1), Q2.8 (D1), Q2.9 (D1); no longer TP6.1
- net VBUS_MIN: now also IC1.1 (VBUS_MIN), TP7.1
- net at R15.2: now also D5.1 (K), Q1.1 (S1), Q1.3 (S2)
- net at R16.2: now also IC1.10 (FLIP)
- net at C6.2: now also IC1.24 (VCCD)
- net GND renamed PD_GND
- net PD_GND: now also D3.3 (GND), D4.2 (A), IC1.19 (GND_1), IC1.22 (GND_2), IC1.25 (GND_3), IC1.6 (ISNK_FINE), Q3.2 (S), TP9.1
- net SAFE_PWR_GATE: no longer names the net of C3.2, C5.2, R10.1, R8.1
- net SAFE_PWR_GATE: now also D6.2 (A), Q2.2 (G1), Q2.4 (G2)
- net VBUS_FET_GATE: no longer names the net of C2.2, C4.2, R15.1, R7.1, R9.1
- net VBUS_FET_GATE: now also D5.2 (A), Q1.2 (G1), Q1.4 (G2); no longer TP8.1
- new net: D6.1 (K), Q2.1 (S1), Q2.3 (S2)
- new net: D7.1 (K), Q3.3 (D)
- new net: D7.2 (A), R19.1
Other:
- note added: "D"
- note added: "Fault LED: on if PD faults (failed negotiation or overvoltage protection fault)"
- note added: "G"
- note added: "If VBUS_IN >= 9V, negotiate highest voltage and power VBUS_OUT Else, negotiate for 5V and power 5V_OUT"
- note added: "NMOS"
- note removed: "- If >= 9V, negotiate highest voltage and power VBUS_OUT - If 5V, power 5V_OUT"
- note removed: "D1"
- note removed: "D2"
- note removed: "G1"
- note removed: "G2"
- note removed: "Testpoints"
- moved on the sheet: C1, C6, C7, C8, C9, R11, R12, R13, R14, R15, R16, R17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
