File: USB_PD_Boost_TestBoard/USB_PD.kicad_sch (KiCad schematic)
At the start: 38 parts, among them IC1 CYPD3177-24LQXQ, Q1 SI7997DP-T1-GE3, Q2 SI7997DP-T1-GE3, Q3 IRLML0030

Commit message: clean up
Parts:
- removed R21: 1k, Resistor_SMD:R_0603_1608Metric_Pad0.98x0.95mm_HandSolder, symbol Device:R_Small
- added R22: 3.3k, Resistor_SMD:R_0603_1608Metric_Pad0.98x0.95mm_HandSolder, symbol Device:R
- renumbered D4 to D5, D5 to D6, D6 to D7, D7 to D8, R9 to R10, R10 to R11, R11 to R12, R12 to R13, R13 to R14, R14 to R15, R15 to R16, R16 to R17, R17 to R18, R18 to R19, R19 to R20, R20 to R21, R7 to R8, R8 to R9, TP15 to TP14, TP16 to TP15, TP17 to TP16, TP18 to TP17, TP19 to TP18, TP20 to TP19
Connections:
- net VBUS: now also R22.1
- net at D8.2 (A): now also R22.2
Other:
- moved on the sheet: C6, D8, Q3
