File: USB_PD_Boost_TestBoard/USB_PD_Boost_TestBoard.kicad_sch (KiCad schematic)
At the start: 35 parts, among them J1 USB_C_Receptacle_USB2.0_16P, J3 575-4, J4 575-4, J5 575-4, J6 575-4, J7 PD_12C

Commit message: something
Parts:
- removed TP4: GND, Connector_PinHeader_2.54mm:PinHeader_1x01_P2.54mm_Vertical, symbol Connector:TestPoint
- TP10, TP11, TP12, TP7, TP8, TP9: footprint TestPoint:TestPoint_Pad_1.0x1.0mm -> Connector_PinHeader_2.54mm:PinHeader_1x01_P2.54mm_Vertical
Changed lines of the file:
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@@
 	(wire
 		(pts
-			(xy 80.01 110.49) (xy 80.01 111.76)
+			(xy 73.66 110.49) (xy 73.66 111.76)
 		)
 		(stroke
@@
 	(wire
 		(pts
-			(xy 73.66 110.49) (xy 73.66 111.76)
-		)
-		(stroke
-			(width 0)
-			(type default)
-		)
-	)
-	(wire
-		(pts
 			(xy 151.13 58.42) (xy 151.13 64.77)
 		)
@@
 	(symbol
 		(lib_id "Connector:TestPoint")
-		(at 80.01 110.49 0)
+		(at 73.66 110.49 0)
 		(unit 1)
 		(exclude_from_sim no)
@@
 		(dnp no)
 		(property "Reference" "TP6"
-			(at 82.55 105.9179 0)
+			(at 76.2 105.9179 0)
 			(effects
 				(font
@@
 		)
 		(property "Value" "GND"
-			(at 78.232 105.156 0)
+			(at 71.882 105.156 0)
 			(effects
 				(font
@@
 		)
 		(property "Footprint" "Connector_PinHeader_2.54mm:PinHeader_1x01_P2.54mm_Vertical"
-			(at 85.09 110.49 0)
+			(at 78.74 110.49 0)
 			(effects
 				(font
@@
 		)
 		(property "Datasheet" "~"
-			(at 85.09 110.49 0)
+			(at 78.74 110.49 0)
 			(effects
 				(font
@@
 		)
 		(property "Description" "test point"
-			(at 80.01 110.49 0)
+			(at 73.66 110.49 0)
 			(effects
 				(font
@@
 			)
 		)
-		(property "Footprint" "TestPoint:TestPoint_Pad_1.0x1.0mm"
+		(property "Footprint" "Connector_PinHeader_2.54mm:PinHeader_1x01_P2.54mm_Vertical"
 			(at 99.06 53.34 0)
 			(effects
@@
 	)
 	(symbol
-		(lib_id "Connector:TestPoint")
-		(at 73.66 110.49 0)
-		(unit 1)
-		(exclude_from_sim no)
-		(in_bom no)
-		(on_board yes)
-		(dnp no)
-		(property "Reference" "TP4"
-			(at 76.2 105.9179 0)
-			(effects
-				(font
-					(size 1.27 1.27)
-				)
-				(justify left)
-				(hide yes)
-			)
-		)
-		(property "Value" "GND"
-			(at 71.882 105.156 0)
-			(effects
-				(font
-					(size 1.27 1.27)
-				)
-				(justify left)
-			)
-		)
-		(property "Footprint" "Connector_PinHeader_2.54mm:PinHeader_1x01_P2.54mm_Vertical"
-			(at 78.74 110.49 0)
-			(effects
-				(font
-					(size 1.27 1.27)
-				)
-				(hide yes)
-			)
-		)
-		(property "Datasheet" "~"
-			(at 78.74 110.49 0)
-			(effects
-				(font
-					(size 1.27 1.27)
-				)
-				(hide yes)
-			)
-		)
-		(property "Description" "test point"
-			(at 73.66 110.49 0)
-			(effects
-				(font
-					(size 1.27 1.27)
-				)
-				(hide yes)
-			)
-		)
-		(pin "1"
-		)
-		(instances
-			(project "USB_PD_Boost_TestBoard"
-				(path "/b6f029de-c5f9-47ba-bc2f-f9cf5cd6ec8c"
-					(reference "TP4")
-					(unit 1)
-				)
-			)
-		)
-	)
-	(symbol
 		(lib_id "Connector_Generic:Conn_01x01")
 		(at 153.67 95.25 0)
@@
 			)
 		)
-		(property "Footprint" "TestPoint:TestPoint_Pad_1.0x1.0mm"
+		(property "Footprint" "Connector_PinHeader_2.54mm:PinHeader_1x01_P2.54mm_Vertical"
 			(at 99.06 41.91 0)
 			(effects
@@
 			)
 		)
-		(property "Footprint" "TestPoint:TestPoint_Pad_1.0x1.0mm"
+		(property "Footprint" "Connector_PinHeader_2.54mm:PinHeader_1x01_P2.54mm_Vertical"
 			(at 99.06 50.8 0)
 			(effects
@@
 	(symbol
 		(lib_id "power:GND")
-		(at 80.01 111.76 0)
+		(at 73.66 111.76 0)
 		(unit 1)
 		(exclude_from_sim no)
@@
 		(fields_autoplaced yes)
 		(property "Reference" "#PWR09"
-			(at 80.01 118.11 0)
+			(at 73.66 118.11 0)
 			(effects
 				(font
@@
 		)
 		(property "Value" "GND"
-			(at 80.01 116.84 0)
+			(at 73.66 116.84 0)
 			(effects
 				(font
@@
 		)
 		(property "Footprint" ""
-			(at 80.01 111.76 0)
+			(at 73.66 111.76 0)
 			(effects
 				(font
@@
 		)
 		(property "Datasheet" ""
-			(at 80.01 111.76 0)
+			(at 73.66 111.76 0)
 			(effects
 				(font
@@
 		)
 		(property "Description" "Power symbol creates a global label with name \"GND\" , ground"
-			(at 80.01 111.76 0)
+			(at 73.66 111.76 0)
 			(effects
 				(font
@@
 			)
 		)
-		(property "Footprint" "TestPoint:TestPoint_Pad_1.0x1.0mm"
+		(property "Footprint" "Connector_PinHeader_2.54mm:PinHeader_1x01_P2.54mm_Vertical"
 			(at 99.06 55.88 0)
 			(effects
@@
 	)
 	(symbol
-		(lib_id "power:GND")
-		(at 73.66 111.76 0)
-		(unit 1)
-		(exclude_from_sim no)
-		(in_bom yes)
-		(on_board yes)
-		(dnp no)
-		(fields_autoplaced yes)
-		(property "Reference" "#PWR07"
-			(at 73.66 118.11 0)
-			(effects
-				(font
-					(size 1.27 1.27)
-				)
-				(hide yes)
-			)
-		)
-		(property "Value" "GND"
-			(at 73.66 116.84 0)
-			(effects
-				(font
-					(size 1.27 1.27)
-				)
-			)
-		)
-		(property "Footprint" ""
-			(at 73.66 111.76 0)
-			(effects
-				(font
-					(size 1.27 1.27)
-				)
-				(hide yes)
-			)
-		)
-		(property "Datasheet" ""
-			(at 73.66 111.76 0)
-			(effects
-				(font
-					(size 1.27 1.27)
-				)
-				(hide yes)
-			)
-		)
-		(property "Description" "Power symbol creates a global label with name \"GND\" , ground"
-			(at 73.66 111.76 0)
-			(effects
-				(font
-					(size 1.27 1.27)
-				)
-				(hide yes)
-			)
-		)
-		(pin "1"
-		)
-		(instances
-			(project "USB_PD_Boost_TestBoard"
-				(path "/b6f029de-c5f9-47ba-bc2f-f9cf5cd6ec8c"
-					(reference "#PWR07")
-					(unit 1)
-				)
-			)
-		)
-	)
-	(symbol
 		(lib_id "Jumper:Jumper_2_Small_Open")
 		(at 118.11 27.94 0)
@@
 			)
 		)
-		(property "Footprint" "TestPoint:TestPoint_Pad_1.0x1.0mm"
+		(property "Footprint" "Connector_PinHeader_2.54mm:PinHeader_1x01_P2.54mm_Vertical"
 			(at 99.06 48.26 0)
 			(effects
@@
 			)
 		)
-		(property "Footprint" "TestPoint:TestPoint_Pad_1.0x1.0mm"
+		(property "Footprint" "Connector_PinHeader_2.54mm:PinHeader_1x01_P2.54mm_Vertical"
 			(at 99.06 44.45 0)
 			(effects

Commit message: fuse holder
Parts:
- F1: footprint UTSVT_Connectors:FUSE_3568 -> Parts:3557-2; symbol utsvt_power:Fuse_3568 -> Device:Fuse; Digikey P/N 36-3568-ND -> 36-3557-2-ND; LCSC P/N (none) -> C3205238; Mouser P/N 534-3568 -> 534-3557-2; P/N 3568 -> 3557-2
- J7, JP1: now left out of the parts list
- R4, R5, R6: LCSC P/N (none) -> C1356479
Changed lines of the file:
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@@
 	)
 	(symbol
-		(lib_id "utsvt_power:Fuse_3568")
+		(lib_id "Device:Fuse")
 		(at 140.97 27.94 90)
 		(unit 1)
@@
 			)
 		)
-		(property "Footprint" "UTSVT_Connectors:FUSE_3568"
+		(property "Footprint" "Parts:3557-2"
 			(at 140.97 29.718 90)
 			(effects
@@
 			)
 		)
-		(property "Datasheet" "kicad-embed://3568-15.pdf"
+		(property "Datasheet" "https://www.mouser.com/datasheet/3/201/1/M65p41.pdf"
 			(at 140.97 27.94 0)
 			(effects
@@
 			)
 		)
-		(property "P/N" "3568"
+		(property "P/N" "3557-2"
 			(at 140.97 27.94 0)
 			(effects
@@
 			)
 		)
-		(property "Mouser P/N" "534-3568 "
+		(property "Mouser P/N" "534-3557-2"
 			(at 140.97 27.94 0)
 			(effects
@@
 			)
 		)
-		(property "Digikey P/N" "36-3568-ND"
+		(property "Digikey P/N" "36-3557-2-ND"
 			(at 140.97 27.94 0)
 			(effects
@@
 			)
 		)
+		(property "LCSC P/N" "C3205238"
+			(at 140.97 27.94 90)
+			(effects
+				(font
+					(size 1.27 1.27)
+				)
+				(hide yes)
+			)
+		)
 		(pin "2"
 		)
@@
 		(unit 1)
 		(exclude_from_sim no)
-		(in_bom yes)
+		(in_bom no)
 		(on_board yes)
 		(dnp no)
@@
 			)
 		)
+		(property "LCSC P/N" "C1356479"
+			(at 166.37 57.15 0)
+			(effects
+				(font
+					(size 1.27 1.27)
+				)
+				(hide yes)
+			)
+		)
 		(pin "1"
 		)
@@
 			)
 		)
+		(property "LCSC P/N" "C1356479"
+			(at 166.37 63.5 0)
+			(effects
+				(font
+					(size 1.27 1.27)
+				)
+				(hide yes)
+			)
+		)
 		(pin "1"
 		)
@@
 		(unit 1)
 		(exclude_from_sim no)
-		(in_bom yes)
+		(in_bom no)
 		(on_board yes)
 		(dnp no)
@@
 			(at 166.37 69.85 0)
 			(effects
+				(font
+					(size 1.27 1.27)
+				)
+				(hide yes)
+			)
+		)
+		(property "LCSC P/N" "C1356479"
+			(at 166.37 69.85 0)
+			(effects

Commit message: comments
Connections:
- net BOOST_VIN: now also F1.3
- net USB_PD_Boost/+USB_PD: now also F1.4
Changed lines of the file:
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@@
 		(pin "1"
+		)
+		(pin "3"
+		)
+		(pin "4"
 		)
 		(instances
