File: USB_PD_Boost_TestBoard/usb_pd_boost.kicad_sch (KiCad schematic)
At the start: 28 parts, among them IC1 TPS55340PWP

Commit message: some stuff
Parts:
- renumbered C1 to C10, C2 to C11, C3 to C12, C6 to C13, C5 to C14, C4 to C15, C7 to C16, C8 to C17, C9 to C18, C10 to C19, C11 to C20, D1 to D7, IC1 to IC2, R6 to R18, R7 to R19, R4 to R20, R5 to R21, R3 to R22, R1 to R23, R2 to R24, TP1 to TP2, TP2 to TP3, TP7 to TP4, TP8 to TP5, TP5 to TP6, TP6 to TP7, TP4 to TP8
Changed lines of the file:
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@@
 		(on_board yes)
 		(dnp no)
-		(property "Reference" "C9"
+		(property "Reference" "C18"
 			(at 198.12 64.77 0)
 			(effects
@@
 			(project "usb_pd_boost"
 				(path "/b6f029de-c5f9-47ba-bc2f-f9cf5cd6ec8c/c44a7706-1e3e-41be-90ad-6eb6c6692006"
-					(reference "C9")
+					(reference "C18")
 					(unit 1)
 				)
@@
 		(on_board yes)
 		(dnp no)
-		(property "Reference" "C3"
+		(property "Reference" "C12"
 			(at 44.958 82.55 0)
 			(effects
@@
 			(project "usb_pd_boost"
 				(path "/b6f029de-c5f9-47ba-bc2f-f9cf5cd6ec8c/c44a7706-1e3e-41be-90ad-6eb6c6692006"
-					(reference "C3")
+					(reference "C12")
 					(unit 1)
 				)
@@
 		(on_board yes)
 		(dnp yes)
-		(property "Reference" "R4"
+		(property "Reference" "R20"
 			(at 59.944 74.93 0)
 			(effects
@@
 			(project ""
 				(path "/b6f029de-c5f9-47ba-bc2f-f9cf5cd6ec8c/c44a7706-1e3e-41be-90ad-6eb6c6692006"
-					(reference "R4")
+					(reference "R20")
 					(unit 1)
 				)
@@
 		(on_board yes)
 		(dnp no)
-		(property "Reference" "TP2"
+		(property "Reference" "TP3"
 			(at 63.5 62.7379 0)
 			(effects
@@
 			(project "usb_pd_boost"
 				(path "/b6f029de-c5f9-47ba-bc2f-f9cf5cd6ec8c/c44a7706-1e3e-41be-90ad-6eb6c6692006"
-					(reference "TP2")
+					(reference "TP3")
 					(unit 1)
 				)
@@
 		(on_board yes)
 		(dnp no)
-		(property "Reference" "C6"
+		(property "Reference" "C13"
 			(at 64.77 81.28 0)
 			(effects
@@
 			(project "usb_pd_boost"
 				(path "/b6f029de-c5f9-47ba-bc2f-f9cf5cd6ec8c/c44a7706-1e3e-41be-90ad-6eb6c6692006"
-					(reference "C6")
+					(reference "C13")
 					(unit 1)
 				)
@@
 		(on_board yes)
 		(dnp no)
-		(property "Reference" "IC1"
+		(property "Reference" "IC2"
 			(at 99.06 58.166 0)
 			(effects
@@
 			(project ""
 				(path "/b6f029de-c5f9-47ba-bc2f-f9cf5cd6ec8c/c44a7706-1e3e-41be-90ad-6eb6c6692006"
-					(reference "IC1")
+					(reference "IC2")
 					(unit 1)
 				)
@@
 		(on_board yes)
 		(dnp no)
-		(property "Reference" "R7"
+		(property "Reference" "R19"
 			(at 45.974 74.93 0)
 			(effects
@@
 			(project "usb_pd_boost"
 				(path "/b6f029de-c5f9-47ba-bc2f-f9cf5cd6ec8c/c44a7706-1e3e-41be-90ad-6eb6c6692006"
-					(reference "R7")
+					(reference "R19")
 					(unit 1)
 				)
@@
 		(on_board yes)
 		(dnp no)
-		(property "Reference" "C5"
+		(property "Reference" "C14"
 			(at 123.698 86.36 0)
 			(effects
@@
 			(project "usb_pd_boost"
 				(path "/b6f029de-c5f9-47ba-bc2f-f9cf5cd6ec8c/c44a7706-1e3e-41be-90ad-6eb6c6692006"
-					(reference "C5")
+					(reference "C14")
 					(unit 1)
 				)
@@
 		(dnp no)
 		(fields_autoplaced yes)
-		(property "Reference" "R1"
+		(property "Reference" "R23"
 			(at 161.29 64.7699 0)
 			(effects
@@
 			(project "usb_pd_boost"
 				(path "/b6f029de-c5f9-47ba-bc2f-f9cf5cd6ec8c/c44a7706-1e3e-41be-90ad-6eb6c6692006"
-					(reference "R1")
+					(reference "R23")
 					(unit 1)
 				)
@@
 		(on_board yes)
 		(dnp no)
-		(property "Reference" "R5"
+		(property "Reference" "R21"
 			(at 130.81 67.564 90)
 			(effects
@@
 			(project ""
 				(path "/b6f029de-c5f9-47ba-bc2f-f9cf5cd6ec8c/c44a7706-1e3e-41be-90ad-6eb6c6692006"
-					(reference "R5")
+					(reference "R21")
 					(unit 1)
 				)
@@
 		(on_board yes)
 		(dnp no)
-		(property "Reference" "C1"
+		(property "Reference" "C10"
 			(at 21.844 89.408 0)
 			(effects
@@
 			(project "usb_pd_boost"
 				(path "/b6f029de-c5f9-47ba-bc2f-f9cf5cd6ec8c/c44a7706-1e3e-41be-90ad-6eb6c6692006"
-					(reference "C1")
+					(reference "C10")
 					(unit 1)
 				)
@@
 		(on_board yes)
 		(dnp no)
-		(property "Reference" "TP6"
+		(property "Reference" "TP7"
 			(at 158.75 70.3579 0)
 			(effects
@@
 			(project "usb_pd_boost"
 				(path "/b6f029de-c5f9-47ba-bc2f-f9cf5cd6ec8c/c44a7706-1e3e-41be-90ad-6eb6c6692006"
-					(reference "TP6")
+					(reference "TP7")
 					(unit 1)
 				)
@@
 		(on_board yes)
 		(dnp no)
-		(property "Reference" "C2"
+		(property "Reference" "C11"
 			(at 32.004 89.408 0)
 			(effects
@@
 			(project "usb_pd_boost"
 				(path "/b6f029de-c5f9-47ba-bc2f-f9cf5cd6ec8c/c44a7706-1e3e-41be-90ad-6eb6c6692006"
-					(reference "C2")
+					(reference "C11")
 					(unit 1)
 				)
@@
 		(on_board yes)
 		(dnp no)
-		(property "Reference" "C11"
+		(property "Reference" "C20"
 			(at 225.298 64.77 0)
 			(effects
@@
 			(project "usb_pd_boost"
 				(path "/b6f029de-c5f9-47ba-bc2f-f9cf5cd6ec8c/c44a7706-1e3e-41be-90ad-6eb6c6692006"
-					(reference "C11")
+					(reference "C20")
 					(unit 1)
 				)
@@
 		(on_board yes)
 		(dnp no)
-		(property "Reference" "C7"
+		(property "Reference" "C16"
 			(at 176.53 64.77 0)
 			(effects
@@
 			(project "usb_pd_boost"
 				(path "/b6f029de-c5f9-47ba-bc2f-f9cf5cd6ec8c/c44a7706-1e3e-41be-90ad-6eb6c6692006"
-					(reference "C7")
+					(reference "C16")
 					(unit 1)
 				)
@@
 		(on_board yes)
 		(dnp no)
-		(property "Reference" "TP8"
+		(property "Reference" "TP5"
 			(at 118.11 79.5019 0)
 			(effects
@@
 			(project "usb_pd_boost"
 				(path "/b6f029de-c5f9-47ba-bc2f-f9cf5cd6ec8c/c44a7706-1e3e-41be-90ad-6eb6c6692006"
-					(reference "TP8")
+					(reference "TP5")
 					(unit 1)
 				)
@@
 		(on_board yes)
 		(dnp no)
-		(property "Reference" "TP7"
+		(property "Reference" "TP4"
 			(at 69.85 71.8819 0)
 			(effects
@@
 			(project "usb_pd_boost"
 				(path "/b6f029de-c5f9-47ba-bc2f-f9cf5cd6ec8c/c44a7706-1e3e-41be-90ad-6eb6c6692006"
-					(reference "TP7")
+					(reference "TP4")
 					(unit 1)
 				)
@@
 		(on_board yes)
 		(dnp no)
-		(property "Reference" "TP4"
+		(property "Reference" "TP8"
 			(at 223.52 53.8481 0)
 			(effects
@@
 			(project "usb_pd_boost"
 				(path "/b6f029de-c5f9-47ba-bc2f-f9cf5cd6ec8c/c44a7706-1e3e-41be-90ad-6eb6c6692006"
-					(reference "TP4")
+					(reference "TP8")
 					(unit 1)
 				)
@@
 		(on_board yes)
 		(dnp no)
-		(property "Reference" "R3"
+		(property "Reference" "R22"
 			(at 130.81 79.756 90)
 			(effects
@@
 			(project "usb_pd_boost"
 				(path "/b6f029de-c5f9-47ba-bc2f-f9cf5cd6ec8c/c44a7706-1e3e-41be-90ad-6eb6c6692006"
-					(reference "R3")
+					(reference "R22")
 					(unit 1)
 				)
@@
 		(dnp no)
 		(fields_autoplaced yes)
-		(property "Reference" "D1"
+		(property "Reference" "D7"
 			(at 138.7475 49.53 0)
 			(effects
@@
 			(project ""
 				(path "/b6f029de-c5f9-47ba-bc2f-f9cf5cd6ec8c/c44a7706-1e3e-41be-90ad-6eb6c6692006"
-					(reference "D1")
+					(reference "D7")
 					(unit 1)
 				)
@@
 		(on_board yes)
 		(dnp no)
-		(property "Reference" "TP1"
+		(property "Reference" "TP2"
 			(at 38.1 51.3079 0)
 			(effects
@@
 			(project ""
 				(path "/b6f029de-c5f9-47ba-bc2f-f9cf5cd6ec8c/c44a7706-1e3e-41be-90ad-6eb6c6692006"
-					(reference "TP1")
+					(reference "TP2")
 					(unit 1)
 				)
@@
 		(on_board yes)
 		(dnp no)
-		(property "Reference" "C10"
+		(property "Reference" "C19"
 			(at 213.868 64.77 0)
 			(effects
@@
 			(project "usb_pd_boost"
 				(path "/b6f029de-c5f9-47ba-bc2f-f9cf5cd6ec8c/c44a7706-1e3e-41be-90ad-6eb6c6692006"
-					(reference "C10")
+					(reference "C19")
 					(unit 1)
 				)
@@
 		(on_board yes)
 		(dnp no)
-		(property "Reference" "C8"
+		(property "Reference" "C17"
 			(at 186.69 64.77 0)
 			(effects
@@
 			(project ""
 				(path "/b6f029de-c5f9-47ba-bc2f-f9cf5cd6ec8c/c44a7706-1e3e-41be-90ad-6eb6c6692006"
-					(reference "C8")
+					(reference "C17")
 					(unit 1)
 				)
@@
 		(on_board yes)
 		(dnp no)
-		(property "Reference" "R6"
+		(property "Reference" "R18"
 			(at 45.72 60.96 0)
 			(effects
@@
 			(project ""
 				(path "/b6f029de-c5f9-47ba-bc2f-f9cf5cd6ec8c/c44a7706-1e3e-41be-90ad-6eb6c6692006"
-					(reference "R6")
+					(reference "R18")
 					(unit 1)
 				)
@@
 		(dnp no)
 		(fields_autoplaced yes)
-		(property "Reference" "R2"
+		(property "Reference" "R24"
 			(at 161.29 80.0099 0)
 			(effects
@@
 			(project ""
 				(path "/b6f029de-c5f9-47ba-bc2f-f9cf5cd6ec8c/c44a7706-1e3e-41be-90ad-6eb6c6692006"
-					(reference "R2")
+					(reference "R24")
 					(unit 1)
 				)
@@
 		(on_board yes)
 		(dnp no)
-		(property "Reference" "C4"
+		(property "Reference" "C15"
 			(at 142.494 86.36 0)
 			(effects
@@
 			(project "usb_pd_boost"
 				(path "/b6f029de-c5f9-47ba-bc2f-f9cf5cd6ec8c/c44a7706-1e3e-41be-90ad-6eb6c6692006"
-					(reference "C4")
+					(reference "C15")
 					(unit 1)
 				)
@@
 		(on_board yes)
 		(dnp no)
-		(property "Reference" "TP5"
+		(property "Reference" "TP6"
 			(at 119.38 51.3079 0)
 			(effects
@@
 			(project "usb_pd_boost"
 				(path "/b6f029de-c5f9-47ba-bc2f-f9cf5cd6ec8c/c44a7706-1e3e-41be-90ad-6eb6c6692006"
-					(reference "TP5")
-					(unit 1)
-				)
+					(reference "TP6")
+					(unit 1)
+				)

Commit message: idk
Parts:
- renumbered R18 to R19, R19 to R20, R20 to R21, R21 to R22, R22 to R23, R23 to R24, R24 to R25, TP2 to TP16, TP3 to TP17, TP4 to TP18, TP5 to TP19, TP6 to TP20, TP7 to TP21, TP8 to TP22
Changed lines of the file:
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@@
 		(on_board yes)
 		(dnp yes)
-		(property "Reference" "R20"
+		(property "Reference" "R21"
 			(at 59.944 74.93 0)
 			(effects
@@
 			(project ""
 				(path "/b6f029de-c5f9-47ba-bc2f-f9cf5cd6ec8c/c44a7706-1e3e-41be-90ad-6eb6c6692006"
-					(reference "R20")
+					(reference "R21")
 					(unit 1)
 				)
@@
 		(on_board yes)
 		(dnp no)
-		(property "Reference" "TP3"
+		(property "Reference" "TP17"
 			(at 63.5 62.7379 0)
 			(effects
@@
 			(project "usb_pd_boost"
 				(path "/b6f029de-c5f9-47ba-bc2f-f9cf5cd6ec8c/c44a7706-1e3e-41be-90ad-6eb6c6692006"
-					(reference "TP3")
+					(reference "TP17")
 					(unit 1)
 				)
@@
 		(on_board yes)
 		(dnp no)
-		(property "Reference" "R19"
+		(property "Reference" "R20"
 			(at 45.974 74.93 0)
 			(effects
@@
 			(project "usb_pd_boost"
 				(path "/b6f029de-c5f9-47ba-bc2f-f9cf5cd6ec8c/c44a7706-1e3e-41be-90ad-6eb6c6692006"
-					(reference "R19")
+					(reference "R20")
 					(unit 1)
 				)
@@
 		(dnp no)
 		(fields_autoplaced yes)
-		(property "Reference" "R23"
+		(property "Reference" "R24"
 			(at 161.29 64.7699 0)
 			(effects
@@
 			(project "usb_pd_boost"
 				(path "/b6f029de-c5f9-47ba-bc2f-f9cf5cd6ec8c/c44a7706-1e3e-41be-90ad-6eb6c6692006"
-					(reference "R23")
+					(reference "R24")
 					(unit 1)
 				)
@@
 		(on_board yes)
 		(dnp no)
-		(property "Reference" "R21"
+		(property "Reference" "R22"
 			(at 130.81 67.564 90)
 			(effects
@@
 			(project ""
 				(path "/b6f029de-c5f9-47ba-bc2f-f9cf5cd6ec8c/c44a7706-1e3e-41be-90ad-6eb6c6692006"
-					(reference "R21")
+					(reference "R22")
 					(unit 1)
 				)
@@
 		(on_board yes)
 		(dnp no)
-		(property "Reference" "TP7"
+		(property "Reference" "TP21"
 			(at 158.75 70.3579 0)
 			(effects
@@
 			(project "usb_pd_boost"
 				(path "/b6f029de-c5f9-47ba-bc2f-f9cf5cd6ec8c/c44a7706-1e3e-41be-90ad-6eb6c6692006"
-					(reference "TP7")
+					(reference "TP21")
 					(unit 1)
 				)
@@
 		(on_board yes)
 		(dnp no)
-		(property "Reference" "TP5"
+		(property "Reference" "TP19"
 			(at 118.11 79.5019 0)
 			(effects
@@
 			(project "usb_pd_boost"
 				(path "/b6f029de-c5f9-47ba-bc2f-f9cf5cd6ec8c/c44a7706-1e3e-41be-90ad-6eb6c6692006"
-					(reference "TP5")
+					(reference "TP19")
 					(unit 1)
 				)
@@
 		(on_board yes)
 		(dnp no)
-		(property "Reference" "TP4"
+		(property "Reference" "TP18"
 			(at 69.85 71.8819 0)
 			(effects
@@
 			(project "usb_pd_boost"
 				(path "/b6f029de-c5f9-47ba-bc2f-f9cf5cd6ec8c/c44a7706-1e3e-41be-90ad-6eb6c6692006"
-					(reference "TP4")
+					(reference "TP18")
 					(unit 1)
 				)
@@
 		(on_board yes)
 		(dnp no)
-		(property "Reference" "TP8"
+		(property "Reference" "TP22"
 			(at 223.52 53.8481 0)
 			(effects
@@
 			(project "usb_pd_boost"
 				(path "/b6f029de-c5f9-47ba-bc2f-f9cf5cd6ec8c/c44a7706-1e3e-41be-90ad-6eb6c6692006"
-					(reference "TP8")
+					(reference "TP22")
 					(unit 1)
 				)
@@
 		(on_board yes)
 		(dnp no)
-		(property "Reference" "R22"
+		(property "Reference" "R23"
 			(at 130.81 79.756 90)
 			(effects
@@
 			(project "usb_pd_boost"
 				(path "/b6f029de-c5f9-47ba-bc2f-f9cf5cd6ec8c/c44a7706-1e3e-41be-90ad-6eb6c6692006"
-					(reference "R22")
+					(reference "R23")
 					(unit 1)
 				)
@@
 		(on_board yes)
 		(dnp no)
-		(property "Reference" "TP2"
+		(property "Reference" "TP16"
 			(at 38.1 51.3079 0)
 			(effects
@@
 			(project ""
 				(path "/b6f029de-c5f9-47ba-bc2f-f9cf5cd6ec8c/c44a7706-1e3e-41be-90ad-6eb6c6692006"
-					(reference "TP2")
+					(reference "TP16")
 					(unit 1)
 				)
@@
 		(on_board yes)
 		(dnp no)
-		(property "Reference" "R18"
+		(property "Reference" "R19"
 			(at 45.72 60.96 0)
 			(effects
@@
 			(project ""
 				(path "/b6f029de-c5f9-47ba-bc2f-f9cf5cd6ec8c/c44a7706-1e3e-41be-90ad-6eb6c6692006"
-					(reference "R18")
+					(reference "R19")
 					(unit 1)
 				)
@@
 		(dnp no)
 		(fields_autoplaced yes)
-		(property "Reference" "R24"
+		(property "Reference" "R25"
 			(at 161.29 80.0099 0)
 			(effects
@@
 			(project ""
 				(path "/b6f029de-c5f9-47ba-bc2f-f9cf5cd6ec8c/c44a7706-1e3e-41be-90ad-6eb6c6692006"
-					(reference "R24")
+					(reference "R25")
 					(unit 1)
 				)
@@
 		(on_board yes)
 		(dnp no)
-		(property "Reference" "TP6"
+		(property "Reference" "TP20"
 			(at 119.38 51.3079 0)
 			(effects
@@
 			(project "usb_pd_boost"
 				(path "/b6f029de-c5f9-47ba-bc2f-f9cf5cd6ec8c/c44a7706-1e3e-41be-90ad-6eb6c6692006"
-					(reference "TP6")
-					(unit 1)
-				)
+					(reference "TP20")
+					(unit 1)
+				)

Commit message: schematic
Parts:
- D8: renamed from D7; footprint B540C-13-F:DIOM7959X250N -> UTSVT_Power:B540C-13-F
- IC2: footprint TPS55340PWP:SOP65P640X120-15N -> UTSVT_Power:TPS55340PWP; symbol TPS55340PWP:TPS55340PWP -> utsvt_power:TPS55340PWP
- L1: footprint SDR1307-100ML:SDR1307100ML -> UTSVT_Power:SDR1307-100ML
- renumbered R19 to R20, R20 to R21, R21 to R22, R22 to R23, R23 to R24, R24 to R25, R25 to R26, TP16 to TP14, TP17 to TP15, TP18 to TP16, TP19 to TP17, TP20 to TP18, TP21 to TP19, TP22 to TP20

Commit message: init layout
Parts:
- removed D8: 5A, UTSVT_Power:B540C-13-F, symbol Device:D_Schottky
- added D8: B540C-13-F, UTSVT_Power:B540C-13-F, symbol utsvt_power:B540C-13-F
Connections:
- net +24V: now also D8.1 (K)
- net at IC2.1 (SW_1), IC2.2 (SW_2), L1.2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: now also D8.2 (A)

Commit message: updated p/n
Parts:
- D8: LCSC P/N (none) -> C72264; P/N (none) -> B540C-13-F
- TP14, TP15, TP16, TP17, TP18, TP19, TP20: now left out of the parts list
Changed lines of the file:
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@@
 		(unit 1)
 		(exclude_from_sim no)
-		(in_bom yes)
+		(in_bom no)
 		(on_board yes)
 		(dnp no)
@@
 		(unit 1)
 		(exclude_from_sim no)
-		(in_bom yes)
+		(in_bom no)
 		(on_board yes)
 		(dnp no)
@@
 			)
 		)
+		(property "LCSC P/N" "C72264"
+			(at 138.43 55.88 0)
+			(effects
+				(font
+					(size 1.27 1.27)
+				)
+				(hide yes)
+			)
+		)
+		(property "P/N" "B540C-13-F"
+			(at 138.43 55.88 0)
+			(effects
+				(font
+					(size 1.27 1.27)
+				)
+				(hide yes)
+			)
+		)
 		(pin "1"
 		)
@@
 		(unit 1)
 		(exclude_from_sim no)
-		(in_bom yes)
+		(in_bom no)
 		(on_board yes)
 		(dnp no)
@@
 		(unit 1)
 		(exclude_from_sim no)
-		(in_bom yes)
+		(in_bom no)
 		(on_board yes)
 		(dnp no)
@@
 		(unit 1)
 		(exclude_from_sim no)
-		(in_bom yes)
+		(in_bom no)
 		(on_board yes)
 		(dnp no)
@@
 		(unit 1)
 		(exclude_from_sim no)
-		(in_bom yes)
+		(in_bom no)
 		(on_board yes)
 		(dnp no)
@@
 		(unit 1)
 		(exclude_from_sim no)
-		(in_bom yes)
+		(in_bom no)
 		(on_board yes)
 		(dnp no)

Commit message: addressed comments, changed PD block a little
Parts:
- renumbered R20 to R21, R21 to R22, R22 to R23, R23 to R24, R24 to R25, R25 to R26, R26 to R27, TP14 to TP19, TP15 to TP20, TP16 to TP21, TP17 to TP22, TP18 to TP23, TP19 to TP24, TP20 to TP25
Changed lines of the file:
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@@
 		(on_board yes)
 		(dnp yes)
-		(property "Reference" "R22"
+		(property "Reference" "R23"
 			(at 59.944 74.93 0)
 			(effects
@@
 			(project ""
 				(path "/b6f029de-c5f9-47ba-bc2f-f9cf5cd6ec8c/5b9bbf7e-f78f-403a-a4be-5024a8867fbc"
-					(reference "R22")
+					(reference "R23")
 					(unit 1)
 				)
@@
 		(on_board yes)
 		(dnp no)
-		(property "Reference" "TP15"
+		(property "Reference" "TP20"
 			(at 63.5 62.7379 0)
 			(effects
@@
 			(project "usb_pd_boost"
 				(path "/b6f029de-c5f9-47ba-bc2f-f9cf5cd6ec8c/5b9bbf7e-f78f-403a-a4be-5024a8867fbc"
-					(reference "TP15")
+					(reference "TP20")
 					(unit 1)
 				)
@@
 		(on_board yes)
 		(dnp no)
-		(property "Reference" "R21"
+		(property "Reference" "R22"
 			(at 45.974 74.93 0)
 			(effects
@@
 			(project "usb_pd_boost"
 				(path "/b6f029de-c5f9-47ba-bc2f-f9cf5cd6ec8c/5b9bbf7e-f78f-403a-a4be-5024a8867fbc"
-					(reference "R21")
+					(reference "R22")
 					(unit 1)
 				)
@@
 		(dnp no)
 		(fields_autoplaced yes)
-		(property "Reference" "R25"
+		(property "Reference" "R26"
 			(at 161.29 64.7699 0)
 			(effects
@@
 			(project "usb_pd_boost"
 				(path "/b6f029de-c5f9-47ba-bc2f-f9cf5cd6ec8c/5b9bbf7e-f78f-403a-a4be-5024a8867fbc"
-					(reference "R25")
+					(reference "R26")
 					(unit 1)
 				)
@@
 		(on_board yes)
 		(dnp no)
-		(property "Reference" "R23"
+		(property "Reference" "R24"
 			(at 130.81 67.564 90)
 			(effects
@@
 			(project ""
 				(path "/b6f029de-c5f9-47ba-bc2f-f9cf5cd6ec8c/5b9bbf7e-f78f-403a-a4be-5024a8867fbc"
-					(reference "R23")
+					(reference "R24")
 					(unit 1)
 				)
@@
 		(on_board yes)
 		(dnp no)
-		(property "Reference" "TP19"
+		(property "Reference" "TP24"
 			(at 158.75 70.3579 0)
 			(effects
@@
 			(project "usb_pd_boost"
 				(path "/b6f029de-c5f9-47ba-bc2f-f9cf5cd6ec8c/5b9bbf7e-f78f-403a-a4be-5024a8867fbc"
-					(reference "TP19")
+					(reference "TP24")
 					(unit 1)
 				)
@@
 		(on_board yes)
 		(dnp no)
-		(property "Reference" "TP17"
+		(property "Reference" "TP22"
 			(at 118.11 79.5019 0)
 			(effects
@@
 			(project "usb_pd_boost"
 				(path "/b6f029de-c5f9-47ba-bc2f-f9cf5cd6ec8c/5b9bbf7e-f78f-403a-a4be-5024a8867fbc"
-					(reference "TP17")
+					(reference "TP22")
 					(unit 1)
 				)
@@
 		(on_board yes)
 		(dnp no)
-		(property "Reference" "TP16"
+		(property "Reference" "TP21"
 			(at 69.85 71.8819 0)
 			(effects
@@
 			(project "usb_pd_boost"
 				(path "/b6f029de-c5f9-47ba-bc2f-f9cf5cd6ec8c/5b9bbf7e-f78f-403a-a4be-5024a8867fbc"
-					(reference "TP16")
+					(reference "TP21")
 					(unit 1)
 				)
@@
 		(on_board yes)
 		(dnp no)
-		(property "Reference" "TP20"
+		(property "Reference" "TP25"
 			(at 223.52 53.8481 0)
 			(effects
@@
 			(project "usb_pd_boost"
 				(path "/b6f029de-c5f9-47ba-bc2f-f9cf5cd6ec8c/5b9bbf7e-f78f-403a-a4be-5024a8867fbc"
-					(reference "TP20")
+					(reference "TP25")
 					(unit 1)
 				)
@@
 		(on_board yes)
 		(dnp no)
-		(property "Reference" "R24"
+		(property "Reference" "R25"
 			(at 130.81 79.756 90)
 			(effects
@@
 			(project "usb_pd_boost"
 				(path "/b6f029de-c5f9-47ba-bc2f-f9cf5cd6ec8c/5b9bbf7e-f78f-403a-a4be-5024a8867fbc"
-					(reference "R24")
+					(reference "R25")
 					(unit 1)
 				)
@@
 		(on_board yes)
 		(dnp no)
-		(property "Reference" "TP14"
+		(property "Reference" "TP19"
 			(at 38.1 51.3079 0)
 			(effects
@@
 			(project ""
 				(path "/b6f029de-c5f9-47ba-bc2f-f9cf5cd6ec8c/5b9bbf7e-f78f-403a-a4be-5024a8867fbc"
-					(reference "TP14")
+					(reference "TP19")
 					(unit 1)
 				)
@@
 		(on_board yes)
 		(dnp no)
-		(property "Reference" "R20"
+		(property "Reference" "R21"
 			(at 45.72 60.96 0)
 			(effects
@@
 			(project ""
 				(path "/b6f029de-c5f9-47ba-bc2f-f9cf5cd6ec8c/5b9bbf7e-f78f-403a-a4be-5024a8867fbc"
-					(reference "R20")
+					(reference "R21")
 					(unit 1)
 				)
@@
 		(dnp no)
 		(fields_autoplaced yes)
-		(property "Reference" "R26"
+		(property "Reference" "R27"
 			(at 161.29 80.0099 0)
 			(effects
@@
 			(project ""
 				(path "/b6f029de-c5f9-47ba-bc2f-f9cf5cd6ec8c/5b9bbf7e-f78f-403a-a4be-5024a8867fbc"
-					(reference "R26")
+					(reference "R27")
 					(unit 1)
 				)
@@
 		(on_board yes)
 		(dnp no)
-		(property "Reference" "TP18"
+		(property "Reference" "TP23"
 			(at 119.38 51.3079 0)
 			(effects
@@
 			(project "usb_pd_boost"
 				(path "/b6f029de-c5f9-47ba-bc2f-f9cf5cd6ec8c/5b9bbf7e-f78f-403a-a4be-5024a8867fbc"
-					(reference "TP18")
-					(unit 1)
-				)
+					(reference "TP23")
+					(unit 1)
+				)
