File: USB_PD_Boost_TestBoard/usb_pd_boost.kicad_sch (KiCad schematic)
At the start: 28 parts, among them IC2 TPS55340PWP

Commit message: comments, load resistors, stuff idk
Parts:
- renumbered R21 to R22, R22 to R23, R23 to R24, R24 to R25, R25 to R26, R26 to R27, R27 to R28
Changed lines of the file:
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@@
 		(on_board yes)
 		(dnp yes)
-		(property "Reference" "R23"
+		(property "Reference" "R24"
 			(at 59.944 74.93 0)
 			(effects
@@
 			(project ""
 				(path "/b6f029de-c5f9-47ba-bc2f-f9cf5cd6ec8c/5b9bbf7e-f78f-403a-a4be-5024a8867fbc"
-					(reference "R23")
+					(reference "R24")
 					(unit 1)
 				)
@@
 		(on_board yes)
 		(dnp no)
-		(property "Reference" "R22"
+		(property "Reference" "R23"
 			(at 45.974 74.93 0)
 			(effects
@@
 			(project "usb_pd_boost"
 				(path "/b6f029de-c5f9-47ba-bc2f-f9cf5cd6ec8c/5b9bbf7e-f78f-403a-a4be-5024a8867fbc"
-					(reference "R22")
+					(reference "R23")
 					(unit 1)
 				)
@@
 		(dnp no)
 		(fields_autoplaced yes)
-		(property "Reference" "R26"
+		(property "Reference" "R27"
 			(at 161.29 64.7699 0)
 			(effects
@@
 			(project "usb_pd_boost"
 				(path "/b6f029de-c5f9-47ba-bc2f-f9cf5cd6ec8c/5b9bbf7e-f78f-403a-a4be-5024a8867fbc"
-					(reference "R26")
+					(reference "R27")
 					(unit 1)
 				)
@@
 		(on_board yes)
 		(dnp no)
-		(property "Reference" "R24"
+		(property "Reference" "R25"
 			(at 130.81 67.564 90)
 			(effects
@@
 			(project ""
 				(path "/b6f029de-c5f9-47ba-bc2f-f9cf5cd6ec8c/5b9bbf7e-f78f-403a-a4be-5024a8867fbc"
-					(reference "R24")
+					(reference "R25")
 					(unit 1)
 				)
@@
 		(on_board yes)
 		(dnp no)
-		(property "Reference" "R25"
+		(property "Reference" "R26"
 			(at 130.81 79.756 90)
 			(effects
@@
 			(project "usb_pd_boost"
 				(path "/b6f029de-c5f9-47ba-bc2f-f9cf5cd6ec8c/5b9bbf7e-f78f-403a-a4be-5024a8867fbc"
-					(reference "R25")
+					(reference "R26")
 					(unit 1)
 				)
@@
 		(on_board yes)
 		(dnp no)
-		(property "Reference" "R21"
+		(property "Reference" "R22"
 			(at 45.72 60.96 0)
 			(effects
@@
 			(project ""
 				(path "/b6f029de-c5f9-47ba-bc2f-f9cf5cd6ec8c/5b9bbf7e-f78f-403a-a4be-5024a8867fbc"
-					(reference "R21")
+					(reference "R22")
 					(unit 1)
 				)
@@
 		(dnp no)
 		(fields_autoplaced yes)
-		(property "Reference" "R27"
+		(property "Reference" "R28"
 			(at 161.29 80.0099 0)
 			(effects
@@
 			(project ""
 				(path "/b6f029de-c5f9-47ba-bc2f-f9cf5cd6ec8c/5b9bbf7e-f78f-403a-a4be-5024a8867fbc"
-					(reference "R27")
-					(unit 1)
-				)
+					(reference "R28")
+					(unit 1)
+				)

Commit message: son
Parts:
- renumbered TP19 to TP21, TP20 to TP22, TP21 to TP23, TP22 to TP24, TP23 to TP25, TP24 to TP26, TP25 to TP27
Changed lines of the file:
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@@
 		(on_board yes)
 		(dnp no)
-		(property "Reference" "TP20"
+		(property "Reference" "TP22"
 			(at 63.5 62.7379 0)
 			(effects
@@
 			(project "usb_pd_boost"
 				(path "/b6f029de-c5f9-47ba-bc2f-f9cf5cd6ec8c/5b9bbf7e-f78f-403a-a4be-5024a8867fbc"
-					(reference "TP20")
+					(reference "TP22")
 					(unit 1)
 				)
@@
 		(on_board yes)
 		(dnp no)
-		(property "Reference" "TP24"
+		(property "Reference" "TP26"
 			(at 158.75 70.3579 0)
 			(effects
@@
 			(project "usb_pd_boost"
 				(path "/b6f029de-c5f9-47ba-bc2f-f9cf5cd6ec8c/5b9bbf7e-f78f-403a-a4be-5024a8867fbc"
-					(reference "TP24")
+					(reference "TP26")
 					(unit 1)
 				)
@@
 		(on_board yes)
 		(dnp no)
-		(property "Reference" "TP22"
+		(property "Reference" "TP24"
 			(at 118.11 79.5019 0)
 			(effects
@@
 			(project "usb_pd_boost"
 				(path "/b6f029de-c5f9-47ba-bc2f-f9cf5cd6ec8c/5b9bbf7e-f78f-403a-a4be-5024a8867fbc"
-					(reference "TP22")
+					(reference "TP24")
 					(unit 1)
 				)
@@
 		(on_board yes)
 		(dnp no)
-		(property "Reference" "TP21"
+		(property "Reference" "TP23"
 			(at 69.85 71.8819 0)
 			(effects
@@
 			(project "usb_pd_boost"
 				(path "/b6f029de-c5f9-47ba-bc2f-f9cf5cd6ec8c/5b9bbf7e-f78f-403a-a4be-5024a8867fbc"
-					(reference "TP21")
+					(reference "TP23")
 					(unit 1)
 				)
@@
 		(on_board yes)
 		(dnp no)
-		(property "Reference" "TP25"
+		(property "Reference" "TP27"
 			(at 223.52 53.8481 0)
 			(effects
@@
 			(project "usb_pd_boost"
 				(path "/b6f029de-c5f9-47ba-bc2f-f9cf5cd6ec8c/5b9bbf7e-f78f-403a-a4be-5024a8867fbc"
-					(reference "TP25")
+					(reference "TP27")
 					(unit 1)
 				)
@@
 		(on_board yes)
 		(dnp no)
-		(property "Reference" "TP19"
+		(property "Reference" "TP21"
 			(at 38.1 51.3079 0)
 			(effects
@@
 			(project ""
 				(path "/b6f029de-c5f9-47ba-bc2f-f9cf5cd6ec8c/5b9bbf7e-f78f-403a-a4be-5024a8867fbc"
-					(reference "TP19")
+					(reference "TP21")
 					(unit 1)
 				)
@@
 		(on_board yes)
 		(dnp no)
-		(property "Reference" "TP23"
+		(property "Reference" "TP25"
 			(at 119.38 51.3079 0)
 			(effects
@@
 			(project "usb_pd_boost"
 				(path "/b6f029de-c5f9-47ba-bc2f-f9cf5cd6ec8c/5b9bbf7e-f78f-403a-a4be-5024a8867fbc"
-					(reference "TP23")
-					(unit 1)
-				)
+					(reference "TP25")
+					(unit 1)
+				)

Commit message: clean up
Parts:
- renumbered D8 to D9, R22 to R23, R23 to R24, R24 to R25, R25 to R26, R26 to R27, R27 to R28, R28 to R29, TP21 to TP20, TP22 to TP21, TP23 to TP22, TP24 to TP23, TP25 to TP24, TP26 to TP25, TP27 to TP26
Changed lines of the file:
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@@
 		(on_board yes)
 		(dnp yes)
-		(property "Reference" "R24"
+		(property "Reference" "R25"
 			(at 59.944 74.93 0)
 			(effects
@@
 			(project ""
 				(path "/b6f029de-c5f9-47ba-bc2f-f9cf5cd6ec8c/5b9bbf7e-f78f-403a-a4be-5024a8867fbc"
-					(reference "R24")
+					(reference "R25")
 					(unit 1)
 				)
@@
 		(on_board yes)
 		(dnp no)
-		(property "Reference" "TP22"
+		(property "Reference" "TP21"
 			(at 63.5 62.7379 0)
 			(effects
@@
 			(project "usb_pd_boost"
 				(path "/b6f029de-c5f9-47ba-bc2f-f9cf5cd6ec8c/5b9bbf7e-f78f-403a-a4be-5024a8867fbc"
-					(reference "TP22")
+					(reference "TP21")
 					(unit 1)
 				)
@@
 		(on_board yes)
 		(dnp no)
-		(property "Reference" "R23"
+		(property "Reference" "R24"
 			(at 45.974 74.93 0)
 			(effects
@@
 			(project "usb_pd_boost"
 				(path "/b6f029de-c5f9-47ba-bc2f-f9cf5cd6ec8c/5b9bbf7e-f78f-403a-a4be-5024a8867fbc"
-					(reference "R23")
+					(reference "R24")
 					(unit 1)
 				)
@@
 		(dnp no)
 		(fields_autoplaced yes)
-		(property "Reference" "R27"
+		(property "Reference" "R28"
 			(at 161.29 64.7699 0)
 			(effects
@@
 			(project "usb_pd_boost"
 				(path "/b6f029de-c5f9-47ba-bc2f-f9cf5cd6ec8c/5b9bbf7e-f78f-403a-a4be-5024a8867fbc"
-					(reference "R27")
+					(reference "R28")
 					(unit 1)
 				)
@@
 		(on_board yes)
 		(dnp no)
-		(property "Reference" "R25"
+		(property "Reference" "R26"
 			(at 130.81 67.564 90)
 			(effects
@@
 			(project ""
 				(path "/b6f029de-c5f9-47ba-bc2f-f9cf5cd6ec8c/5b9bbf7e-f78f-403a-a4be-5024a8867fbc"
-					(reference "R25")
+					(reference "R26")
 					(unit 1)
 				)
@@
 		(on_board yes)
 		(dnp no)
-		(property "Reference" "TP26"
+		(property "Reference" "TP25"
 			(at 158.75 70.3579 0)
 			(effects
@@
 			(project "usb_pd_boost"
 				(path "/b6f029de-c5f9-47ba-bc2f-f9cf5cd6ec8c/5b9bbf7e-f78f-403a-a4be-5024a8867fbc"
-					(reference "TP26")
+					(reference "TP25")
 					(unit 1)
 				)
@@
 		(dnp no)
 		(fields_autoplaced yes)
-		(property "Reference" "D8"
+		(property "Reference" "D9"
 			(at 138.7475 49.53 0)
 			(effects
@@
 			(project ""
 				(path "/b6f029de-c5f9-47ba-bc2f-f9cf5cd6ec8c/5b9bbf7e-f78f-403a-a4be-5024a8867fbc"
-					(reference "D8")
+					(reference "D9")
 					(unit 1)
 				)
@@
 		(on_board yes)
 		(dnp no)
-		(property "Reference" "TP24"
+		(property "Reference" "TP23"
 			(at 118.11 79.5019 0)
 			(effects
@@
 			(project "usb_pd_boost"
 				(path "/b6f029de-c5f9-47ba-bc2f-f9cf5cd6ec8c/5b9bbf7e-f78f-403a-a4be-5024a8867fbc"
-					(reference "TP24")
+					(reference "TP23")
 					(unit 1)
 				)
@@
 		(on_board yes)
 		(dnp no)
-		(property "Reference" "TP23"
+		(property "Reference" "TP22"
 			(at 69.85 71.8819 0)
 			(effects
@@
 			(project "usb_pd_boost"
 				(path "/b6f029de-c5f9-47ba-bc2f-f9cf5cd6ec8c/5b9bbf7e-f78f-403a-a4be-5024a8867fbc"
-					(reference "TP23")
+					(reference "TP22")
 					(unit 1)
 				)
@@
 		(on_board yes)
 		(dnp no)
-		(property "Reference" "TP27"
+		(property "Reference" "TP26"
 			(at 223.52 53.8481 0)
 			(effects
@@
 			(project "usb_pd_boost"
 				(path "/b6f029de-c5f9-47ba-bc2f-f9cf5cd6ec8c/5b9bbf7e-f78f-403a-a4be-5024a8867fbc"
-					(reference "TP27")
+					(reference "TP26")
 					(unit 1)
 				)
@@
 		(on_board yes)
 		(dnp no)
-		(property "Reference" "R26"
+		(property "Reference" "R27"
 			(at 130.81 79.756 90)
 			(effects
@@
 			(project "usb_pd_boost"
 				(path "/b6f029de-c5f9-47ba-bc2f-f9cf5cd6ec8c/5b9bbf7e-f78f-403a-a4be-5024a8867fbc"
-					(reference "R26")
+					(reference "R27")
 					(unit 1)
 				)
@@
 		(on_board yes)
 		(dnp no)
-		(property "Reference" "TP21"
+		(property "Reference" "TP20"
 			(at 38.1 51.3079 0)
 			(effects
@@
 			(project ""
 				(path "/b6f029de-c5f9-47ba-bc2f-f9cf5cd6ec8c/5b9bbf7e-f78f-403a-a4be-5024a8867fbc"
-					(reference "TP21")
+					(reference "TP20")
 					(unit 1)
 				)
@@
 		(on_board yes)
 		(dnp no)
-		(property "Reference" "R22"
+		(property "Reference" "R23"
 			(at 45.72 60.96 0)
 			(effects
@@
 			(project ""
 				(path "/b6f029de-c5f9-47ba-bc2f-f9cf5cd6ec8c/5b9bbf7e-f78f-403a-a4be-5024a8867fbc"
-					(reference "R22")
+					(reference "R23")
 					(unit 1)
 				)
@@
 		(dnp no)
 		(fields_autoplaced yes)
-		(property "Reference" "R28"
+		(property "Reference" "R29"
 			(at 161.29 80.0099 0)
 			(effects
@@
 			(project ""
 				(path "/b6f029de-c5f9-47ba-bc2f-f9cf5cd6ec8c/5b9bbf7e-f78f-403a-a4be-5024a8867fbc"
-					(reference "R28")
+					(reference "R29")
 					(unit 1)
 				)
@@
 		(on_board yes)
 		(dnp no)
-		(property "Reference" "TP25"
+		(property "Reference" "TP24"
 			(at 119.38 51.3079 0)
 			(effects
@@
 			(project "usb_pd_boost"
 				(path "/b6f029de-c5f9-47ba-bc2f-f9cf5cd6ec8c/5b9bbf7e-f78f-403a-a4be-5024a8867fbc"
-					(reference "TP25")
-					(unit 1)
-				)
+					(reference "TP24")
+					(unit 1)
+				)
