File: USB_PD_Boost_TestBoard/USB_PD_Boost_TestBoard.kicad_pcb (KiCad board)
At the start: 2 copper layers, 54.7 x 63.4 mm, 87 parts, among them IC1 CYPD3177-24LQXQ, IC2 TPS55340PWP, J1 USB_C_Receptacle_USB2.0_16P, J2 575-4, J3 575-4, Q1 SI7997DP-T1-GE3, Q2 SI7997DP-T1-GE3, Q3 IRLML0030

Commit message: updated p/n
Parts:
- moved TP5 0.71 mm to (151.4, 118.6)
Changed lines of the file:
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@@
 	(footprint "Connector_PinHeader_2.54mm:PinHeader_1x01_P2.54mm_Vertical"
 		(layer "F.Cu")
-		(at 152.1206 118.5926)
+		(at 151.408759 118.5926)
 		(descr "Through hole straight pin header, 1x01, 2.54mm pitch, single row")
 		(tags "Through hole pin header THT 1x01 2.54mm single row")

Commit message: comments, load resistors, stuff idk
Parts:
- removed the D3 at (145.9, 127.2)
- removed the R19 at (134.2, 133.2)
- removed the R2 at (117.0, 99.5)
- removed the TP3 at (103.7, 126.3)
- removed the TP4 at (107.8, 126.3)
- added D1: VBUS_IN, LED_SMD:LED_0603_1608Metric_Pad1.05x0.95mm_HandSolder, F.Cu at (194.9, 102.5)
- added F1: 5A, UTSVT_Connectors:FUSE_3568, F.Cu at (107.3, 105.2)
- added J2: PD_I2C, Connector_PinHeader_2.54mm:PinHeader_1x02_P2.54mm_Vertical, F.Cu at (138.7, 126.0)
- added J5: 575-4, UTSVT_Connectors:5754, F.Cu at (158.0, 92.6)
- added J6: 575-4, UTSVT_Connectors:5754, F.Cu at (169.7, 92.6)
- added JP1: BoostJumper, Connector_PinHeader_2.54mm:PinHeader_1x02_P2.54mm_Vertical, F.Cu at (106.8, 118.1)
- added R1: 2.49k, Resistor_SMD:R_0603_1608Metric_Pad0.98x0.95mm_HandSolder, F.Cu at (190.5, 102.4)
- added R21: 1k, Resistor_SMD:R_0603_1608Metric_Pad0.98x0.95mm_HandSolder, F.Cu at (128.8, 134.2)
- added R5: 33, Parts:RES_PWR263S-35, F.Cu at (162.6, 118.1)
- added R6: 33, Parts:RES_PWR263S-35, F.Cu at (162.6, 130.6)
- added TP1: CC2, Connector_PinHeader_2.54mm:PinHeader_1x01_P2.54mm_Vertical, F.Cu at (190.6, 85.1)
- added TP10: ISINK_FINE, TestPoint:TestPoint_Pad_1.0x1.0mm, F.Cu at (193.4, 119.1)
- added TP11: PD_GPIO_1, Connector_PinHeader_2.54mm:PinHeader_1x01_P2.54mm_Vertical, F.Cu at (190.6, 94.3)
- added TP12: PD_HPI_INT, Connector_PinHeader_2.54mm:PinHeader_1x01_P2.54mm_Vertical, F.Cu at (190.6, 98.9)
- added TP16: PD_1V8, Connector_PinHeader_2.54mm:PinHeader_1x01_P2.54mm_Vertical, F.Cu at (201.3, 85.1)
- added TP2: CC1, Connector_PinHeader_2.54mm:PinHeader_1x01_P2.54mm_Vertical, F.Cu at (190.6, 89.7)
- added TP5: SAFE_PWR_EN, TestPoint:TestPoint_Pad_1.0x1.0mm, F.Cu at (187.3, 116.0)
- R4: value 0 -> 33; footprint Resistor_SMD:R_0603_1608Metric_Pad0.98x0.95mm_HandSolder -> Parts:RES_PWR263S-35
- TP6: value VBUS_MAX -> VBUS_FET_EN
- TP7: value VBUS_MIN -> VBUS_MAX
- TP8: value ISINK_COARSE -> VBUS_MIN
- TP9: value ISINK_FINE -> ISINK_COARSE
- moved TP9 89.9 mm to (193.4, 116.0), turned to 0 degrees
- moved TP8 86.8 mm to (190.4, 119.1), turned to 0 degrees
- moved TP7 82.7 mm to (190.4, 116.0), turned to 0 degrees
- moved TP6 79.6 mm to (187.3, 119.1), turned to 0 degrees
- moved H2 75.2 mm to (76.1, 81.3)
- moved H4 75.2 mm to (76.1, 138.3)
- moved TP4 51.9 mm to (178.1, 133.7)
- moved TP23 49.0 mm to (190.8, 126.8)
- moved TP25 49.0 mm to (190.8, 140.4)
- moved R4 43.4 mm to (162.6, 105.5)
- moved TP3 42.6 mm to (101.8, 132.8)
- moved H1 34.9 mm to (68.4, 81.2)
- moved H3 34.9 mm to (68.4, 138.1)
- moved TP13 21.1 mm to (145.8, 138.9)
- moved TP14 19.8 mm to (101.8, 118.3), turned to 90 degrees
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- renumbered D1 to D2, D2 to D3, J2 to J3, J3 to J4, R8 to R10, R9 to R11, R10 to R12, R11 to R13, R12 to R14, R13 to R15, R14 to R16, R15 to R17, R16 to R18, R17 to R19, R1 to R2, R18 to R20, R20 to R22, R21 to R23, R22 to R24, R23 to R25, R24 to R26, R25 to R27, R26 to R28, R5 to R7, R6 to R8, R7 to R9, TP5 to TP13, TP10 to TP14, TP11 to TP15, TP12 to TP17, TP13 to TP18, TP14 to TP19, TP15 to TP20, TP16 to TP21, TP17 to TP22, TP18 to TP23, TP19 to TP24, TP20 to TP25, TP1 to TP3, TP2 to TP4
Connections:
- net /USB_PD/SCL renamed /USB_PD/PD_SCL
- net /USB_PD/SDA renamed /USB_PD/PD_SDA
- net Net-(IC1-VCCD) renamed /USB_PD/PD_1V8
- net VBUS_IN renamed /VBUS_IN
- C10 pad 1: /BOOST_VIN -> /USB_PD_Boost/+USB_PD
- C11 pad 1: /BOOST_VIN -> /USB_PD_Boost/+USB_PD
- C12 pad 1: /BOOST_VIN -> /USB_PD_Boost/+USB_PD
- C7 pad 1: PD_3V3 -> /USB_PD/PD_3V3
- C8 pad 1: PD_3V3 -> /USB_PD/PD_3V3
- C9 pad 1: PD_3V3 -> /USB_PD/PD_3V3
- IC1 pad 2: PD_3V3 -> /USB_PD/PD_3V3
- IC1 pad 23: PD_3V3 -> /USB_PD/PD_3V3
- IC2 pad 3: /BOOST_VIN -> /USB_PD_Boost/+USB_PD
- J1 pad A6: /D+ -> unconnected-(J1-D+-PadA6)
- J1 pad A7: /D- -> unconnected-(J1-D--PadA7)
- J1 pad B6: /D+ -> unconnected-(J1-D+-PadB6)
- J1 pad B7: /D- -> unconnected-(J1-D--PadB7)
- J3 pad 1: Net-(J2-Pin_1) -> /BOOST_VIN
- L1 pad 1: /BOOST_VIN -> /USB_PD_Boost/+USB_PD
- R13 pad 1: PD_3V3 -> /USB_PD/PD_3V3
- R14 pad 1: PD_3V3 -> /USB_PD/PD_3V3
- R18 pad 1: PD_3V3 -> /USB_PD/PD_3V3
- R19 pad 1: PD_3V3 -> /USB_PD/PD_3V3
- R20 pad 1: PD_3V3 -> /USB_PD/PD_3V3
- R22 pad 1: /BOOST_VIN -> /USB_PD_Boost/+USB_PD
- R4 pad 1: /PD_VOUT -> GND
- R4 pad 2: /BOOST_VIN -> /BOOST_24V_OUT
- TP17 pad 1: PD_3V3 -> /USB_PD/PD_3V3
- TP19 pad 1: /BOOST_VIN -> /USB_PD_Boost/+USB_PD
- TP6 pad 1: PD_3V3 -> /USB_PD/VBUS_FET_EN
- TP7 pad 1: /USB_PD/VBUS_MIN -> /USB_PD/PD_3V3
- TP8 pad 1: /USB_PD/ISINK_COARSE -> /USB_PD/VBUS_MIN
- TP9 pad 1: GND -> /USB_PD/ISINK_COARSE
Routing:
- net /D+: track 5.58 -> 0.00 mm
- net /D-: track 5.52 -> 0.00 mm
- net /CC1: track 2.62 -> 0.00 mm
- net /CC2: track 2.42 -> 0.00 mm
Other:
- board outline removed

Commit message: son
Parts:
- added TP4: GND, Connector_PinHeader_2.54mm:PinHeader_1x01_P2.54mm_Vertical, F.Cu at (166.3, 83.4)
- added TP6: GND, Connector_PinHeader_2.54mm:PinHeader_1x01_P2.54mm_Vertical, F.Cu at (107.3, 83.4)
- R1: value 2.49k -> 3.3k
- moved H4 98.4 mm to (174.3, 143.7)
- moved H2 98.4 mm to (174.4, 82.2)
- moved TP12 94.8 mm to (99.1, 127.8)
- moved TP11 94.6 mm to (99.1, 122.3)
- moved TP9 91.4 mm to (99.1, 111.3)
- moved TP10 91.3 mm to (99.1, 116.8)
- moved TP14 82.3 mm to (120.4, 141.9)
- moved TP13 78.4 mm to (128.3, 141.9)
- moved TP7 76.4 mm to (111.6, 126.1)
- moved TP8 75.9 mm to (111.6, 123.4)
- moved TP1 67.9 mm to (145.6, 136.1)
- moved TP27 65.7 mm to (158.1, 83.4)
- moved TP18 65.0 mm to (145.6, 118.6)
- moved TP25 60.6 mm to (142.4, 90.2)
- moved TP2 60.5 mm to (145.6, 130.2)
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- renumbered TP8 to TP10, TP9 to TP11, TP10 to TP12, TP11 to TP13, TP12 to TP14, TP13 to TP15, TP14 to TP16, TP15 to TP17, TP16 to TP18, TP17 to TP19, TP18 to TP20, TP19 to TP21, TP20 to TP22, TP21 to TP23, TP22 to TP24, TP23 to TP25, TP24 to TP26, TP25 to TP27, TP4 to TP5, TP5 to TP7, TP6 to TP8, TP7 to TP9
Other:
- board outline added: 83.6 x 68.1 mm

Commit message: early layout stuff
Parts:
- removed J2: PD_I2C, Connector_PinHeader_2.54mm:PinHeader_1x02_P2.54mm_Vertical
- added J7: PD_12C, Connector_PinHeader_2.54mm:PinHeader_1x03_P2.54mm_Vertical, F.Cu at (142.9, 125.0)
- moved D1 40.6 mm to (110.1, 144.7), turned to -90 degrees
- moved R1 39.0 mm to (111.9, 144.7), turned to -90 degrees
- moved TP15 30.6 mm to (115.1, 144.7)
- moved D4 21.0 mm to (127.1, 138.6), turned to 0 degrees
- moved C1 19.0 mm to (121.6, 137.1)
- moved TP20 17.3 mm to (128.7, 134.1)
- moved TP14 15.3 mm to (135.4, 144.7)
- moved R7 14.3 mm to (134.0, 122.8), turned to 0 degrees
- moved R8 14.2 mm to (134.0, 124.5), turned to 0 degrees
- moved J1 12.6 mm to (124.6, 145.9)
- moved TP18 10.3 mm to (135.4, 118.6)
- moved TP1 9.10 mm to (142.9, 144.7)
- moved TP2 8.20 mm to (142.9, 138.0)
- moved TP13 8.08 mm to (135.4, 138.0)
- moved TP19 6.49 mm to (142.9, 118.6)
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Routing:
- net Net-(D5-A): track 0.00 -> 25.9 mm
- net Net-(D6-A): track 0.00 -> 22.0 mm
- net Net-(D5-K): track 0.00 -> 14.0 mm
- net /VBUS_IN: track 0.00 -> 11.7 mm
- net /BOOST_24V_OUT: track 0.00 -> 10.3 mm
- net /USB_PD_Boost/+USB_PD: track 0.00 -> 10.0 mm
- net /USB_PD/VBUS_MIN: track 0.00 -> 9.83 mm, vias 0 -> 2
- net /USB_PD/PD_3V3: track 0.00 -> 9.42 mm
- net Net-(D6-K): track 0.00 -> 8.28 mm
- net Net-(IC2-EN): track 0.00 -> 7.73 mm
- net GND: track 0.00 -> 7.14 mm, vias 0 -> 9
- net /USB_PD/ISINK_COARSE: track 0.00 -> 6.62 mm, vias 0 -> 2
- net Net-(D7-K): track 0.00 -> 5.79 mm
- net /USB_PD/SAFE_PWR_EN: track 0.00 -> 5.25 mm
- net /USB_PD/VBUS_FET_EN: track 0.00 -> 4.97 mm
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- added copper zone on F.Cu, net /BOOST_24V_OUT
- added copper zone on F.Cu, net /BOOST_VIN
- added copper zone on B.Cu, net /DISSIPATION
- added copper zone on F.Cu, net /DISSIPATION
- added copper zone on F.Cu, net /PD_VOUT
- added copper zone on F.Cu, net /USB_PD_Boost/+USB_PD
- added copper zone on F.Cu, net /VBUS_IN
- added copper zone on B.Cu, net GND
- added copper zone on F.Cu, net Net-(D8-A)
Other:
- board size 83.6 x 68.1 mm -> 83.6 x 69.8 mm
- board text added: "1V8"
- board text added: "3V3"

Commit message: more layout
Parts:
- moved D1 29.8 mm to (139.9, 144.0)
- moved TP14 26.7 mm to (108.6, 143.9)
- moved R1 26.1 mm to (137.9, 144.0)
- moved TP13 20.8 mm to (115.4, 143.9)
- moved TP5 20.2 mm to (146.1, 143.9)
- moved TP15 19.0 mm to (134.1, 143.9)
- moved TP1 15.9 mm to (148.4, 129.8)
- moved TP2 14.1 mm to (148.5, 125.0)
- moved TP3 6.36 mm to (103.2, 138.7)
- moved D2 4.84 mm to (98.6, 132.7), turned to 180 degrees
- moved TP7 4.67 mm to (106.9, 126.2)
- moved TP8 4.67 mm to (106.9, 123.4)
- moved TP17 4.66 mm to (98.6, 138.7)
- moved R2 4.60 mm to (98.6, 134.5), turned to 180 degrees
Routing:
- net /USB_PD/PD_3V3: track 9.42 -> 92.9 mm, vias 0 -> 5
- net Net-(IC2-EN): track 7.73 -> 56.3 mm, vias 0 -> 1
- net /VBUS_IN: track 11.7 -> 57.6 mm, vias 0 -> 3
- net /PD_VOUT: track 0.00 -> 45.7 mm, vias 0 -> 4
- net /CC1: track 3.14 -> 44.6 mm, vias 0 -> 2
- net /CC2: track 2.51 -> 43.2 mm, vias 0 -> 2
- net /USB_PD/PD_HPI_INT: track 0.00 -> 38.9 mm, vias 0 -> 1
- net Net-(IC2-SS): track 2.38 -> 40.0 mm, vias 0 -> 1
- net Net-(IC2-FB): track 4.71 -> 37.6 mm, vias 0 -> 1
- net /USB_PD/PD_GPIO_1: track 0.00 -> 32.8 mm, vias 0 -> 1
- net Net-(IC2-COMP): track 4.85 -> 34.5 mm, vias 0 -> 1
- net /USB_PD/ISINK_COARSE: track 6.62 -> 33.3 mm, vias 2 -> 4
- net /USB_PD/VBUS_MIN: track 9.83 -> 32.1 mm, vias 2 -> 4
- net /PD_5V_OUT: track 4.01 -> 26.0 mm, vias 0 -> 2
- net /USB_PD/SAFE_PWR_EN: track 5.25 -> 24.3 mm, vias 0 -> 2
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
Commit message: cooking or no??
Parts:
- moved R3 32.9 mm to (158.6, 140.9), turned to 0 degrees
- moved D3 32.8 mm to (158.6, 142.7), turned to 0 degrees
- moved TP3 6.53 mm to (102.9, 145.2)
- moved D7 3.09 mm to (134.1, 133.8)
- moved TP5 2.56 mm to (148.3, 145.2)
- moved TP20 2.53 mm to (130.8, 135.3)
- moved D2 2.36 mm to (98.5, 135.1)
- moved R2 2.36 mm to (98.5, 136.9)
- moved TP7 2.16 mm to (106.9, 128.3)
- moved H4 2.02 mm to (175.8, 146.6)
- moved H2 2.01 mm to (175.9, 80.9)
- moved C3 1.45 mm to (115.1, 137.0)
- moved R12 1.45 mm to (115.1, 138.8)
- moved H3 1.45 mm to (97.3, 146.6)
- moved C4 1.45 mm to (115.1, 114.7)
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Routing:
- net /BOOST_24V_OUT: track 10.3 -> 26.1 mm, vias 0 -> 2
- net GND: track 14.1 -> 20.2 mm, vias 14 -> 144
- net Net-(IC2-SS): track 40.0 -> 42.3 mm
- net /USB_PD/PD_1V8: track 9.51 -> 11.6 mm
- net Net-(D3-A): track 0.00 -> 1.77 mm
- net /VBUS_IN: track 57.6 -> 56.0 mm
- net Net-(IC2-EN): track 56.3 -> 57.0 mm
- net /USB_PD/PD_HPI_INT: track 38.9 -> 38.3 mm
- net /PD_5V_OUT: track 26.0 -> 25.4 mm
- net /PD_VOUT: track 45.7 -> 45.1 mm
- net /USB_PD/PD_FAULT: track 9.28 -> 8.99 mm, vias 0 -> 2
Other:
- board size 83.6 x 69.8 mm -> 85.2 x 72.4 mm
- board text added: "24V OUT"
- board text added: "5V PWR PATH"
- board text added: "BOOST"
- board text added: "BOOST_VIN"
- board text added: "BOOST_VOUT"
- board text added: "CC1"
- board text added: "CC2"
- board text added: "COMP"
- board text added: "EN"
- board text added: "FAULT"
- board text added: "FB"
- board text added: "FUSE"
- board text added: "GND"
- board text added: "HPI_INT"
- board text added: "I_COARSE"
- board text added: "I_FINE"
- board text added: "LOAD"
- board text added: "PD 5V"
- board text added: "PD VOUT"
- board text added: "PD-> BOOST"
- board text added: "PD_GPIO"
- board text added: "SCL|SDA|GND"
- board text added: "SS"
- board text added: "SW"
- board text added: "USB PD"
- board text added: "VBUS"
- board text added: "VBUS PWR PATH"
- board text added: "VIN"
- board text added: "VOUT"
- board text added: "V_MAX"
- board text added: "V_MIN"

Commit message: something
Parts:
- removed TP4: GND, Connector_PinHeader_2.54mm:PinHeader_1x01_P2.54mm_Vertical
- TP10, TP11, TP12, TP20, TP7, TP8, TP9: footprint TestPoint:TestPoint_Pad_1.0x1.0mm -> Connector_PinHeader_2.54mm:PinHeader_1x01_P2.54mm_Vertical
- moved R3 58.7 mm to (164.5, 82.5)
- moved D3 58.7 mm to (164.5, 84.3)
- moved TP8 2.90 mm to (107.5, 121.8)
- moved TP7 2.48 mm to (107.5, 130.7)
- moved TP20 1.82 mm to (129.0, 135.1)
- moved D2 1.57 mm to (98.5, 133.5)
- moved R2 1.57 mm to (98.5, 135.3)
- moved TP17 1.57 mm to (98.6, 138.4)
Routing:
- net /USB_PD_Boost/+USB_PD: track 28.0 -> 31.6 mm
- net /BOOST_24V_OUT: track 26.1 -> 29.1 mm
- net /USB_PD/SAFE_PWR_EN: track 24.6 -> 26.9 mm
- net /USB_PD/VBUS_MIN: track 32.1 -> 34.3 mm, vias 4 -> 3
- net /USB_PD/VBUS_FET_EN: track 23.9 -> 26.1 mm
- net /USB_PD/PD_3V3: track 92.9 -> 90.9 mm, vias 5 -> 4
- net /USB_PD/PD_1V8: track 11.6 -> 12.5 mm
- net /PD_5V_OUT: track 25.4 -> 24.7 mm
- net /USB_PD/ISINK_COARSE: vias 4 -> 3
Other:
- board text added: "LOAD TESTING"
- board text added: "SETPOINTS"
- board text added: "USB PD + Boost Testboard 2026 RevX"
- board text removed: "LOAD"
- board text removed: "VOUT"

Commit message: some tweaks
Routing:
- net /USB_PD/PD_HPI_INT: track 38.3 -> 37.4 mm
- net /VBUS_IN: track 56.0 -> 56.9 mm
- net /USB_PD/PD_GPIO_1: track 32.8 -> 32.1 mm
- net Net-(IC2-EN): track 57.0 -> 57.6 mm
- net Net-(IC2-SS): track 42.3 -> 42.9 mm
Other:
- outline, holes or cut-outs redrawn
- board text added: "INPUT"
- board text removed: "FUSE"
