File: USB_PD_Boost_TestBoard/USB_PD_Boost_TestBoard.kicad_pcb (KiCad board)
At the start: 2 copper layers, 85.2 x 72.4 mm, 100 parts, among them IC1 CYPD3177-24LQXQ, IC2 TPS55340PWP, J1 USB_C_Receptacle_USB2.0_16P, J3 575-4, J4 575-4, J5 575-4, J6 575-4, J7 PD_12C, Q1 SI7997DP-T1-GE3, Q2 SI7997DP-T1-GE3, Q3 IRLML0030

Commit message: fuse holder
Parts:
- F1: footprint UTSVT_Connectors:FUSE_3568 -> Parts:3557-2
- moved F1 0.55 mm to (111.3, 104.4)
Routing:
- net GND: track 20.2 -> 22.9 mm, vias 144 -> 147
Other:
- board text added: "OUTPUT"

Commit message: comments
Parts:
- moved TP7 1.68 mm to (105.8, 130.7)
- moved TP8 1.68 mm to (105.8, 121.8)
- moved C10 0.28 mm to (126.1, 106.5)
- moved C11 0.28 mm to (123.4, 106.5)
- moved C12 0.16 mm to (128.8, 106.4)
Connections:
- F1 pad 3: (no net) -> /BOOST_VIN
- F1 pad 4: (no net) -> /USB_PD_Boost/+USB_PD
Routing:
- net GND: track 22.9 -> 17.4 mm, vias 147 -> 155
- net /VBUS_IN: track 56.9 -> 53.4 mm
- net Net-(IC2-EN): track 57.6 -> 55.0 mm, vias 1 -> 2
- net /USB_PD/SAFE_PWR_EN: track 26.7 -> 28.7 mm
- net /CC2: track 43.5 -> 45.4 mm
- net /USB_PD/PD_3V3: track 90.9 -> 92.8 mm
- net /USB_PD/VBUS_FET_EN: track 26.1 -> 27.6 mm
- net /USB_PD/PD_1V8: track 12.5 -> 11.3 mm
- net /USB_PD_Boost/+USB_PD: track 31.5 -> 30.6 mm, vias 0 -> 2
- net /CC1: track 44.6 -> 45.3 mm

Commit message: addressed reviews
Parts:
- moved TP16 12.8 mm to (104.9, 117.2)
- moved TP10 6.32 mm to (97.7, 124.3)
- moved TP11 6.32 mm to (97.7, 129.8)
- moved TP12 6.32 mm to (97.7, 135.3)
- moved TP9 6.32 mm to (97.7, 118.8)
- moved TP17 6.29 mm to (104.6, 136.6)
- moved R2 6.14 mm to (104.5, 134.0)
- moved D2 6.11 mm to (104.5, 132.1)
- moved TP8 3.18 mm to (104.4, 124.7)
- moved TP7 2.44 mm to (104.4, 128.7)
- moved F1 1.51 mm to (109.8, 104.3)
Routing:
- net /PD_VOUT: track 44.8 -> 36.3 mm
- net /PD_5V_OUT: track 24.7 -> 19.7 mm, vias 2 -> 1
- net /USB_PD/PD_3V3: track 92.8 -> 88.1 mm
- net /USB_PD/VBUS_FET_EN: track 27.6 -> 25.7 mm, vias 2 -> 1
- net /USB_PD/SAFE_PWR_EN: track 28.7 -> 27.3 mm, vias 2 -> 1
- net /USB_PD/VBUS_MIN: track 34.3 -> 33.5 mm, vias 3 -> 2
- net /USB_PD/ISINK_COARSE: track 33.3 -> 33.7 mm, vias 3 -> 2
- net GND: vias 155 -> 160
Other:
- board text added: "BOOST INPUT FUSE"
- board text added: "PD->BOOST JUMPER"
- board text removed: "PD-> BOOST"

Commit message: clean up
Parts:
- removed the R21 at (134.1, 132.1)
- added D2: VBUS_IN, LED_SMD:LED_0603_1608Metric_Pad1.05x0.95mm_HandSolder, F.Cu at (104.5, 119.9)
- added LOGO1: LHRS, UTSVT_Logos:LHRs_LOGO, F.Cu at (144.3, 139.4)
- added R2: 3.3k, Resistor_SMD:R_0603_1608Metric_Pad0.98x0.95mm_HandSolder, F.Cu at (104.5, 118.2)
- added R22: 3.3k, Resistor_SMD:R_0603_1608Metric_Pad0.98x0.95mm_HandSolder, F.Cu at (134.1, 132.1)
- F1: footprint Parts:3557-2 -> UTSVT_Power:Fuse-3557-2
- moved TP15 1.60 mm to (104.6, 115.6)
- moved TP16 1.18 mm to (104.6, 137.8)
- moved R3 1.18 mm to (104.5, 135.1)
- moved D3 1.18 mm to (104.5, 133.3)
- moved TP7 0.22 mm to (104.6, 124.7)
- moved TP6 0.20 mm to (104.6, 128.7)
- renumbered D2 to D3, D3 to D4, D4 to D5, D5 to D6, D6 to D7, D7 to D8, D8 to D9, J7 to J2, R9 to R10, R10 to R11, R11 to R12, R12 to R13, R13 to R14, R14 to R15, R15 to R16, R16 to R17, R17 to R18, R18 to R19, R19 to R20, R20 to R21, R22 to R23, R23 to R24, R24 to R25, R25 to R26, R26 to R27, R27 to R28, R28 to R29, R2 to R3, R3 to R4, R4 to R5, R5 to R6, R6 to R7, R7 to R8, R8 to R9, TP3 to TP1, TP11 to TP10, TP12 to TP11, TP13 to TP12, TP14 to TP13, TP15 to TP14, TP16 to TP15, TP17 to TP16, TP18 to TP17, TP19 to TP18, TP20 to TP19, TP5 to TP2, TP21 to TP20, TP22 to TP21, TP23 to TP22, TP24 to TP23, TP25 to TP24, TP26 to TP25, TP27 to TP26, TP6 to TP3, TP1 to TP4, TP2 to TP5, TP7 to TP6, TP8 to TP7, TP9 to TP8, TP10 to TP9
Routing:
- net /PD_VOUT: track 36.3 -> 40.1 mm
- net Net-(D2-A): track 0.00 -> 1.59 mm
- net GND: vias 160 -> 161
Other:
- board text added: "USB PD + Boost Testboard Michael Adeluyi 2026 RevX"
- board text added: "^ REMOVE PD JUMPER WHILE USING ^"
- board text removed: "USB PD + Boost Testboard 2026 RevX"
