File: PowerPath_TestBoard/PowerPath/12VBuck.kicad_sch (KiCad schematic)
At the start: 12 parts, among them U1 LMR51635XDDCR

Commit message: reviewed lakshay, ready for lil shah
Parts:
- removed C1: 2.2u, Capacitor_SMD:C_0805_2012Metric_Pad1.18x1.45mm_HandSolder, symbol Device:C_Small
- removed C2: 100n, Resistor_SMD:R_0201_0603Metric_Pad0.64x0.40mm_HandSolder, symbol Device:C_Small
- removed C3, C4: 47u, Capacitor_SMD:C_1210_3225Metric_Pad1.33x2.70mm_HandSolder, symbol Device:C_Small
- removed L1: 10u, Inductor_SMD:L_TDK_VLP8040, symbol Device:L_Small
- removed R2: 10.2k, Resistor_SMD:R_0603_1608Metric, symbol Device:R_Small
- removed TP5: V_in_24V, TestPoint:TestPoint_THTPad_D3.0mm_Drill1.5mm, symbol Connector:TestPoint
- removed TP6: FB, TestPoint:TestPoint_THTPad_D3.0mm_Drill1.5mm, symbol Connector:TestPoint
- removed TP7: CB, TestPoint:TestPoint_THTPad_D3.0mm_Drill1.5mm, symbol Connector:TestPoint
- removed TP8: SW, TestPoint:TestPoint_THTPad_D3.0mm_Drill1.5mm, symbol Connector:TestPoint
- removed U1: LMR51635XDDCR, utsvt_ics:DDC0006A-MFG, symbol 2026-04-25_18-34-12:LMR51635XDDCR
- added C10, C9: 47u, Capacitor_SMD:C_1210_3225Metric_Pad1.33x2.70mm_HandSolder, symbol Device:C_Small
- added C11: 2.2u, Capacitor_SMD:C_0805_2012Metric_Pad1.18x1.45mm_HandSolder, symbol Device:C_Small
- added C12: 100n, Resistor_SMD:R_0201_0603Metric_Pad0.64x0.40mm_HandSolder, symbol Device:C_Small
- added L3: 15u, Inductor_SMD:L_TDK_VLP8040, symbol Device:L_Small
- added R4: 10.2k, Resistor_SMD:R_0603_1608Metric, symbol Device:R_Small
- added TP11: CB, TestPoint:TestPoint_THTPad_D3.0mm_Drill1.5mm, symbol Connector:TestPoint
- added TP14: FB, TestPoint:TestPoint_THTPad_D3.0mm_Drill1.5mm, symbol Connector:TestPoint
- added TP15: SW, TestPoint:TestPoint_THTPad_D3.0mm_Drill1.5mm, symbol Connector:TestPoint
- added TP9: V_in_24V, TestPoint:TestPoint_THTPad_D3.0mm_Drill1.5mm, symbol Connector:TestPoint
- added U3: LMR51635XDDCR, utsvt_ics:DDC0006A-MFG, symbol 2026-04-25_18-34-12:LMR51635XDDCR
- R1: value 53.6k -> 143k; LCSC P/N C23074 -> C22877; P/N 0603WAF5362T5E -> 0603WAF1433T5E
Connections:
- net CB: now also C12.1, TP11.1, U3.6 (CB)
- net FB: now also R4.1, TP14.1, U3.1 (FB)
- net GND: now also C10.2, C11.2, C9.2, R4.2, U3.4 (GND)
- net SW: now also C12.2, L3.1, TP15.1, U3.5 (SW)
- net V_in_24V: now also C11.1, TP9.1, U3.2 (EN), U3.3 (VIN)
- net V_out_5V renamed V_out_12V
- net V_out_12V: now also C10.1, C9.1, L3.2
Other:
- note added: "12V Vout"
- note added: "24V-12V Buck Converter"
- note removed: "24V-5V Buck Converter"
- note removed: "5V Vout"
