File: PowerPath_TestBoard/PowerPath/3V3Buck.kicad_sch (KiCad schematic)
At the start: 12 parts, among them U1 LMR51635XDDCR

Commit message: reviewed lakshay, ready for lil shah
Parts:
- removed C1: 2.2u, Capacitor_SMD:C_0805_2012Metric_Pad1.18x1.45mm_HandSolder, symbol Device:C_Small
- removed C2: 100n, Resistor_SMD:R_0201_0603Metric_Pad0.64x0.40mm_HandSolder, symbol Device:C_Small
- removed R1: 53.6k, Resistor_SMD:R_0603_1608Metric, symbol Device:R_Small
- removed R2: 10.2k, Resistor_SMD:R_0603_1608Metric, symbol Device:R_Small
- removed TP5: V_in_24V, TestPoint:TestPoint_THTPad_D3.0mm_Drill1.5mm, symbol Connector:TestPoint
- removed TP6: FB, TestPoint:TestPoint_THTPad_D3.0mm_Drill1.5mm, symbol Connector:TestPoint
- removed TP7: CB, TestPoint:TestPoint_THTPad_D3.0mm_Drill1.5mm, symbol Connector:TestPoint
- removed TP8: SW, TestPoint:TestPoint_THTPad_D3.0mm_Drill1.5mm, symbol Connector:TestPoint
- added C6, C7: 47u, Capacitor_SMD:C_1210_3225Metric_Pad1.33x2.70mm_HandSolder, symbol Device:C_Small
- added R6: 31.6k, Resistor_SMD:R_0603_1608Metric, symbol Device:R_Small
- added R7: 10.2k, Resistor_SMD:R_0603_1608Metric, symbol Device:R_Small
- added TP16: V_in_24V, TestPoint:TestPoint_THTPad_D3.0mm_Drill1.5mm, symbol Connector:TestPoint
- added TP17: CB, TestPoint:TestPoint_THTPad_D3.0mm_Drill1.5mm, symbol Connector:TestPoint
- added TP18: FB, TestPoint:TestPoint_THTPad_D3.0mm_Drill1.5mm, symbol Connector:TestPoint
- added TP19: SW, TestPoint:TestPoint_THTPad_D3.0mm_Drill1.5mm, symbol Connector:TestPoint
- C3: value 47u -> 2.2u; footprint Capacitor_SMD:C_1210_3225Metric_Pad1.33x2.70mm_HandSolder -> Capacitor_SMD:C_0805_2012Metric_Pad1.18x1.45mm_HandSolder; LCSC P/N C77101 -> C1771; P/N GRM32ER61C476KE15L -> CL21F225ZAFNNNE
- C4: value 47u -> 100n; footprint Capacitor_SMD:C_1210_3225Metric_Pad1.33x2.70mm_HandSolder -> Resistor_SMD:R_0201_0603Metric_Pad0.64x0.40mm_HandSolder; LCSC P/N C77101 -> C14663; P/N GRM32ER61C476KE15L -> MLASH168SB7104KTNA01
- L1: value 10u -> 5.6u; footprint Inductor_SMD:L_TDK_VLP8040 -> Inductor_SMD:L_TDK_SLF6025; LCSC P/N C354639 -> C2997651; P/N CKCS8040-10uH/M -> PNLS6045-5R6M 5.6UH
- U1: footprint utsvt_ics:DDC0006A-MFG -> breh:DDC0006A-MFG
Connections:
- net CB: now also C4.1, TP17.1
- net FB: now also R6.2, R7.1, TP18.1
- net GND: now also C6.2, C7.2, R7.2; no longer C4.2
- net SW: now also C4.2, TP19.1
- net V_in_24V: now also C3.1, TP16.1
- removed net V_out_5V: C3.1, C4.1, L1.2
- new net V_out_3V3: C6.1, C7.1, L1.2, R6.1
Other:
- note added: "24V-3.3V Buck Converter"
- note added: "3.3V Vout"
- note removed: "24V-5V Buck Converter"
- note removed: "5V Vout"
