File: PowerPath_TestBoard/PowerPath/LDO.kicad_sch (KiCad schematic)
At the start: 5 parts, among them U1 MCP1826S_LDO

Commit message: reviewed lakshay, ready for lil shah
Parts:
- C7, C8: P/N (none) -> GRM21BR61H106KE43L
Changed lines of the file:
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@@
+			)
+		)
+		(property "P/N" "GRM21BR61H106KE43L"
+			(at 62.23 52.07 0)
+			(effects
+				(font
+					(size 1.27 1.27)
+				)
+				(hide yes)
 			)
 		)
@@
 			(at 36.83 52.07 0)
 			(effects
+				(font
+					(size 1.27 1.27)
+				)
+				(hide yes)
+			)
+		)
+		(property "P/N" "GRM21BR61H106KE43L"
+			(at 36.83 52.07 0)
+			(effects
