File: PowerPath_TestBoard/PowerPath/PowerPath.kicad_sch (KiCad schematic)
At the start: 29 parts, among them J1 +24V_Ext, J2 GND, J3 +V_in_24V, J4 GND, J5 +Vin_5V, J6 GND

Commit message: reviewed lakshay, ready for lil shah
Parts:
- removed J4, J6: GND, 575-4:5754, symbol Connector_Generic:Conn_01x01
- removed TP11: +Vout_5V, TestPoint:TestPoint_THTPad_D3.0mm_Drill1.5mm, symbol Connector:TestPoint
- removed TP9: V_in_24V, TestPoint:TestPoint_THTPad_D3.0mm_Drill1.5mm, symbol Connector:TestPoint
- added D11, D9: LED, LED_SMD:LED_0603_1608Metric, symbol Device:LED
- added F1: 1A, UTSVT_Connectors:FUSE_3568, symbol utsvt_power:Fuse_3568
- added JP10, JP11, JP12, JP13, JP14, JP15, JP4, JP5, JP6, JP7, JP8, JP9: PP to Buck, Connector_PinHeader_1.00mm:PinHeader_1x02_P1.00mm_Vertical, symbol Jumper:SolderJumper_2_Open
- added JP3: Buck to LDO, Connector_PinHeader_1.00mm:PinHeader_1x02_P1.00mm_Vertical, symbol Jumper:SolderJumper_2_Open
- added R10: 10k, Resistor_SMD:R_0603_1608Metric, symbol Device:R
- added R11, R16: 1k, Bourns_DPAK_1k:RES_PWR163_BRN, symbol Device:R
- added R14, R17, R18: 470, Bourns_DPAK_470:RES_PWR263S_BRN, symbol Device:R
- added R19, R22, R24: 100, Bourns_DPAK_100:RES_PWR163_BRN, symbol Device:R
- added R21: 330, Bourns_DPAK_200:RES_PWR163_BRN, symbol Device:R
- added R25, R26: 50, Bourns_DPAK_50:BO_PWR163, symbol Device:R
- added R28: 200, Bourns_DPAK_200:RES_PWR163_BRN, symbol Device:R
- added R3: 22k, Resistor_SMD:R_0603_1608Metric, symbol Device:R
- added TP16: 12V_Out, TestPoint:TestPoint_THTPad_D3.0mm_Drill1.5mm, symbol Connector:TestPoint
- D3, D4, D5, D6, D7, D8: footprint (none) -> LED_SMD:LED_0603_1608Metric; LCSC P/N (none) -> C84263; P/N (none) -> NCD0603R1
- JP1: footprint Jumper:SolderJumper-2_P1.3mm_Open_RoundedPad1.0x1.5mm -> Connector_PinHeader_1.00mm:PinHeader_1x02_P1.00mm_Vertical
- JP2: value Buck to LDO -> PP to Buck; footprint Jumper:SolderJumper-2_P1.3mm_Open_RoundedPad1.0x1.5mm -> Connector_PinHeader_1.00mm:PinHeader_1x02_P1.00mm_Vertical
- R4, R5, R6: value 22.1k -> 22k; footprint (none) -> Resistor_SMD:R_0603_1608Metric; LCSC P/N (none) -> C31850; P/N (none) -> CRCW060322K0FKEAHP
- R7, R8: value 2.21k -> 2.2k; footprint (none) -> Resistor_SMD:R_0603_1608Metric; LCSC P/N (none) -> C4190; P/N (none) -> 0603WAF2201T5E
- R9: value 2.21k -> 1k; footprint (none) -> Resistor_SMD:R_0603_1608Metric; LCSC P/N (none) -> C4190; P/N (none) -> 0603WAF2201T5E
Connections:
- net +24V_Ext: now also F1.2; no longer J1.1 (Pin_1)
- net +V_out_5V_Buck: now also JP3.1 (A); no longer JP2.1 (A)
- net +Vin_5V: now also JP13.2 (B), JP3.2 (B), JP8.2 (B), JP9.2 (B); no longer JP2.2 (B)
- net 24V_OUT: now also JP2.1 (A), JP15.2 (B), JP4.2 (B), JP5.2 (B)
- net GND: now also D11.1 (K), D9.1 (K), R11.2, R14.2, R16.2, R17.2, R18.2, R19.2, R21.2, R22.2, R24.2, R25.2, R26.2, R28.2
- net +Vout_5V renamed +Vout_3V3
- net +Vout_3V3: now also JP10.2 (B), JP11.2 (B), JP14.2 (B)
- new net: F1.1, J1.1 (Pin_1)
- new net: D11.2 (A), R10.2
- new net: JP6.1 (A), R16.1
- new net: JP12.1 (A), R24.1
- new net: JP4.1 (A), R11.1
- new net: JP10.1 (A), R21.1
- new net: JP13.1 (A), R25.1
- new net: D9.2 (A), R3.2
- new net: JP11.1 (A), R22.1
- new net: JP8.1 (A), R18.1
- new net: JP14.1 (A), R26.1
- new net: JP7.1 (A), R17.1
- new net: JP5.1 (A), R14.1
- new net: JP9.1 (A), R19.1
- new net: JP15.1 (A), R28.1
- new net 12VBuck/V_in_24V: JP2.2 (B), R3.1
- new net V_out_12V: JP12.2 (B), JP6.2 (B), JP7.2 (B), R10.1, TP16.1
Other:
- added sheet 12VBuck (12VBuck.kicad_sch)
- note added: "12V loads: 1kΩ → 12mA, 0.144W 470Ω → 25.5mA, 0.306W 100Ω → 120mA, 1.44W"
- note added: "24V Resistor Calculations: R = (12V - 2V) / 1.0mA R = 10V / 0.001A R = 10k"
- note added: "24V Resistor Calculations: R = (24V - 2V) / 1.0mA R = 22V / 0.001A R = 22000Ω"
- note added: "24V loads: 1kΩ → 24mA, 0.576W 470Ω → 51mA, 1.23W 200Ω → 120mA, 2.88W"
- note added: "3.3V loads: 330Ω → 10mA, 0.033W 100Ω → 33mA, 0.109W 50Ω → 66mA, 0.218W"
- note added: "3v3 Resistor calculation: R = (3.3V - 2V) / 1.3mA R = 1.3V / 0.0013A R = 1000Ω"
- note added: "5V Resistor calculation: R = (5V - 2V) / 1.36mA R = 3V / 0.00136A R ≈ 2205Ω -> 2.2k"
- note added: "5V loads: 470Ω → 10.6mA, 0.053W 100Ω → 50mA, 0.25W 50Ω → 100mA, 0.5W"
- note added: "GND Connector"
- note added: "Load Resistor Testing - 12V"
- note added: "Load Resistor Testing - 24V"
- note added: "Load Resistor Testing - 3V3"
- note added: "Load Resistor Testing - 5V"
- note removed: "Buck Connectors"
- note removed: "Debug LEDs"
- note removed: "LDO Connectors"
- note removed: "PP Connectors"
- note removed: "Solder Jumper"
- moved on the sheet: D3, D4, D5, D6, D7, D8, J1, J2, J3, J5, JP1, R4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
