File: PowerPath_TestBoard/PowerPath/PowerProtection.kicad_sch (KiCad schematic)
At the start: 17 parts, among them U7 LM76202QPWPRQ1

Commit message: reviewed lakshay, ready for lil shah
Parts:
- C20, C23: LCSC P/N (none) -> C3840574
- R12: LCSC P/N (none) -> C4107995
- R13: LCSC P/N (none) -> C2076662
- R15: LCSC P/N (none) -> C844348
- R20: LCSC P/N (none) -> C4062016
- R30: LCSC P/N (none) -> C4332876
- U7: LCSC P/N (none) -> C1849484
Changed lines of the file:
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@@
+			)
+		)
+		(property "LCSC P/N" "C3840574"
+			(at 29.21 36.83 0)
+			(effects
+				(font
+					(size 1.27 1.27)
+				)
+				(hide yes)
 			)
 		)
@@
 			)
 		)
+		(property "LCSC P/N" "C4062016"
+			(at 129.54 92.71 0)
+			(effects
+				(font
+					(size 1.27 1.27)
+				)
+				(hide yes)
+			)
+		)
 		(pin "1"
 		)
@@
 			)
 		)
+		(property "LCSC P/N" "C844348"
+			(at 21.59 123.19 0)
+			(effects
+				(font
+					(size 1.27 1.27)
+				)
+				(hide yes)
+			)
+		)
 		(pin "1"
 		)
@@
 		)
 		(property "P/N" "GRM21BR61H106KE43K"
+			(at 130.81 38.1 0)
+			(effects
+				(font
+					(size 1.27 1.27)
+				)
+				(hide yes)
+			)
+		)
+		(property "LCSC P/N" "C3840574"
 			(at 130.81 38.1 0)
 			(effects
@@
 			)
 		)
+		(property "LCSC P/N" "C4332876"
+			(at 142.24 36.83 0)
+			(effects
+				(font
+					(size 1.27 1.27)
+				)
+				(hide yes)
+			)
+		)
 		(pin "1"
 		)
@@
 			)
 		)
+		(property "LCSC P/N" "C1849484"
+			(at 67.31 31.75 0)
+			(effects
+				(font
+					(size 1.27 1.27)
+				)
+				(hide yes)
+			)
+		)
 		(pin "12"
 		)
@@
 			)
 		)
+		(property "LCSC P/N" "C2076662"
+			(at 21.59 113.03 0)
+			(effects
+				(font
+					(size 1.27 1.27)
+				)
+				(hide yes)
+			)
+		)
 		(pin "1"
 		)
@@
 			(at 21.59 102.87 0)
 			(effects
+				(font
+					(size 1.27 1.27)
+				)
+				(hide yes)
+			)
+		)
+		(property "LCSC P/N" "C4107995"
+			(at 21.59 102.87 0)
+			(effects
