File: PowerPath_TestBoard/PowerPath/testgainga.kicad_sch (KiCad schematic)
At the start: 12 parts, among them U1 LMR51635XDDCR

Commit message: reviewed lakshay, ready for lil shah
Parts:
- TP5, TP6, TP7, TP8: footprint TestPoint:TestPoint_THTPad_D3.0mm_Drill1.5mm -> (none)
Changed lines of the file:
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@@
 			)
 			(project "5VBuck"
-				(path "/ad6c7df0-eb90-4670-9aa8-3e2007aefc2d/ae63f0a9-78b8-4efb-b2ee-a2699a24d705"
+				(path "/ad6c7df0-eb90-4670-9aa8-3e2007aefc2d/4ce3c563-64ba-4b6e-b334-e3956b5d5a33"
+					(reference "L1")
+					(unit 1)
+				)
+				(path "/ad6c7df0-eb90-4670-9aa8-3e2007aefc2d/c59a1097-f91e-4d56-b57d-869363ca5893"
 					(reference "L1")
 					(unit 1)
@@
 			)
 			(project "5VBuck"
-				(path "/ad6c7df0-eb90-4670-9aa8-3e2007aefc2d/ae63f0a9-78b8-4efb-b2ee-a2699a24d705"
+				(path "/ad6c7df0-eb90-4670-9aa8-3e2007aefc2d/4ce3c563-64ba-4b6e-b334-e3956b5d5a33"
+					(reference "R2")
+					(unit 1)
+				)
+				(path "/ad6c7df0-eb90-4670-9aa8-3e2007aefc2d/c59a1097-f91e-4d56-b57d-869363ca5893"
 					(reference "R2")
 					(unit 1)
@@
 			)
 			(project "5VBuck"
-				(path "/ad6c7df0-eb90-4670-9aa8-3e2007aefc2d/ae63f0a9-78b8-4efb-b2ee-a2699a24d705"
+				(path "/ad6c7df0-eb90-4670-9aa8-3e2007aefc2d/4ce3c563-64ba-4b6e-b334-e3956b5d5a33"
+					(reference "C1")
+					(unit 1)
+				)
+				(path "/ad6c7df0-eb90-4670-9aa8-3e2007aefc2d/c59a1097-f91e-4d56-b57d-869363ca5893"
 					(reference "C1")
 					(unit 1)
@@
 			)
 		)
-		(property "Footprint" "TestPoint:TestPoint_THTPad_D3.0mm_Drill1.5mm"
+		(property "Footprint" ""
 			(at 186.69 85.09 0)
 			(effects
@@
 		(instances
 			(project "PowerPath"
-				(path "/ad6c7df0-eb90-4670-9aa8-3e2007aefc2d/ae63f0a9-78b8-4efb-b2ee-a2699a24d705"
+				(path "/ad6c7df0-eb90-4670-9aa8-3e2007aefc2d/4ce3c563-64ba-4b6e-b334-e3956b5d5a33"
+					(reference "TP6")
+					(unit 1)
+				)
+				(path "/ad6c7df0-eb90-4670-9aa8-3e2007aefc2d/c59a1097-f91e-4d56-b57d-869363ca5893"
 					(reference "TP6")
 					(unit 1)
@@
 			)
 			(project "5VBuck"
-				(path "/ad6c7df0-eb90-4670-9aa8-3e2007aefc2d/ae63f0a9-78b8-4efb-b2ee-a2699a24d705"
+				(path "/ad6c7df0-eb90-4670-9aa8-3e2007aefc2d/4ce3c563-64ba-4b6e-b334-e3956b5d5a33"
+					(reference "C2")
+					(unit 1)
+				)
+				(path "/ad6c7df0-eb90-4670-9aa8-3e2007aefc2d/c59a1097-f91e-4d56-b57d-869363ca5893"
 					(reference "C2")
 					(unit 1)
@@
 			)
 			(project "5VBuck"
-				(path "/ad6c7df0-eb90-4670-9aa8-3e2007aefc2d/ae63f0a9-78b8-4efb-b2ee-a2699a24d705"
+				(path "/ad6c7df0-eb90-4670-9aa8-3e2007aefc2d/4ce3c563-64ba-4b6e-b334-e3956b5d5a33"
+					(reference "U1")
+					(unit 1)
+				)
+				(path "/ad6c7df0-eb90-4670-9aa8-3e2007aefc2d/c59a1097-f91e-4d56-b57d-869363ca5893"
 					(reference "U1")
 					(unit 1)
@@
 			)
 		)
-		(property "Footprint" "TestPoint:TestPoint_THTPad_D3.0mm_Drill1.5mm"
+		(property "Footprint" ""
 			(at 173.99 85.09 0)
 			(effects
@@
 		(instances
 			(project ""
-				(path "/ad6c7df0-eb90-4670-9aa8-3e2007aefc2d/ae63f0a9-78b8-4efb-b2ee-a2699a24d705"
+				(path "/ad6c7df0-eb90-4670-9aa8-3e2007aefc2d/4ce3c563-64ba-4b6e-b334-e3956b5d5a33"
+					(reference "TP5")
+					(unit 1)
+				)
+				(path "/ad6c7df0-eb90-4670-9aa8-3e2007aefc2d/c59a1097-f91e-4d56-b57d-869363ca5893"
 					(reference "TP5")
 					(unit 1)
@@
 			)
 			(project "5VBuck"
-				(path "/ad6c7df0-eb90-4670-9aa8-3e2007aefc2d/ae63f0a9-78b8-4efb-b2ee-a2699a24d705"
+				(path "/ad6c7df0-eb90-4670-9aa8-3e2007aefc2d/4ce3c563-64ba-4b6e-b334-e3956b5d5a33"
+					(reference "#FLG01")
+					(unit 1)
+				)
+				(path "/ad6c7df0-eb90-4670-9aa8-3e2007aefc2d/c59a1097-f91e-4d56-b57d-869363ca5893"
 					(reference "#FLG01")
 					(unit 1)
@@
 			)
 		)
-		(property "Footprint" "TestPoint:TestPoint_THTPad_D3.0mm_Drill1.5mm"
+		(property "Footprint" ""
 			(at 186.69 97.79 0)
 			(effects
@@
 		(instances
 			(project "PowerPath"
-				(path "/ad6c7df0-eb90-4670-9aa8-3e2007aefc2d/ae63f0a9-78b8-4efb-b2ee-a2699a24d705"
+				(path "/ad6c7df0-eb90-4670-9aa8-3e2007aefc2d/4ce3c563-64ba-4b6e-b334-e3956b5d5a33"
+					(reference "TP8")
+					(unit 1)
+				)
+				(path "/ad6c7df0-eb90-4670-9aa8-3e2007aefc2d/c59a1097-f91e-4d56-b57d-869363ca5893"
 					(reference "TP8")
 					(unit 1)
@@
 			)
 			(project "5VBuck"
-				(path "/ad6c7df0-eb90-4670-9aa8-3e2007aefc2d/ae63f0a9-78b8-4efb-b2ee-a2699a24d705"
+				(path "/ad6c7df0-eb90-4670-9aa8-3e2007aefc2d/4ce3c563-64ba-4b6e-b334-e3956b5d5a33"
+					(reference "C4")
+					(unit 1)
+				)
+				(path "/ad6c7df0-eb90-4670-9aa8-3e2007aefc2d/c59a1097-f91e-4d56-b57d-869363ca5893"
 					(reference "C4")
 					(unit 1)
@@
 			)
 			(project "5VBuck"
-				(path "/ad6c7df0-eb90-4670-9aa8-3e2007aefc2d/ae63f0a9-78b8-4efb-b2ee-a2699a24d705"
+				(path "/ad6c7df0-eb90-4670-9aa8-3e2007aefc2d/4ce3c563-64ba-4b6e-b334-e3956b5d5a33"
+					(reference "#FLG02")
+					(unit 1)
+				)
+				(path "/ad6c7df0-eb90-4670-9aa8-3e2007aefc2d/c59a1097-f91e-4d56-b57d-869363ca5893"
 					(reference "#FLG02")
 					(unit 1)
@@
 			)
 			(project "5VBuck"
-				(path "/ad6c7df0-eb90-4670-9aa8-3e2007aefc2d/ae63f0a9-78b8-4efb-b2ee-a2699a24d705"
+				(path "/ad6c7df0-eb90-4670-9aa8-3e2007aefc2d/4ce3c563-64ba-4b6e-b334-e3956b5d5a33"
+					(reference "R1")
+					(unit 1)
+				)
+				(path "/ad6c7df0-eb90-4670-9aa8-3e2007aefc2d/c59a1097-f91e-4d56-b57d-869363ca5893"
 					(reference "R1")
 					(unit 1)
@@
 			)
 			(project "5VBuck"
-				(path "/ad6c7df0-eb90-4670-9aa8-3e2007aefc2d/ae63f0a9-78b8-4efb-b2ee-a2699a24d705"
+				(path "/ad6c7df0-eb90-4670-9aa8-3e2007aefc2d/4ce3c563-64ba-4b6e-b334-e3956b5d5a33"
+					(reference "C3")
+					(unit 1)
+				)
+				(path "/ad6c7df0-eb90-4670-9aa8-3e2007aefc2d/c59a1097-f91e-4d56-b57d-869363ca5893"
 					(reference "C3")
 					(unit 1)
@@
 			)
 		)
-		(property "Footprint" "TestPoint:TestPoint_THTPad_D3.0mm_Drill1.5mm"
+		(property "Footprint" ""
 			(at 173.99 97.79 0)
 			(effects
@@
 		(instances
 			(project "PowerPath"
-				(path "/ad6c7df0-eb90-4670-9aa8-3e2007aefc2d/ae63f0a9-78b8-4efb-b2ee-a2699a24d705"
+				(path "/ad6c7df0-eb90-4670-9aa8-3e2007aefc2d/4ce3c563-64ba-4b6e-b334-e3956b5d5a33"
 					(reference "TP7")
 					(unit 1)
+				)
+				(path "/ad6c7df0-eb90-4670-9aa8-3e2007aefc2d/c59a1097-f91e-4d56-b57d-869363ca5893"
+					(reference "TP7")
+					(unit 1)
