File: 100PinMCU_TestBoard/100PinMCU_ESP32_TestBoard/LDO.kicad_sch (KiCad schematic)
At the start: 5 parts, among them U1 MCP1826S

Commit message: esp32 design block will be updated later
Parts:
- renumbered C2 to C10, C1 to C9, D1 to D12, U1 to U2
Changed lines of the file:
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@@
 		(dnp no)
 		(fields_autoplaced yes)
-		(property "Reference" "C2"
+		(property "Reference" "C10"
 			(at 168.275 68.5735 0)
 			(effects
@@
 			(project "LDO"
 				(path "/abcdaa41-14f3-4587-9aac-314b09095246/ab199eb4-16ff-472f-a198-e557cdece1a6"
-					(reference "C2")
+					(reference "C10")
 					(unit 1)
 				)
@@
 		(dnp no)
 		(fields_autoplaced yes)
-		(property "Reference" "U1"
+		(property "Reference" "U2"
 			(at 152.4 56.515 0)
 			(effects
@@
 			(project ""
 				(path "/abcdaa41-14f3-4587-9aac-314b09095246/ab199eb4-16ff-472f-a198-e557cdece1a6"
-					(reference "U1")
+					(reference "U2")
 					(unit 1)
 				)
@@
 		(dnp no)
 		(fields_autoplaced yes)
-		(property "Reference" "D1"
+		(property "Reference" "D12"
 			(at 133.604 57.15 0)
 			(effects
@@
 			(project ""
 				(path "/abcdaa41-14f3-4587-9aac-314b09095246/ab199eb4-16ff-472f-a198-e557cdece1a6"
-					(reference "D1")
+					(reference "D12")
 					(unit 1)
 				)
@@
 		(dnp no)
 		(fields_autoplaced yes)
-		(property "Reference" "C1"
+		(property "Reference" "C9"
 			(at 142.875 68.5735 0)
 			(effects
@@
 			(project "LDO"
 				(path "/abcdaa41-14f3-4587-9aac-314b09095246/ab199eb4-16ff-472f-a198-e557cdece1a6"
-					(reference "C1")
-					(unit 1)
-				)
+					(reference "C9")
+					(unit 1)
+				)
