File: 100PinMCU_TestBoard/100PinMCU_ESP32_TestBoard/100PinMCU_ESP32_TestBoard.kicad_sch (KiCad schematic)
At the start: 32 parts, among them J1 Conn_02x06_Odd_Even, J2 Conn_01x06, J3 Conn_01x02, J4 Conn_01x02

Commit message: footprints fixed actually
Parts:
- D1, D2, D3, D4, D5: footprint Diode_SMD:D_0603_1608Metric_Pad1.05x0.95mm_HandSolderDiode_SMD:D_0603_1608Metric_Pad1.05x0.95mm_HandSolder -> Diode_SMD:D_0603_1608Metric_Pad1.05x0.95mm_HandSolder
Other:
- moved on the sheet: D5, R8, TP5
Changed lines of the file:
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@@
 	)
 	(junction
-		(at 266.065 38.735)
+		(at 210.82 38.735)
 		(diameter 0)
 		(color 0 0 0 0)
@@
 	)
 	(junction
-		(at 266.065 24.765)
+		(at 210.82 24.765)
 		(diameter 0)
 		(color 0 0 0 0)
@@
 	(wire
 		(pts
-			(xy 266.065 38.735) (xy 266.065 43.815)
+			(xy 210.82 38.735) (xy 210.82 43.815)
 		)
 		(stroke
@@
 	(wire
 		(pts
-			(xy 266.065 21.59) (xy 266.065 24.765)
+			(xy 210.82 21.59) (xy 210.82 24.765)
 		)
 		(stroke
@@
 	(wire
 		(pts
-			(xy 266.065 46.355) (xy 266.065 48.895)
+			(xy 210.82 46.355) (xy 210.82 48.895)
 		)
 		(stroke
@@
 	(wire
 		(pts
-			(xy 266.065 34.925) (xy 266.065 38.735)
+			(xy 210.82 34.925) (xy 210.82 38.735)
 		)
 		(stroke
@@
 	(wire
 		(pts
-			(xy 266.065 24.765) (xy 266.065 27.305)
+			(xy 210.82 24.765) (xy 210.82 27.305)
 		)
 		(stroke
@@
 			)
 		)
-		(property "Footprint" "Diode_SMD:D_0603_1608Metric_Pad1.05x0.95mm_HandSolderDiode_SMD:D_0603_1608Metric_Pad1.05x0.95mm_HandSolder"
+		(property "Footprint" "Diode_SMD:D_0603_1608Metric_Pad1.05x0.95mm_HandSolder"
 			(at 80.645 174.625 0)
 			(effects
@@
 			)
 		)
-		(property "Footprint" "Diode_SMD:D_0603_1608Metric_Pad1.05x0.95mm_HandSolderDiode_SMD:D_0603_1608Metric_Pad1.05x0.95mm_HandSolder"
+		(property "Footprint" "Diode_SMD:D_0603_1608Metric_Pad1.05x0.95mm_HandSolder"
 			(at 50.8 174.625 0)
 			(effects
@@
 	(symbol
 		(lib_id "power:+3.3V")
-		(at 266.065 21.59 0)
+		(at 210.82 21.59 0)
 		(unit 1)
 		(exclude_from_sim no)
@@
 		(fields_autoplaced yes)
 		(property "Reference" "#PWR018"
-			(at 266.065 25.4 0)
+			(at 210.82 25.4 0)
 			(effects
 				(font
@@
 		)
 		(property "Value" "+3.3V"
-			(at 266.065 16.51 0)
+			(at 210.82 16.51 0)
 			(effects
 				(font
@@
 		)
 		(property "Footprint" ""
-			(at 266.065 21.59 0)
+			(at 210.82 21.59 0)
 			(effects
 				(font
@@
 		)
 		(property "Datasheet" ""
-			(at 266.065 21.59 0)
+			(at 210.82 21.59 0)
 			(effects
 				(font
@@
 		)
 		(property "Description" "Power symbol creates a global label with name \"+3.3V\""
-			(at 266.065 21.59 0)
+			(at 210.82 21.59 0)
 			(effects
 				(font
@@
 	(symbol
 		(lib_id "Device:R_US")
-		(at 266.065 31.115 0)
+		(at 210.82 31.115 0)
 		(mirror y)
 		(unit 1)
@@
 		(fields_autoplaced yes)
 		(property "Reference" "R8"
-			(at 267.97 29.8449 0)
+			(at 212.725 29.8449 0)
 			(effects
 				(font
@@
 		)
 		(property "Value" "1k"
-			(at 267.97 32.3849 0)
+			(at 212.725 32.3849 0)
 			(effects
 				(font
@@
 		)
 		(property "Footprint" "Resistor_SMD:R_0603_1608Metric_Pad0.98x0.95mm_HandSolder"
-			(at 265.049 31.369 90)
+			(at 209.804 31.369 90)
 			(effects
 				(font
@@
 		)
 		(property "Datasheet" "~"
-			(at 266.065 31.115 0)
+			(at 210.82 31.115 0)
 			(effects
 				(font
@@
 		)
 		(property "Description" "Resistor, US symbol"
-			(at 266.065 31.115 0)
+			(at 210.82 31.115 0)
 			(effects
 				(font
@@
 	(symbol
 		(lib_id "power:GND")
-		(at 266.065 48.895 0)
+		(at 210.82 48.895 0)
 		(mirror y)
 		(unit 1)
@@
 		(fields_autoplaced yes)
 		(property "Reference" "#PWR019"
-			(at 266.065 55.245 0)
+			(at 210.82 55.245 0)
 			(effects
 				(font
@@
 		)
 		(property "Value" "GND"
-			(at 266.065 53.975 0)
+			(at 210.82 53.975 0)
 			(effects
 				(font
@@
 		)
 		(property "Footprint" ""
-			(at 266.065 48.895 0)
+			(at 210.82 48.895 0)
 			(effects
 				(font
@@
 		)
 		(property "Datasheet" ""
-			(at 266.065 48.895 0)
+			(at 210.82 48.895 0)
 			(effects
 				(font
@@
 		)
 		(property "Description" "Power symbol creates a global label with name \"GND\" , ground"
-			(at 266.065 48.895 0)
+			(at 210.82 48.895 0)
 			(effects
 				(font
@@
 	(symbol
 		(lib_id "Connector:TestPoint")
-		(at 266.065 24.765 270)
+		(at 210.82 24.765 270)
 		(unit 1)
 		(exclude_from_sim no)
@@
 		(fields_autoplaced yes)
 		(property "Reference" "TP5"
-			(at 271.78 23.4949 90)
+			(at 216.535 23.4949 90)
 			(effects
 				(font
@@
 		)
 		(property "Value" "TestPoint"
-			(at 271.78 26.0349 90)
+			(at 216.535 26.0349 90)
 			(effects
 				(font
@@
 		)
 		(property "Footprint" "TestPoint:TestPoint_Loop_D1.80mm_Drill1.0mm_Beaded"
-			(at 266.065 29.845 0)
+			(at 210.82 29.845 0)
 			(effects
 				(font
@@
 		)
 		(property "Datasheet" "~"
-			(at 266.065 29.845 0)
+			(at 210.82 29.845 0)
 			(effects
 				(font
@@
 		)
 		(property "Description" "test point"
-			(at 266.065 24.765 0)
+			(at 210.82 24.765 0)
 			(effects
 				(font
@@
 			)
 		)
-		(property "Footprint" "Diode_SMD:D_0603_1608Metric_Pad1.05x0.95mm_HandSolderDiode_SMD:D_0603_1608Metric_Pad1.05x0.95mm_HandSolder"
+		(property "Footprint" "Diode_SMD:D_0603_1608Metric_Pad1.05x0.95mm_HandSolder"
 			(at 60.96 174.625 0)
 			(effects
@@
 			)
 		)
-		(property "Footprint" "Diode_SMD:D_0603_1608Metric_Pad1.05x0.95mm_HandSolderDiode_SMD:D_0603_1608Metric_Pad1.05x0.95mm_HandSolder"
+		(property "Footprint" "Diode_SMD:D_0603_1608Metric_Pad1.05x0.95mm_HandSolder"
 			(at 71.12 174.625 0)
 			(effects
@@
 	(symbol
 		(lib_id "Device:LED")
-		(at 266.065 42.545 270)
+		(at 210.82 42.545 270)
 		(mirror x)
 		(unit 1)
@@
 		(dnp no)
 		(property "Reference" "D5"
-			(at 261.366 38.227 0)
+			(at 206.121 38.227 0)
 			(effects
 				(font
@@
 		)
 		(property "Value" "LED"
-			(at 263.906 38.227 0)
+			(at 208.661 38.227 0)
 			(effects
 				(font
@@
 			)
 		)
-		(property "Footprint" "Diode_SMD:D_0603_1608Metric_Pad1.05x0.95mm_HandSolderDiode_SMD:D_0603_1608Metric_Pad1.05x0.95mm_HandSolder"
-			(at 266.065 42.545 0)
+		(property "Footprint" "Diode_SMD:D_0603_1608Metric_Pad1.05x0.95mm_HandSolder"
+			(at 210.82 42.545 0)
 			(effects
 				(font
@@
 		)
 		(property "Datasheet" "~"
-			(at 266.065 42.545 0)
+			(at 210.82 42.545 0)
 			(effects
 				(font
@@
 		)
 		(property "Description" "Light emitting diode"
-			(at 266.065 42.545 0)
+			(at 210.82 42.545 0)
 			(effects
 				(font
@@
 		)
 		(property "Sim.Pins" "1=K 2=A"
-			(at 266.065 42.545 0)
+			(at 210.82 42.545 0)
 			(effects
 				(font
