File: 100PinMCU_TestBoard/100PinMCU_ESP32_TestBoard/100PinMCU_ESP32_TestBoard.kicad_sch (KiCad schematic)
At the start: 32 parts, among them J1 Conn_02x06_Odd_Even, J2 Conn_01x06, J3 Conn_01x02, J4 Conn_01x02

Commit message: lakshay comments addressed footprint p/n in progress
Parts:
- removed J1: Conn_02x06_Odd_Even, Connector_PinHeader_2.54mm:PinHeader_2x06_P2.54mm_Vertical, symbol Connector_Generic:Conn_02x06_Odd_Even
- removed J3, J4: Conn_01x02, Connector_PinHeader_2.54mm:PinHeader_1x02_P2.54mm_Vertical, symbol Connector_Generic:Conn_01x02
- removed JP1, JP2, JP3, JP8: Jumper_2_Bridged, Jumper:SolderJumper-2_P1.3mm_Bridged2Bar_Pad1.0x1.5mm, symbol Jumper:Jumper_2_Bridged
- added C29: 10uF, Capacitor_SMD:C_0805_2012Metric, symbol Device:C
- added D16: D_Schottky, Diode_SMD:D_SOD-123, symbol Device:D_Schottky
- added D20: TPD2EUSB30DRTR, UTSVT_ICs:TPD2EUSB30DRTR, symbol USB_PD_Symbols:TPD2EUSB30DRTR
- added J3, J4: LogicAnalyzer, UTSVT_Connectors:CONN_SFH11-xxxC-D05-ST-XX_SUL, symbol utsvt_connectors:LogicAnalyzer
- added J7: USB_C_Receptacle_USB2.0_16P, UTSVT_Connectors:USB_C_Receptacle_GCT_USB4105-xx-A_16P_TopMnt_Horizontal, symbol UTSVT-Connectors:USB_C_Receptacle_USB2.0_16P
- added J8: Conn_01x04, symbol Connector_Generic:Conn_01x04
- added R26, R27: 5.1k, Resistor_SMD:R_0603_1608Metric_Pad0.98x0.95mm_HandSolder, symbol Device:R
- D1, D2, D3, D4, D5: LCSC P/N (none) -> C7371904
- JP4, JP5, JP6, JP7, JP9: footprint Jumper:SolderJumper-2_P1.3mm_Bridged2Bar_Pad1.0x1.5mm -> Connector_PinHeader_2.54mm:PinHeader_1x02_P2.54mm_Vertical
Connections:
- net FDCAN1_RX: now also J3.5 (CH5)
- net FDCAN1_TX: now also J3.6 (CH4)
- net GND: now also C29.1, D20.3 (GND), J3.1 (GND), J4.1 (GND), J7.A1 (GND), J7.A12 (GND), J7.B1 (GND), J7.B12 (GND), J7.S1 (SHIELD), J7.S2 (Shield), J7.S3 (Shield), J7.S4 (Shield), R26.1, R27.1
- net GPIO1: now also J3.4 (CH6)
- net I2C2_SCL: now also J3.9 (CH1)
- net I2C2_SDA: now also J3.10 (CH0)
- net SPI1_MISO: now also J4.9 (CH1)
- net SPI1_MOSI: now also J4.10 (CH0)
- net SPI1_NSS: now also J4.7 (CH3)
- net SPI1_SCK: now also J4.8 (CH2)
- net UART_RX: now also J3.7 (CH3)
- net UART_TX: now also J3.8 (CH2)
- new net CAN_H1: J8.1 (Pin_1)
- new net CAN_H2: J8.2 (Pin_2)
- new net CAN_L1: J8.3 (Pin_3)
- new net CAN_L2: J8.4 (Pin_4)
- new net CC1: J7.A5 (CC1), R26.2
- new net CC2: J7.B5 (CC2), R27.2
- new net D+: D20.1 (D+), J7.A6 (D+), J7.B6 (D+)
- new net D-: D20.2 (D-), J7.A7 (D-), J7.B7 (D-)
- new net GPIO2: J3.3 (CH7)
- new net VBUS: C29.2, D16.1 (K)
- new net VBUS_IN: D16.2 (A), J7.A4 (VBUS), J7.A9 (VBUS), J7.B4 (VBUS), J7.B9 (VBUS)
- no-connect marks 60 -> 53
Other:
- removed sheet USB_PD
- sheet 100PinMCU ports: added none; removed PC13, PC14-OSC32_IN, PC15-OSC32_OUT
- note added: "5.5V working 7V breakdown 8V clamping"
- note added: "Pulldowns for 5V USB-C PD"
- note added: "USB Protection"
- note added: "USB-C Port"
- note removed: "Logic Analyzer"
- moved on the sheet: D5, J2, JP10, R8, TP5
