File: 100PinMCU_TestBoard/100PinMCU_ESP32_TestBoard/ESP32.kicad_sch (KiCad schematic)
At the start: 21 parts, among them J5 USB_C_Receptacle_USB2.0_16P, SW1 BOOT Switch, SW2 RESET Button, U1 ESP32-C6-MINI-1

Commit message: footprints fixed actually
Parts:
- D9: footprint Diode_SMD:D_0603_1608Metric_Pad1.05x0.95mm_HandSolderDiode_SMD:D_0603_1608Metric_Pad1.05x0.95mm_HandSolder -> Diode_SMD:D_0603_1608Metric_Pad1.05x0.95mm_HandSolder
- J5: footprint utsvt_connectors:USB_C_Receptacle_GCT_USB4105-xx-A_16P_TopMnt_Horizontal -> UTSVT_Connectors:USB_C_Receptacle_GCT_USB4105-xx-A_16P_TopMnt_Horizontal
- SW1: footprint utsvt_esp32:450406020024 -> UTSVT_Esp32:450406020024
- SW2: footprint utsvt_esp32:TL3365AF180QG -> UTSVT_Esp32:TL3365AF180QG
- U1: footprint utsvt_special:ESP32-C6-MINI-1 -> RF_Module:ESP32-C6-MINI-1
Changed lines of the file:
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@@
 			)
 		)
-		(property "Footprint" "utsvt_special:ESP32-C6-MINI-1"
+		(property "Footprint" "RF_Module:ESP32-C6-MINI-1"
 			(at 158.75 78.74 0)
 			(effects
@@
 			)
 		)
-		(property "Footprint" "utsvt_esp32:TL3365AF180QG"
+		(property "Footprint" "UTSVT_Esp32:TL3365AF180QG"
 			(at 167.64 27.94 0)
 			(effects
@@
 			)
 		)
-		(property "Footprint" "utsvt_connectors:USB_C_Receptacle_GCT_USB4105-xx-A_16P_TopMnt_Horizontal"
+		(property "Footprint" "UTSVT_Connectors:USB_C_Receptacle_GCT_USB4105-xx-A_16P_TopMnt_Horizontal"
 			(at 35.56 87.63 0)
 			(effects
@@
 			)
 		)
-		(property "Footprint" "utsvt_esp32:450406020024"
+		(property "Footprint" "UTSVT_Esp32:450406020024"
 			(at 118.11 34.29 0)
 			(effects
@@
 			)
 		)
-		(property "Footprint" "Diode_SMD:D_0603_1608Metric_Pad1.05x0.95mm_HandSolderDiode_SMD:D_0603_1608Metric_Pad1.05x0.95mm_HandSolder"
+		(property "Footprint" "Diode_SMD:D_0603_1608Metric_Pad1.05x0.95mm_HandSolder"
 			(at 210.82 24.13 0)
 			(effects
