File: 100PinMCU_TestBoard/ESP32.kicad_sch (KiCad schematic)
At the start: 34 parts, among them J2 Conn_01x06, J3 LogicAnalyzer, J4 LogicAnalyzer, J7 USB_C_Receptacle_USB2.0_16P, J8 Conn_01x04

Commit message: pre japan flight
Parts:
- removed C29: 10uF, Capacitor_SMD:C_0805_2012Metric, symbol Device:C
- removed D1, D2, D3, D4, D5: LED, Diode_SMD:D_0603_1608Metric_Pad1.05x0.95mm_HandSolder, symbol Device:LED
- removed D16: D_Schottky, Diode_SMD:D_SOD-123, symbol Device:D_Schottky
- removed D20: TPD2EUSB30DRTR, UTSVT_ICs:TPD2EUSB30DRTR, symbol USB_PD_Symbols:TPD2EUSB30DRTR
- removed J2: Conn_01x06, Connector_PinHeader_2.54mm:PinHeader_1x06_P2.54mm_Vertical, symbol Connector_Generic:Conn_01x06
- removed J3, J4: LogicAnalyzer, UTSVT_Connectors:CONN_SFH11-xxxC-D05-ST-XX_SUL, symbol utsvt_connectors:LogicAnalyzer
- removed J7: USB_C_Receptacle_USB2.0_16P, UTSVT_Connectors:USB_C_Receptacle_GCT_USB4105-xx-A_16P_TopMnt_Horizontal, symbol UTSVT-Connectors:USB_C_Receptacle_USB2.0_16P
- removed J8: Conn_01x04, symbol Connector_Generic:Conn_01x04
- removed JP10: Jumper_2_Open, Jumper:SolderJumper-2_P1.3mm_Open_Pad1.0x1.5mm, symbol Jumper:Jumper_2_Open
- removed JP4, JP5, JP6, JP7, JP9: Jumper_2_Bridged, Connector_PinHeader_2.54mm:PinHeader_1x02_P2.54mm_Vertical, symbol Jumper:Jumper_2_Bridged
- removed R1, R2, R3, R4, R7, R8: 1k, Resistor_SMD:R_0603_1608Metric_Pad0.98x0.95mm_HandSolder, symbol Device:R_US
- removed R26, R27: 5.1k, Resistor_SMD:R_0603_1608Metric_Pad0.98x0.95mm_HandSolder, symbol Device:R
- removed R5, R6: 4.7k, Resistor_SMD:R_0603_1608Metric_Pad0.98x0.95mm_HandSolder, symbol Device:R_US
- removed TP1, TP2, TP3, TP4, TP5: TestPoint, TestPoint:TestPoint_Loop_D1.80mm_Drill1.0mm_Beaded, symbol Connector:TestPoint
- added C6, C7: 10uF, Capacitor_SMD:C_0805_2012Metric_Pad1.18x1.45mm_HandSolder, symbol Device:C
- added C8, C9: 0.1uF, Capacitor_SMD:C_0603_1608Metric_Pad1.08x0.95mm_HandSolder, symbol Device:C
- added D10: SP0503BAHT, Package_TO_SOT_SMD:SOT-143, symbol utsvt_ics:SP0503BAH
- added D11: ESP_PWR, Diode_SMD:D_0603_1608Metric_Pad1.05x0.95mm_HandSolder, symbol Device:LED
- added D12: ESP_LED1, Diode_SMD:D_0603_1608Metric_Pad1.05x0.95mm_HandSolder, symbol Device:LED
- added D13: ESP_LED2, Diode_SMD:D_0603_1608Metric_Pad1.05x0.95mm_HandSolder, symbol Device:LED
- added D9: 1N5819HW-7-F, Diode_SMD:D_SOD-123, symbol Device:D_Schottky
- added J6: USB_C_Receptacle_USB2.0_16P, UTSVT_Connectors:USB_C_Receptacle_GCT_USB4105-xx-A_16P_TopMnt_Horizontal, symbol utsvt_connectors:USB_C_Receptacle_USB2.0_16P
- added R13, R14: 5.1k, Resistor_SMD:R_0603_1608Metric_Pad0.98x0.95mm_HandSolder, symbol Device:R
- added R15, R16, R17: 10k, Resistor_SMD:R_0603_1608Metric_Pad0.98x0.95mm_HandSolder, symbol Device:R
- added R18, R19, R20: 1k, Resistor_SMD:R_0603_1608Metric_Pad0.98x0.95mm_HandSolder, symbol Device:R
- added SW1: BOOT Switch, UTSVT_Esp32:450406020024, symbol Switch:SW_SPDT
- added SW2: RESET Button, UTSVT_Esp32:TL3365AF180QG, symbol Switch:SW_Push
- added U1: ESP32-C6-MINI-1, RF_Module:ESP32-C6-MINI-1, symbol utsvt_special:ESP32-C6-MINI-1/U
Connections:
- net GND: now also C6.2, C9.2, D10.1 (A), D11.1 (K), D12.1 (K), D13.1 (K), J6.A1 (GND), J6.A12 (GND), J6.B1 (GND), J6.B12 (GND), J6.S1 (SHIELD), J6.S2 (Shield), J6.S3 (Shield), J6.S4 (Shield), R13.2, R14.2, SW1.3 (C), SW2.2, U1.1 (GND), U1.11 (GND), U1.14 (GND), U1.2 (GND), U1.36 (GND), U1.37 (GND), U1.38 (GND), U1.39 (GND), U1.40 (GND), U1.41 (GND), U1.42 (GND), U1.43 (GND), U1.44 (GND), U1.45 (GND), U1.46 (GND), U1.47 (GND), U1.48 (GND), U1.49 (GND), U1.50 (GND), U1.51 (GND), U1.52 (GND), U1.53 (GND)
- new net: D12.2 (A), R19.2
- new net: R17.1, U1.22 (GPIO8)
- new net: D13.2 (A), R20.2
- new net: R15.2, SW1.2 (B)
- new net: J6.B5 (CC2), R14.1
- new net: J6.A5 (CC1), R13.1
- new net: D11.2 (A), R18.2
- new net +3.3V_ESP: C7.1, C7.2, C8.1, C8.2, R16.1, R17.2, R18.1, SW1.1 (A), U1.3 (3V3)
- new net +5V_LDO_IN: C6.1, D9.1 (K)
- new net BOOT: R15.1, U1.23 (GPIO9)
- new net ESP_GPIO1: U1.19 (GPIO14)
- new net ESP_GPIO2: U1.20 (GPIO15)
- new net ESP_GPIO3: U1.24 (GPIO18)
- new net ESP_GPIO4: U1.25 (GPIO19)
- new net ESP_RESET: C9.1, R16.2, SW2.1, U1.8 (EN/CHIP_PU)
- new net ESP_UART_RX: U1.31 (U0TXD/GPIO16)
- new net ESP_UART_TX: U1.30 (U0RXD/GPIO17)
- new net LED1: R19.1, U1.26 (GPIO20)
- new net LED2: R20.1, U1.27 (GPIO21)
- new net USB_D+: D10.2 (K), J6.A6 (D+), J6.B6 (D+), U1.18 (GPIO13/USB_D+)
- new net USB_D-: D10.3 (K), J6.A7 (D-), J6.B7 (D-), U1.17 (GPIO12/USB_D-)
- new net VBUSB: D10.4 (K), D9.2 (A), J6.A4 (VBUS), J6.A9 (VBUS), J6.B4 (VBUS), J6.B9 (VBUS)
- no-connect marks 53 -> 12
Other:
- removed sheet 100PinMCU
- removed sheet CAN_Transceiver
- removed sheet CAN_Transceiver1
- removed sheet ESP32
- removed sheet LDO
- note added: "+3.3V turns it on normally"
- note added: "BOOT Switch"
- note added: "Connect this to a GPIO pin on the MCU THROUGH A RESISTOR to allow the MCU to reboot the ESP32"
- note added: "ESD Protection"
- note added: "ESP LEDs"
- note added: "ESP32 Design Block"
- note added: "From MUX design block"
- note added: "GND puts it in BOOT mode"
- note added: "MUX Power"
- note added: "Other notes: The GPIO can be used for whatever you like, but it is recommended you connect at least two to your MCU directly"
- note added: "Outside requirements: there must be an LDO and MUX design block on your schematic. The +5V_LDO_IN should be routed to the power input of the LDO design block. The output of that LDO, +3.3V_USB, should then be wired to one of the inputs of the MUX the other input to the MUX should be your main board +3.3V The output from this MUX must be routed back to the ESP design block as +3.3V_MUX_OUT input"
- note added: "README"
- note added: "RESET Button"
- note added: "THE UART LINES ARE MCU RELATIVE. READ THE NOTE BY THE UART LINES."
- note added: "The TX/RX lines are relative to MCU, so connect ESP_UART_RX to MCU's UART_RX and ESP_UART_TX to MCU's UART_TX"
- note added: "This block is used to integrate the ESP32 MCU for debugging/wireless communication purposes."
- note added: "USB Receptacle"
- note added: "USB_D+/- lines should be routed as differential pair (90 ohm impedance)"
- note added: "Wire to LDO design block"
- note removed: "5.5V working 7V breakdown 8V clamping"
- note removed: "Pulldowns for 5V USB-C PD"
- note removed: "USB Protection"
- note removed: "USB-C Port"
