File: 100PinMCU_TestBoard/ESP32.kicad_sch (KiCad schematic)
At the start: 21 parts, among them J10 USB_C_Receptacle_USB2.0_16P, SW3 BOOT Switch, SW4 RESET Button, U4 ESP32-C6-MINI-1

Commit message: erc
Parts:
- renumbered C30 to C1, C31 to C2, C32 to C3, C33 to C4, D22 to D10, D18 to D6, D19 to D7, D20 to D8, D21 to D9, J10 to J7, R30 to R11, R31 to R12, R32 to R13, R33 to R14, R34 to R15, R35 to R16, R36 to R17, R37 to R18, SW3 to SW1, SW4 to SW2, U4 to U1
Changed lines of the file:
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@@
 		(dnp no)
 		(fields_autoplaced yes)
-		(property "Reference" "R36"
+		(property "Reference" "R17"
 			(at 200.66 29.21 90)
 			(effects
@@
 			(project "100PinMCU_ESP32_TestBoard"
 				(path "/abcdaa41-14f3-4587-9aac-314b09095246/9d06ac8a-c506-4496-a533-5f4a7c9f87a1"
-					(reference "R36")
+					(reference "R17")
 					(unit 1)
 				)
@@
 		(on_board yes)
 		(dnp no)
-		(property "Reference" "C30"
+		(property "Reference" "C1"
 			(at 74.168 78.486 0)
 			(effects
@@
 			(project "100PinMCU_ESP32_TestBoard"
 				(path "/abcdaa41-14f3-4587-9aac-314b09095246/9d06ac8a-c506-4496-a533-5f4a7c9f87a1"
-					(reference "C30")
+					(reference "C1")
 					(unit 1)
 				)
@@
 		(dnp no)
 		(fields_autoplaced yes)
-		(property "Reference" "U4"
+		(property "Reference" "U1"
 			(at 158.3533 78.74 0)
 			(effects
@@
 			(project "100PinMCU_ESP32_TestBoard"
 				(path "/abcdaa41-14f3-4587-9aac-314b09095246/9d06ac8a-c506-4496-a533-5f4a7c9f87a1"
-					(reference "U4")
+					(reference "U1")
 					(unit 1)
 				)
@@
 		(on_board yes)
 		(dnp no)
-		(property "Reference" "C32"
+		(property "Reference" "C3"
 			(at 145.034 72.644 0)
 			(effects
@@
 			(project "100PinMCU_ESP32_TestBoard"
 				(path "/abcdaa41-14f3-4587-9aac-314b09095246/9d06ac8a-c506-4496-a533-5f4a7c9f87a1"
-					(reference "C32")
+					(reference "C3")
 					(unit 1)
 				)
@@
 		(dnp no)
 		(fields_autoplaced yes)
-		(property "Reference" "D19"
+		(property "Reference" "D7"
 			(at 74.93 135.89 90)
 			(effects
@@
 			(project "100PinMCU_ESP32_TestBoard"
 				(path "/abcdaa41-14f3-4587-9aac-314b09095246/9d06ac8a-c506-4496-a533-5f4a7c9f87a1"
-					(reference "D19")
+					(reference "D7")
 					(unit 1)
 				)
@@
 		(dnp no)
 		(fields_autoplaced yes)
-		(property "Reference" "#PWR033"
+		(property "Reference" "#PWR022"
 			(at 127 33.02 0)
 			(effects
@@
 			(project "100PinMCU_ESP32_TestBoard"
 				(path "/abcdaa41-14f3-4587-9aac-314b09095246/9d06ac8a-c506-4496-a533-5f4a7c9f87a1"
-					(reference "#PWR033")
+					(reference "#PWR022")
 					(unit 1)
 				)
@@
 		(on_board yes)
 		(dnp no)
-		(property "Reference" "#PWR032"
+		(property "Reference" "#PWR021"
 			(at 43.18 146.05 0)
 			(effects
@@
 			(project "100PinMCU_ESP32_TestBoard"
 				(path "/abcdaa41-14f3-4587-9aac-314b09095246/9d06ac8a-c506-4496-a533-5f4a7c9f87a1"
-					(reference "#PWR032")
+					(reference "#PWR021")
 					(unit 1)
 				)
@@
 		(on_board yes)
 		(dnp no)
-		(property "Reference" "R37"
+		(property "Reference" "R18"
 			(at 200.66 42.418 90)
 			(effects
@@
 			(project "100PinMCU_ESP32_TestBoard"
 				(path "/abcdaa41-14f3-4587-9aac-314b09095246/9d06ac8a-c506-4496-a533-5f4a7c9f87a1"
-					(reference "R37")
+					(reference "R18")
 					(unit 1)
 				)
@@
 		(on_board yes)
 		(dnp no)
-		(property "Reference" "C31"
+		(property "Reference" "C2"
 			(at 135.636 72.644 0)
 			(effects
@@
 			(project "100PinMCU_ESP32_TestBoard"
 				(path "/abcdaa41-14f3-4587-9aac-314b09095246/9d06ac8a-c506-4496-a533-5f4a7c9f87a1"
-					(reference "C31")
+					(reference "C2")
 					(unit 1)
 				)
@@
 		(on_board yes)
 		(dnp no)
-		(property "Reference" "D22"
+		(property "Reference" "D10"
 			(at 211.074 42.164 0)
 			(effects
@@
 			(project "100PinMCU_ESP32_TestBoard"
 				(path "/abcdaa41-14f3-4587-9aac-314b09095246/9d06ac8a-c506-4496-a533-5f4a7c9f87a1"
-					(reference "D22")
+					(reference "D10")
 					(unit 1)
 				)
@@
 		(on_board yes)
 		(dnp no)
-		(property "Reference" "SW4"
+		(property "Reference" "SW2"
 			(at 167.64 26.416 0)
 			(effects
@@
 			(project "100PinMCU_ESP32_TestBoard"
 				(path "/abcdaa41-14f3-4587-9aac-314b09095246/9d06ac8a-c506-4496-a533-5f4a7c9f87a1"
-					(reference "SW4")
+					(reference "SW2")
 					(unit 1)
 				)
@@
 		(on_board yes)
 		(dnp no)
-		(property "Reference" "R34"
+		(property "Reference" "R15"
 			(at 197.104 101.854 90)
 			(effects
@@
 			(project "100PinMCU_ESP32_TestBoard"
 				(path "/abcdaa41-14f3-4587-9aac-314b09095246/9d06ac8a-c506-4496-a533-5f4a7c9f87a1"
-					(reference "R34")
+					(reference "R15")
 					(unit 1)
 				)
@@
 		(dnp no)
 		(fields_autoplaced yes)
-		(property "Reference" "R32"
+		(property "Reference" "R13"
 			(at 107.95 29.21 90)
 			(effects
@@
 			(project "100PinMCU_ESP32_TestBoard"
 				(path "/abcdaa41-14f3-4587-9aac-314b09095246/9d06ac8a-c506-4496-a533-5f4a7c9f87a1"
-					(reference "R32")
+					(reference "R13")
 					(unit 1)
 				)
@@
 		(on_board yes)
 		(dnp no)
-		(property "Reference" "#PWR036"
+		(property "Reference" "#PWR025"
 			(at 189.23 25.4 0)
 			(effects
@@
 			(project "100PinMCU_ESP32_TestBoard"
 				(path "/abcdaa41-14f3-4587-9aac-314b09095246/9d06ac8a-c506-4496-a533-5f4a7c9f87a1"
-					(reference "#PWR036")
+					(reference "#PWR025")
 					(unit 1)
 				)
@@
 		(on_board yes)
 		(dnp no)
-		(property "Reference" "R31"
+		(property "Reference" "R12"
 			(at 50.038 81.28 90)
 			(effects
@@
 			(project "100PinMCU_ESP32_TestBoard"
 				(path "/abcdaa41-14f3-4587-9aac-314b09095246/9d06ac8a-c506-4496-a533-5f4a7c9f87a1"
-					(reference "R31")
+					(reference "R12")
 					(unit 1)
 				)
@@
 		(on_board yes)
 		(dnp no)
-		(property "Reference" "R33"
+		(property "Reference" "R14"
 			(at 151.384 25.654 0)
 			(effects
@@
 			(project "100PinMCU_ESP32_TestBoard"
 				(path "/abcdaa41-14f3-4587-9aac-314b09095246/9d06ac8a-c506-4496-a533-5f4a7c9f87a1"
-					(reference "R33")
+					(reference "R14")
 					(unit 1)
 				)
@@
 		(dnp no)
 		(fields_autoplaced yes)
-		(property "Reference" "#PWR034"
+		(property "Reference" "#PWR023"
 			(at 156.21 72.39 0)
 			(effects
@@
 			(project "100PinMCU_ESP32_TestBoard"
 				(path "/abcdaa41-14f3-4587-9aac-314b09095246/9d06ac8a-c506-4496-a533-5f4a7c9f87a1"
-					(reference "#PWR034")
+					(reference "#PWR023")
 					(unit 1)
 				)
@@
 		(on_board yes)
 		(dnp no)
-		(property "Reference" "D18"
+		(property "Reference" "D6"
 			(at 61.722 66.04 0)
 			(effects
@@
 			(project "100PinMCU_ESP32_TestBoard"
 				(path "/abcdaa41-14f3-4587-9aac-314b09095246/9d06ac8a-c506-4496-a533-5f4a7c9f87a1"
-					(reference "D18")
+					(reference "D6")
 					(unit 1)
 				)
@@
 		(on_board yes)
 		(dnp no)
-		(property "Reference" "C33"
+		(property "Reference" "C4"
 			(at 153.924 35.814 0)
 			(effects
@@
 			(project "100PinMCU_ESP32_TestBoard"
 				(path "/abcdaa41-14f3-4587-9aac-314b09095246/9d06ac8a-c506-4496-a533-5f4a7c9f87a1"
-					(reference "C33")
+					(reference "C4")
 					(unit 1)
 				)
@@
 		(on_board yes)
 		(dnp no)
-		(property "Reference" "R30"
+		(property "Reference" "R11"
 			(at 50.292 76.2 90)
 			(effects
@@
 			(project "100PinMCU_ESP32_TestBoard"
 				(path "/abcdaa41-14f3-4587-9aac-314b09095246/9d06ac8a-c506-4496-a533-5f4a7c9f87a1"
-					(reference "R30")
+					(reference "R11")
 					(unit 1)
 				)
@@
 		(dnp no)
 		(fields_autoplaced yes)
-		(property "Reference" "J10"
+		(property "Reference" "J7"
 			(at 31.75 64.77 0)
 			(effects
@@
 			(project "100PinMCU_ESP32_TestBoard"
 				(path "/abcdaa41-14f3-4587-9aac-314b09095246/9d06ac8a-c506-4496-a533-5f4a7c9f87a1"
-					(reference "J10")
+					(reference "J7")
 					(unit 1)
 				)
@@
 		(on_board yes)
 		(dnp no)
-		(property "Reference" "D21"
+		(property "Reference" "D9"
 			(at 210.82 27.94 0)
 			(effects
@@
 			(project "100PinMCU_ESP32_TestBoard"
 				(path "/abcdaa41-14f3-4587-9aac-314b09095246/9d06ac8a-c506-4496-a533-5f4a7c9f87a1"
-					(reference "D21")
+					(reference "D9")
 					(unit 1)
 				)
@@
 		(on_board yes)
 		(dnp no)
-		(property "Reference" "SW3"
+		(property "Reference" "SW1"
 			(at 117.348 26.416 0)
 			(effects
@@
 			(project "100PinMCU_ESP32_TestBoard"
 				(path "/abcdaa41-14f3-4587-9aac-314b09095246/9d06ac8a-c506-4496-a533-5f4a7c9f87a1"
-					(reference "SW3")
+					(reference "SW1")
 					(unit 1)
 				)
@@
 		(dnp no)
 		(fields_autoplaced yes)
-		(property "Reference" "R35"
+		(property "Reference" "R16"
 			(at 200.66 19.05 90)
 			(effects
@@
 			(project "100PinMCU_ESP32_TestBoard"
 				(path "/abcdaa41-14f3-4587-9aac-314b09095246/9d06ac8a-c506-4496-a533-5f4a7c9f87a1"
-					(reference "R35")
+					(reference "R16")
 					(unit 1)
 				)
@@
 		(on_board yes)
 		(dnp no)
-		(property "Reference" "D20"
+		(property "Reference" "D8"
 			(at 210.82 17.78 0)
 			(effects
@@
 			(project "100PinMCU_ESP32_TestBoard"
 				(path "/abcdaa41-14f3-4587-9aac-314b09095246/9d06ac8a-c506-4496-a533-5f4a7c9f87a1"
-					(reference "D20")
+					(reference "D8")
 					(unit 1)
 				)
@@
 		(on_board yes)
 		(dnp no)
-		(property "Reference" "#PWR037"
+		(property "Reference" "#PWR026"
 			(at 208.28 109.22 0)
 			(effects
@@
 			(project "100PinMCU_ESP32_TestBoard"
 				(path "/abcdaa41-14f3-4587-9aac-314b09095246/9d06ac8a-c506-4496-a533-5f4a7c9f87a1"
-					(reference "#PWR037")
+					(reference "#PWR026")
 					(unit 1)
 				)
@@
 		(dnp no)
 		(fields_autoplaced yes)
-		(property "Reference" "#PWR035"
+		(property "Reference" "#PWR024"
 			(at 157.48 26.67 0)
 			(effects
@@
 			(project "100PinMCU_ESP32_TestBoard"
 				(path "/abcdaa41-14f3-4587-9aac-314b09095246/9d06ac8a-c506-4496-a533-5f4a7c9f87a1"
-					(reference "#PWR035")
-					(unit 1)
-				)
+					(reference "#PWR024")
+					(unit 1)
+				)

Commit message: mcu layout
Connections:
- net +3.3V_ESP: no longer C2.2, C3.2
- net GND: now also C2.2, C3.2
Changed lines of the file:
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@@
-	)
-	(junction
-		(at 156.21 80.01)
-		(diameter 0)
-		(color 0 0 0 0)
 	)
 	(junction
@@
 	)
 	(junction
-		(at 148.59 80.01)
-		(diameter 0)
-		(color 0 0 0 0)
-	)
-	(junction
 		(at 71.12 72.39)
 		(diameter 0)
@@
 		(color 0 0 0 0)
 	)
+	(junction
+		(at 139.7 81.28)
+		(diameter 0)
+		(color 0 0 0 0)
+	)
 	(no_connect
 		(at 184.15 129.54)
@@
 	(wire
 		(pts
-			(xy 156.21 80.01) (xy 156.21 69.85)
-		)
-		(stroke
-			(width 0)
-			(type default)
-		)
-	)
-	(wire
-		(pts
 			(xy 148.59 69.85) (xy 148.59 71.12)
 		)
@@
 	(wire
 		(pts
-			(xy 139.7 80.01) (xy 139.7 78.74)
+			(xy 139.7 78.74) (xy 139.7 81.28)
 		)
 		(stroke
@@
 	(wire
 		(pts
+			(xy 139.7 81.28) (xy 148.59 81.28)
+		)
+		(stroke
+			(width 0)
+			(type default)
+		)
+	)
+	(wire
+		(pts
 			(xy 31.75 110.49) (xy 31.75 111.76)
 		)
@@
 	(wire
 		(pts
-			(xy 139.7 80.01) (xy 148.59 80.01)
-		)
-		(stroke
-			(width 0)
-			(type default)
-		)
-	)
-	(wire
-		(pts
 			(xy 48.26 92.71) (xy 46.99 92.71)
 		)
@@
 	(wire
 		(pts
-			(xy 148.59 80.01) (xy 156.21 80.01)
-		)
-		(stroke
-			(width 0)
-			(type default)
-		)
-	)
-	(wire
-		(pts
 			(xy 218.44 39.37) (xy 218.44 40.64)
 		)
@@
 	(wire
 		(pts
+			(xy 137.16 81.28) (xy 139.7 81.28)
+		)
+		(stroke
+			(width 0)
+			(type default)
+		)
+	)
+	(wire
+		(pts
 			(xy 43.18 142.24) (xy 43.18 146.05)
 		)
@@
 	(wire
 		(pts
-			(xy 148.59 78.74) (xy 148.59 80.01)
+			(xy 148.59 78.74) (xy 148.59 81.28)
 		)
 		(stroke
@@
 	(wire
 		(pts
-			(xy 156.21 80.01) (xy 156.21 81.28)
+			(xy 156.21 69.85) (xy 156.21 81.28)
 		)
 		(stroke
@@
 		(effects
 			(font
+				(size 1.27 1.27)
+			)
+			(justify right)
+		)
+	)
+	(hierarchical_label "GND"
+		(shape input)
+		(at 137.16 81.28 180)
+		(effects
+			(font

Commit message: schem fixes + some semblance of layout ish
Parts:
- D6: value 1N5819HW-7-F -> D_Schottky; Mouser Part Number (none) -> 1N5819HW-7-F; P/N 1N5819HW-7-F -> BAT760-7
Changed lines of the file:
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@@
+	)
+	(symbol
+		(lib_id "Device:D_Schottky")
+		(at 60.96 72.39 0)
+		(mirror y)
+		(unit 1)
+		(exclude_from_sim no)
+		(in_bom yes)
+		(on_board yes)
+		(dnp no)
+		(property "Reference" "D6"
+			(at 60.96 69.85 0)
+			(effects
+				(font
+					(size 1.27 1.27)
+				)
+			)
+		)
+		(property "Value" "D_Schottky"
+			(at 60.96 67.31 0)
+			(effects
+				(font
+					(size 1.27 1.27)
+				)
+			)
+		)
+		(property "Footprint" "Diode_SMD:D_SOD-123"
+			(at 60.96 72.39 0)
+			(effects
+				(font
+					(size 1.27 1.27)
+				)
+				(hide yes)
+			)
+		)
+		(property "Datasheet" "~"
+			(at 60.96 72.39 0)
+			(effects
+				(font
+					(size 1.27 1.27)
+				)
+				(hide yes)
+			)
+		)
+		(property "Description" "Schottky diode"
+			(at 60.96 72.39 0)
+			(effects
+				(font
+					(size 1.27 1.27)
+				)
+				(hide yes)
+			)
+		)
+		(property "P/N" "BAT760-7"
+			(at 60.96 72.39 0)
+			(effects
+				(font
+					(size 1.27 1.27)
+				)
+				(hide yes)
+			)
+		)
+		(property "Sim.Type" ""
+			(at 60.96 72.39 0)
+			(effects
+				(font
+					(size 1.27 1.27)
+				)
+				(hide yes)
+			)
+		)
+		(property "Inventory" ""
+			(at 60.96 72.39 0)
+			(effects
+				(font
+					(size 1.27 1.27)
+				)
+				(hide yes)
+			)
+		)
+		(property "Color" ""
+			(at 60.96 72.39 0)
+			(effects
+				(font
+					(size 1.27 1.27)
+				)
+			)
+		)
+		(property "If" ""
+			(at 60.96 72.39 0)
+			(effects
+				(font
+					(size 1.27 1.27)
+				)
+			)
+		)
+		(property "Mfg" ""
+			(at 60.96 72.39 0)
+			(effects
+				(font
+					(size 1.27 1.27)
+				)
+			)
+		)
+		(property "Vf" ""
+			(at 60.96 72.39 0)
+			(effects
+				(font
+					(size 1.27 1.27)
+				)
+			)
+		)
+		(property "Mouser Part Number" "1N5819HW-7-F"
+			(at 60.96 72.39 0)
+			(effects
+				(font
+					(size 1.27 1.27)
+				)
+				(hide yes)
+			)
+		)
+		(property "LCSC P/N" "C82544"
+			(at 60.96 72.39 0)
+			(effects
+				(font
+					(size 1.27 1.27)
+				)
+				(hide yes)
+			)
+		)
+		(pin "2"
+		)
+		(pin "1"
+		)
+		(instances
+			(project "100PinMCU_ESP32_TestBoard"
+				(path "/abcdaa41-14f3-4587-9aac-314b09095246/9d06ac8a-c506-4496-a533-5f4a7c9f87a1"
+					(reference "D6")
+					(unit 1)
+				)
+			)
+		)
 	)
 	(symbol
@@
 					(unit 1)
 				)
-			)
-		)
-	)
-	(symbol
-		(lib_id "Device:D_Schottky")
-		(at 60.96 72.39 180)
-		(unit 1)
-		(exclude_from_sim no)
-		(in_bom yes)
-		(on_board yes)
-		(dnp no)
-		(property "Reference" "D6"
-			(at 61.722 66.04 0)
-			(effects
-				(font
-					(size 1.27 1.27)
-				)
-			)
-		)
-		(property "Value" "1N5819HW-7-F"
-			(at 61.722 68.58 0)
-			(effects
-				(font
-					(size 1.27 1.27)
-				)
-			)
-		)
-		(property "Footprint" "Diode_SMD:D_SOD-123"
-			(at 60.96 72.39 0)
-			(effects
-				(font
-					(size 1.27 1.27)
-				)
-				(hide yes)
-			)
-		)
-		(property "Datasheet" "kicad-embed://DIOD-S-A0011683586-1.pdf"
-			(at 60.96 72.39 0)
-			(effects
-				(font
-					(size 1.27 1.27)
-				)
-				(hide yes)
-			)
-		)
-		(property "Description" "Schottky diode"
-			(at 60.96 72.39 0)
-			(effects
-				(font
-					(size 1.27 1.27)
-				)
-				(hide yes)
-			)
-		)
-		(property "P/N" "1N5819HW-7-F"
-			(at 60.96 72.39 0)
-			(effects
-				(font
-					(size 1.27 1.27)
-				)
-				(hide yes)
-			)
-		)
-		(property "LCSC P/N" "C82544"
-			(at 60.96 72.39 0)
-			(effects
-				(font
-					(size 1.27 1.27)
-				)
-				(hide yes)
-			)
-		)
-		(pin "2"
-		)
-		(pin "1"
-		)
-		(instances
-			(project "100PinMCU_ESP32_TestBoard"
-				(path "/abcdaa41-14f3-4587-9aac-314b09095246/9d06ac8a-c506-4496-a533-5f4a7c9f87a1"
-					(reference "D6")
-					(unit 1)
-				)

Commit message: more layout but me go sleep now
Parts:
- removed D7: SP0503BAHT, Package_TO_SOT_SMD:SOT-143, symbol utsvt_ics:SP0503BAH
- added D7: TPD2EUSB30DRTR, UTSVT_ICs:TPD2EUSB30DRTR, symbol USB_PD_Symbols:TPD2EUSB30DRTR
Connections:
- net GND: now also D7.3 (GND)
- net USB_D+: now also D7.2 (D-)
- net USB_D-: now also D7.1 (D+)
Other:
- note added: "5.5V working 7V breakdown 8V clamping"
Changed lines of the file:
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@@
+		)
+	)
+	(text "5.5V working\n7V breakdown\n8V clamping"
+		(exclude_from_sim no)
+		(at 71.12 148.59 0)
+		(effects
+			(font
+				(size 1.27 1.27)
+				(thickness 0.1588)
+			)
+			(justify left top)
 		)
 	)
@@
 	(wire
 		(pts
-			(xy 80.01 144.78) (xy 83.82 144.78)
+			(xy 57.15 144.78) (xy 64.77 144.78)
 		)
 		(stroke
@@
 	(wire
 		(pts
-			(xy 60.96 144.78) (xy 69.85 144.78)
-		)
-		(stroke
-			(width 0)
-			(type default)
-		)
-	)
-	(wire
-		(pts
 			(xy 175.26 33.02) (xy 175.26 38.1)
 		)
@@
 	(wire
 		(pts
-			(xy 60.96 147.32) (xy 69.85 147.32)
-		)
-		(stroke
-			(width 0)
-			(type default)
-		)
-	)
-	(wire
-		(pts
 			(xy 184.15 114.3) (xy 196.85 114.3)
 		)
@@
 	(wire
 		(pts
-			(xy 60.96 142.24) (xy 69.85 142.24)
-		)
-		(stroke
-			(width 0)
-			(type default)
-		)
-	)
-	(wire
-		(pts
 			(xy 142.24 33.02) (xy 157.48 33.02)
 		)
@@
 	(wire
 		(pts
+			(xy 90.17 142.24) (xy 92.71 142.24)
+		)
+		(stroke
+			(width 0)
+			(type default)
+		)
+	)
+	(wire
+		(pts
 			(xy 139.7 71.12) (xy 139.7 69.85)
 		)
@@
 	(wire
 		(pts
-			(xy 83.82 144.78) (xy 83.82 148.59)
-		)
-		(stroke
-			(width 0)
-			(type default)
-		)
-	)
-	(wire
-		(pts
 			(xy 184.15 111.76) (xy 196.85 111.76)
 		)
@@
 		(pts
 			(xy 48.26 92.71) (xy 46.99 92.71)
+		)
+		(stroke
+			(width 0)
+			(type default)
+		)
+	)
+	(wire
+		(pts
+			(xy 57.15 142.24) (xy 64.77 142.24)
 		)
 		(stroke
@@
 		)
 	)
+	(label "USB_D+"
+		(at 57.15 144.78 0)
+		(effects
+			(font
+				(size 1.27 1.27)
+			)
+			(justify left bottom)
+		)
+	)
 	(label "BOOT"
 		(at 97.79 34.29 0)
@@
 		)
 	)
-	(label "USB_D+"
-		(at 60.96 147.32 0)
+	(label "USB_D-"
+		(at 57.15 142.24 0)
 		(effects
 			(font
@@
 		)
 	)
-	(label "USB_D-"
-		(at 60.96 144.78 0)
-		(effects
-			(font
-				(size 1.27 1.27)
-			)
-			(justify left bottom)
-		)
-	)
 	(label "ESP_RESET"
 		(at 142.24 33.02 0)
@@
 			)
 			(justify right bottom)
-		)
-	)
-	(label "VBUSB"
-		(at 60.96 142.24 0)
-		(effects
-			(font
-				(size 1.27 1.27)
-			)
-			(justify left bottom)
 		)
 	)
@@
 		)
 	)
+	(hierarchical_label "GND"
+		(shape input)
+		(at 92.71 142.24 270)
+		(effects
+			(font
+				(size 1.27 1.27)
+			)
+			(justify right)
+		)
+	)
 	(hierarchical_label "ESP_GPIO4"
 		(shape bidirectional)
@@
 		(shape input)
 		(at 218.44 26.67 270)
-		(effects
-			(font
-				(size 1.27 1.27)
-			)
-			(justify right)
-		)
-	)
-	(hierarchical_label "GND"
-		(shape input)
-		(at 83.82 148.59 270)
 		(effects
 			(font
@@
 	)
 	(symbol
-		(lib_id "utsvt_ics:SP0503BAH")
-		(at 74.93 144.78 90)
-		(unit 1)
-		(exclude_from_sim no)
-		(in_bom yes)
-		(on_board yes)
-		(dnp no)
-		(fields_autoplaced yes)
-		(property "Reference" "D7"
-			(at 74.93 135.89 90)
-			(effects
-				(font
-					(size 1.27 1.27)
-				)
-			)
-		)
-		(property "Value" "SP0503BAHT"
-			(at 74.93 138.43 90)
-			(effects
-				(font
-					(size 1.27 1.27)
-				)
-			)
-		)
-		(property "Footprint" "Package_TO_SOT_SMD:SOT-143"
-			(at 76.2 139.065 0)
-			(effects
-				(font
-					(size 1.27 1.27)
-				)
-				(justify left)
-				(hide yes)
-			)
-		)
-		(property "Datasheet" "kicad-embed://Littelfuse-TVS-Diode-Array-SP05-Datasheet.pdf"
-			(at 71.755 141.605 0)
-			(effects
-				(font
-					(size 1.27 1.27)
-				)
-				(hide yes)
-			)
-		)
-		(property "Description" ""
-			(at 74.93 144.78 0)
-			(effects
-				(font
-					(size 1.27 1.27)
-				)
-				(hide yes)
-			)
-		)
-		(property "Mouser Part Number" "576-SP0503BAHTG "
-			(at 74.93 144.78 0)
-			(effects
-				(font
-					(size 1.27 1.27)
-				)
-				(hide yes)
-			)
-		)
-		(property "P/N" "SP0503BAHTG"
-			(at 74.93 144.78 0)
-			(effects
-				(font
-					(size 1.27 1.27)
-				)
-				(hide yes)
-			)
-		)
-		(property "LCSC P/N" "C7074"
-			(at 74.93 144.78 90)
-			(effects
-				(font
-					(size 1.27 1.27)
-				)
-				(hide yes)
-			)
-		)
-		(pin "3"
-		)
-		(pin "4"
-		)
-		(pin "1"
-		)
-		(pin "2"
-		)
-		(instances
-			(project "100PinMCU_ESP32_TestBoard"
-				(path "/abcdaa41-14f3-4587-9aac-314b09095246/9d06ac8a-c506-4496-a533-5f4a7c9f87a1"
-					(reference "D7")
-					(unit 1)
-				)
-			)
-		)
-	)
-	(symbol
 		(lib_id "power:+3.3V")
 		(at 127 29.21 0)
@@
 					(unit 1)
 				)
+			)
+		)
+	)
+	(symbol
+		(lib_id "USB_PD_Symbols:TPD2EUSB30DRTR")
+		(at 64.77 142.24 0)
+		(unit 1)
+		(exclude_from_sim no)
+		(in_bom yes)
+		(on_board yes)
+		(dnp no)
+		(fields_autoplaced yes)
+		(property "Reference" "D7"
+			(at 77.47 134.62 0)
+			(effects
+				(font
+					(size 1.27 1.27)
+				)
+			)
+		)
+		(property "Value" "TPD2EUSB30DRTR"
+			(at 77.47 137.16 0)
+			(effects
+				(font
+					(size 1.27 1.27)
+				)
+			)
+		)
+		(property "Footprint" "UTSVT_ICs:TPD2EUSB30DRTR"
+			(at 86.36 237.16 0)
+			(effects
+				(font
+					(size 1.27 1.27)
+				)
+				(justify left top)
+				(hide yes)
+			)
+		)
+		(property "Datasheet" "kicad-embed://sf-000234749.pdf"
+			(at 86.36 337.16 0)
+			(effects
+				(font
+					(size 1.27 1.27)
+				)
+				(justify left top)
+				(hide yes)
+			)
+		)
+		(property "Description" "Texas Instruments TPD2EUSB30DRTR Dual Bi-Directional TVS Diode Array, 45W peak, 3-Pin SOT"
+			(at 64.77 142.24 0)
+			(effects
+				(font
+					(size 1.27 1.27)
+				)
+				(hide yes)
+			)
+		)
+		(property "Height" "0.5"
+			(at 86.36 537.16 0)
+			(effects
+				(font
+					(size 1.27 1.27)
+				)
+				(justify left top)
+				(hide yes)
+			)
+		)
+		(property "Mouser Part Number" "595-TPD2EUSB30DRTR"
+			(at 86.36 637.16 0)
+			(effects
+				(font
+					(size 1.27 1.27)
+				)
+				(justify left top)
+				(hide yes)
+			)
+		)
+		(property "Mouser Price/Stock" "https://www.mouser.co.uk/ProductDetail/Texas-Instruments/TPD2EUSB30DRTR?qs=%2Fqzd9s%252BcLd6bPJi5HXCDvw%3D%3D"
+			(at 86.36 737.16 0)
+			(effects
+				(font
+					(size 1.27 1.27)
+				)
+				(justify left top)
+				(hide yes)
+			)
+		)
+		(property "Manufacturer_Name" "Texas Instruments"
+			(at 86.36 837.16 0)
+			(effects
+				(font
+					(size 1.27 1.27)
+				)
+				(justify left top)
+				(hide yes)
+			)
+		)
+		(property "P/N" "TPD2EUSB30DRTR"
+			(at 86.36 937.16 0)
+			(effects
+				(font
+					(size 1.27 1.27)
+				)
+				(justify left top)
+				(hide yes)
+			)
+		)
+		(property "LCSC P/N" "C97502"
+			(at 64.77 142.24 0)
+			(effects
+				(font
+					(size 1.27 1.27)
+				)
+				(hide yes)
+			)
+		)
+		(pin "2"
+		)
+		(pin "1"
+		)
+		(pin "3"
+		)
+		(instances
+			(project "100PinMCU_ESP32_TestBoard"
+				(path "/abcdaa41-14f3-4587-9aac-314b09095246/9d06ac8a-c506-4496-a533-5f4a7c9f87a1"
+					(reference "D7")
+					(unit 1)
+				)

Commit message: she's an onion now
Connections:
- net USB_D+: now also D7.1 (D+); no longer D7.2 (D-)
- net USB_D-: now also D7.2 (D-); no longer D7.1 (D+)
Changed lines of the file:
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@@
-		)
-	)
-	(label "USB_D+"
-		(at 57.15 144.78 0)
-		(effects
-			(font
-				(size 1.27 1.27)
-			)
-			(justify left bottom)
 		)
 	)
@@
 		)
 	)
-	(label "USB_D-"
-		(at 57.15 142.24 0)
-		(effects
-			(font
-				(size 1.27 1.27)
-			)
-			(justify left bottom)
-		)
-	)
 	(label "LED1"
 		(at 194.31 121.92 180)
@@
 			)
 			(justify right bottom)
+		)
+	)
+	(label "USB_D+"
+		(at 57.15 142.24 0)
+		(effects
+			(font
+				(size 1.27 1.27)
+			)
+			(justify left bottom)
 		)
 	)
@@
 		)
 	)
+	(label "USB_D-"
+		(at 57.15 144.78 0)
+		(effects
+			(font
+				(size 1.27 1.27)
+			)
+			(justify left bottom)
+		)
+	)
