File: 100PinMCU_TestBoard/100PinMCU_ESP32_TestBoard.kicad_sch (KiCad schematic)
At the start: 34 parts, among them J1 LogicAnalyzer, J2 LogicAnalyzer, J3 ADC_Breakout, J5 USB_C_Receptacle_USB2.0_16P, J8 CAN_Breakout

Commit message: pre board
Parts:
- J8: footprint (none) -> Connector_PinHeader_2.54mm:PinHeader_1x04_P2.54mm_Vertical
Changed lines of the file:
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@@
 			)
 		)
-		(property "Footprint" ""
+		(property "Footprint" "Connector_PinHeader_2.54mm:PinHeader_1x04_P2.54mm_Vertical"
 			(at 33.655 168.91 0)
 			(effects
