File: 100PinMCU_TestBoard/100PinMCU_ESP32_TestBoard.kicad_sch (KiCad schematic)
At the start: 32 parts, among them J1 LogicAnalyzer_1, J2 LogicAnalyzer_2, J3 CAN_Breakout, J4 ADC_Breakout, J5 CAN_2, J6 CAN_1

Commit message: erc
Parts:
- renumbered D7 to D2, D2 to D3, D3 to D4, D4 to D5, J4 to J1, J1 to J2, J6 to J3, J5 to J4, J2 to J5, J3 to J6, JP8 to JP5, JP9 to JP7, R15 to R1, R7 to R10, R16 to R2, R5 to R4, R12 to R5, R4 to R6, R9 to R7, R6 to R9, TP4 to TP1, TP5 to TP2, TP2 to TP3, TP3 to TP4
Connections:
- no-connect marks 46 -> 50
