File: 100PinMCU_TestBoard/USB-C.kicad_sch (KiCad schematic)
At the start: 6 parts, among them J7 USB_C_Receptacle_USB2.0_16P

Commit message: erc
Parts:
- renumbered C1 to C29, D5 to D16, D6 to D17, J7 to J9, R10 to R28, R11 to R29
Changed lines of the file:
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@@
 		(on_board yes)
 		(dnp no)
-		(property "Reference" "D6"
+		(property "Reference" "D17"
 			(at 59.69 28.575 0)
 			(effects
@@
 			(project "100PinMCU_ESP32_TestBoard"
 				(path "/abcdaa41-14f3-4587-9aac-314b09095246/941bc526-dbd8-4c9d-9757-597be17aacce"
-					(reference "D6")
+					(reference "D17")
 					(unit 1)
 				)
@@
 		(on_board yes)
 		(dnp no)
-		(property "Reference" "J7"
+		(property "Reference" "J9"
 			(at 71.374 26.924 0)
 			(effects
@@
 			(project "100PinMCU_ESP32_TestBoard"
 				(path "/abcdaa41-14f3-4587-9aac-314b09095246/941bc526-dbd8-4c9d-9757-597be17aacce"
-					(reference "J7")
+					(reference "J9")
 					(unit 1)
 				)
@@
 		(dnp no)
 		(fields_autoplaced yes)
-		(property "Reference" "#PWR025"
+		(property "Reference" "#PWR031"
 			(at 87.63 79.375 0)
 			(effects
@@
 			(project "100PinMCU_ESP32_TestBoard"
 				(path "/abcdaa41-14f3-4587-9aac-314b09095246/941bc526-dbd8-4c9d-9757-597be17aacce"
-					(reference "#PWR025")
+					(reference "#PWR031")
 					(unit 1)
 				)
@@
 		(on_board yes)
 		(dnp no)
-		(property "Reference" "R10"
+		(property "Reference" "R28"
 			(at 33.274 52.07 90)
 			(effects
@@
 			(project "100PinMCU_ESP32_TestBoard"
 				(path "/abcdaa41-14f3-4587-9aac-314b09095246/941bc526-dbd8-4c9d-9757-597be17aacce"
-					(reference "R10")
+					(reference "R28")
 					(unit 1)
 				)
@@
 		(dnp no)
 		(fields_autoplaced yes)
-		(property "Reference" "D5"
+		(property "Reference" "D16"
 			(at 43.18 74.93 0)
 			(effects
@@
 			(project "100PinMCU_ESP32_TestBoard"
 				(path "/abcdaa41-14f3-4587-9aac-314b09095246/941bc526-dbd8-4c9d-9757-597be17aacce"
-					(reference "D5")
+					(reference "D16")
 					(unit 1)
 				)
@@
 		(on_board yes)
 		(dnp no)
-		(property "Reference" "#PWR019"
+		(property "Reference" "#PWR028"
 			(at 37.465 62.865 0)
 			(effects
@@
 			(project "100PinMCU_ESP32_TestBoard"
 				(path "/abcdaa41-14f3-4587-9aac-314b09095246/941bc526-dbd8-4c9d-9757-597be17aacce"
-					(reference "#PWR019")
+					(reference "#PWR028")
 					(unit 1)
 				)
@@
 		(on_board yes)
 		(dnp no)
-		(property "Reference" "R11"
+		(property "Reference" "R29"
 			(at 41.529 52.07 90)
 			(effects
@@
 			(project "100PinMCU_ESP32_TestBoard"
 				(path "/abcdaa41-14f3-4587-9aac-314b09095246/941bc526-dbd8-4c9d-9757-597be17aacce"
-					(reference "R11")
+					(reference "R29")
 					(unit 1)
 				)
@@
 		(on_board yes)
 		(dnp no)
-		(property "Reference" "#PWR021"
+		(property "Reference" "#PWR030"
 			(at 58.42 91.44 0)
 			(effects
@@
 			(project "100PinMCU_ESP32_TestBoard"
 				(path "/abcdaa41-14f3-4587-9aac-314b09095246/941bc526-dbd8-4c9d-9757-597be17aacce"
-					(reference "#PWR021")
+					(reference "#PWR030")
 					(unit 1)
 				)
@@
 		(on_board yes)
 		(dnp no)
-		(property "Reference" "#PWR020"
+		(property "Reference" "#PWR029"
 			(at 53.34 50.165 0)
 			(effects
@@
 			(project "100PinMCU_ESP32_TestBoard"
 				(path "/abcdaa41-14f3-4587-9aac-314b09095246/941bc526-dbd8-4c9d-9757-597be17aacce"
-					(reference "#PWR020")
+					(reference "#PWR029")
 					(unit 1)
 				)
@@
 		(on_board yes)
 		(dnp no)
-		(property "Reference" "#PWR018"
+		(property "Reference" "#PWR027"
 			(at 29.21 62.865 0)
 			(effects
@@
 			(project "100PinMCU_ESP32_TestBoard"
 				(path "/abcdaa41-14f3-4587-9aac-314b09095246/941bc526-dbd8-4c9d-9757-597be17aacce"
-					(reference "#PWR018")
+					(reference "#PWR027")
 					(unit 1)
 				)
@@
 		(on_board yes)
 		(dnp no)
-		(property "Reference" "C1"
+		(property "Reference" "C29"
 			(at 56.3372 41.1734 0)
 			(effects
@@
 			(project "100PinMCU_ESP32_TestBoard"
 				(path "/abcdaa41-14f3-4587-9aac-314b09095246/941bc526-dbd8-4c9d-9757-597be17aacce"
-					(reference "C1")
+					(reference "C29")
 					(unit 1)
 				)
