File: 100PinMCU_TestBoard/Power_Mux.kicad_sch (KiCad schematic)
At the start: 6 parts, among them U1 TPS2117DRLR

Commit message: erc
Parts:
- renumbered C1 to C30, C2 to C31, C3 to C32, C4 to C33, R1 to R30, U1 to U4
Changed lines of the file:
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@@
 		(on_board yes)
 		(dnp no)
-		(property "Reference" "C4"
+		(property "Reference" "C33"
 			(at 91.8972 57.2516 0)
 			(effects
@@
 			(project "power-mux-block"
 				(path "/abcdaa41-14f3-4587-9aac-314b09095246/8bbc384d-f945-48c6-90d4-966a04218661"
-					(reference "C4")
+					(reference "C33")
 					(unit 1)
 				)
@@
 		(on_board yes)
 		(dnp no)
-		(property "Reference" "R1"
+		(property "Reference" "R30"
 			(at 78.994 67.564 0)
 			(effects
@@
 			(project "power-mux-block"
 				(path "/abcdaa41-14f3-4587-9aac-314b09095246/8bbc384d-f945-48c6-90d4-966a04218661"
-					(reference "R1")
+					(reference "R30")
 					(unit 1)
 				)
@@
 		(on_board yes)
 		(dnp no)
-		(property "Reference" "C1"
+		(property "Reference" "C30"
 			(at 24.5872 44.5516 0)
 			(effects
@@
 			(project "power-mux-block"
 				(path "/abcdaa41-14f3-4587-9aac-314b09095246/8bbc384d-f945-48c6-90d4-966a04218661"
-					(reference "C1")
+					(reference "C30")
 					(unit 1)
 				)
@@
 		(dnp no)
 		(fields_autoplaced yes)
-		(property "Reference" "U1"
+		(property "Reference" "U4"
 			(at 60.96 44.45 0)
 			(effects
@@
 			(project ""
 				(path "/abcdaa41-14f3-4587-9aac-314b09095246/8bbc384d-f945-48c6-90d4-966a04218661"
-					(reference "U1")
+					(reference "U4")
 					(unit 1)
 				)
@@
 		(on_board yes)
 		(dnp no)
-		(property "Reference" "C3"
+		(property "Reference" "C32"
 			(at 42.3672 67.4116 0)
 			(effects
@@
 			(project "power-mux-block"
 				(path "/abcdaa41-14f3-4587-9aac-314b09095246/8bbc384d-f945-48c6-90d4-966a04218661"
-					(reference "C3")
+					(reference "C32")
 					(unit 1)
 				)
@@
 		(on_board yes)
 		(dnp no)
-		(property "Reference" "C2"
+		(property "Reference" "C31"
 			(at 38.5572 44.5516 0)
 			(effects
@@
 			(project "power-mux-block"
 				(path "/abcdaa41-14f3-4587-9aac-314b09095246/8bbc384d-f945-48c6-90d4-966a04218661"
-					(reference "C2")
-					(unit 1)
-				)
+					(reference "C31")
+					(unit 1)
+				)

Commit message: clark
Parts:
- U4: footprint pretty:TPS2117DRLR -> UTSVT_Power:TPS2117DRLR
Changed lines of the file:
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@@
 			)
 		)
-		(property "Footprint" "pretty:TPS2117DRLR"
+		(property "Footprint" "UTSVT_Power:TPS2117DRLR"
 			(at 60.96 62.23 0)
 			(effects
