File: 100PinMCU_TestBoard/100PinMCU.kicad_sch (KiCad schematic)
At the start: 28 parts, among them J1 SWD_Header_02x02, U2 STM32G491VET6, Y1 Crystal

Commit message: pre japan flight
Parts:
- renumbered C1 to C16, C2 to C17, C14 to C18, C3 to C19, C9 to C20, C4 to C21, C10 to C22, C5 to C23, C12 to C24, C6 to C25, C13 to C26, C7 to C27, C8 to C28, C11 to C29, D2 to D16, D1 to D17, FB2 to FB1, FB1 to FB2, J1 to J7, R4 to R23, R5 to R24, R1 to R25, R3 to R26, R2 to R27, U2 to U3
Changed lines of the file:
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@@
 		(dnp no)
 		(fields_autoplaced yes)
-		(property "Reference" "C12"
+		(property "Reference" "C24"
 			(at 213.995 60.9599 0)
 			(effects
@@
 			(project "PS-100PinMCU"
 				(path "/abcdaa41-14f3-4587-9aac-314b09095246/840885ae-57ff-4136-b869-7c6178ab9d24"
-					(reference "C12")
+					(reference "C24")
 					(unit 1)
 				)
@@
 		(dnp no)
 		(fields_autoplaced yes)
-		(property "Reference" "R1"
+		(property "Reference" "R25"
 			(at 182.245 105.4099 0)
 			(effects
@@
 			(project "PS-100PinMCU"
 				(path "/abcdaa41-14f3-4587-9aac-314b09095246/840885ae-57ff-4136-b869-7c6178ab9d24"
-					(reference "R1")
+					(reference "R25")
 					(unit 1)
 				)
@@
 		(dnp no)
 		(fields_autoplaced yes)
-		(property "Reference" "U2"
+		(property "Reference" "U3"
 			(at 93.345 28.575 0)
 			(effects
@@
 			(project ""
 				(path "/abcdaa41-14f3-4587-9aac-314b09095246/840885ae-57ff-4136-b869-7c6178ab9d24"
-					(reference "U2")
+					(reference "U3")
 					(unit 1)
 				)
@@
 		(dnp no)
 		(fields_autoplaced yes)
-		(property "Reference" "R2"
+		(property "Reference" "R27"
 			(at 234.95 114.9349 0)
 			(effects
@@
 			(project "PS-100PinMCU"
 				(path "/abcdaa41-14f3-4587-9aac-314b09095246/840885ae-57ff-4136-b869-7c6178ab9d24"
-					(reference "R2")
+					(reference "R27")
 					(unit 1)
 				)
@@
 		(dnp no)
 		(fields_autoplaced yes)
-		(property "Reference" "R4"
+		(property "Reference" "R23"
 			(at 138.43 21.59 90)
 			(effects
@@
 			(project ""
 				(path "/abcdaa41-14f3-4587-9aac-314b09095246/840885ae-57ff-4136-b869-7c6178ab9d24"
-					(reference "R4")
+					(reference "R23")
 					(unit 1)
 				)
@@
 		(dnp no)
 		(fields_autoplaced yes)
-		(property "Reference" "C10"
+		(property "Reference" "C22"
 			(at 199.39 60.9599 0)
 			(effects
@@
 			(project "PS-100PinMCU"
 				(path "/abcdaa41-14f3-4587-9aac-314b09095246/840885ae-57ff-4136-b869-7c6178ab9d24"
-					(reference "C10")
+					(reference "C22")
 					(unit 1)
 				)
@@
 		(on_board yes)
 		(dnp no)
-		(property "Reference" "R5"
+		(property "Reference" "R24"
 			(at 138.43 33.02 90)
 			(effects
@@
 			(project ""
 				(path "/abcdaa41-14f3-4587-9aac-314b09095246/840885ae-57ff-4136-b869-7c6178ab9d24"
-					(reference "R5")
+					(reference "R24")
 					(unit 1)
 				)
@@
 		(dnp no)
 		(fields_autoplaced yes)
-		(property "Reference" "C4"
+		(property "Reference" "C21"
 			(at 194.31 35.5599 0)
 			(effects
@@
 			(project "PS-100PinMCU"
 				(path "/abcdaa41-14f3-4587-9aac-314b09095246/840885ae-57ff-4136-b869-7c6178ab9d24"
-					(reference "C4")
+					(reference "C21")
 					(unit 1)
 				)
@@
 		(dnp no)
 		(fields_autoplaced yes)
-		(property "Reference" "C9"
+		(property "Reference" "C20"
 			(at 184.15 60.9599 0)
 			(effects
@@
 			(project "PS-100PinMCU"
 				(path "/abcdaa41-14f3-4587-9aac-314b09095246/840885ae-57ff-4136-b869-7c6178ab9d24"
-					(reference "C9")
+					(reference "C20")
 					(unit 1)
 				)
@@
 		(on_board yes)
 		(dnp no)
-		(property "Reference" "R3"
+		(property "Reference" "R26"
 			(at 225.806 94.996 90)
 			(effects
@@
 			(project "PS-100PinMCU"
 				(path "/abcdaa41-14f3-4587-9aac-314b09095246/840885ae-57ff-4136-b869-7c6178ab9d24"
-					(reference "R3")
+					(reference "R26")
 					(unit 1)
 				)
@@
 		(dnp no)
 		(fields_autoplaced yes)
-		(property "Reference" "C1"
+		(property "Reference" "C16"
 			(at 33.655 46.3549 0)
 			(effects
@@
 			(project ""
 				(path "/abcdaa41-14f3-4587-9aac-314b09095246/840885ae-57ff-4136-b869-7c6178ab9d24"
-					(reference "C1")
+					(reference "C16")
 					(unit 1)
 				)
@@
 		(dnp no)
 		(fields_autoplaced yes)
-		(property "Reference" "C6"
+		(property "Reference" "C25"
 			(at 219.71 35.5599 0)
 			(effects
@@
 			(project "PS-100PinMCU"
 				(path "/abcdaa41-14f3-4587-9aac-314b09095246/840885ae-57ff-4136-b869-7c6178ab9d24"
-					(reference "C6")
+					(reference "C25")
 					(unit 1)
 				)
@@
 		(dnp no)
 		(fields_autoplaced yes)
-		(property "Reference" "C7"
+		(property "Reference" "C27"
 			(at 232.41 35.5599 0)
 			(effects
@@
 			(project "PS-100PinMCU"
 				(path "/abcdaa41-14f3-4587-9aac-314b09095246/840885ae-57ff-4136-b869-7c6178ab9d24"
-					(reference "C7")
+					(reference "C27")
 					(unit 1)
 				)
@@
 		(dnp no)
 		(fields_autoplaced yes)
-		(property "Reference" "C2"
+		(property "Reference" "C17"
 			(at 46.355 46.3549 0)
 			(effects
@@
 			(project ""
 				(path "/abcdaa41-14f3-4587-9aac-314b09095246/840885ae-57ff-4136-b869-7c6178ab9d24"
-					(reference "C2")
+					(reference "C17")
 					(unit 1)
 				)
@@
 		(dnp no)
 		(fields_autoplaced yes)
-		(property "Reference" "D1"
+		(property "Reference" "D17"
 			(at 247.015 109.2199 90)
 			(effects
@@
 			(project "PS-100PinMCU"
 				(path "/abcdaa41-14f3-4587-9aac-314b09095246/840885ae-57ff-4136-b869-7c6178ab9d24"
-					(reference "D1")
+					(reference "D17")
 					(unit 1)
 				)
@@
 		(on_board yes)
 		(dnp no)
-		(property "Reference" "FB2"
+		(property "Reference" "FB1"
 			(at 101.092 188.595 90)
 			(effects
@@
 			(project "PS-100PinMCU"
 				(path "/abcdaa41-14f3-4587-9aac-314b09095246/840885ae-57ff-4136-b869-7c6178ab9d24"
-					(reference "FB2")
+					(reference "FB1")
 					(unit 1)
 				)
@@
 		(dnp no)
 		(fields_autoplaced yes)
-		(property "Reference" "C3"
+		(property "Reference" "C19"
 			(at 183.515 35.5599 0)
 			(effects
@@
 			(project "PS-100PinMCU"
 				(path "/abcdaa41-14f3-4587-9aac-314b09095246/840885ae-57ff-4136-b869-7c6178ab9d24"
-					(reference "C3")
+					(reference "C19")
 					(unit 1)
 				)
@@
 		(dnp no)
 		(fields_autoplaced yes)
-		(property "Reference" "D2"
+		(property "Reference" "D16"
 			(at 236.22 105.0924 90)
 			(effects
@@
 			(project "PS-100PinMCU"
 				(path "/abcdaa41-14f3-4587-9aac-314b09095246/840885ae-57ff-4136-b869-7c6178ab9d24"
-					(reference "D2")
+					(reference "D16")
 					(unit 1)
 				)
@@
 		(on_board yes)
 		(dnp no)
-		(property "Reference" "J1"
+		(property "Reference" "J7"
 			(at 156.718 16.002 0)
 			(effects
@@
 			(project ""
 				(path "/abcdaa41-14f3-4587-9aac-314b09095246/840885ae-57ff-4136-b869-7c6178ab9d24"
-					(reference "J1")
+					(reference "J7")
 					(unit 1)
 				)
@@
 		(dnp no)
 		(fields_autoplaced yes)
-		(property "Reference" "C13"
+		(property "Reference" "C26"
 			(at 229.235 60.9599 0)
 			(effects
@@
 			(project "PS-100PinMCU"
 				(path "/abcdaa41-14f3-4587-9aac-314b09095246/840885ae-57ff-4136-b869-7c6178ab9d24"
-					(reference "C13")
+					(reference "C26")
 					(unit 1)
 				)
@@
 		(dnp no)
 		(fields_autoplaced yes)
-		(property "Reference" "FB1"
+		(property "Reference" "FB2"
 			(at 259.6642 48.895 90)
 			(effects
@@
 			(project ""
 				(path "/abcdaa41-14f3-4587-9aac-314b09095246/840885ae-57ff-4136-b869-7c6178ab9d24"
-					(reference "FB1")
+					(reference "FB2")
 					(unit 1)
 				)
@@
 		(on_board yes)
 		(dnp no)
-		(property "Reference" "C14"
+		(property "Reference" "C18"
 			(at 182.626 115.6716 0)
 			(effects
@@
 			(project "PS-100PinMCU"
 				(path "/abcdaa41-14f3-4587-9aac-314b09095246/840885ae-57ff-4136-b869-7c6178ab9d24"
-					(reference "C14")
+					(reference "C18")
 					(unit 1)
 				)
@@
 		(dnp no)
 		(fields_autoplaced yes)
-		(property "Reference" "C11"
+		(property "Reference" "C29"
 			(at 269.24 62.2299 0)
 			(effects
@@
 			(project "PS-100PinMCU"
 				(path "/abcdaa41-14f3-4587-9aac-314b09095246/840885ae-57ff-4136-b869-7c6178ab9d24"
-					(reference "C11")
+					(reference "C29")
 					(unit 1)
 				)
@@
 		(dnp no)
 		(fields_autoplaced yes)
-		(property "Reference" "C5"
+		(property "Reference" "C23"
 			(at 207.01 35.5599 0)
 			(effects
@@
 			(project "PS-100PinMCU"
 				(path "/abcdaa41-14f3-4587-9aac-314b09095246/840885ae-57ff-4136-b869-7c6178ab9d24"
-					(reference "C5")
+					(reference "C23")
 					(unit 1)
 				)
@@
 		(on_board yes)
 		(dnp no)
-		(property "Reference" "C8"
+		(property "Reference" "C28"
 			(at 245.237 35.433 0)
 			(effects
@@
 			(project "PS-100PinMCU"
 				(path "/abcdaa41-14f3-4587-9aac-314b09095246/840885ae-57ff-4136-b869-7c6178ab9d24"
-					(reference "C8")
+					(reference "C28")
 					(unit 1)
 				)

Commit message: pre board
Parts:
- D16: footprint (none) -> Diode_SMD:D_0603_1608Metric_Pad1.05x0.95mm_HandSolder
- FB1, FB2: footprint (none) -> Inductor_SMD:L_0603_1608Metric_Pad1.05x0.95mm_HandSolder
- J7: footprint 878320406:CONN04_878320406_MOL -> UTSVT_Connectors:CONN04_878320406_MOL
- R23, R24, R27: footprint (none) -> Resistor_SMD:R_0603_1608Metric_Pad0.98x0.95mm_HandSolder
- Reset1: footprint TL3365AF180QG:TL3365AF180QG -> UTSVT_Esp32:TL3365AF180QG
- S1: footprint 450406020024:450406020024 -> UTSVT_Esp32:450406020024
- U3: footprint LQFP_491VET6_STM:LQFP_491VET6_STM -> UTSVT_ICs:LQFP_491VET6_STM
Changed lines of the file:
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@@
 			)
 		)
-		(property "Footprint" "LQFP_491VET6_STM:LQFP_491VET6_STM"
+		(property "Footprint" "UTSVT_ICs:LQFP_491VET6_STM"
 			(at 57.785 38.735 0)
 			(effects
@@
 			)
 		)
-		(property "Footprint" ""
+		(property "Footprint" "Resistor_SMD:R_0603_1608Metric_Pad0.98x0.95mm_HandSolder"
 			(at 233.426 116.459 90)
 			(effects
@@
 			)
 		)
-		(property "Footprint" ""
+		(property "Footprint" "Resistor_SMD:R_0603_1608Metric_Pad0.98x0.95mm_HandSolder"
 			(at 138.684 28.321 90)
 			(effects
@@
 			)
 		)
-		(property "Footprint" ""
+		(property "Footprint" "Resistor_SMD:R_0603_1608Metric_Pad0.98x0.95mm_HandSolder"
 			(at 138.684 30.861 90)
 			(effects
@@
 			)
 		)
-		(property "Footprint" ""
+		(property "Footprint" "Inductor_SMD:L_0603_1608Metric_Pad1.05x0.95mm_HandSolder"
 			(at 98.425 187.833 90)
 			(effects
@@
 			)
 		)
-		(property "Footprint" ""
+		(property "Footprint" "Diode_SMD:D_0603_1608Metric_Pad1.05x0.95mm_HandSolder"
 			(at 232.41 104.775 0)
 			(effects
@@
 			)
 		)
-		(property "Footprint" "878320406:CONN04_878320406_MOL"
+		(property "Footprint" "UTSVT_Connectors:CONN04_878320406_MOL"
 			(at 156.845 22.225 0)
 			(effects
@@
 			)
 		)
-		(property "Footprint" ""
+		(property "Footprint" "Inductor_SMD:L_0603_1608Metric_Pad1.05x0.95mm_HandSolder"
 			(at 259.715 57.658 90)
 			(effects
@@
 			)
 		)
-		(property "Footprint" "450406020024:450406020024"
+		(property "Footprint" "UTSVT_Esp32:450406020024"
 			(at 280.035 4.14 0)
 			(effects
@@
 			)
 		)
-		(property "Footprint" "TL3365AF180QG:TL3365AF180QG"
+		(property "Footprint" "UTSVT_Esp32:TL3365AF180QG"
 			(at 197.485 115.57 0)
 			(effects

Commit message: add mux
Parts:
- renumbered J7 to J9, R23 to R25, R24 to R26, R25 to R27, R26 to R28, R27 to R29
Changed lines of the file:
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@@
 		(dnp no)
 		(fields_autoplaced yes)
-		(property "Reference" "R25"
+		(property "Reference" "R27"
 			(at 182.245 105.4099 0)
 			(effects
@@
 			(project "PS-100PinMCU"
 				(path "/abcdaa41-14f3-4587-9aac-314b09095246/840885ae-57ff-4136-b869-7c6178ab9d24"
-					(reference "R25")
+					(reference "R27")
 					(unit 1)
 				)
@@
 		(dnp no)
 		(fields_autoplaced yes)
-		(property "Reference" "R27"
+		(property "Reference" "R29"
 			(at 234.95 114.9349 0)
 			(effects
@@
 			(project "PS-100PinMCU"
 				(path "/abcdaa41-14f3-4587-9aac-314b09095246/840885ae-57ff-4136-b869-7c6178ab9d24"
-					(reference "R27")
+					(reference "R29")
 					(unit 1)
 				)
@@
 		(dnp no)
 		(fields_autoplaced yes)
-		(property "Reference" "R23"
+		(property "Reference" "R25"
 			(at 138.43 21.59 90)
 			(effects
@@
 			(project ""
 				(path "/abcdaa41-14f3-4587-9aac-314b09095246/840885ae-57ff-4136-b869-7c6178ab9d24"
-					(reference "R23")
+					(reference "R25")
 					(unit 1)
 				)
@@
 		(on_board yes)
 		(dnp no)
-		(property "Reference" "R24"
+		(property "Reference" "R26"
 			(at 138.43 33.02 90)
 			(effects
@@
 			(project ""
 				(path "/abcdaa41-14f3-4587-9aac-314b09095246/840885ae-57ff-4136-b869-7c6178ab9d24"
-					(reference "R24")
+					(reference "R26")
 					(unit 1)
 				)
@@
 		(on_board yes)
 		(dnp no)
-		(property "Reference" "R26"
+		(property "Reference" "R28"
 			(at 225.806 94.996 90)
 			(effects
@@
 			(project "PS-100PinMCU"
 				(path "/abcdaa41-14f3-4587-9aac-314b09095246/840885ae-57ff-4136-b869-7c6178ab9d24"
-					(reference "R26")
+					(reference "R28")
 					(unit 1)
 				)
@@
 		(on_board yes)
 		(dnp no)
-		(property "Reference" "J7"
+		(property "Reference" "J9"
 			(at 156.718 16.002 0)
 			(effects
@@
 			(project ""
 				(path "/abcdaa41-14f3-4587-9aac-314b09095246/840885ae-57ff-4136-b869-7c6178ab9d24"
-					(reference "J7")
-					(unit 1)
-				)
+					(reference "J9")
+					(unit 1)
+				)

Commit message: save before laptop dies
Parts:
- R25, R26, R27, R28, R29: symbol Device:R_US -> Device:R
Changed lines of the file:
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@@
 	)
 	(symbol
-		(lib_id "Device:R_US")
+		(lib_id "Device:R")
 		(at 179.705 106.68 180)
 		(unit 1)
@@
 		(fields_autoplaced yes)
 		(property "Reference" "R27"
-			(at 182.245 105.4099 0)
+			(at 181.61 105.4099 0)
 			(effects
 				(font
@@
 		)
 		(property "Value" "10k"
-			(at 182.245 107.9499 0)
+			(at 181.61 107.9499 0)
 			(effects
 				(font
@@
 		)
 		(property "Footprint" "Resistor_SMD:R_0603_1608Metric_Pad0.98x0.95mm_HandSolder"
-			(at 178.689 106.426 90)
+			(at 181.483 106.68 90)
 			(effects
 				(font
@@
 			)
 		)
-		(property "Description" "Resistor, US symbol"
+		(property "Description" "Resistor"
 			(at 179.705 106.68 0)
 			(effects
@@
 	)
 	(symbol
-		(lib_id "Device:R_US")
+		(lib_id "Device:R")
 		(at 232.41 116.205 0)
 		(unit 1)
@@
 		)
 		(property "Footprint" "Resistor_SMD:R_0603_1608Metric_Pad0.98x0.95mm_HandSolder"
-			(at 233.426 116.459 90)
+			(at 230.632 116.205 90)
 			(effects
 				(font
@@
 			)
 		)
-		(property "Description" "Resistor, US symbol"
+		(property "Description" "Resistor"
 			(at 232.41 116.205 0)
 			(effects
@@
 	)
 	(symbol
-		(lib_id "Device:R_US")
+		(lib_id "Device:R")
 		(at 138.43 27.305 90)
 		(mirror x)
@@
 		)
 		(property "Footprint" "Resistor_SMD:R_0603_1608Metric_Pad0.98x0.95mm_HandSolder"
-			(at 138.684 28.321 90)
+			(at 138.43 25.527 90)
 			(effects
 				(font
@@
 			)
 		)
-		(property "Description" "Resistor, US symbol"
+		(property "Description" "Resistor"
 			(at 138.43 27.305 0)
 			(effects
@@
 	)
 	(symbol
-		(lib_id "Device:R_US")
+		(lib_id "Device:R")
 		(at 138.43 29.845 90)
 		(mirror x)
@@
 		)
 		(property "Footprint" "Resistor_SMD:R_0603_1608Metric_Pad0.98x0.95mm_HandSolder"
-			(at 138.684 30.861 90)
+			(at 138.43 28.067 90)
 			(effects
 				(font
@@
 			)
 		)
-		(property "Description" "Resistor, US symbol"
+		(property "Description" "Resistor"
 			(at 138.43 29.845 0)
 			(effects
@@
 	)
 	(symbol
-		(lib_id "Device:R_US")
+		(lib_id "Device:R")
 		(at 226.695 99.06 90)
 		(mirror x)
@@
 		)
 		(property "Footprint" "Resistor_SMD:R_0603_1608Metric_Pad0.98x0.95mm_HandSolder"
-			(at 226.949 100.076 90)
+			(at 226.695 97.282 90)
 			(effects
 				(font
@@
 			)
 		)
-		(property "Description" "Resistor, US symbol"
+		(property "Description" "Resistor"
 			(at 226.695 99.06 0)
 			(effects

Commit message: erc
Parts:
- renumbered C16 to C15, C17 to C16, C18 to C17, C19 to C18, C20 to C19, C21 to C20, C22 to C21, C23 to C22, C24 to C23, C25 to C24, C26 to C25, C27 to C26, C28 to C27, C29 to C28, D16 to D14, D17 to D15, J9 to J8, R25 to R23, R26 to R24, R27 to R25, R28 to R26, R29 to R27
Changed lines of the file:
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@@
 		(dnp no)
 		(fields_autoplaced yes)
-		(property "Reference" "C24"
+		(property "Reference" "C23"
 			(at 213.995 60.9599 0)
 			(effects
@@
 			(project "PS-100PinMCU"
 				(path "/abcdaa41-14f3-4587-9aac-314b09095246/840885ae-57ff-4136-b869-7c6178ab9d24"
-					(reference "C24")
+					(reference "C23")
 					(unit 1)
 				)
@@
 		(dnp no)
 		(fields_autoplaced yes)
-		(property "Reference" "R27"
+		(property "Reference" "R25"
 			(at 181.61 105.4099 0)
 			(effects
@@
 			(project "PS-100PinMCU"
 				(path "/abcdaa41-14f3-4587-9aac-314b09095246/840885ae-57ff-4136-b869-7c6178ab9d24"
-					(reference "R27")
+					(reference "R25")
 					(unit 1)
 				)
@@
 		(dnp no)
 		(fields_autoplaced yes)
-		(property "Reference" "R29"
+		(property "Reference" "R27"
 			(at 234.95 114.9349 0)
 			(effects
@@
 			(project "PS-100PinMCU"
 				(path "/abcdaa41-14f3-4587-9aac-314b09095246/840885ae-57ff-4136-b869-7c6178ab9d24"
-					(reference "R29")
+					(reference "R27")
 					(unit 1)
 				)
@@
 		(dnp no)
 		(fields_autoplaced yes)
-		(property "Reference" "R25"
+		(property "Reference" "R23"
 			(at 138.43 21.59 90)
 			(effects
@@
 			(project ""
 				(path "/abcdaa41-14f3-4587-9aac-314b09095246/840885ae-57ff-4136-b869-7c6178ab9d24"
-					(reference "R25")
+					(reference "R23")
 					(unit 1)
 				)
@@
 		(dnp no)
 		(fields_autoplaced yes)
-		(property "Reference" "C22"
+		(property "Reference" "C21"
 			(at 199.39 60.9599 0)
 			(effects
@@
 			(project "PS-100PinMCU"
 				(path "/abcdaa41-14f3-4587-9aac-314b09095246/840885ae-57ff-4136-b869-7c6178ab9d24"
-					(reference "C22")
+					(reference "C21")
 					(unit 1)
 				)
@@
 		(on_board yes)
 		(dnp no)
-		(property "Reference" "R26"
+		(property "Reference" "R24"
 			(at 138.43 33.02 90)
 			(effects
@@
 			(project ""
 				(path "/abcdaa41-14f3-4587-9aac-314b09095246/840885ae-57ff-4136-b869-7c6178ab9d24"
-					(reference "R26")
+					(reference "R24")
 					(unit 1)
 				)
@@
 		(dnp no)
 		(fields_autoplaced yes)
-		(property "Reference" "C21"
+		(property "Reference" "C20"
 			(at 194.31 35.5599 0)
 			(effects
@@
 			(project "PS-100PinMCU"
 				(path "/abcdaa41-14f3-4587-9aac-314b09095246/840885ae-57ff-4136-b869-7c6178ab9d24"
-					(reference "C21")
+					(reference "C20")
 					(unit 1)
 				)
@@
 		(dnp no)
 		(fields_autoplaced yes)
-		(property "Reference" "C20"
+		(property "Reference" "C19"
 			(at 184.15 60.9599 0)
 			(effects
@@
 			(project "PS-100PinMCU"
 				(path "/abcdaa41-14f3-4587-9aac-314b09095246/840885ae-57ff-4136-b869-7c6178ab9d24"
-					(reference "C20")
+					(reference "C19")
 					(unit 1)
 				)
@@
 		(on_board yes)
 		(dnp no)
-		(property "Reference" "R28"
+		(property "Reference" "R26"
 			(at 225.806 94.996 90)
 			(effects
@@
 			(project "PS-100PinMCU"
 				(path "/abcdaa41-14f3-4587-9aac-314b09095246/840885ae-57ff-4136-b869-7c6178ab9d24"
-					(reference "R28")
+					(reference "R26")
 					(unit 1)
 				)
@@
 		(dnp no)
 		(fields_autoplaced yes)
-		(property "Reference" "C16"
+		(property "Reference" "C15"
 			(at 33.655 46.3549 0)
 			(effects
@@
 			(project ""
 				(path "/abcdaa41-14f3-4587-9aac-314b09095246/840885ae-57ff-4136-b869-7c6178ab9d24"
-					(reference "C16")
+					(reference "C15")
 					(unit 1)
 				)
@@
 		(dnp no)
 		(fields_autoplaced yes)
-		(property "Reference" "C25"
+		(property "Reference" "C24"
 			(at 219.71 35.5599 0)
 			(effects
@@
 			(project "PS-100PinMCU"
 				(path "/abcdaa41-14f3-4587-9aac-314b09095246/840885ae-57ff-4136-b869-7c6178ab9d24"
-					(reference "C25")
+					(reference "C24")
 					(unit 1)
 				)
@@
 		(dnp no)
 		(fields_autoplaced yes)
-		(property "Reference" "C27"
+		(property "Reference" "C26"
 			(at 232.41 35.5599 0)
 			(effects
@@
 			(project "PS-100PinMCU"
 				(path "/abcdaa41-14f3-4587-9aac-314b09095246/840885ae-57ff-4136-b869-7c6178ab9d24"
-					(reference "C27")
+					(reference "C26")
 					(unit 1)
 				)
@@
 		(dnp no)
 		(fields_autoplaced yes)
-		(property "Reference" "C17"
+		(property "Reference" "C16"
 			(at 46.355 46.3549 0)
 			(effects
@@
 			(project ""
 				(path "/abcdaa41-14f3-4587-9aac-314b09095246/840885ae-57ff-4136-b869-7c6178ab9d24"
-					(reference "C17")
+					(reference "C16")
 					(unit 1)
 				)
@@
 		(dnp no)
 		(fields_autoplaced yes)
-		(property "Reference" "D17"
+		(property "Reference" "D15"
 			(at 247.015 109.2199 90)
 			(effects
@@
 			(project "PS-100PinMCU"
 				(path "/abcdaa41-14f3-4587-9aac-314b09095246/840885ae-57ff-4136-b869-7c6178ab9d24"
-					(reference "D17")
+					(reference "D15")
 					(unit 1)
 				)
@@
 		(dnp no)
 		(fields_autoplaced yes)
-		(property "Reference" "C19"
+		(property "Reference" "C18"
 			(at 183.515 35.5599 0)
 			(effects
@@
 			(project "PS-100PinMCU"
 				(path "/abcdaa41-14f3-4587-9aac-314b09095246/840885ae-57ff-4136-b869-7c6178ab9d24"
-					(reference "C19")
+					(reference "C18")
 					(unit 1)
 				)
@@
 		(dnp no)
 		(fields_autoplaced yes)
-		(property "Reference" "D16"
+		(property "Reference" "D14"
 			(at 236.22 105.0924 90)
 			(effects
@@
 			(project "PS-100PinMCU"
 				(path "/abcdaa41-14f3-4587-9aac-314b09095246/840885ae-57ff-4136-b869-7c6178ab9d24"
-					(reference "D16")
+					(reference "D14")
 					(unit 1)
 				)
@@
 		(on_board yes)
 		(dnp no)
-		(property "Reference" "J9"
+		(property "Reference" "J8"
 			(at 156.718 16.002 0)
 			(effects
@@
 			(project ""
 				(path "/abcdaa41-14f3-4587-9aac-314b09095246/840885ae-57ff-4136-b869-7c6178ab9d24"
-					(reference "J9")
+					(reference "J8")
 					(unit 1)
 				)
@@
 		(dnp no)
 		(fields_autoplaced yes)
-		(property "Reference" "C26"
+		(property "Reference" "C25"
 			(at 229.235 60.9599 0)
 			(effects
@@
 			(project "PS-100PinMCU"
 				(path "/abcdaa41-14f3-4587-9aac-314b09095246/840885ae-57ff-4136-b869-7c6178ab9d24"
-					(reference "C26")
+					(reference "C25")
 					(unit 1)
 				)
@@
 		(on_board yes)
 		(dnp no)
-		(property "Reference" "C18"
+		(property "Reference" "C17"
 			(at 182.626 115.6716 0)
 			(effects
@@
 			(project "PS-100PinMCU"
 				(path "/abcdaa41-14f3-4587-9aac-314b09095246/840885ae-57ff-4136-b869-7c6178ab9d24"
-					(reference "C18")
+					(reference "C17")
 					(unit 1)
 				)
@@
 		(dnp no)
 		(fields_autoplaced yes)
-		(property "Reference" "C29"
+		(property "Reference" "C28"
 			(at 269.24 62.2299 0)
 			(effects
@@
 			(project "PS-100PinMCU"
 				(path "/abcdaa41-14f3-4587-9aac-314b09095246/840885ae-57ff-4136-b869-7c6178ab9d24"
-					(reference "C29")
+					(reference "C28")
 					(unit 1)
 				)
@@
 		(dnp no)
 		(fields_autoplaced yes)
-		(property "Reference" "C23"
+		(property "Reference" "C22"
 			(at 207.01 35.5599 0)
 			(effects
@@
 			(project "PS-100PinMCU"
 				(path "/abcdaa41-14f3-4587-9aac-314b09095246/840885ae-57ff-4136-b869-7c6178ab9d24"
-					(reference "C23")
+					(reference "C22")
 					(unit 1)
 				)
@@
 		(on_board yes)
 		(dnp no)
-		(property "Reference" "C28"
+		(property "Reference" "C27"
 			(at 245.237 35.433 0)
 			(effects
@@
 			(project "PS-100PinMCU"
 				(path "/abcdaa41-14f3-4587-9aac-314b09095246/840885ae-57ff-4136-b869-7c6178ab9d24"
-					(reference "C28")
+					(reference "C27")
 					(unit 1)
 				)

Commit message: schem fixes + some semblance of layout ish
Parts:
- added J10: SWD_PinHeader, Connector_PinHeader_2.54mm:PinHeader_1x04_P2.54mm_Vertical, symbol Connector_Generic:Conn_01x04
Connections:
- net 3V3: now also J10.1 (Pin_1)
- net GND: now also J10.2 (Pin_2)
- net at J8.3 (Pin_3), R23.2: now also J8.4 (Pin_4), R24.2, J10.3 (Pin_3), J10.4 (Pin_4)
Other:
- moved on the sheet: C15, C16, C17, C28, D14, D15, FB1, FB2, J8, R23, R24, R25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
