File: 100PinMCU_TestBoard/100PinMCU_ESP32_TestBoard.kicad_pcb (KiCad board)
At the start: 2 copper layers, 134 parts, among them IC1 TCAN3413DR, IC2 TCAN3413DR, IC3 CYPD3177-24LQXQ, J1 Conn_02x06_Odd_Even, J2 Conn_01x06, J3 Conn_01x02, J4 Conn_01x02, J5 USB_C_Receptacle_USB2.0_16P, J6 SWD_Header_02x02, Q1 SI7997DP-T1-GE3, Q2 SI7997DP-T1-GE3, SW1 BOOT Switch, SW2 RESET Button, U1 ESP32-C6-MINI-1, U2 MCP1826S, U3 STM32G491VET6, Y1 Crystal

Commit message: pre board
Parts:
- removed the C15 at (154.9, 48.1)
- removed C30, C31, C32, C33, C34, C35: 1uF, Capacitor_SMD:C_0603_1608Metric_Pad1.08x0.95mm_HandSolder
- removed C36, C37: 0.1uF, Capacitor_SMD:C_0603_1608Metric_Pad1.08x0.95mm_HandSolder
- removed the D14 at (283.5, 50.2)
- removed the D15 at (162.9, 60.9)
- removed D18, D19: SMBJ10A-E3_52, Diode_SMD:D_SMB
- removed IC3: CYPD3177-24LQXQ, UTSVT_ICs:CYPD3177-24LQXQ
- removed the J3 at (141.3, 66.4)
- removed J4: Conn_01x02, Connector_PinHeader_2.54mm:PinHeader_1x02_P2.54mm_Vertical
- removed the J6 at (265.4, 47.1)
- removed the JP1 at (132.5, 48.6)
- removed the JP2 at (132.5, 52.2)
- removed the JP3 at (132.5, 55.7)
- removed the JP8 at (136.8, 55.7)
- removed Q1, Q2: SI7997DP-T1-GE3, UTSVT_ICs:SI7997DP-T1-GE3
- removed the R21 at (167.9, 48.1)
- removed the R22 at (167.9, 50.6)
- removed R28, R29, R34: 1k, Resistor_SMD:R_0603_1608Metric_Pad0.98x0.95mm_HandSolder
- removed R30: 10k, Resistor_SMD:R_0603_1608Metric_Pad0.98x0.95mm_HandSolder
- removed R31, R36: 49.9k, Resistor_SMD:R_0603_1608Metric_Pad0.98x0.95mm_HandSolder
- removed R32, R33, R35: 5.1k, Resistor_SMD:R_0603_1608Metric_Pad0.98x0.95mm_HandSolder
- removed R37: 4.7k, Resistor_SMD:R_0603_1608Metric_Pad0.98x0.95mm_HandSolder
- removed R38, R39: 2.2k, Resistor_SMD:R_0603_1608Metric_Pad0.98x0.95mm_HandSolder
- added C1: 10uF, Capacitor_SMD:C_0805_2012Metric, F.Cu at (156.3, 133.3)
- added D5: TPD2EUSB30DRTR, UTSVT_ICs:TPD2EUSB30DRTR, F.Cu at (155.5, 136.2)
- added D6: D_Schottky, Diode_SMD:D_SOD-123, F.Cu at (152.7, 130.2)
- added J2: LogicAnalyzer, UTSVT_Connectors:CONN_SFH11-xxxC-D05-ST-XX_SUL, F.Cu at (143.8, 122.4)
- added J5: USB_C_Receptacle_USB2.0_16P, UTSVT_Connectors:USB_C_Receptacle_GCT_USB4105-xx-A_16P_TopMnt_Horizontal, F.Cu at (143.9, 133.8)
- added J7: SWD_Header_02x02, UTSVT_Connectors:CONN04_878320406_MOL, F.Cu at (178.1, 127.1)
- added J8: CAN_Breakout, Connector_PinHeader_2.54mm:PinHeader_1x04_P2.54mm_Vertical, F.Cu at (137.7, 166.0)
- added R8: 5.1k, Resistor_SMD:R_0603_1608Metric_Pad0.98x0.95mm_HandSolder, F.Cu at (151.9, 133.1)
- added R9: 5.1k, Resistor_SMD:R_0603_1608Metric_Pad0.98x0.95mm_HandSolder, F.Cu at (151.9, 135.6)
- C17: value 0.1uF -> 26p
- C18: value 10uF -> 0.1uF; footprint Capacitor_SMD:C_0805_2012Metric -> Capacitor_SMD:C_0603_1608Metric_Pad1.08x0.95mm_HandSolder
- C19: value 0.1uF -> 10uF; footprint Capacitor_SMD:C_0603_1608Metric_Pad1.08x0.95mm_HandSolder -> Capacitor_SMD:C_0805_2012Metric
- C23, C25: value 1uF -> 0.1uF
- C24, C26: value 0.1uF -> 1uF
- C29: value 10uF -> 0.1uF; footprint Capacitor_SMD:C_0805_2012Metric_Pad1.18x1.45mm_HandSolder -> Capacitor_SMD:C_0603_1608Metric_Pad1.08x0.95mm_HandSolder
- C6: renamed from C5; footprint Capacitor_SMD:C_0805_2012Metric -> Capacitor_SMD:C_0805_2012Metric_Pad1.18x1.45mm_HandSolder
- C7: renamed from C6; footprint Capacitor_SMD:C_0805_2012Metric -> Capacitor_SMD:C_0805_2012Metric_Pad1.18x1.45mm_HandSolder
- C8: renamed from C7; footprint Capacitor_SMD:C_0603_1608Metric -> Capacitor_SMD:C_0603_1608Metric_Pad1.08x0.95mm_HandSolder
- C9: renamed from C8; footprint Capacitor_SMD:C_0603_1608Metric -> Capacitor_SMD:C_0603_1608Metric_Pad1.08x0.95mm_HandSolder
- D16: value TPD2EUSB30DRTR -> LED; footprint UTSVT_ICs:TPD2EUSB30DRTR -> Diode_SMD:D_0603_1608Metric_Pad1.05x0.95mm_HandSolder
- D17: value SMBJ24A-E3_52 -> D_TVS; footprint Diode_SMD:D_SMB -> Diode_SMD:D_SOD-323
- J1: value Conn_02x06_Odd_Even -> LogicAnalyzer; footprint Connector_PinHeader_2.54mm:PinHeader_2x06_P2.54mm_Vertical -> UTSVT_Connectors:CONN_SFH11-xxxC-D05-ST-XX_SUL
- J3: renamed from J2; value Conn_01x06 -> ADC_Breakout
- JP1: renamed from JP4; footprint Jumper:SolderJumper-2_P1.3mm_Bridged2Bar_Pad1.0x1.5mm -> Connector_PinHeader_2.54mm:PinHeader_1x02_P2.54mm_Vertical
- JP2: renamed from JP5; footprint Jumper:SolderJumper-2_P1.3mm_Bridged2Bar_Pad1.0x1.5mm -> Connector_PinHeader_2.54mm:PinHeader_1x02_P2.54mm_Vertical
- JP3: renamed from JP6; footprint Jumper:SolderJumper-2_P1.3mm_Bridged2Bar_Pad1.0x1.5mm -> Connector_PinHeader_2.54mm:PinHeader_1x02_P2.54mm_Vertical
- JP4: renamed from JP7; footprint Jumper:SolderJumper-2_P1.3mm_Bridged2Bar_Pad1.0x1.5mm -> Connector_PinHeader_2.54mm:PinHeader_1x02_P2.54mm_Vertical
- JP5: renamed from JP9; footprint Jumper:SolderJumper-2_P1.3mm_Bridged2Bar_Pad1.0x1.5mm -> Connector_PinHeader_2.54mm:PinHeader_1x02_P2.54mm_Vertical
- R23, R24: value 10k -> 22
- R25: value 1k -> 10k
- R26: value 5.1k -> 10k
- R27: value 5.1k -> 1k
- TP1: value TestPoint -> 3V3_ESP
- TP2: value TestPoint -> ESP_TX
- TP3: value TestPoint -> ESP_RX
- TP4: value TestPoint -> GND_ESP
- TP5: value TestPoint -> 3V3_LED
- moved U3 192.6 mm to (75.6, 97.3)
- moved R27 133.9 mm to (126.8, 175.0)
- moved R24 123.9 mm to (126.8, 172.5)
- moved R23 123.9 mm to (126.8, 170.0)
- moved D16 121.5 mm to (131.2, 165.0)
- moved S1 118.3 mm to (166.6, 128.3)
- moved Reset1 116.0 mm to (177.9, 113.3)
- moved FB1 115.3 mm to (126.8, 164.9)
- moved FB2 115.3 mm to (126.8, 167.5)
- moved D17 115.0 mm to (179.3, 132.9)
- moved R26 103.9 mm to (171.4, 121.5)
- moved C29 83.3 mm to (171.4, 116.5)
- moved C19 79.8 mm to (174.9, 132.9)
- moved C21 73.5 mm to (162.7, 121.5)
- moved C26 73.5 mm to (167.1, 121.5)
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- renumbered C9 to C10, C10 to C11, C11 to C12, C12 to C13, C13 to C14, C14 to C15, C1 to C2, C2 to C3, C3 to C4, C4 to C5, D8 to D10, D9 to D11, D10 to D12, D11 to D13, D12 to D14, D13 to D15, D5 to D7, D6 to D8, D7 to D9, J5 to J6, JP10 to JP6, JP11 to JP7, JP12 to JP8, R8 to R10, R9 to R11, R10 to R12, R11 to R13, R12 to R14, R13 to R15, R14 to R16, R15 to R17, R16 to R18, R17 to R19, R18 to R20, R19 to R21, R20 to R22
Connections:
- net /100PinMCU/PB12 renamed /FDCAN2_RX
- net /100PinMCU/PB13 renamed /FDCAN2_TX
- net /CAN_Transceiver/CAN_H renamed /CAN_H1
- net /CAN_Transceiver/CAN_L renamed /CAN_L1
- net /CAN_Transceiver1/CAN_H renamed /CAN_H2
- net /CAN_Transceiver1/CAN_L renamed /CAN_L2
- C16 pad 2: Net-(U3-PF0-OSC_IN) -> Net-(U3-PF1-OSC_OUT)
- C17 pad 1: /100PinMCU/PG10-NRST -> GND
- C17 pad 2: GND -> Net-(U3-PF0-OSC_IN)
- C18 pad 1: /100PinMCU/3V3 -> /100PinMCU/PG10-NRST
- C19 pad 1: /100PinMCU/VDDA -> /100PinMCU/3V3
- C19 pad 2: /100PinMCU/GNDA -> GND
- C20 pad 1: /100PinMCU/3V3 -> /100PinMCU/VDDA
- C20 pad 2: GND -> /100PinMCU/GNDA
- C21 pad 1: /100PinMCU/VDDA -> /100PinMCU/3V3
- C21 pad 2: /100PinMCU/GNDA -> GND
- C22 pad 1: /100PinMCU/3V3 -> /100PinMCU/VDDA
- C22 pad 2: GND -> /100PinMCU/GNDA
- C23 pad 1: /100PinMCU/VDDA -> /100PinMCU/3V3
- C23 pad 2: /100PinMCU/GNDA -> GND
- C24 pad 1: /100PinMCU/3V3 -> /100PinMCU/VDDA
- C24 pad 2: GND -> /100PinMCU/GNDA
- C25 pad 1: /100PinMCU/VDDA -> /100PinMCU/3V3
- C25 pad 2: /100PinMCU/GNDA -> GND
- C26 pad 1: /100PinMCU/3V3 -> /100PinMCU/VDDA
- C26 pad 2: GND -> /100PinMCU/GNDA
- C28 pad 1: /100PinMCU/VDDA -> /100PinMCU/3V3
- C28 pad 2: /100PinMCU/GNDA -> GND
- C29 pad 1: VBUS_IN -> /100PinMCU/VDDA
- C29 pad 2: GND -> /100PinMCU/GNDA
- D16 pad 1: /100PinMCU/USB_DP -> Net-(D16-K)
- D16 pad 2: /100PinMCU/USB_DM -> Net-(D16-A)
- D17 pad 1: VBUS_IN -> GND
- D17 pad 2: GND -> Net-(D16-A)
- J1 pad 1: /I2C2_SDA -> GND
- J1 pad 10: /SPI1_NSS -> /I2C2_SDA
- J1 pad 2: /I2C2_SCL -> unconnected-(J1-NC-Pad2)
- J1 pad 3: /UART_TX -> /GPIO2
- J1 pad 4: /UART_RX -> /GPIO1
- J1 pad 5: /FDCAN1_TX -> /FDCAN1_RX
- J1 pad 6: /FDCAN1_RX -> /FDCAN1_TX
- J1 pad 7: /SPI1_MOSI -> /UART_RX
- J1 pad 8: /SPI1_MISO -> /UART_TX
- J1 pad 9: /SPI1_SCK -> /I2C2_SCL
- JP6 pad 1: +3.3V -> /LDO/Vout
- JP6 pad 2: /LDO/Vout -> +3.3V
- R23 pad 1: /100PinMCU/PG10-NRST -> /100PinMCU/SWCLK
- R23 pad 2: /100PinMCU/3V3 -> Net-(J7-Pin_3)
- R24 pad 1: /100PinMCU/BOOT -> /100PinMCU/SWDIO
- R24 pad 2: Net-(D14-A) -> Net-(J7-Pin_4)
- R25 pad 1: Net-(D14-K) (its old number) -> /100PinMCU/PG10-NRST
- R25 pad 2: GND -> /100PinMCU/3V3
- R26 pad 1: /USB_PD/CC1 -> /BOOT
- R26 pad 2: GND -> Net-(D16-A)
- R27 pad 1: /USB_PD/CC2 -> Net-(D16-K)
- R6 pad 1: /I2C2_SCL -> +3.3V
- R6 pad 2: +3.3V -> /I2C2_SCL
- S1 pad 2: Net-(D14-A) -> Net-(D16-A)
- U1 pad 19: /ESP32/ESP_GPIO1 -> /100PinMCU/PG10-NRST
- U1 pad 20: /ESP32/ESP_GPIO2 -> /BOOT
- U1 pad 24: /ESP32/ESP_GPIO3 -> /100PinMCU/PC0
- U1 pad 25: /ESP32/ESP_GPIO4 -> /100PinMCU/PC1
- U3 pad 65: /100PinMCU/PC6 -> /GPIO2
- U3 pad 7: /100PinMCU/PC13 -> unconnected-(U3-PC13-Pad7)
- U3 pad 72: /100PinMCU/USB_DM -> /D-
- U3 pad 73: /100PinMCU/USB_DP -> /D+
- U3 pad 8: /100PinMCU/PC14-OSC32_IN -> unconnected-(U3-PC14-OSC32_IN-Pad8)
- U3 pad 9: /100PinMCU/PC15-OSC32_OUT -> unconnected-(U3-PC15-OSC32_OUT-Pad9)
- U3 pad 95: /100PinMCU/BOOT -> /BOOT

Commit message: during flight
Parts:
- moved D7 225.4 mm to (52.6, 35.5), turned to -90 degrees
- moved D1 209.5 mm to (71.1, 83.6), turned to -90 degrees
- moved D2 206.5 mm to (73.7, 83.6), turned to -90 degrees
- moved D3 203.6 mm to (76.2, 83.7), turned to -90 degrees
- moved D4 200.7 mm to (78.7, 83.6), turned to -90 degrees
- moved D17 164.9 mm to (40.4, 44.0)
- moved R27 163.0 mm to (36.9, 39.0), turned to 180 degrees
- moved D11 157.9 mm to (125.6, 48.1), turned to 180 degrees
- moved D16 155.2 mm to (40.4, 39.1)
- moved R26 148.7 mm to (44.5, 44.0), turned to 180 degrees
- moved C19 147.0 mm to (47.1, 60.1), turned to 90 degrees
- moved S1 146.4 mm to (41.6, 52.1)
- moved C27 146.0 mm to (34.7, 60.2), turned to 90 degrees
- moved C23 145.7 mm to (31.8, 60.1), turned to 90 degrees
- moved C28 144.0 mm to (37.8, 60.2), turned to 90 degrees
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Connections:
- J1 pad 10: /I2C2_SDA -> unconnected-(J1-CH0-Pad10)
- J1 pad 3: /GPIO2 -> unconnected-(J1-CH7-Pad3)
- J1 pad 4: /GPIO1 -> /GPIO2
- J1 pad 9: /I2C2_SCL -> /BOOT
- J2 pad 10: /SPI1_MOSI -> /I2C2_SDA
- J2 pad 4: unconnected-(J2-CH6-Pad4) -> /GPIO1
- J2 pad 5: unconnected-(J2-CH5-Pad5) -> /SPI1_NSS
- J2 pad 6: /BOOT -> /SPI1_SCK
- J2 pad 7: /SPI1_NSS -> /SPI1_MISO
- J2 pad 8: /SPI1_SCK -> /SPI1_MOSI
- J2 pad 9: /SPI1_MISO -> /I2C2_SCL
Routing:
- net +3.3V: track 0.00 -> 229.7 mm, vias 0 -> 5
- net GND: track 0.00 -> 178.9 mm
- net /100PinMCU/3V3: track 0.00 -> 120.0 mm, vias 0 -> 2
- net /100PinMCU/PD2: track 0.00 -> 110.2 mm, vias 0 -> 2
- net /100PinMCU/PG10-NRST: track 0.00 -> 105.9 mm, vias 0 -> 2
- net /BOOT: track 0.00 -> 90.3 mm, vias 0 -> 6
- net /100PinMCU/PC0: track 0.00 -> 84.6 mm, vias 0 -> 2
- net /100PinMCU/PC1: track 0.00 -> 83.0 mm, vias 0 -> 2
- net +3.3V_ESP: track 0.00 -> 58.5 mm, vias 0 -> 2
- net /100PinMCU/VDDA: track 0.00 -> 55.8 mm
- net /D+: track 0.00 -> 53.6 mm, vias 0 -> 2
- net /D-: track 0.00 -> 49.7 mm, vias 0 -> 2
- net /I2C2_SDA: track 0.00 -> 46.0 mm, vias 0 -> 2
- net /100PinMCU/PA10: track 0.00 -> 40.3 mm, vias 0 -> 2
- net /100PinMCU/PA9: track 0.00 -> 34.5 mm, vias 0 -> 2
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- added copper zone on B.Cu, net GND
- added copper zone on F.Cu, net GND
Other:
- board outline added: 110.5 x 74.5 mm

Commit message: mount fuji tmrw
Parts:
- added J4: CAN1_Conn, Connector_PinHeader_1.00mm:PinHeader_1x02_P1.00mm_Vertical, F.Cu at (68.0, 38.1)
- added J9: CAN_Breakout, Connector_PinHeader_1.00mm:PinHeader_1x04_P1.00mm_Vertical, F.Cu at (70.9, 38.1)
- added R28: 0, Resistor_SMD:R_0603_1608Metric_Pad0.98x0.95mm_HandSolder, F.Cu at (73.5, 37.0)
- added R29: 0, Resistor_SMD:R_0603_1608Metric_Pad0.98x0.95mm_HandSolder, F.Cu at (68.0, 42.0)
- J8: value CAN_Breakout -> CAN2_Conn; footprint Connector_PinHeader_2.54mm:PinHeader_1x04_P2.54mm_Vertical -> Connector_PinHeader_1.00mm:PinHeader_1x02_P1.00mm_Vertical
- moved J8 21.1 mm to (73.5, 40.1)
Connections:
- J8 pad 1: /CAN_H1 -> /CAN_H2
- J8 pad 2: /CAN_H2 -> /CAN_L2
Routing:
- net /CAN_L2: track 6.80 -> 56.9 mm, vias 0 -> 2
- net /CAN_H2: track 6.72 -> 50.0 mm, vias 0 -> 2
- net /CAN_H1: track 7.64 -> 25.4 mm
- net /CAN_L1: track 8.46 -> 19.3 mm

Commit message: separate subcircuits
Parts:
- removed TP5: 3V3_LED, TestPoint:TestPoint_Loop_D1.80mm_Drill1.0mm_Beaded
- added C30: 0.1uF, Capacitor_SMD:C_0603_1608Metric_Pad1.08x0.95mm_HandSolder, F.Cu at (161.4, 183.0)
- added C31: 0.1uF, Capacitor_SMD:C_0603_1608Metric_Pad1.08x0.95mm_HandSolder, F.Cu at (161.4, 185.5)
- added C32: 0.1uF, Capacitor_SMD:C_0603_1608Metric_Pad1.08x0.95mm_HandSolder, F.Cu at (161.4, 188.0)
- added C33: 0.1uF, Capacitor_SMD:C_0603_1608Metric_Pad1.08x0.95mm_HandSolder, F.Cu at (161.4, 190.5)
- added JP9: TRM, Connector_PinHeader_2.54mm:PinHeader_1x02_P2.54mm_Vertical, F.Cu at (214.8, 79.8)
- added R30: 10k, Resistor_SMD:R_0603_1608Metric_Pad0.98x0.95mm_HandSolder, F.Cu at (161.4, 193.0)
- added U4: TPS2117DRLR, UTSVT_Power:TPS2117DRLR, F.Cu at (165.9, 183.6)
- C1: footprint Capacitor_SMD:C_0805_2012Metric -> Capacitor_SMD:C_0805_2012Metric_Pad1.18x1.45mm_HandSolder
- C12: value 10u -> 0.1u; footprint Capacitor_SMD:C_0805_2012Metric_Pad1.18x1.45mm_HandSolder -> Capacitor_SMD:C_0603_1608Metric_Pad1.08x0.95mm_HandSolder
- C15: value 0.1u -> 26p
- C17: value 26p -> 0.1uF
- C18, C29: value 0.1uF -> 10uF; footprint Capacitor_SMD:C_0603_1608Metric_Pad1.08x0.95mm_HandSolder -> Capacitor_SMD:C_0805_2012Metric
- C19: value 10uF -> 0.1uF; footprint Capacitor_SMD:C_0805_2012Metric -> Capacitor_SMD:C_0603_1608Metric_Pad1.08x0.95mm_HandSolder
- C2: value 10u -> 10uF
- C23, C25: value 0.1uF -> 1uF
- C24, C26: value 1uF -> 0.1uF
- C3, C4: value 0.1u -> 0.1uF
- C5: value 0.1u -> 10u; footprint Capacitor_SMD:C_0603_1608Metric_Pad1.08x0.95mm_HandSolder -> Capacitor_SMD:C_0805_2012Metric_Pad1.18x1.45mm_HandSolder
- C6, C7: value 10uF -> 0.1u; footprint Capacitor_SMD:C_0805_2012Metric_Pad1.18x1.45mm_HandSolder -> Capacitor_SMD:C_0603_1608Metric_Pad1.08x0.95mm_HandSolder
- C8: value 0.1uF -> 0.1u
- C9: value 0.1uF -> 10u; footprint Capacitor_SMD:C_0603_1608Metric_Pad1.08x0.95mm_HandSolder -> Capacitor_SMD:C_0805_2012Metric_Pad1.18x1.45mm_HandSolder
- D10: value SP0503BAHT -> ESP_LED2; footprint Package_TO_SOT_SMD:SOT-143 -> Diode_SMD:D_0603_1608Metric_Pad1.05x0.95mm_HandSolder
- D11: value ESP_PWR -> CDSOT23-T24CAN; footprint Diode_SMD:D_0603_1608Metric_Pad1.05x0.95mm_HandSolder -> UTSVT_Passives:CDSOT23-T24CAN
- D12: value ESP_LED1 -> SBA130CH-AU_R1_000A1; footprint Diode_SMD:D_0603_1608Metric_Pad1.05x0.95mm_HandSolder -> Diode_SMD:D_SOD-323_HandSoldering
- D13: value ESP_LED2 -> CDSOT23-T24CAN; footprint Diode_SMD:D_0603_1608Metric_Pad1.05x0.95mm_HandSolder -> UTSVT_Passives:CDSOT23-T24CAN
- D14: value SBA130CH-AU_R1_000A1 -> LED; footprint Diode_SMD:D_SOD-323_HandSoldering -> Diode_SMD:D_0603_1608Metric_Pad1.05x0.95mm_HandSolder
- D15: value CDSOT23-T24CAN -> D_TVS; footprint UTSVT_Passives:CDSOT23-T24CAN -> Diode_SMD:D_SOD-323
- D16: value LED -> TPD2EUSB30DRTR; footprint Diode_SMD:D_0603_1608Metric_Pad1.05x0.95mm_HandSolder -> UTSVT_ICs:TPD2EUSB30DRTR
- D17: value D_TVS -> D_Schottky; footprint Diode_SMD:D_SOD-323 -> Diode_SMD:D_SOD-123
- D2: value LED -> 3V3
- D5: value TPD2EUSB30DRTR -> LED; footprint UTSVT_ICs:TPD2EUSB30DRTR -> Diode_SMD:D_0603_1608Metric_Pad1.05x0.95mm_HandSolder
- D6: value D_Schottky -> 1N5819HW-7-F
- D7: value LED -> SP0503BAHT; footprint Diode_SMD:D_0603_1608Metric_Pad1.05x0.95mm_HandSolder -> Package_TO_SOT_SMD:SOT-143
- D8: value CDSOT23-T24CAN -> ESP_PWR; footprint UTSVT_Passives:CDSOT23-T24CAN -> Diode_SMD:D_0603_1608Metric_Pad1.05x0.95mm_HandSolder
- D9: value 1N5819HW-7-F -> ESP_LED1; footprint Diode_SMD:D_SOD-123 -> Diode_SMD:D_0603_1608Metric_Pad1.05x0.95mm_HandSolder
- J1: value LogicAnalyzer -> ADC_Breakout; footprint UTSVT_Connectors:CONN_SFH11-xxxC-D05-ST-XX_SUL -> Connector_PinHeader_2.54mm:PinHeader_1x06_P2.54mm_Vertical
- J2: value LogicAnalyzer -> LogicAnalyzer_1
- J3: value ADC_Breakout -> CAN_1; footprint Connector_PinHeader_2.54mm:PinHeader_1x06_P2.54mm_Vertical -> Connector_PinHeader_1.00mm:PinHeader_1x02_P1.00mm_Vertical
- J4: value CAN1_Conn -> CAN_2
- J5: value USB_C_Receptacle_USB2.0_16P -> LogicAnalyzer_2; footprint UTSVT_Connectors:USB_C_Receptacle_GCT_USB4105-xx-A_16P_TopMnt_Horizontal -> UTSVT_Connectors:CONN_SFH11-xxxC-D05-ST-XX_SUL
- J6: value USB_C_Receptacle_USB2.0_16P -> CAN_Breakout; footprint UTSVT_Connectors:USB_C_Receptacle_GCT_USB4105-xx-A_16P_TopMnt_Horizontal -> Connector_PinHeader_2.54mm:PinHeader_1x04_P2.54mm_Vertical
- J7: value SWD_Header_02x02 -> USB_C_Receptacle_USB2.0_16P; footprint UTSVT_Connectors:CONN04_878320406_MOL -> UTSVT_Connectors:USB_C_Receptacle_GCT_USB4105-xx-A_16P_TopMnt_Horizontal
- J8: value CAN2_Conn -> SWD_Header_02x02; footprint Connector_PinHeader_1.00mm:PinHeader_1x02_P1.00mm_Vertical -> UTSVT_Connectors:CONN04_878320406_MOL
- J9: value CAN_Breakout -> USB_C_Receptacle_USB2.0_16P; footprint Connector_PinHeader_1.00mm:PinHeader_1x04_P1.00mm_Vertical -> UTSVT_Connectors:USB_C_Receptacle_GCT_USB4105-xx-A_16P_TopMnt_Horizontal
- JP1: value Jumper_2_Bridged -> ESP_PWR; footprint Connector_PinHeader_2.54mm:PinHeader_1x02_P2.54mm_Vertical -> Jumper:SolderJumper-2_P1.3mm_Open_TrianglePad1.0x1.5mm
- JP2: value Jumper_2_Bridged -> ESP_RST_EN
- JP3: value Jumper_2_Bridged -> ESP_TX_EN
- JP4: value Jumper_2_Bridged -> ESP_RX_EN
- JP5: value Jumper_2_Bridged -> MCU_PWR; footprint Connector_PinHeader_2.54mm:PinHeader_1x02_P2.54mm_Vertical -> Jumper:SolderJumper-2_P1.3mm_Open_TrianglePad1.0x1.5mm
- JP6: value Jumper_2_Open -> CAN_H_LOOPBACK; footprint Jumper:SolderJumper-2_P1.3mm_Open_Pad1.0x1.5mm -> Connector_PinHeader_2.54mm:PinHeader_1x02_P2.54mm_Vertical
- JP7: value TRM -> CAN_L_LOOPBACK
- R1: value 1k -> 16k
- R11, R12: value 60 -> 5.1k
- R13, R14: value 5.1k -> 10k
- R16, R17: value 10k -> 1k
- R19, R20: value 1k -> 60
- R2, R4: value 1k -> 4.7k
- R28, R29: value 0 -> 5.1k
- R5, R6: value 4.7k -> 1k
- R8: value 5.1k -> 4.7k
- R9: value 5.1k -> 1k
- TP1: value 3V3_ESP -> GND_ESP
- TP2: value ESP_TX -> 3V3
- TP3: value ESP_RX -> ESP_TX
- TP4: value GND_ESP -> ESP_RX
- moved D7 253.2 mm to (274.7, 157.1), turned to 0 degrees
- moved D6 240.7 mm to (275.5, 153.1)
- moved C1 239.7 mm to (270.2, 152.9), turned to 0 degrees
- moved C2 239.2 mm to (270.2, 155.9), turned to 0 degrees
- moved R11 235.7 mm to (277.4, 124.8), turned to 0 degrees
- moved C4 235.5 mm to (277.4, 122.2), turned to 0 degrees
- moved D16 235.4 mm to (275.3, 22.5)
- moved R12 234.2 mm to (277.4, 127.3)
- moved C3 234.1 mm to (277.4, 119.7), turned to 0 degrees
- moved D8 233.9 mm to (265.6, 152.7), turned to 0 degrees
- moved D17 225.0 mm to (265.1, 32.8)
- moved C5 222.0 mm to (275.3, 79.7), turned to 0 degrees
- moved C29 220.2 mm to (274.5, 32.6), turned to 0 degrees
- moved IC1 215.5 mm to (272.5, 74.9), turned to 0 degrees
- moved J7 212.5 mm to (248.9, 156.7), turned to 0 degrees
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Connections:
- C1 pad 1: GND -> /ESP32/+5V_LDO_IN
- C1 pad 2: /5V_VBUS -> GND
- C10 pad 2: Net-(D14-K) -> +3.3V
- C11 pad 1: GND -> +3.3V
- C11 pad 2: /LDO/Vout -> GND
- C14 pad 1: +3.3V -> GND
- C14 pad 2: GND -> Net-(C14-Pad2)
- C15 pad 2: Net-(C15-Pad2) -> Net-(U3-PF1-OSC_OUT)
- C16 pad 2: Net-(U3-PF1-OSC_OUT) -> Net-(U3-PF0-OSC_IN)
- C17 pad 1: GND -> /100PinMCU/PG10-NRST
- C17 pad 2: Net-(U3-PF0-OSC_IN) -> GND
- C18 pad 1: /100PinMCU/PG10-NRST -> /100PinMCU/3V3
- C19 pad 1: /100PinMCU/3V3 -> /100PinMCU/VDDA
- C19 pad 2: GND -> /100PinMCU/GNDA
- C2 pad 1: +3.3V -> +3.3V_ESP
- C2 pad 2: GND -> +3.3V_ESP
- C20 pad 1: /100PinMCU/VDDA -> /100PinMCU/3V3
- C20 pad 2: /100PinMCU/GNDA -> GND
- C21 pad 1: /100PinMCU/3V3 -> /100PinMCU/VDDA
- C21 pad 2: GND -> /100PinMCU/GNDA
- C22 pad 1: /100PinMCU/VDDA -> /100PinMCU/3V3
- C22 pad 2: /100PinMCU/GNDA -> GND
- C23 pad 1: /100PinMCU/3V3 -> /100PinMCU/VDDA
- C23 pad 2: GND -> /100PinMCU/GNDA
- C24 pad 1: /100PinMCU/VDDA -> /100PinMCU/3V3
- C24 pad 2: /100PinMCU/GNDA -> GND
- C25 pad 1: /100PinMCU/3V3 -> /100PinMCU/VDDA
- C25 pad 2: GND -> /100PinMCU/GNDA
- C26 pad 1: /100PinMCU/VDDA -> /100PinMCU/3V3
- C26 pad 2: /100PinMCU/GNDA -> GND
- C28 pad 1: /100PinMCU/3V3 -> /100PinMCU/VDDA
- C28 pad 2: GND -> /100PinMCU/GNDA
- C29 pad 1: /100PinMCU/VDDA -> GND
- C29 pad 2: /100PinMCU/GNDA -> /Power_Mux/VIN_2
- C3 pad 1: +3.3V -> +3.3V_ESP
- C3 pad 2: GND -> +3.3V_ESP
- C4 pad 1: +3.3V -> /ESP32/ESP_RESET
- C5 pad 1: GND -> +3.3V
- C5 pad 2: Net-(C5-Pad2) -> GND
- C6 pad 1: /ESP32/+5V_LDO_IN -> +3.3V
- C7 pad 1: +3.3V_ESP -> +3.3V
- C7 pad 2: +3.3V_ESP -> GND
- C8 pad 1: +3.3V_ESP -> GND
- C8 pad 2: +3.3V_ESP -> Net-(C8-Pad2)
- C9 pad 1: /ESP32/ESP_RESET -> GND
- C9 pad 2: GND -> Net-(D12-K)
- D10 pad 2: /ESP32/USB_D+ -> Net-(D10-A)
- D11 pad 1: GND -> /CAN_H1
- D11 pad 2: Net-(D11-A) -> /CAN_L1
- D12 pad 1: GND -> Net-(D12-K)
- D12 pad 2: Net-(D12-A) -> /LDO/Vin
- D13 pad 1: GND -> /CAN_H2
- D13 pad 2: Net-(D13-A) -> /CAN_L2
- D14 pad 2: /ESP32/+5V_LDO_IN -> Net-(D14-A)
- D15 pad 1: /CAN_H2 -> GND
- D15 pad 2: /CAN_L2 -> Net-(D14-A)
- D16 pad 1: Net-(D16-K) -> /D+
- D16 pad 2: Net-(D16-A) -> /D-
- D17 pad 1: GND -> /Power_Mux/VIN_2
- D17 pad 2: Net-(D16-A) -> /USB-C/VBUS_IN
- D5 pad 1: /D+ -> GND
- D5 pad 2: /D- -> Net-(D5-A)
- D6 pad 1: /5V_VBUS -> /ESP32/+5V_LDO_IN
- D6 pad 2: /VBUS_IN -> /ESP32/VBUSB
- D7 pad 2: Net-(D7-A) -> /ESP32/USB_D+
- D8 pad 1: /CAN_H1 -> GND
- D8 pad 2: /CAN_L1 -> Net-(D8-A)
- D9 pad 1: /ESP32/+5V_LDO_IN -> GND
- D9 pad 2: /ESP32/VBUSB -> Net-(D9-A)
- J1 pad 1: GND -> /100PinMCU/GNDA
- J1 pad 2: unconnected-(J1-NC-Pad2) -> /ADC3_IN4
- J1 pad 3: unconnected-(J1-CH7-Pad3) -> /ADC3_IN3
- J1 pad 4: /GPIO2 -> /ADC3_IN2
- J1 pad 5: /FDCAN1_RX -> /ADC3_IN1
- J1 pad 6: /FDCAN1_TX -> /100PinMCU/VDDA
- J2 pad 10: /I2C2_SDA -> unconnected-(J2-CH0-Pad10)
- J2 pad 4: /GPIO1 -> /GPIO2
- J2 pad 5: /SPI1_NSS -> /FDCAN1_RX
- J2 pad 6: /SPI1_SCK -> /FDCAN1_TX
- J2 pad 7: /SPI1_MISO -> /UART_RX
- J2 pad 8: /SPI1_MOSI -> /UART_TX
- J2 pad 9: /I2C2_SCL -> /BOOT
- J3 pad 1: /100PinMCU/VDDA -> /CAN_H1
- J3 pad 2: /ADC3_IN1 -> /CAN_L1
- J4 pad 1: /CAN_H1 -> /CAN_H2
- J4 pad 2: /CAN_L1 -> /CAN_L2
- J8 pad 1: /CAN_H2 -> /100PinMCU/3V3
- J8 pad 2: /CAN_L2 -> GND
- JP1 pad 1: /100PinMCU/3V3 -> +3.3V_ESP
- JP5 pad 1: +3.3V -> /100PinMCU/3V3
- JP5 pad 2: +3.3V_ESP -> +3.3V
- JP6 pad 1: /LDO/Vout -> /CAN_H1
- JP6 pad 2: +3.3V -> /CAN_H2
- JP7 pad 1: Net-(JP7-A) -> /CAN_L1
- JP7 pad 2: /CAN_L1 -> /CAN_L2
- JP8 pad 2: /CAN_L2 -> /CAN_L1
- R1 pad 1: /100PinMCU/PE8 -> /ESP32/+5V_LDO_IN
- R1 pad 2: Net-(D1-A) -> /Power_Mux/PR1
- R10 pad 1: +3.3V -> /100PinMCU/PE14
- R10 pad 2: Net-(D7-A) -> Net-(D5-A)
- R11 pad 1: /CAN_H1 -> Net-(J7-CC1)
- R11 pad 2: Net-(C5-Pad2) -> GND
- R12 pad 1: Net-(C5-Pad2) -> Net-(J7-CC2)
- R12 pad 2: Net-(JP7-A) -> GND
- R13 pad 1: Net-(J6-CC1) -> /ESP32/BOOT
- R13 pad 2: GND -> Net-(SW1-B)
- R14 pad 1: Net-(J6-CC2) -> +3.3V_ESP
- R14 pad 2: GND -> /ESP32/ESP_RESET
- R15 pad 1: /ESP32/BOOT -> Net-(U1-GPIO8)
- R15 pad 2: Net-(SW1-B) -> +3.3V_ESP
- R16 pad 2: /ESP32/ESP_RESET -> Net-(D8-A)
- R17 pad 1: Net-(U1-GPIO8) -> /ESP32/LED1
- R17 pad 2: +3.3V_ESP -> Net-(D9-A)
- R18 pad 1: +3.3V_ESP -> /ESP32/LED2
- R18 pad 2: Net-(D11-A) -> Net-(D10-A)
- R19 pad 1: /ESP32/LED1 -> /CAN_H1
- R19 pad 2: Net-(D12-A) -> Net-(C8-Pad2)
- R2 pad 1: /100PinMCU/PE11 -> /Power_Mux/PR1
- R2 pad 2: Net-(D2-A) -> GND
- R20 pad 1: /ESP32/LED2 -> Net-(C8-Pad2)
- R20 pad 2: Net-(D13-A) -> Net-(JP8-A)
- R21 pad 2: Net-(C15-Pad2) -> Net-(C14-Pad2)
- R22 pad 1: Net-(C15-Pad2) -> Net-(C14-Pad2)
- R22 pad 2: Net-(JP8-A) -> Net-(JP9-A)
- R23 pad 2: Net-(J7-Pin_3) -> Net-(J8-Pin_3)
- R24 pad 2: Net-(J7-Pin_4) -> Net-(J8-Pin_4)
- R26 pad 2: Net-(D16-A) -> Net-(D14-A)
- R27 pad 1: Net-(D16-K) -> Net-(D14-K)
- R28 pad 1: /CAN_H1 -> GND
- R28 pad 2: /CAN_H2 -> /USB-C/CC2
- R29 pad 1: /CAN_L1 -> GND
- R29 pad 2: /CAN_L2 -> /USB-C/CC1
- R3 pad 1: /100PinMCU/PE12 -> /100PinMCU/PE8
- R3 pad 2: Net-(D3-A) -> Net-(D1-A)
- R4 pad 1: /100PinMCU/PE14 -> +3.3V
- R4 pad 2: Net-(D4-A) -> /I2C2_SCL
- R5 pad 2: /I2C2_SDA -> Net-(D2-A)
- R6 pad 1: +3.3V -> /100PinMCU/PE11
- R6 pad 2: /I2C2_SCL -> Net-(D3-A)
- R8 pad 1: GND -> +3.3V
- R8 pad 2: /CC2 -> /I2C2_SDA
- R9 pad 1: GND -> /100PinMCU/PE12
- R9 pad 2: /CC1 -> Net-(D4-A)
- S1 pad 2: Net-(D16-A) -> Net-(D14-A)
- TP1 pad 1: +3.3V -> GND
- TP2 pad 1: /ESP32/ESP_UART_TX -> +3.3V
- TP3 pad 1: /ESP32/ESP_UART_RX -> /ESP32/ESP_UART_TX
- TP4 pad 1: GND -> /ESP32/ESP_UART_RX
- TP_3.3V1 pad 1: /LDO/Vout -> +3.3V
- U2 pad 1: Net-(D14-K) -> Net-(D12-K)
- U2 pad 3: /LDO/Vout -> +3.3V
Routing:
- net +3.3V: track 229.7 -> 0.00 mm, vias 5 -> 0
- net GND: track 178.9 -> 0.00 mm
- net /100PinMCU/3V3: track 120.0 -> 0.00 mm, vias 2 -> 0
- net /100PinMCU/PD2: track 110.2 -> 0.00 mm, vias 2 -> 0
- net /100PinMCU/PG10-NRST: track 105.9 -> 0.00 mm, vias 2 -> 0
- net /BOOT: track 90.3 -> 0.00 mm, vias 6 -> 0
- net /100PinMCU/PC0: track 84.6 -> 0.00 mm, vias 2 -> 0
- net /100PinMCU/PC1: track 83.0 -> 0.00 mm, vias 2 -> 0
- net +3.3V_ESP: track 58.5 -> 0.00 mm, vias 2 -> 0
- net /CAN_L2: track 56.9 -> 0.00 mm, vias 2 -> 0
- net /100PinMCU/VDDA: track 55.8 -> 0.00 mm
- net /D+: track 53.6 -> 0.00 mm, vias 2 -> 0
- net /CAN_H2: track 50.0 -> 0.00 mm, vias 2 -> 0
- net /D-: track 49.7 -> 0.00 mm, vias 2 -> 0
- net /I2C2_SDA: track 46.0 -> 0.00 mm, vias 2 -> 0
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- removed copper zone on B.Cu, net GND
- removed copper zone on F.Cu, net GND
Other:
- board outline removed

Commit message: can layout
Parts:
- J3, J4: footprint Connector_PinHeader_1.00mm:PinHeader_1x02_P1.00mm_Vertical -> Connector_PinHeader_2.54mm:PinHeader_1x02_P2.54mm_Vertical
- R28, R29: moved to B.Cu
- moved C5 67.7 mm to (208.0, 87.2), turned to 90 degrees
- moved C6 57.9 mm to (210.0, 87.2), turned to 90 degrees
- moved IC1 57.3 mm to (216.5, 87.2)
- moved C7 55.6 mm to (211.8, 87.2), turned to 90 degrees
- moved D11 52.9 mm to (222.5, 87.2)
- moved JP8 46.8 mm to (225.0, 91.2), turned to -90 degrees
- moved R19 44.0 mm to (222.2, 84.5)
- moved R20 40.8 mm to (225.5, 87.2), turned to -90 degrees
- moved C8 40.6 mm to (226.0, 84.5), turned to 180 degrees
- moved J3 31.1 mm to (230.0, 87.0)
- moved J4 24.3 mm to (230.5, 74.2)
- moved C29 22.3 mm to (253.2, 26.0), turned to -90 degrees
- moved R22 17.3 mm to (225.8, 74.2), turned to -90 degrees
- moved C14 16.9 mm to (226.2, 71.5), turned to 180 degrees
- moved R29 16.3 mm to (262.5, 20.5), turned to -90 degrees
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
Commit message: mcu layout
Parts:
- C17, C21, C25, C28, FB1, FB2, R11, R12, R23, R24, R25, R26, R27: moved to B.Cu
- moved D12 269.0 mm to (227.8, 19.8)
- moved C9 268.6 mm to (224.5, 22.5), turned to 90 degrees
- moved C10 268.0 mm to (224.5, 26.5), turned to -90 degrees
- moved U2 266.3 mm to (230.1, 24.5)
- moved TP_3.3V1 252.7 mm to (226.2, 30.5), turned to 180 degrees
- moved C33 171.4 mm to (196.4, 22.8), turned to 90 degrees
- moved R30 170.5 mm to (202.3, 27.5)
- moved C31 166.6 mm to (202.3, 24.0)
- moved C32 166.1 mm to (195.6, 25.5), turned to 180 degrees
- moved R2 165.2 mm to (197.2, 29.0), turned to 180 degrees
- moved R1 164.4 mm to (197.2, 27.2)
- moved U4 163.0 mm to (199.0, 24.0)
- moved C30 162.5 mm to (202.3, 25.8)
- moved Reset1 71.0 mm to (109.8, 175.2), turned to 180 degrees
- moved U3 68.6 mm to (125.7, 165.2)
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Connections:
- C2 pad 2: +3.3V_ESP -> GND
- C3 pad 2: +3.3V_ESP -> GND
Routing:
- net Net-(U3-PF0-OSC_IN): track 0.00 -> 7.11 mm
- net Net-(U3-PF1-OSC_OUT): track 0.00 -> 6.90 mm
- net GND: track 0.00 -> 1.77 mm
Other:
- copper layers 2 -> 4
- board text added: "change this chud diode to the other one :("
- board text added: "pin headers for swd too"

Commit message: all subcircuits layout
Parts:
- removed TP4: ESP_RX, TestPoint:TestPoint_Loop_D1.80mm_Drill1.0mm_Beaded
- R4, R5, R7, R8: moved to B.Cu
- TP1: value GND_ESP -> GND
- TP3: value ESP_TX -> GND
- moved J2 245.4 mm to (227.3, 148.6)
- moved J5 245.4 mm to (227.3, 157.7)
- moved JP3 209.0 mm to (270.0, 112.5), turned to -90 degrees
- moved R7 205.9 mm to (248.8, 111.2)
- moved R4 205.3 mm to (239.8, 158.7), turned to 90 degrees
- moved JP4 204.4 mm to (270.0, 108.8), turned to -90 degrees
- moved R8 202.3 mm to (238.5, 162.2), turned to 180 degrees
- moved JP5 201.9 mm to (230.0, 29.8)
- moved TP1 201.6 mm to (236.8, 24.8)
- moved TP2 201.4 mm to (236.8, 30.0)
- moved R5 200.2 mm to (229.5, 30.5), turned to -90 degrees
- moved JP1 198.2 mm to (245.5, 109.8), turned to 180 degrees
- moved TP3 196.0 mm to (242.8, 119.2)
- moved D2 196.0 mm to (230.0, 32.0), turned to 180 degrees
- moved JP2 184.8 mm to (241.2, 113.2), turned to 90 degrees
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Connections:
- C10 pad 2: +3.3V -> /LDO/Vout
- C18 pad 1: /100PinMCU/3V3 -> +3.3V
- C20 pad 1: /100PinMCU/3V3 -> +3.3V
- C22 pad 1: /100PinMCU/3V3 -> +3.3V
- C24 pad 1: /100PinMCU/3V3 -> +3.3V
- C26 pad 1: /100PinMCU/3V3 -> +3.3V
- C27 pad 1: /100PinMCU/3V3 -> +3.3V
- FB2 pad 1: /100PinMCU/3V3 -> +3.3V
- J8 pad 1: /100PinMCU/3V3 -> +3.3V
- JP5 pad 1: /100PinMCU/3V3 -> /LDO/Vout
- R25 pad 2: /100PinMCU/3V3 -> +3.3V
- S1 pad 3: /100PinMCU/3V3 -> +3.3V
- TP3 pad 1: /ESP32/ESP_UART_TX -> GND
- TP_3.3V1 pad 1: +3.3V -> /LDO/Vout
- U2 pad 3: +3.3V -> /LDO/Vout
- U3 pad 100: /100PinMCU/3V3 -> +3.3V
- U3 pad 24: /100PinMCU/3V3 -> +3.3V
- U3 pad 49: /100PinMCU/3V3 -> +3.3V
- U3 pad 6: /100PinMCU/3V3 -> +3.3V
- U3 pad 64: /100PinMCU/3V3 -> +3.3V
- U3 pad 75: /100PinMCU/3V3 -> +3.3V
Other:
- board text added: "LEDs"
- board text added: "unhide fab layer silks for all jumpers + leds + tps"

Commit message: schem fixes + some semblance of layout ish
Parts:
- added J10: SWD_PinHeader, Connector_PinHeader_2.54mm:PinHeader_1x04_P2.54mm_Vertical, F.Cu at (40.3, 106.6)
- D6: value 1N5819HW-7-F -> D_Schottky
- moved JP6 229.2 mm to (47.3, 97.6)
- moved J6 228.7 mm to (55.8, 98.1), turned to 180 degrees
- moved C7 223.8 mm to (27.1, 93.8)
- moved C8 223.8 mm to (41.3, 91.0)
- moved D11 223.8 mm to (37.8, 93.8)
- moved IC1 223.8 mm to (31.8, 93.8)
- moved JP8 223.8 mm to (40.3, 97.8)
- moved R19 223.8 mm to (37.6, 91.0)
- moved R20 223.8 mm to (40.8, 93.8)
- moved C6 222.7 mm to (27.0, 97.4), turned to -90 degrees
- moved J3 221.6 mm to (47.3, 92.1), turned to 90 degrees
- moved C5 214.7 mm to (33.3, 97.9), turned to 180 degrees
- moved JP7 194.7 mm to (81.6, 97.3)
- moved C13 193.2 mm to (61.0, 93.5)
- moved C14 193.2 mm to (75.3, 90.7)
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Connections:
- J8 pad 3: Net-(J8-Pin_3) -> Net-(J10-Pin_3)
- J8 pad 4: Net-(J8-Pin_4) -> Net-(J10-Pin_3)
- R23 pad 2: Net-(J8-Pin_3) -> Net-(J10-Pin_3)
- R24 pad 2: Net-(J8-Pin_4) -> Net-(J10-Pin_3)
Routing:
- net +3.3V: track 0.00 -> 44.5 mm, vias 0 -> 3
- net GND: track 1.77 -> 16.9 mm
- net /100PinMCU/VDDA: track 0.00 -> 12.5 mm, vias 0 -> 1
- net /100PinMCU/GNDA: track 0.00 -> 11.6 mm, vias 0 -> 1
- net /100PinMCU/PG10-NRST: track 0.00 -> 6.77 mm, vias 0 -> 2
- net /LDO/Vout: track 0.00 -> 6.01 mm
- net /CAN_L2: track 0.00 -> 5.88 mm
- net /CAN_L1: track 0.00 -> 5.87 mm
- net Net-(D12-K): track 0.00 -> 5.39 mm
- net /CAN_H1: track 0.00 -> 4.29 mm
- net /CAN_H2: track 0.00 -> 4.25 mm
- net Net-(C8-Pad2): track 0.00 -> 3.96 mm
- net Net-(C14-Pad2): track 0.00 -> 3.96 mm
- net Net-(D2-A): track 0.00 -> 3.33 mm, vias 0 -> 1
- net Net-(JP8-A): track 0.00 -> 3.29 mm
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Other:
- board text removed: "LEDs"
- board text removed: "pin headers for swd too"
