File: 100PinMCU_TestBoard/100PinMCU_ESP32_TestBoard.kicad_pcb (KiCad board)
At the start: 4 copper layers, 116 parts, among them IC1 TCAN3413DR, IC2 TCAN3413DR, J1 ADC_Breakout, J10 SWD_PinHeader, J2 LogicAnalyzer_1, J3 CAN_1, J4 CAN_2, J5 LogicAnalyzer_2, J6 CAN_Breakout, J7 USB_C_Receptacle_USB2.0_16P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

Commit message: more layout but me go sleep now
Parts:
- C23, D17: moved to B.Cu
- D7: value SP0503BAHT -> TPD2EUSB30DRTR; footprint Package_TO_SOT_SMD:SOT-143 -> UTSVT_ICs:TPD2EUSB30DRTR
- moved J1 88.5 mm to (129.5, 115.9)
- moved JP6 83.0 mm to (127.5, 76.2), turned to 180 degrees
- moved D1 81.6 mm to (136.1, 115.4)
- moved R3 81.6 mm to (136.2, 113.7)
- moved D3 80.5 mm to (140.1, 115.4)
- moved R6 80.5 mm to (140.1, 113.7)
- moved R9 79.5 mm to (144.2, 113.7)
- moved D4 79.5 mm to (144.1, 115.4)
- moved D5 78.5 mm to (148.2, 115.4)
- moved R10 78.5 mm to (148.2, 113.7)
- moved R13 76.0 mm to (190.3, 85.5)
- moved SW1 76.0 mm to (196.6, 89.5)
- moved R15 76.0 mm to (188.6, 85.5)
- moved U1 75.1 mm to (186.4, 75.9)
- moved JP3 74.3 mm to (198.9, 77.4)
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Connections:
- D7 pad 1: GND -> /ESP32/USB_D-
- D7 pad 3: /ESP32/USB_D- -> GND
Routing:
- net +3.3V: track 44.5 -> 127.1 mm
- net /I2C2_SDA: track 0.00 -> 51.3 mm, vias 0 -> 3
- net /FDCAN1_TX: track 0.00 -> 46.1 mm, vias 0 -> 2
- net /FDCAN1_RX: track 0.00 -> 46.1 mm
- net /100PinMCU/SWDIO: track 0.00 -> 41.3 mm, vias 0 -> 1
- net /D-: track 0.00 -> 39.9 mm, vias 0 -> 2
- net /100PinMCU/SWCLK: track 0.00 -> 39.1 mm, vias 0 -> 1
- net /D+: track 0.00 -> 38.7 mm
- net /I2C2_SCL: track 0.00 -> 38.2 mm, vias 0 -> 2
- net /BOOT: track 0.00 -> 36.0 mm, vias 0 -> 1
- net /SPI1_MISO: track 0.00 -> 34.3 mm
- net /CAN_L2: track 5.88 -> 39.2 mm, vias 0 -> 1
- net /CAN_H2: track 4.25 -> 36.6 mm, vias 0 -> 1
- net /FDCAN2_TX: track 0.00 -> 32.1 mm, vias 0 -> 2
- net /100PinMCU/GNDA: track 11.6 -> 43.5 mm, vias 1 -> 2
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- added copper zone on B.Cu, net GND
- added copper zone on F.Cu, net GND
Other:
- board outline added: 113.5 x 49.1 mm
- board text added: "CAN1"
- board text added: "CAN2"
- board text added: "DEBUG"
- board text added: "EXT"
- board text added: "H L"
- board text added: "H1"
- board text added: "H2"
- board text added: "INPUT"
- board text added: "L1"
- board text added: "L2"
- board text added: "LOOPBACK"
- board text added: "SCL MISO NSS X GND"
- board text added: "SDA MOSI SCK GPIO1 X"
- board text added: "STM USB"
- board text added: "TERM"
- board text added: "USR"

Commit message: she's an onion now
Parts:
- added H1: MountingHole_Pad, MountingHole:MountingHole_3.2mm_M3_Pad_TopBottom, F.Cu at (87.3, 116.3)
- added H2: MountingHole_Pad, MountingHole:MountingHole_3.2mm_M3_Pad_TopBottom, F.Cu at (87.3, 72.7)
- added H3: MountingHole_Pad, MountingHole:MountingHole_3.2mm_M3_Pad_TopBottom, F.Cu at (197.1, 72.7)
- added H4: MountingHole_Pad, MountingHole:MountingHole_3.2mm_M3_Pad_TopBottom, F.Cu at (197.1, 116.2)
- C17, D17, R23, R24, R25, R26, R27, R4, R8: moved to F.Cu
- moved SW1 114.1 mm to (109.8, 163.6), turned to 180 degrees
- moved R13 109.6 mm to (116.4, 166.5), turned to 90 degrees
- moved R15 104.2 mm to (116.4, 160.7), turned to 90 degrees
- moved R7 89.8 mm to (265.9, 86.9)
- moved C2 89.8 mm to (265.6, 84.9)
- moved C3 89.8 mm to (267.6, 84.9)
- moved C4 89.8 mm to (266.6, 95.7)
- moved JP2 89.8 mm to (262.1, 92.2)
- moved R14 89.8 mm to (266.6, 97.4)
- moved SW2 89.8 mm to (266.6, 90.8)
- moved TP3 89.8 mm to (262.0, 96.8)
- moved JP1 89.8 mm to (262.6, 85.4)
- moved C30 79.7 mm to (249.6, 145.1)
- moved C31 79.7 mm to (249.6, 143.3)
- moved C32 79.7 mm to (242.8, 144.8)
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Connections:
- D7 pad 1: /ESP32/USB_D- -> /ESP32/USB_D+
- D7 pad 2: /ESP32/USB_D+ -> /ESP32/USB_D-
Routing:
- net +3.3V: track 127.1 -> 60.1 mm, vias 3 -> 14
- net /100PinMCU/PG10-NRST: track 6.77 -> 37.3 mm
- net /ESP32/ESP_UART_TX: track 0.00 -> 15.6 mm
- net /ESP32/ESP_UART_RX: track 0.00 -> 13.7 mm
- net /ESP32/VBUSB: track 0.00 -> 11.7 mm, vias 0 -> 2
- net /ESP32/USB_D+: track 0.00 -> 9.80 mm
- net /ESP32/USB_D-: track 0.00 -> 9.76 mm
- net /I2C2_SCL: track 38.2 -> 47.3 mm
- net GND: track 16.9 -> 24.2 mm, vias 1 -> 6
- net Net-(SW1-B): track 0.00 -> 6.90 mm
- net /100PinMCU/PE14: track 21.8 -> 28.5 mm
- net Net-(J10-Pin_3): track 15.6 -> 22.2 mm, vias 1 -> 0
- net /D+: track 38.7 -> 32.4 mm, vias 0 -> 2
- net /D-: track 39.9 -> 34.4 mm
- net +3.3V_ESP: track 0.00 -> 4.52 mm
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- added copper zone on B.Cu, net +3.3V
- added copper zone on In1.Cu, net +3.3V
- added copper zone on In2.Cu, net GND
- removed copper zone on B.Cu, net GND
Other:
- board size 113.5 x 49.1 mm -> 116.8 x 50.6 mm
- board text added: "3.3V"
- board text added: "BOOT LED"
- board text added: "CANH"
- board text added: "CANL"
- board text added: "ESP LEDs"
- board text added: "ESP USB"
- board text added: "GND"
- board text added: "GND X CAN_RX UART_RX BOOT"
- board text added: "LED1"
- board text added: "LED2"
- board text added: "PE11"
- board text added: "PE12"
- board text added: "PE14"
- board text added: "PE8"
- board text added: "PWR"
- board text added: "STM BOOT"
- board text added: "STM LEDs"
- board text added: "STM RESET"
- board text added: "STM32G4"
- board text added: "SWCLK"
- board text added: "SWCLK 3.3V"
- board text added: "SWDIO"
- board text added: "SWDIO GND"
- board text added: "UART RX"
- board text added: "UART TX"
- board text added: "VDDA ADC1 ADC2 ADC3 ADC4 GNDA"
- board text added: "X GPIO2 CAN_TX UART_TX X"
- board text removed: "change this chud diode to the other one :("
- board text removed: "unhide fab layer silks for all jumpers + leds + tps"

Commit message: initial layout (yes I will add funny silkscreen tmrw)
Parts:
- R5, R7: moved to F.Cu
- moved SW1 94.0 mm to (181.1, 102.3), turned to 90 degrees
- moved R13 93.4 mm to (187.1, 105.4)
- moved R15 91.9 mm to (187.1, 101.9)
- moved R30 89.1 mm to (182.0, 88.7), turned to 180 degrees
- moved R2 88.3 mm to (174.7, 94.2)
- moved C33 86.4 mm to (174.7, 90.0), turned to 180 degrees
- moved C32 86.2 mm to (174.6, 92.1)
- moved C30 85.7 mm to (182.0, 92.3)
- moved C31 85.7 mm to (182.0, 90.5)
- moved U4 85.3 mm to (178.3, 91.7)
- moved R1 84.2 mm to (178.5, 94.2), turned to 180 degrees
- moved R7 74.7 mm to (191.4, 93.0), turned to -90 degrees
- moved C4 73.5 mm to (193.1, 93.0), turned to -90 degrees
- moved TP3 73.2 mm to (191.2, 78.3)
- moved R14 71.9 mm to (194.8, 93.0), turned to 90 degrees
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Routing:
- net /100PinMCU/PC1: track 0.00 -> 74.6 mm, vias 0 -> 2
- net /100PinMCU/PC0: track 0.00 -> 71.7 mm, vias 0 -> 2
- net /BOOT: track 31.7 -> 102.5 mm, vias 2 -> 3
- net /100PinMCU/PG10-NRST: track 37.3 -> 107.6 mm, vias 2 -> 4
- net +3.3V_ESP: track 4.52 -> 66.6 mm, vias 0 -> 4
- net /100PinMCU/PD2: track 0.00 -> 62.0 mm, vias 0 -> 1
- net /100PinMCU/PA10: track 0.00 -> 59.8 mm, vias 0 -> 2
- net /100PinMCU/PA9: track 0.00 -> 56.6 mm, vias 0 -> 2
- net /FDCAN1_TX: track 49.2 -> 82.5 mm, vias 2 -> 3
- net /ESP32/USB_D+: track 9.80 -> 42.3 mm
- net /ESP32/USB_D-: track 9.76 -> 40.9 mm
- net /UART_TX: track 0.00 -> 29.7 mm, vias 0 -> 1
- net /UART_RX: track 0.00 -> 28.8 mm, vias 0 -> 1
- net /Power_Mux/VIN_2: track 2.64 -> 29.2 mm
- net /FDCAN1_RX: track 46.1 -> 72.7 mm
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Other:
- board size 116.8 x 50.6 mm -> 117.6 x 50.6 mm
- board text added: "ESP BOOT"
- board text added: "ESP RESET"
- board text added: "LDO"
- board text added: "PWR MUX"
- board text added: "RESET EN"
- board text added: "Rev X 2026: 100 Pin MCU Jolyn, Ravi & Surabhi"
- board text added: "VOUT"

Commit message: oops my edge cuts were weird
Parts:
- moved H1 0.22 mm to (87.6, 116.4)
- moved H4 0.14 mm to (198.3, 116.4)
- moved H2 0.14 mm to (87.6, 72.6)
- moved H3 0.10 mm to (198.3, 72.6)
Other:
- board size 117.6 x 50.6 mm -> 117.5 x 50.6 mm
Changed lines of the file:
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@@
 	(footprint "MountingHole:MountingHole_3.2mm_M3_Pad_TopBottom"
 		(layer "F.Cu")
-		(at 198.2 116.3)
+		(at 198.3 116.4)
 		(descr "Mounting Hole 3.2mm, M3, generated by kicad-footprint-generator mountinghole.py")
 		(tags "mountinghole M3")
@@
 	(footprint "MountingHole:MountingHole_3.2mm_M3_Pad_TopBottom"
 		(layer "F.Cu")
-		(at 198.3 72.7)
+		(at 198.3 72.6)
 		(descr "Mounting Hole 3.2mm, M3, generated by kicad-footprint-generator mountinghole.py")
 		(tags "mountinghole M3")
@@
 	(footprint "MountingHole:MountingHole_3.2mm_M3_Pad_TopBottom"
 		(layer "F.Cu")
-		(at 87.7 72.7)
+		(at 87.6 72.6)
 		(descr "Mounting Hole 3.2mm, M3, generated by kicad-footprint-generator mountinghole.py")
 		(tags "mountinghole M3")
@@
 	(footprint "MountingHole:MountingHole_3.2mm_M3_Pad_TopBottom"
 		(layer "F.Cu")
-		(at 87.8 116.3)
+		(at 87.6 116.4)
 		(descr "Mounting Hole 3.2mm, M3, generated by kicad-footprint-generator mountinghole.py")
 		(tags "mountinghole M3")
@@
 	)
 	(gr_line
-		(start 84.2 116.8)
-		(end 84.2 72.225)
+		(start 198.5 119.8)
+		(end 87.4 119.8)
 		(stroke
 			(width 0.05)
@@
 		(layer "Edge.Cuts")
 	)
-	(gr_arc
-		(start 201.8 116.8)
-		(mid 200.92132 118.92132)
-		(end 198.8 119.8)
+	(gr_line
+		(start 87.4 69.2)
+		(end 198.5 69.2)
 		(stroke
 			(width 0.05)
@@
 	)
 	(gr_arc
-		(start 84.2 72.225)
-		(mid 85.07868 70.10368)
-		(end 87.2 69.225)
+		(start 201.7 116.6)
+		(mid 200.762742 118.862742)
+		(end 198.5 119.8)
 		(stroke
 			(width 0.05)
@@
 	)
 	(gr_line
-		(start 201.8 72.225)
-		(end 201.8 116.8)
+		(start 84.2 116.6)
+		(end 84.2 72.4)
 		(stroke
 			(width 0.05)
@@
 		(layer "Edge.Cuts")
 	)
-	(gr_line
-		(start 198.8 119.8)
-		(end 87.2 119.8)
+	(gr_arc
+		(start 87.4 119.8)
+		(mid 85.137258 118.862742)
+		(end 84.2 116.6)
 		(stroke
 			(width 0.05)
@@
 		(layer "Edge.Cuts")
 	)
-	(gr_line
-		(start 87.2 69.225)
-		(end 198.8 69.225)
+	(gr_arc
+		(start 84.2 72.4)
+		(mid 85.137258 70.137258)
+		(end 87.4 69.2)
 		(stroke
 			(width 0.05)
@@
 	)
 	(gr_arc
-		(start 198.8 69.225)
-		(mid 200.92132 70.10368)
-		(end 201.8 72.225)
+		(start 198.5 69.2)
+		(mid 200.762742 70.137258)
+		(end 201.7 72.4)
 		(stroke
 			(width 0.05)
@@
 		(layer "Edge.Cuts")
 	)
-	(gr_arc
-		(start 87.2 119.8)
-		(mid 85.07868 118.92132)
-		(end 84.2 116.8)
+	(gr_line
+		(start 201.7 72.4)
+		(end 201.7 116.6)
 		(stroke
 			(width 0.05)
@@
 	)
 	(gr_text "UART\nTX"
-		(at 188.3 114.4 0)
+		(at 188.3 114.6 0)
 		(layer "F.SilkS" knockout)
 		(effects
@@
 	)
 	(gr_text "UART\nRX"
-		(at 188.1 118.4 0)
+		(at 188.1 118.5 0)
 		(layer "F.SilkS" knockout)
 		(effects
@@
 		)
 	)
+	(dimension
+		(type orthogonal)
+		(layer "Dwgs.User")
+		(pts
+			(xy 84.2 75.9) (xy 201.8 76)
+		)
+		(height -10.8)
+		(orientation 0)
+		(format
+			(prefix "")
+			(suffix "")
+			(units 3)
+			(units_format 0)
+			(precision 4)
+			(suppress_zeroes yes)
+		)
+		(style
+			(thickness 0.1)
+			(arrow_length 1.27)
+			(text_position_mode 0)
+			(arrow_direction outward)
+			(extension_height 0.58642)
+			(extension_offset 0.5)
+			(keep_text_aligned yes)
+		)
+		(gr_text "117.6"
+			(at 143 63.95 0)
+			(layer "Dwgs.User")
+			(effects
+				(font
+					(size 1 1)
+					(thickness 0.15)
+				)
+			)
+		)
+	)
+	(dimension
+		(type orthogonal)
+		(layer "Dwgs.User")
+		(pts
+			(xy 91.7 69.2) (xy 91.5 119.8)
+		)
+		(height -9)
+		(orientation 1)
+		(format
+			(prefix "")
+			(suffix "")
+			(units 3)
+			(units_format 0)
+			(precision 4)
+			(suppress_zeroes yes)
+		)
+		(style
+			(thickness 0.1)
+			(arrow_length 1.27)
+			(text_position_mode 0)
+			(arrow_direction outward)
+			(extension_height 0.58642)
+			(extension_offset 0.5)
+			(keep_text_aligned yes)
+		)
+		(gr_text "50.6"
+			(at 81.55 94.5 90)
+			(layer "Dwgs.User")
+			(effects
+				(font
+					(size 1 1)
+					(thickness 0.15)
+				)
+			)
+		)
+	)

Commit message: ravi comments addressed
Parts:
- added G***: LHRs_LOGO, UTSVT_Logos:LHRs_LOGO, B.Cu at (171.7, 115.5)
- moved C29 7.09 mm to (167.6, 82.8)
- moved C1 6.24 mm to (184.9, 81.0)
- moved D16 5.36 mm to (162.3, 79.2)
- moved D7 5.28 mm to (179.8, 79.2)
- moved D6 1.73 mm to (184.4, 78.3), turned to 180 degrees
- moved J9 0.90 mm to (162.8, 72.0)
- moved R28 0.90 mm to (161.1, 72.0)
- moved R29 0.90 mm to (164.1, 72.0)
- moved J7 0.84 mm to (180.3, 72.0)
- moved R11 0.84 mm to (181.6, 72.2)
- moved R12 0.84 mm to (178.6, 72.2)
- moved D17 0.65 mm to (166.8, 80.0), turned to 180 degrees
Routing:
- net /LDO/Vout: track 24.8 -> 0.00 mm
- net /Power_Mux/VIN_2: track 29.2 -> 8.13 mm, vias 0 -> 2
- net /ESP32/+5V_LDO_IN: track 26.2 -> 10.5 mm, vias 2 -> 4
- net /ESP32/VBUSB: track 12.5 -> 3.99 mm
- net /USB-C/VBUS_IN: track 12.3 -> 5.96 mm
- net /ESP32/USB_D+: track 42.3 -> 36.9 mm
- net /100PinMCU/PG10-NRST: track 107.6 -> 112.8 mm, vias 4 -> 3
- net /ESP32/USB_D-: track 40.9 -> 36.5 mm
- net +3.3V: track 60.1 -> 56.3 mm, vias 16 -> 15
- net /100PinMCU/SWCLK: track 38.1 -> 41.2 mm
- net /D+: track 32.4 -> 35.3 mm, vias 2 -> 0
- net /I2C2_SDA: track 57.8 -> 54.9 mm
- net /D-: track 34.4 -> 36.4 mm, vias 2 -> 0
- net Net-(U3-PF0-OSC_IN): track 7.11 -> 5.61 mm
- net /USB-C/CC2: track 2.81 -> 3.62 mm
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- added copper zone on In1.Cu, net /ESP32/+5V_LDO_IN
- added copper zone on B.Cu, net /ESP32/VBUSB
- added copper zone on F.Cu, net /LDO/Vout
- added copper zone on In2.Cu, net /Power_Mux/VIN_2
- added copper zone on B.Cu, net /USB-C/VBUS_IN
Other:
- board text added: "GPIO 20"
- board text added: "GPIO 21"
- board text removed: "LED1"
- board text removed: "LED2"

Commit message: silkscreen + gerbers
Parts:
- added G***: LOGO, LOGO, B.Cu at (186.7, 98.5)
- added G***: LOGO, LOGO, B.Cu at (159.1, 109.5)
Other:
- board text added: "ee yes pee"
- board text added: "he's just like me fr"
- board text added: "wait which way does this go again?"
- board text added: "will ravi notice maid-ravi before ordering?"
