File: 100PinMCU_TestBoard/100PinMCU_ESP32_TestBoard.kicad_pcb (KiCad board)
At the start: 4 copper layers, 117.5 x 50.6 mm, 123 parts, among them IC1 TCAN3413DR, IC2 TCAN3413DR, J1 ADC_Breakout, J10 SWD_PinHeader, J2 LogicAnalyzer_1, J3 CAN_1, J4 CAN_2, J5 LogicAnalyzer_2, J6 CAN_Breakout, J7 USB_C_Receptacle_USB2.0_16P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

Commit message: almost pulled a prat
Routing:
- net GND: track 41.8 -> 60.4 mm, vias 12 -> 17
- net +3.3V: track 56.3 -> 59.0 mm, vias 15 -> 16
- net +3.3V_ESP: track 66.6 -> 64.8 mm
- net (no net): vias 122 -> 138
