File: 48PinMCU_TestBoard/CAN_Transceiver.kicad_sch (KiCad schematic)
At the start: 9 parts, among them IC1 TCAN3413DR

Commit message: fixes made
Parts:
- JP1: footprint Connector_PinHeader_2.54mm:PinHeader_2x14_P2.54mm_Vertical -> Connector_PinHeader_2.54mm:PinHeader_1x02_P2.54mm_Vertical
Changed lines of the file:
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@@
+		)
+	)
+	(hierarchical_label "GND"
+		(shape input)
+		(at 93.98 72.39 0)
+		(effects
+			(font
+				(size 1.27 1.27)
+			)
+			(justify left)
 		)
 	)
@@
 		)
 	)
+	(hierarchical_label "GND"
+		(shape input)
+		(at 114.3 67.31 0)
+		(effects
+			(font
+				(size 1.27 1.27)
+			)
+			(justify left)
+		)
+	)
 	(hierarchical_label "CAN_L"
 		(shape bidirectional)
@@
 		(shape input)
 		(at 177.8 44.45 0)
-		(effects
-			(font
-				(size 1.27 1.27)
-			)
-			(justify left)
-		)
-	)
-	(hierarchical_label "GND"
-		(shape input)
-		(at 93.98 72.39 0)
-		(effects
-			(font
-				(size 1.27 1.27)
-			)
-			(justify left)
-		)
-	)
-	(hierarchical_label "GND"
-		(shape input)
-		(at 114.3 67.31 0)
 		(effects
 			(font
@@
 			)
 		)
-		(property "Footprint" "Connector_PinHeader_2.54mm:PinHeader_2x14_P2.54mm_Vertical"
+		(property "Footprint" "Connector_PinHeader_2.54mm:PinHeader_1x02_P2.54mm_Vertical"
 			(at 180.34 69.85 0)
 			(effects
@@
 		)
 		(instances
-			(project ""
-				(path "/69b823fd-c065-40ff-9bb9-c5835555f3eb/9d9eae1e-c713-4323-9845-a569cff8d5d3"
-					(reference "JP2")
-					(unit 1)
-				)
-			)
-			(project ""
-				(path "/81d906df-a099-480a-8398-28a8e913d125"
-					(reference "JP1")
-					(unit 1)
-				)
-			)
-			(project ""
+			(project "48PinMCU_TestBoard"
 				(path "/9cc459e0-f86d-41bb-8426-cce80d92e44c/b2b34277-6380-4c83-b190-63063b84f81a"
 					(reference "JP1")
 					(unit 1)
-				)
-			)
-			(project "CAN_Transceiver"
-				(path "/a09f9696-80ee-4697-8aaa-225f287b667b"
-					(reference "JP1")
-					(unit 1)

Commit message: All fixes fixed
Parts:
- renumbered C26 to C23, C27 to C24, C28 to C27, D10 to D18, IC1 to IC2, JP1 to JP15, R18 to R30, R19 to R31
Changed lines of the file:
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@@
 		(on_board yes)
 		(dnp no)
-		(property "Reference" "C27"
+		(property "Reference" "C24"
 			(at 40.64 58.42 0)
 			(effects
@@
 			(project ""
 				(path "/9cc459e0-f86d-41bb-8426-cce80d92e44c/b2b34277-6380-4c83-b190-63063b84f81a"
-					(reference "C27")
+					(reference "C24")
 					(unit 1)
 				)
@@
 		(dnp no)
 		(fields_autoplaced yes)
-		(property "Reference" "IC1"
+		(property "Reference" "IC2"
 			(at 92.71 48.26 0)
 			(effects
@@
 			(project ""
 				(path "/9cc459e0-f86d-41bb-8426-cce80d92e44c/b2b34277-6380-4c83-b190-63063b84f81a"
-					(reference "IC1")
+					(reference "IC2")
 					(unit 1)
 				)
@@
 		(dnp no)
 		(fields_autoplaced yes)
-		(property "Reference" "JP1"
+		(property "Reference" "JP15"
 			(at 180.34 63.5 0)
 			(effects
@@
 			(project "48PinMCU_TestBoard"
 				(path "/9cc459e0-f86d-41bb-8426-cce80d92e44c/b2b34277-6380-4c83-b190-63063b84f81a"
-					(reference "JP1")
+					(reference "JP15")
 					(unit 1)
 				)
@@
 		(dnp no)
 		(fields_autoplaced yes)
-		(property "Reference" "D10"
+		(property "Reference" "D18"
 			(at 161.29 31.75 0)
 			(effects
@@
 			(project ""
 				(path "/9cc459e0-f86d-41bb-8426-cce80d92e44c/b2b34277-6380-4c83-b190-63063b84f81a"
-					(reference "D10")
+					(reference "D18")
 					(unit 1)
 				)
@@
 		(on_board yes)
 		(dnp no)
-		(property "Reference" "C28"
+		(property "Reference" "C27"
 			(at 52.578 58.42 0)
 			(effects
@@
 			(project ""
 				(path "/9cc459e0-f86d-41bb-8426-cce80d92e44c/b2b34277-6380-4c83-b190-63063b84f81a"
-					(reference "C28")
+					(reference "C27")
 					(unit 1)
 				)
@@
 		(on_board yes)
 		(dnp no)
-		(property "Reference" "C26"
+		(property "Reference" "C23"
 			(at 29.718 58.42 0)
 			(effects
@@
 			(project ""
 				(path "/9cc459e0-f86d-41bb-8426-cce80d92e44c/b2b34277-6380-4c83-b190-63063b84f81a"
-					(reference "C26")
+					(reference "C23")
 					(unit 1)
 				)
@@
 		(on_board yes)
 		(dnp no)
-		(property "Reference" "R19"
+		(property "Reference" "R31"
 			(at 166.37 64.77 90)
 			(effects
@@
 			(project ""
 				(path "/9cc459e0-f86d-41bb-8426-cce80d92e44c/b2b34277-6380-4c83-b190-63063b84f81a"
-					(reference "R19")
+					(reference "R31")
 					(unit 1)
 				)
@@
 		(on_board yes)
 		(dnp no)
-		(property "Reference" "R18"
+		(property "Reference" "R30"
 			(at 140.97 64.77 90)
 			(effects
@@
 			(project ""
 				(path "/9cc459e0-f86d-41bb-8426-cce80d92e44c/b2b34277-6380-4c83-b190-63063b84f81a"
-					(reference "R18")
-					(unit 1)
-				)
+					(reference "R30")
+					(unit 1)
+				)
