File: 48PinMCU_TestBoard/LDO.kicad_sch (KiCad schematic)
At the start: 4 parts, among them U3 MCP1826S

Commit message: All fixes fixed
Parts:
- renumbered D9 to D17
Changed lines of the file:
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@@
 		(dnp no)
 		(fields_autoplaced yes)
-		(property "Reference" "D9"
+		(property "Reference" "D17"
 			(at 47.244 39.37 0)
 			(effects
@@
 			(project ""
 				(path "/9cc459e0-f86d-41bb-8426-cce80d92e44c/ede07d47-91ad-43c5-ac5b-8c9172101cbc"
-					(reference "D9")
+					(reference "D17")
 					(unit 1)
 				)
