File: 48PinMCU_TestBoard/ESP32.kicad_sch (KiCad schematic)
At the start: 24 parts, among them J2 USB_C_Receptacle_USB2.0_16P, SW3 BOOT Switch, SW4 RESET Button, U2 ESP32-C6-MINI-1

Commit message: fixes made
Parts:
- removed C17: 10uF, Capacitor_SMD:C_0805_2012Metric_Pad1.18x1.45mm_HandSolder, symbol Device:C
- removed C18: 0.1uF, Capacitor_SMD:C_0603_1608Metric_Pad1.08x0.95mm_HandSolder, symbol Device:C
- SW4: footprint UTSVT_Special:450406020024 -> UTSVT_ESP32:TL3365AF180QG

Commit message: All fixes fixed
Parts:
- renumbered C16 to C18, D3 to D11, D4 to D12, D5 to D13, D6 to D14, D7 to D15, D8 to D16, J2 to J6, R6 to R19, R7 to R20, R8 to R21, R9 to R22, R10 to R23, R11 to R24, R12 to R25, R21 to R26, R13 to R27, R14 to R28
Connections:
- net VBUSB: no longer D15.2 (A), J6.A4 (VBUS), J6.A9 (VBUS), J6.B4 (VBUS), J6.B9 (VBUS)
- new net VBUS: D15.2 (A), J6.A4 (VBUS), J6.A9 (VBUS), J6.B4 (VBUS), J6.B9 (VBUS)
Changed lines of the file:
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@@
 		)
 	)
-	(label "VBUSB"
+	(label "VBUS"
 		(at 78.74 29.21 0)
 		(effects
@@
 		(on_board yes)
 		(dnp no)
-		(property "Reference" "R8"
+		(property "Reference" "R21"
 			(at 73.406 122.936 90)
 			(effects
@@
 			(project ""
 				(path "/9cc459e0-f86d-41bb-8426-cce80d92e44c/34d16e22-f6a7-4a85-a60f-fa2e3b96ee10"
-					(reference "R8")
+					(reference "R21")
 					(unit 1)
 				)
@@
 		(on_board yes)
 		(dnp no)
-		(property "Reference" "C16"
+		(property "Reference" "C18"
 			(at 103.378 35.306 0)
 			(effects
@@
 			(project ""
 				(path "/9cc459e0-f86d-41bb-8426-cce80d92e44c/34d16e22-f6a7-4a85-a60f-fa2e3b96ee10"
-					(reference "C16")
+					(reference "C18")
 					(unit 1)
 				)
@@
 		(on_board yes)
 		(dnp no)
-		(property "Reference" "D4"
+		(property "Reference" "D12"
 			(at 87.63 110.49 0)
 			(effects
@@
 			(project ""
 				(path "/9cc459e0-f86d-41bb-8426-cce80d92e44c/34d16e22-f6a7-4a85-a60f-fa2e3b96ee10"
-					(reference "D4")
+					(reference "D12")
 					(unit 1)
 				)
@@
 		(on_board yes)
 		(dnp no)
-		(property "Reference" "R9"
+		(property "Reference" "R22"
 			(at 73.66 134.366 90)
 			(effects
@@
 			(project ""
 				(path "/9cc459e0-f86d-41bb-8426-cce80d92e44c/34d16e22-f6a7-4a85-a60f-fa2e3b96ee10"
-					(reference "R9")
+					(reference "R22")
 					(unit 1)
 				)
@@
 		(on_board yes)
 		(dnp no)
-		(property "Reference" "D6"
+		(property "Reference" "D14"
 			(at 87.63 133.858 0)
 			(effects
@@
 			(project ""
 				(path "/9cc459e0-f86d-41bb-8426-cce80d92e44c/34d16e22-f6a7-4a85-a60f-fa2e3b96ee10"
-					(reference "D6")
+					(reference "D14")
 					(unit 1)
 				)
@@
 		(on_board yes)
 		(dnp no)
-		(property "Reference" "R14"
+		(property "Reference" "R28"
 			(at 227.584 101.854 90)
 			(effects
@@
 			(project ""
 				(path "/9cc459e0-f86d-41bb-8426-cce80d92e44c/34d16e22-f6a7-4a85-a60f-fa2e3b96ee10"
-					(reference "R14")
+					(reference "R28")
 					(unit 1)
 				)
@@
 		(dnp no)
 		(fields_autoplaced yes)
-		(property "Reference" "R12"
+		(property "Reference" "R25"
 			(at 137.16 29.21 90)
 			(effects
@@
 			(project ""
 				(path "/9cc459e0-f86d-41bb-8426-cce80d92e44c/34d16e22-f6a7-4a85-a60f-fa2e3b96ee10"
-					(reference "R12")
+					(reference "R25")
 					(unit 1)
 				)
@@
 		(on_board yes)
 		(dnp no)
-		(property "Reference" "R11"
+		(property "Reference" "R24"
 			(at 79.248 38.1 90)
 			(effects
@@
 			(project ""
 				(path "/9cc459e0-f86d-41bb-8426-cce80d92e44c/34d16e22-f6a7-4a85-a60f-fa2e3b96ee10"
-					(reference "R11")
+					(reference "R24")
 					(unit 1)
 				)
@@
 		(on_board yes)
 		(dnp no)
-		(property "Reference" "R13"
+		(property "Reference" "R27"
 			(at 180.594 25.654 0)
 			(effects
@@
 			(project ""
 				(path "/9cc459e0-f86d-41bb-8426-cce80d92e44c/34d16e22-f6a7-4a85-a60f-fa2e3b96ee10"
-					(reference "R13")
+					(reference "R27")
 					(unit 1)
 				)
@@
 		(on_board yes)
 		(dnp no)
-		(property "Reference" "D7"
+		(property "Reference" "D15"
 			(at 90.932 22.86 0)
 			(effects
@@
 			(project ""
 				(path "/9cc459e0-f86d-41bb-8426-cce80d92e44c/34d16e22-f6a7-4a85-a60f-fa2e3b96ee10"
-					(reference "D7")
+					(reference "D15")
 					(unit 1)
 				)
@@
 		(on_board yes)
 		(dnp no)
-		(property "Reference" "R10"
+		(property "Reference" "R23"
 			(at 79.502 33.02 90)
 			(effects
@@
 			(project ""
 				(path "/9cc459e0-f86d-41bb-8426-cce80d92e44c/34d16e22-f6a7-4a85-a60f-fa2e3b96ee10"
-					(reference "R10")
+					(reference "R23")
 					(unit 1)
 				)
@@
 		(on_board yes)
 		(dnp no)
-		(property "Reference" "R21"
+		(property "Reference" "R26"
 			(at 150.114 76.454 0)
 			(effects
@@
 			(project "48PinMCU_TestBoard"
 				(path "/9cc459e0-f86d-41bb-8426-cce80d92e44c/34d16e22-f6a7-4a85-a60f-fa2e3b96ee10"
-					(reference "R21")
+					(reference "R26")
 					(unit 1)
 				)
@@
 		(dnp no)
 		(fields_autoplaced yes)
-		(property "Reference" "J2"
+		(property "Reference" "J6"
 			(at 60.96 21.59 0)
 			(effects
@@
 			(project ""
 				(path "/9cc459e0-f86d-41bb-8426-cce80d92e44c/34d16e22-f6a7-4a85-a60f-fa2e3b96ee10"
-					(reference "J2")
+					(reference "J6")
 					(unit 1)
 				)
@@
 		(on_board yes)
 		(dnp no)
-		(property "Reference" "D5"
+		(property "Reference" "D13"
 			(at 87.376 121.666 0)
 			(effects
@@
 			(project ""
 				(path "/9cc459e0-f86d-41bb-8426-cce80d92e44c/34d16e22-f6a7-4a85-a60f-fa2e3b96ee10"
-					(reference "D5")
+					(reference "D13")
 					(unit 1)
 				)
@@
 		(dnp no)
 		(fields_autoplaced yes)
-		(property "Reference" "R7"
+		(property "Reference" "R20"
 			(at 73.66 111.76 90)
 			(effects
@@
 			(project ""
 				(path "/9cc459e0-f86d-41bb-8426-cce80d92e44c/34d16e22-f6a7-4a85-a60f-fa2e3b96ee10"
-					(reference "R7")
+					(reference "R20")
 					(unit 1)
 				)
@@
 		(dnp no)
 		(fields_autoplaced yes)
-		(property "Reference" "R6"
+		(property "Reference" "R19"
 			(at 73.66 100.33 90)
 			(effects
@@
 			(project ""
 				(path "/9cc459e0-f86d-41bb-8426-cce80d92e44c/34d16e22-f6a7-4a85-a60f-fa2e3b96ee10"
-					(reference "R6")
+					(reference "R19")
 					(unit 1)
 				)
@@
 		(on_board yes)
 		(dnp no)
-		(property "Reference" "D3"
+		(property "Reference" "D11"
 			(at 87.63 99.06 0)
 			(effects
@@
 			(project ""
 				(path "/9cc459e0-f86d-41bb-8426-cce80d92e44c/34d16e22-f6a7-4a85-a60f-fa2e3b96ee10"
-					(reference "D3")
+					(reference "D11")
 					(unit 1)
 				)
@@
 		(on_board yes)
 		(dnp no)
-		(property "Reference" "#PWR0101"
+		(property "Reference" "#PWR030"
 			(at 238.76 109.22 0)
 			(effects
@@
 			(project ""
 				(path "/9cc459e0-f86d-41bb-8426-cce80d92e44c/34d16e22-f6a7-4a85-a60f-fa2e3b96ee10"
-					(reference "#PWR0101")
+					(reference "#PWR030")
 					(unit 1)
 				)
@@
 		(dnp no)
 		(fields_autoplaced yes)
-		(property "Reference" "D8"
+		(property "Reference" "D16"
 			(at 236.22 24.13 0)
 			(effects
@@
 			(project ""
 				(path "/9cc459e0-f86d-41bb-8426-cce80d92e44c/34d16e22-f6a7-4a85-a60f-fa2e3b96ee10"
-					(reference "D8")
-					(unit 1)
-				)
+					(reference "D16")
+					(unit 1)
+				)

Commit message: preliminary layout blocks
Parts:
- removed R26: 10k, Resistor_SMD:R_0603_1608Metric_Pad0.98x0.95mm_HandSolder, symbol Device:R
Connections:
- net VBUSB is gone; now on net VBUS: R20.1
Changed lines of the file:
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@@
-	)
-	(junction
-		(at 156.21 86.36)
-		(diameter 0)
-		(color 0 0 0 0)
 	)
 	(junction
@@
 	(wire
 		(pts
-			(xy 156.21 86.36) (xy 158.75 86.36)
+			(xy 149.86 86.36) (xy 158.75 86.36)
 		)
 		(stroke
@@
 	(wire
 		(pts
-			(xy 156.21 82.55) (xy 156.21 86.36)
-		)
-		(stroke
-			(width 0)
-			(type default)
-		)
-	)
-	(wire
-		(pts
 			(xy 100.33 105.41) (xy 100.33 116.84)
 		)
@@
 		(pts
 			(xy 100.33 31.75) (xy 100.33 29.21)
-		)
-		(stroke
-			(width 0)
-			(type default)
-		)
-	)
-	(wire
-		(pts
-			(xy 149.86 86.36) (xy 156.21 86.36)
-		)
-		(stroke
-			(width 0)
-			(type default)
-		)
-	)
-	(wire
-		(pts
-			(xy 156.21 71.12) (xy 156.21 74.93)
 		)
 		(stroke
@@
 		)
 	)
-	(label "VBUSB"
+	(label "VBUS"
 		(at 60.96 116.84 0)
 		(effects
@@
 			)
 			(justify left)
-		)
-	)
-	(hierarchical_label "+3.3V_ESP"
-		(shape input)
-		(at 156.21 71.12 180)
-		(effects
-			(font
-				(size 1.27 1.27)
-			)
-			(justify right)
 		)
 	)
@@
 					(unit 1)
 				)
-			)
-		)
-	)
-	(symbol
-		(lib_id "Device:R")
-		(at 156.21 78.74 0)
-		(unit 1)
-		(exclude_from_sim no)
-		(in_bom yes)
-		(on_board yes)
-		(dnp no)
-		(property "Reference" "R26"
-			(at 150.114 76.454 0)
-			(effects
-				(font
-					(size 1.27 1.27)
-				)
-				(justify left)
-			)
-		)
-		(property "Value" "10k"
-			(at 150.114 78.994 0)
-			(effects
-				(font
-					(size 1.27 1.27)
-				)
-				(justify left)
-			)
-		)
-		(property "Footprint" "Resistor_SMD:R_0603_1608Metric_Pad0.98x0.95mm_HandSolder"
-			(at 154.432 78.74 90)
-			(effects
-				(font
-					(size 1.27 1.27)
-				)
-				(hide yes)
-			)
-		)
-		(property "Datasheet" "kicad-embed://dcrcwe3.pdf"
-			(at 156.21 78.74 0)
-			(effects
-				(font
-					(size 1.27 1.27)
-				)
-				(hide yes)
-			)
-		)
-		(property "Description" "resistor"
-			(at 156.21 78.74 0)
-			(effects
-				(font
-					(size 1.27 1.27)
-				)
-				(hide yes)
-			)
-		)
-		(property "P/N" "CRCW060310K0FKEI "
-			(at 156.21 78.74 90)
-			(effects
-				(font
-					(size 1.27 1.27)
-				)
-				(hide yes)
-			)
-		)
-		(property "LCSC P/N" "C25804"
-			(at 156.21 78.74 90)
-			(effects
-				(font
-					(size 1.27 1.27)
-					(thickness 0.1588)
-				)
-				(hide yes)
-			)
-		)
-		(pin "1"
-		)
-		(pin "2"
-		)
-		(instances
-			(project "48PinMCU_TestBoard"
-				(path "/9cc459e0-f86d-41bb-8426-cce80d92e44c/34d16e22-f6a7-4a85-a60f-fa2e3b96ee10"
-					(reference "R26")
-					(unit 1)
-				)

Commit message: added bypass caps in series with ESP DC input
Parts:
- added C17: 0.1uF, Capacitor_SMD:C_0603_1608Metric_Pad1.08x0.95mm_HandSolder, symbol Device:C
- added C31: 10uF, Capacitor_SMD:C_0805_2012Metric_Pad1.18x1.45mm_HandSolder, symbol Device:C
Connections:
- net +3.3V_ESP: now also C17.1, C31.1
- net GND: now also C17.2, C31.2
