File: PowerPath_TestBoard/PowerPath.kicad_sch (KiCad schematic)
At the start: 41 parts, among them J1 24V Test, J2 +24V_Ext, J3 12V Test, J4 5V Test, J5 3V Test, J6 +V_in_24V, J7 GND, J8 +Vin_5V, J9 +3V3_Ext

Commit message: addressed all final comments, review?
Parts:
- removed F1: 5A, UTSVT_Connectors:FUSE_3568, symbol utsvt_power:Fuse_3568
- removed J9: +3V3_Ext, UTSVT_Connectors:5754, symbol Connector_Generic:Conn_01x01
- removed TP2: Fault, TestPoint:TestPoint_THTPad_D3.0mm_Drill1.5mm, symbol Connector:TestPoint
- removed TP3: IMON, TestPoint:TestPoint_THTPad_D3.0mm_Drill1.5mm, symbol Connector:TestPoint
- added F1: 5A, UTSVT_Power:Fuse-3557-2, symbol utsvt_power:Fuse_3557_2
- added H1, H2, H3, H4: MountingHole, MountingHole:MountingHole_3mm_Pad_TopBottom, symbol Mechanical:MountingHole
- renumbered J3 to J4, J4 to J5, J5 to J6, J6 to J7, J7 to J8, J8 to J9, TP4 to TP2, TP5 to TP3, TP6 to TP4, TP7 to TP5, TP8 to TP6
Connections:
- net +24V_Ext: now also F1.2
- net +24V_Ext_In: now also F1.1
- net 24V_OUT renamed Vout_24V
Other:
- sheet PowerProtection ports: added Vin, Vout; removed 24V_Ext, 24V_OUT, Fault, IMON_OUT
