File: PowerPath_TestBoard/PowerPath.kicad_sch (KiCad schematic)
At the start: 42 parts, among them J1 24V Test, J2 +24V_Ext, J4 12V Test, J5 5V Test, J6 3V Test, J7 +V_in_24V, J8 GND, J9 +Vin_5V

Commit message: finished tony's review, should be good?
Parts:
- removed H1, H2, H3, H4: MountingHole, MountingHole:MountingHole_3mm_Pad_TopBottom, symbol Mechanical:MountingHole
- added H1, H2, H3, H5: MountingHole_Pad_MP, MountingHole:MountingHole_3mm_Pad_TopBottom, symbol Mechanical:MountingHole_Pad_MP
- added TP20, TP21: GND, TestPoint:TestPoint_THTPad_D3.0mm_Drill1.5mm, symbol Connector:TestPoint
Connections:
- net GND: now also TP20.1, TP21.1
- no-connect marks 0 -> 4
