File: PowerPath_TestBoard/LDO.kicad_sch (KiCad schematic)
At the start: 5 parts, among them U1 MCP1826S_LDO

Commit message: addressed all reviews, starting layout
Parts:
- renumbered C7 to C6, C8 to C7, D1 to D11, U1 to U2
Changed lines of the file:
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@@
 		(dnp no)
 		(fields_autoplaced yes)
-		(property "Reference" "C8"
+		(property "Reference" "C7"
 			(at 64.77 50.7935 0)
 			(effects
@@
 			(project "LDO"
 				(path "/ad6c7df0-eb90-4670-9aa8-3e2007aefc2d/8ef5b44a-1ea6-4b34-80bc-234862ce4b8d"
-					(reference "C8")
+					(reference "C7")
 					(unit 1)
 				)
@@
 		(dnp no)
 		(fields_autoplaced yes)
-		(property "Reference" "U1"
+		(property "Reference" "U2"
 			(at 49.53 39.37 0)
 			(effects
@@
 			(project ""
 				(path "/ad6c7df0-eb90-4670-9aa8-3e2007aefc2d/8ef5b44a-1ea6-4b34-80bc-234862ce4b8d"
-					(reference "U1")
+					(reference "U2")
 					(unit 1)
 				)
@@
 		(dnp no)
 		(fields_autoplaced yes)
-		(property "Reference" "D1"
+		(property "Reference" "D11"
 			(at 30.734 39.37 0)
 			(effects
@@
 			(project ""
 				(path "/ad6c7df0-eb90-4670-9aa8-3e2007aefc2d/8ef5b44a-1ea6-4b34-80bc-234862ce4b8d"
-					(reference "D1")
+					(reference "D11")
 					(unit 1)
 				)
@@
 		(dnp no)
 		(fields_autoplaced yes)
-		(property "Reference" "C7"
+		(property "Reference" "C6"
 			(at 39.37 50.7935 0)
 			(effects
@@
 			(project "LDO"
 				(path "/ad6c7df0-eb90-4670-9aa8-3e2007aefc2d/8ef5b44a-1ea6-4b34-80bc-234862ce4b8d"
-					(reference "C7")
-					(unit 1)
-				)
+					(reference "C6")
+					(unit 1)
+				)

Commit message: addressed all final comments, review?
Parts:
- TP_3.3V1: footprint TestPoint:TestPoint_Loop_D1.80mm_Drill1.0mm_Beaded -> TestPoint:TestPoint_THTPad_D3.0mm_Drill1.5mm
- renumbered C6 to C1, C7 to C2, D11 to D9, U2 to U1
Changed lines of the file:
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@@
 		(dnp no)
 		(fields_autoplaced yes)
-		(property "Reference" "C7"
+		(property "Reference" "C2"
 			(at 64.77 50.7935 0)
 			(effects
@@
 			(project "LDO"
 				(path "/ad6c7df0-eb90-4670-9aa8-3e2007aefc2d/8ef5b44a-1ea6-4b34-80bc-234862ce4b8d"
-					(reference "C7")
+					(reference "C2")
 					(unit 1)
 				)
@@
 			)
 		)
-		(property "Footprint" "TestPoint:TestPoint_Loop_D1.80mm_Drill1.0mm_Beaded"
+		(property "Footprint" "TestPoint:TestPoint_THTPad_D3.0mm_Drill1.5mm"
 			(at 67.31 45.72 0)
 			(effects
@@
 		(dnp no)
 		(fields_autoplaced yes)
-		(property "Reference" "U2"
+		(property "Reference" "U1"
 			(at 49.53 39.37 0)
 			(effects
@@
 			(project ""
 				(path "/ad6c7df0-eb90-4670-9aa8-3e2007aefc2d/8ef5b44a-1ea6-4b34-80bc-234862ce4b8d"
-					(reference "U2")
+					(reference "U1")
 					(unit 1)
 				)
@@
 		(on_board yes)
 		(dnp no)
-		(property "Reference" "D11"
+		(property "Reference" "D9"
 			(at 30.734 39.37 0)
 			(effects
@@
 			(project ""
 				(path "/ad6c7df0-eb90-4670-9aa8-3e2007aefc2d/8ef5b44a-1ea6-4b34-80bc-234862ce4b8d"
-					(reference "D11")
+					(reference "D9")
 					(unit 1)
 				)
@@
 		(dnp no)
 		(fields_autoplaced yes)
-		(property "Reference" "C6"
+		(property "Reference" "C1"
 			(at 39.37 50.7935 0)
 			(effects
@@
 			(project "LDO"
 				(path "/ad6c7df0-eb90-4670-9aa8-3e2007aefc2d/8ef5b44a-1ea6-4b34-80bc-234862ce4b8d"
-					(reference "C6")
-					(unit 1)
-				)
+					(reference "C1")
+					(unit 1)
+				)
