File: PowerPath_TestBoard/PowerProtection.kicad_sch (KiCad schematic)
At the start: 17 parts, among them U7 LM76202QPWPRQ1

Commit message: addressed all reviews, starting layout
Parts:
- renumbered C20 to C1, C25 to C3, C5 to C4, C23 to C5, D2 to D9, R13 to R10, R15 to R11, R27 to R12, R20 to R13, R30 to R14, R1 to R15, R31 to R16, R23 to R17, R12 to R9, U7 to U1
Changed lines of the file:
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@@
 		(dnp no)
 		(fields_autoplaced yes)
-		(property "Reference" "#PWR024"
+		(property "Reference" "#PWR017"
 			(at 99.06 57.15 0)
 			(effects
@@
 			(project "PeripheralSOM"
 				(path "/ad6c7df0-eb90-4670-9aa8-3e2007aefc2d/338d1821-4309-4081-b4a8-79e8861ff3c2"
-					(reference "#PWR024")
+					(reference "#PWR017")
 					(unit 1)
 				)
@@
 		(on_board yes)
 		(dnp yes)
-		(property "Reference" "R31"
+		(property "Reference" "R16"
 			(at 153.67 28.448 90)
 			(effects
@@
 			(project "PeripheralSOM"
 				(path "/ad6c7df0-eb90-4670-9aa8-3e2007aefc2d/338d1821-4309-4081-b4a8-79e8861ff3c2"
-					(reference "R31")
+					(reference "R16")
 					(unit 1)
 				)
@@
 		(dnp no)
 		(fields_autoplaced yes)
-		(property "Reference" "C25"
+		(property "Reference" "C3"
 			(at 110.49 46.355 0)
 			(effects
@@
 			(project "BPS-PeripheralSOM"
 				(path "/ad6c7df0-eb90-4670-9aa8-3e2007aefc2d/338d1821-4309-4081-b4a8-79e8861ff3c2"
-					(reference "C25")
+					(reference "C3")
 					(unit 1)
 				)
@@
 		(dnp no)
 		(fields_autoplaced yes)
-		(property "Reference" "#PWR030"
+		(property "Reference" "#PWR018"
 			(at 120.65 50.8 0)
 			(effects
@@
 			(project "PeripheralSOM"
 				(path "/ad6c7df0-eb90-4670-9aa8-3e2007aefc2d/338d1821-4309-4081-b4a8-79e8861ff3c2"
-					(reference "#PWR030")
+					(reference "#PWR018")
 					(unit 1)
 				)
@@
 		(dnp no)
 		(fields_autoplaced yes)
-		(property "Reference" "#PWR022"
+		(property "Reference" "#PWR016"
 			(at 52.07 49.53 0)
 			(effects
@@
 			(project ""
 				(path "/ad6c7df0-eb90-4670-9aa8-3e2007aefc2d/338d1821-4309-4081-b4a8-79e8861ff3c2"
-					(reference "#PWR022")
+					(reference "#PWR016")
 					(unit 1)
 				)
@@
 		(on_board yes)
 		(dnp no)
-		(property "Reference" "#FLG0102"
+		(property "Reference" "#FLG05"
 			(at 130.81 29.845 0)
 			(effects
@@
 			(project "PeripheralSOM"
 				(path "/ad6c7df0-eb90-4670-9aa8-3e2007aefc2d/338d1821-4309-4081-b4a8-79e8861ff3c2"
-					(reference "#FLG0102")
+					(reference "#FLG05")
 					(unit 1)
 				)
@@
 		(on_board yes)
 		(dnp no)
-		(property "Reference" "C20"
+		(property "Reference" "C1"
 			(at 32.2072 35.6616 0)
 			(effects
@@
 			(project "BPS-PeripheralSOM"
 				(path "/ad6c7df0-eb90-4670-9aa8-3e2007aefc2d/338d1821-4309-4081-b4a8-79e8861ff3c2"
-					(reference "C20")
+					(reference "C1")
 					(unit 1)
 				)
@@
 		(dnp no)
 		(fields_autoplaced yes)
-		(property "Reference" "#PWR05"
+		(property "Reference" "#PWR019"
 			(at 157.48 86.36 0)
 			(effects
@@
 			(project "PeripheralSOM"
 				(path "/ad6c7df0-eb90-4670-9aa8-3e2007aefc2d/338d1821-4309-4081-b4a8-79e8861ff3c2"
-					(reference "#PWR05")
+					(reference "#PWR019")
 					(unit 1)
 				)
@@
 		(dnp no)
 		(fields_autoplaced yes)
-		(property "Reference" "R20"
+		(property "Reference" "R13"
 			(at 132.08 91.4399 0)
 			(effects
@@
 			(project "BPS-PeripheralSOM"
 				(path "/ad6c7df0-eb90-4670-9aa8-3e2007aefc2d/338d1821-4309-4081-b4a8-79e8861ff3c2"
-					(reference "R20")
+					(reference "R13")
 					(unit 1)
 				)
@@
 		(dnp no)
 		(fields_autoplaced yes)
-		(property "Reference" "R15"
+		(property "Reference" "R11"
 			(at 24.13 121.9199 0)
 			(effects
@@
 			(project "BPS-PeripheralSOM"
 				(path "/ad6c7df0-eb90-4670-9aa8-3e2007aefc2d/338d1821-4309-4081-b4a8-79e8861ff3c2"
-					(reference "R15")
+					(reference "R11")
 					(unit 1)
 				)
@@
 		(on_board yes)
 		(dnp no)
-		(property "Reference" "#FLG0101"
+		(property "Reference" "#FLG04"
 			(at 29.21 29.845 0)
 			(effects
@@
 			(project "BPS-PeripheralSOM"
 				(path "/ad6c7df0-eb90-4670-9aa8-3e2007aefc2d/338d1821-4309-4081-b4a8-79e8861ff3c2"
-					(reference "#FLG0101")
+					(reference "#FLG04")
 					(unit 1)
 				)
@@
 		(on_board yes)
 		(dnp no)
-		(property "Reference" "C23"
+		(property "Reference" "C5"
 			(at 133.8072 36.9316 0)
 			(effects
@@
 			(project "BPS-PeripheralSOM"
 				(path "/ad6c7df0-eb90-4670-9aa8-3e2007aefc2d/338d1821-4309-4081-b4a8-79e8861ff3c2"
-					(reference "C23")
+					(reference "C5")
 					(unit 1)
 				)
@@
 		(on_board yes)
 		(dnp no)
-		(property "Reference" "R1"
+		(property "Reference" "R15"
 			(at 147.828 87.7316 0)
 			(effects
@@
 			(project "PeripheralSOM"
 				(path "/ad6c7df0-eb90-4670-9aa8-3e2007aefc2d/338d1821-4309-4081-b4a8-79e8861ff3c2"
-					(reference "R1")
+					(reference "R15")
 					(unit 1)
 				)
@@
 		(dnp no)
 		(fields_autoplaced yes)
-		(property "Reference" "R23"
+		(property "Reference" "R17"
 			(at 160.02 88.265 0)
 			(effects
@@
 			(project "PeripheralSOM"
 				(path "/ad6c7df0-eb90-4670-9aa8-3e2007aefc2d/338d1821-4309-4081-b4a8-79e8861ff3c2"
-					(reference "R23")
+					(reference "R17")
 					(unit 1)
 				)
@@
 		(on_board yes)
 		(dnp no)
-		(property "Reference" "C5"
+		(property "Reference" "C4"
 			(at 123.6472 36.9316 0)
 			(effects
@@
 			(project "PeripheralSOM"
 				(path "/ad6c7df0-eb90-4670-9aa8-3e2007aefc2d/338d1821-4309-4081-b4a8-79e8861ff3c2"
-					(reference "C5")
+					(reference "C4")
 					(unit 1)
 				)
@@
 		(dnp no)
 		(fields_autoplaced yes)
-		(property "Reference" "R27"
+		(property "Reference" "R12"
 			(at 39.37 67.945 0)
 			(effects
@@
 			(project "PeripheralSOM"
 				(path "/ad6c7df0-eb90-4670-9aa8-3e2007aefc2d/338d1821-4309-4081-b4a8-79e8861ff3c2"
-					(reference "R27")
+					(reference "R12")
 					(unit 1)
 				)
@@
 		(on_board yes)
 		(dnp no)
-		(property "Reference" "D2"
+		(property "Reference" "D9"
 			(at 54.356 36.068 90)
 			(effects
@@
 			(project "BPS-PeripheralSOM"
 				(path "/ad6c7df0-eb90-4670-9aa8-3e2007aefc2d/338d1821-4309-4081-b4a8-79e8861ff3c2"
-					(reference "D2")
+					(reference "D9")
 					(unit 1)
 				)
@@
 		(dnp no)
 		(fields_autoplaced yes)
-		(property "Reference" "R30"
+		(property "Reference" "R14"
 			(at 144.78 35.5599 0)
 			(effects
@@
 			(project ""
 				(path "/ad6c7df0-eb90-4670-9aa8-3e2007aefc2d/338d1821-4309-4081-b4a8-79e8861ff3c2"
-					(reference "R30")
+					(reference "R14")
 					(unit 1)
 				)
@@
 		(dnp no)
 		(fields_autoplaced yes)
-		(property "Reference" "U7"
+		(property "Reference" "U1"
 			(at 82.55 24.13 0)
 			(effects
@@
 			(project "BPS-PeripheralSOM"
 				(path "/ad6c7df0-eb90-4670-9aa8-3e2007aefc2d/338d1821-4309-4081-b4a8-79e8861ff3c2"
-					(reference "U7")
+					(reference "U1")
 					(unit 1)
 				)
@@
 		(on_board yes)
 		(dnp no)
-		(property "Reference" "#PWR092"
+		(property "Reference" "#PWR020"
 			(at 158.75 49.53 0)
 			(effects
@@
 			(project "PeripheralSOM"
 				(path "/ad6c7df0-eb90-4670-9aa8-3e2007aefc2d/338d1821-4309-4081-b4a8-79e8861ff3c2"
-					(reference "#PWR092")
+					(reference "#PWR020")
 					(unit 1)
 				)
@@
 		(dnp no)
 		(fields_autoplaced yes)
-		(property "Reference" "R13"
+		(property "Reference" "R10"
 			(at 24.13 111.7599 0)
 			(effects
@@
 			(project "BPS-PeripheralSOM"
 				(path "/ad6c7df0-eb90-4670-9aa8-3e2007aefc2d/338d1821-4309-4081-b4a8-79e8861ff3c2"
-					(reference "R13")
+					(reference "R10")
 					(unit 1)
 				)
@@
 		(on_board yes)
 		(dnp no)
-		(property "Reference" "R12"
+		(property "Reference" "R9"
 			(at 23.368 101.7016 0)
 			(effects
@@
 			(project "BPS-PeripheralSOM"
 				(path "/ad6c7df0-eb90-4670-9aa8-3e2007aefc2d/338d1821-4309-4081-b4a8-79e8861ff3c2"
-					(reference "R12")
-					(unit 1)
-				)
+					(reference "R9")
+					(unit 1)
+				)

Commit message: addressed all final comments, review?
Parts:
- removed C1: 10uF, Capacitor_SMD:C_0805_2012Metric_Pad1.18x1.45mm_HandSolder, symbol Device:C
- removed C2: 1uF, Capacitor_SMD:C_0603_1608Metric_Pad1.08x0.95mm_HandSolder, symbol Device:C
- removed D9: TVS, Diode_SMD:D_SOD-323_HandSoldering, symbol Diode:SD12_SOD323
- removed R10: 590, Resistor_SMD:R_0603_1608Metric_Pad0.98x0.95mm_HandSolder, symbol Device:R
- removed R11: 2.1k, Resistor_SMD:R_0603_1608Metric_Pad0.98x0.95mm_HandSolder, symbol Device:R
- removed R12, R15, R17: 10k, Resistor_SMD:R_0603_1608Metric_Pad0.98x0.95mm_HandSolder, symbol Device:R
- removed R13: 402k, Resistor_SMD:R_0603_1608Metric_Pad0.98x0.95mm_HandSolder, symbol Device:R
- removed R14: 24m, Resistor_SMD:R_0603_1608Metric_Pad0.98x0.95mm_HandSolder, symbol Device:R
- removed R16: 100k, Resistor_SMD:R_0603_1608Metric_Pad0.98x0.95mm_HandSolder, symbol Device:R
- removed R9: 45.3k, Resistor_SMD:R_0603_1608Metric_Pad0.98x0.95mm_HandSolder, symbol Device:R
- removed U1: LM76202QPWPRQ1, UTSVT_Power:LM76202QPWPRQ1, symbol utsvt_power:LM76202QPWPRQ1
- added C6: 10n, Capacitor_SMD:C_0603_1608Metric_Pad1.08x0.95mm_HandSolder, symbol ECE319H:C
- added C7: 10u, Capacitor_SMD:C_0805_2012Metric_Pad1.18x1.45mm_HandSolder, symbol Device:C
- added IC1: LM74502DDFR, UTSVT_Power:SOT65P280X110-8N, symbol UTSVT_ICs:LM74502HDDFR
- added Q1, Q2: PSMN012-100YS, PSMN012-100YS:TO127P600X120-5N, symbol Simulation_SPICE:NMOS
- added R10: 1k, Resistor_SMD:R_0603_1608Metric_Pad0.98x0.95mm_HandSolder, symbol Device:R_US
- added R11: 33, Resistor_SMD:R_0603_1608Metric_Pad0.98x0.95mm_HandSolder, symbol Device:R_US
- added R12: 223k, Resistor_SMD:R_0603_1608Metric_Pad0.98x0.95mm_HandSolder, symbol Device:R_US
- added R13: 137k, Resistor_SMD:R_0603_1608Metric_Pad0.98x0.95mm_HandSolder, symbol Device:R_US
- added R14, R15, R9: 10k, Resistor_SMD:R_0603_1608Metric_Pad0.98x0.95mm_HandSolder, symbol Device:R_US
- added TP14, TP15, TP16, TP17, TP18, TP19: 24V_OUT, TestPoint:TestPoint_THTPad_D3.0mm_Drill1.5mm, symbol Connector:TestPoint
- C3: value 100nF -> 0.1u; Mouser Part Number (none) -> 963-HMK107B7104KA-T; P/N MLASH168SB7104KTNA01 -> HMK107B7104KA-T
- C4: value 1uF -> 1u; Mouser Part Number (none) -> 963-UMK107BJ105KA-T; P/N MLASU168SB5105KTNA01 -> UMK107BJ105KA-T
- C5: value 10uF -> 220n; footprint Capacitor_SMD:C_0805_2012Metric_Pad1.18x1.45mm_HandSolder -> Capacitor_SMD:C_0603_1608Metric_Pad1.08x0.95mm_HandSolder; LCSC P/N C3840574 -> (none); Mouser Part Number (none) -> 963-MSASU168SB7224KT; P/N GRM21BR61H106KE43K -> MSASU168SB7224KTNB25
- D10: value TVS -> SMAF4758A; footprint Diode_SMD:D_SOD-123F -> UTSVT_Passives:SODFL5026X125N; LCSC P/N C2649858 -> (none); Mouser Part Number (none) -> 833-SMAF4758A-TP; P/N SMF3.3 -> SMAF4758A-TP
Connections:
- net IMON_OUT is gone; now on an unnamed net: D10.1 (K)
- net RTN is gone; now on net GND: C3.2
- net GND: now also C4.1, C6.2, C7.2, IC1.2 (GND), R14.1, R15.2; no longer C4.2, C5.2
- net Vin: now reaches C3.1
- net Vin: now also Q1.5 (D), R12.1, R13.2, R14.2, R9.2
- net 24V_OUT: no longer names the net of C5.1
- net 24V_OUT: now also C4.2, IC1.5 (VS), R9.1, TP14.1; no longer C4.1
- new net: C5.2, IC1.4 (VCAP), TP19.1
- new net: IC1.7 (OV), R12.2, R15.1, TP17.1
- new net: IC1.1 (EN/UVLO), R13.1, TP18.1
- new net: IC1.6 (GATE), R11.2
- new net: C6.1, R10.1
- new net Vout: C7.1, Q2.5 (D)
- new net gate: Q1.4 (G), Q2.4 (G), R10.2, R11.1, TP15.1
- new net source: IC1.8 (SRC), Q1.1 (S), Q1.2 (S), Q1.3 (S), Q2.1 (S), Q2.2 (S), Q2.3 (S), TP16.1
- no-connect marks 2 -> 0
Other:
- note added: "1.235 is Enable/UVLO falling threshold on data sheet"
- note added: "Overvoltage Protection: 29.03V Vovr = (R2 * Vov)/(R1 + R2) Vov = Vovr * (R1 + R2) / R2 29.13 = 1.25 * (223k + 10k) / 10k"
- note added: "gate"
- note added: "source"
- note removed: "20.88 ms ramp time"
- note removed: "Current Monitoring"
- note removed: "DNP until validated"
- note removed: "Functional Mode Selection"
- note removed: "ILim(A) = 12/R(k) 1.2A = 12/10kΩ"
- note removed: "OVP set to 27v for buck max voltage of 28v"
- note removed: "Overcurrent Protection"
- note removed: "Pullups"
- note removed: "RTN!=GND Conecting GND to RTN turns off RPP!"
- note removed: "SHDN has weak internal pullup - pulled up to MCU voltage after initial power on"
- note removed: "Set to circuit breaker (latchoff) Use 0 ohm resistor for auto-retry (540ms)"
- note removed: "Typical gain: 78.28 uA/A Vout @ 1.3A = 2.407v R(imon) = 23.7 mΩ"
- note removed: "Under/Overvoltage Protection"

Commit message: added p/n for missing fields
Parts:
- C6: P/N (none) -> MCASU168SB7103KTNA01
Changed lines of the file:
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@@
+			)
+		)
+		(property "Part #" ""
+			(at 54.61 81.28 0)
+			(effects
+				(font
+					(size 1.27 1.27)
+				)
+				(hide yes)
 			)
 		)
@@
 			)
 		)
+		(property "Part #" ""
+			(at 68.58 48.26 0)
+			(effects
+				(font
+					(size 1.27 1.27)
+				)
+				(hide yes)
+			)
+		)
 		(pin "1"
 		)
@@
 		)
 		(property "Description" "test point"
+			(at 57.15 86.36 0)
+			(effects
+				(font
+					(size 1.27 1.27)
+				)
+				(hide yes)
+			)
+		)
+		(property "Part #" ""
 			(at 57.15 86.36 0)
 			(effects
@@
 			)
 		)
+		(property "Part #" ""
+			(at 90.17 43.18 90)
+			(effects
+				(font
+					(size 1.27 1.27)
+				)
+				(hide yes)
+			)
+		)
 		(pin "4"
 		)
@@
 			)
 		)
+		(property "Part #" ""
+			(at 43.18 58.42 0)
+			(effects
+				(font
+					(size 1.27 1.27)
+				)
+				(hide yes)
+			)
+		)
 		(pin "1"
 		)
@@
 		)
 		(property "Description" "test point"
+			(at 93.98 81.28 0)
+			(effects
+				(font
+					(size 1.27 1.27)
+				)
+				(hide yes)
+			)
+		)
+		(property "Part #" ""
 			(at 93.98 81.28 0)
 			(effects
@@
 			)
 		)
+		(property "Part #" ""
+			(at 102.87 95.25 0)
+			(effects
+				(font
+					(size 1.27 1.27)
+				)
+				(hide yes)
+			)
+		)
 		(pin "1"
 		)
@@
 			)
 		)
+		(property "Part #" ""
+			(at 34.29 46.99 0)
+			(effects
+				(font
+					(size 1.27 1.27)
+				)
+				(hide yes)
+			)
+		)
 		(pin "1"
 		)
@@
 		)
 		(property "P/N" "CRCW0603137KFKEA"
+			(at 97.79 88.9 90)
+			(effects
+				(font
+					(size 1.27 1.27)
+				)
+				(hide yes)
+			)
+		)
+		(property "Part #" ""
 			(at 97.79 88.9 90)
 			(effects
@@
 			)
 		)
+		(property "Part #" ""
+			(at 46.99 77.47 0)
+			(effects
+				(font
+					(size 1.27 1.27)
+				)
+				(hide yes)
+			)
+		)
 		(pin "1"
 		)
@@
 			)
 		)
+		(property "Part #" ""
+			(at 63.5 43.18 90)
+			(effects
+				(font
+					(size 1.27 1.27)
+				)
+				(hide yes)
+			)
+		)
 		(pin "1"
 		)
@@
 			)
 		)
+		(property "Part #" ""
+			(at 72.39 60.96 0)
+			(effects
+				(font
+					(size 1.27 1.27)
+				)
+				(hide yes)
+			)
+		)
 		(pin "1"
 		)
@@
 			)
 		)
+		(property "Part #" ""
+			(at 58.42 77.47 0)
+			(effects
+				(font
+					(size 1.27 1.27)
+				)
+				(hide yes)
+			)
+		)
 		(pin "1"
 		)
@@
 		)
 		(property "Description" "test point"
+			(at 78.74 40.64 0)
+			(effects
+				(font
+					(size 1.27 1.27)
+				)
+				(hide yes)
+			)
+		)
+		(property "Part #" ""
 			(at 78.74 40.64 0)
 			(effects
@@
 			)
 		)
+		(property "Part #" ""
+			(at 67.31 53.34 90)
+			(effects
+				(font
+					(size 1.27 1.27)
+				)
+				(hide yes)
+			)
+		)
 		(pin "1"
 		)
@@
 		)
 		(property "Description" "Unpolarized capacitor"
+			(at 62.23 59.69 0)
+			(effects
+				(font
+					(size 1.27 1.27)
+				)
+				(hide yes)
+			)
+		)
+		(property "P/N" "MCASU168SB7103KTNA01"
+			(at 62.23 59.69 0)
+			(effects
+				(font
+					(size 1.27 1.27)
+				)
+				(hide yes)
+			)
+		)
+		(property "Part #" ""
 			(at 62.23 59.69 0)
 			(effects
@@
 			)
 		)
+		(property "Part #" ""
+			(at 92.71 88.9 0)
+			(effects
+				(font
+					(size 1.27 1.27)
+				)
+				(hide yes)
+			)
+		)
 		(pin "1"
 		)
@@
 		)
 		(property "Vf" ""
+			(at 109.22 46.99 0)
+			(effects
+				(font
+					(size 1.27 1.27)
+				)
+				(hide yes)
+			)
+		)
+		(property "Part #" ""
 			(at 109.22 46.99 0)
 			(effects
@@
 			)
 		)
+		(property "Part #" ""
+			(at 104.14 81.28 90)
+			(effects
+				(font
+					(size 1.27 1.27)
+				)
+				(hide yes)
+			)
+		)
 		(pin "1"
 		)
@@
 		)
 		(property "P/N" "SMAF4758A-TP"
+			(at 43.18 83.82 90)
+			(effects
+				(font
+					(size 1.27 1.27)
+				)
+				(hide yes)
+			)
+		)
+		(property "Part #" ""
 			(at 43.18 83.82 90)
 			(effects
@@
 			)
 		)
+		(property "Part #" ""
+			(at 36.83 81.28 0)
+			(effects
+				(font
+					(size 1.27 1.27)
+				)
+				(hide yes)
+			)
+		)
 		(pin "2"
 		)
@@
 			(at 97.79 73.66 0)
 			(effects
+				(font
+					(size 1.27 1.27)
+				)
+				(hide yes)
+			)
+		)
+		(property "Part #" ""
+			(at 97.79 73.66 0)
+			(effects
