File: PowerPath_TestBoard/PowerProtection.kicad_sch (KiCad schematic)
At the start: 20 parts, among them IC1 LM74502DDFR, Q1 PSMN012-100YS, Q2 PSMN012-100YS

Commit message: updated with new comments + new gen gebers
Parts:
- C6: P/N (none) -> EMK107SD103KA-T
- C7: footprint Capacitor_SMD:C_0603_1608Metric_Pad1.08x0.95mm_HandSolder -> Capacitor_SMD:C_0805_2012Metric_Pad1.18x1.45mm_HandSolder
Changed lines of the file:
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@@
+			)
+		)
+		(property "P/N" "EMK107SD103KA-T"
+			(at 62.23 59.69 0)
+			(effects
+				(font
+					(size 1.27 1.27)
+				)
+				(hide yes)
 			)
 		)
@@
 			)
 		)
-		(property "Footprint" "Capacitor_SMD:C_0603_1608Metric_Pad1.08x0.95mm_HandSolder"
+		(property "Footprint" "Capacitor_SMD:C_0805_2012Metric_Pad1.18x1.45mm_HandSolder"
 			(at 110.1852 50.8 0)
 			(effects
