File: PowerPath_TestBoard/testiung.kicad_sch (KiCad schematic)
At the start: 20 parts, among them IC1 LM74502DDFR, Q1 PSMN012-100YS, Q2 PSMN012-100YS

Commit message: updated with PP + gen gebers
Parts:
- removed TP19, TP20, TP21, TP22: +V_out_5V, TestPoint:TestPoint_THTPad_D3.0mm_Drill1.5mm, symbol Connector:TestPoint
- D2: renamed from D10; footprint SMBJ30CD:DIONM5436X244N -> UTSVT_Power:SMBJ30CD
- renumbered C3 to C1, C4 to C2, C5 to C3, C6 to C4, C7 to C5, D11 to D1, R9 to R1, R10 to R3, R11 to R4, R13 to R5, R12 to R6, R14 to R7
Connections:
- net Vin: now also Q1.1 (D); no longer Q1.5 (D)
- net Vout: now also Q2.1 (D); no longer Q2.5 (D)
- net gate: now also Q1.2 (G), Q2.2 (G); no longer Q1.4 (G), Q2.4 (G)
- net source: no longer Q1.1 (S), Q1.2 (S), Q2.1 (S), Q2.2 (S)
Other:
- moved on the sheet: Q2
