File: PowerPath_TestBoard/12VBuck.kicad_sch (KiCad schematic)
At the start: 12 parts, among them U1 LMR51635XDDCR

Commit message: addressed all reviews, starting layout
Parts:
- removed C1: 2.2u, Capacitor_SMD:C_0805_2012Metric_Pad1.18x1.45mm_HandSolder, symbol Device:C_Small
- removed C2: 100n, Resistor_SMD:R_0201_0603Metric_Pad0.64x0.40mm_HandSolder, symbol Device:C_Small
- removed C3, C4: 47u, Capacitor_SMD:C_1210_3225Metric_Pad1.33x2.70mm_HandSolder, symbol Device:C_Small
- removed R1: 53.6k, Resistor_SMD:R_0603_1608Metric, symbol Device:R_Small
- removed R2: 10.2k, Resistor_SMD:R_0603_1608Metric, symbol Device:R_Small
- removed TP5: V_in_24V, TestPoint:TestPoint_THTPad_D3.0mm_Drill1.5mm, symbol Connector:TestPoint
- removed TP6: FB, TestPoint:TestPoint_THTPad_D3.0mm_Drill1.5mm, symbol Connector:TestPoint
- removed TP7: CB, TestPoint:TestPoint_THTPad_D3.0mm_Drill1.5mm, symbol Connector:TestPoint
- removed TP8: SW, TestPoint:TestPoint_THTPad_D3.0mm_Drill1.5mm, symbol Connector:TestPoint
- removed U1: LMR51635XDDCR, utsvt_ics:DDC0006A-MFG, symbol 2026-04-25_18-34-12:LMR51635XDDCR
- added C10, C11: 47u, Capacitor_SMD:C_1210_3225Metric_Pad1.33x2.70mm_HandSolder, symbol Device:C_Small
- added C8: 2.2u, Capacitor_SMD:C_0805_2012Metric_Pad1.18x1.45mm_HandSolder, symbol Device:C_Small
- added C9: 100n, Capacitor_SMD:C_0603_1608Metric, symbol Device:C_Small
- added R18: 143k, Resistor_SMD:R_0603_1608Metric, symbol Device:R_Small
- added R19: 10.2k, Resistor_SMD:R_0603_1608Metric, symbol Device:R_Small
- added TP10: CB, TestPoint:TestPoint_THTPad_D3.0mm_Drill1.5mm, symbol Connector:TestPoint
- added TP11: FB, TestPoint:TestPoint_THTPad_D3.0mm_Drill1.5mm, symbol Connector:TestPoint
- added TP12: SW, TestPoint:TestPoint_THTPad_D3.0mm_Drill1.5mm, symbol Connector:TestPoint
- added TP9: V_in_24V, TestPoint:TestPoint_THTPad_D3.0mm_Drill1.5mm, symbol Connector:TestPoint
- added U3: LMR51635XDDCR, utsvt_ics:DDC0006A-MFG, symbol 2026-04-25_18-34-12:LMR51635XDDCR
- L1: value 10u -> 15u; LCSC P/N C354639 -> C2849555; P/N CKCS8040-10uH/M -> PNLS8040-150M 15UH
Connections:
- net CB: now also C9.1, TP10.1, U3.6 (CB)
- net FB: now also R18.2, R19.1, TP11.1, U3.1 (FB)
- net GND: now also C10.2, C11.2, C8.2, R19.2, U3.4 (GND)
- net SW: now also C9.2, TP12.1, U3.5 (SW)
- net V_in_24V: now also C8.1, TP9.1, U3.2 (EN), U3.3 (VIN)
- net V_out_5V renamed V_out_12V
- net V_out_12V: now also C10.1, C11.1, R18.1
Other:
- note added: "12V Vout"
- note added: "24V-12V Buck Converter"
- note removed: "24V-5V Buck Converter"
- note removed: "5V Vout"

Commit message: addressed final rounds of schematic comments, inital layouting
Parts:
- U3: footprint utsvt_ics:DDC0006A-MFG -> UTSVT_ICs:DDC0006A-MFG
Changed lines of the file:
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@@
 			)
 		)
-		(property "Footprint" "utsvt_ics:DDC0006A-MFG"
+		(property "Footprint" "UTSVT_ICs:DDC0006A-MFG"
 			(at 114.3 81.28 0)
 			(effects

Commit message: addressed all final comments, review?
Parts:
- renumbered R18 to R16, R19 to R17, TP12 to TP10, TP9 to TP7, TP10 to TP8, TP11 to TP9, U3 to U2
Changed lines of the file:
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@@
 		(dnp no)
 		(fields_autoplaced yes)
-		(property "Reference" "#FLG07"
+		(property "Reference" "#FLG05"
 			(at 149.86 79.375 0)
 			(effects
@@
 			(project "PS-Buck"
 				(path "/ad6c7df0-eb90-4670-9aa8-3e2007aefc2d/41c72b07-cf60-4ca9-96a7-6ae96aaa0c90"
-					(reference "#FLG07")
+					(reference "#FLG05")
 					(unit 1)
 				)
@@
 		(on_board yes)
 		(dnp no)
-		(property "Reference" "TP9"
+		(property "Reference" "TP7"
 			(at 229.87 123.6979 0)
 			(effects
@@
 			(project "PowerPath"
 				(path "/ad6c7df0-eb90-4670-9aa8-3e2007aefc2d/41c72b07-cf60-4ca9-96a7-6ae96aaa0c90"
-					(reference "TP9")
+					(reference "TP7")
 					(unit 1)
 				)
@@
 		(on_board yes)
 		(dnp no)
-		(property "Reference" "TP11"
+		(property "Reference" "TP9"
 			(at 242.57 123.6979 0)
 			(effects
@@
 			(project "PowerPath"
 				(path "/ad6c7df0-eb90-4670-9aa8-3e2007aefc2d/41c72b07-cf60-4ca9-96a7-6ae96aaa0c90"
-					(reference "TP11")
+					(reference "TP9")
 					(unit 1)
 				)
@@
 		(on_board yes)
 		(dnp no)
-		(property "Reference" "TP10"
+		(property "Reference" "TP8"
 			(at 229.87 136.3979 0)
 			(effects
@@
 			(project "PowerPath"
 				(path "/ad6c7df0-eb90-4670-9aa8-3e2007aefc2d/41c72b07-cf60-4ca9-96a7-6ae96aaa0c90"
-					(reference "TP10")
+					(reference "TP8")
 					(unit 1)
 				)
@@
 		(dnp no)
 		(fields_autoplaced yes)
-		(property "Reference" "U3"
+		(property "Reference" "U2"
 			(at 129.54 71.12 0)
 			(effects
@@
 			(project "PS-Buck"
 				(path "/ad6c7df0-eb90-4670-9aa8-3e2007aefc2d/41c72b07-cf60-4ca9-96a7-6ae96aaa0c90"
-					(reference "U3")
+					(reference "U2")
 					(unit 1)
 				)
@@
 		(on_board yes)
 		(dnp no)
-		(property "Reference" "TP12"
+		(property "Reference" "TP10"
 			(at 242.57 136.3979 0)
 			(effects
@@
 			(project "PowerPath"
 				(path "/ad6c7df0-eb90-4670-9aa8-3e2007aefc2d/41c72b07-cf60-4ca9-96a7-6ae96aaa0c90"
-					(reference "TP12")
+					(reference "TP10")
 					(unit 1)
 				)
@@
 		(dnp no)
 		(fields_autoplaced yes)
-		(property "Reference" "#FLG09"
+		(property "Reference" "#FLG07"
 			(at 181.61 84.455 0)
 			(effects
@@
 			(project "PS-Buck"
 				(path "/ad6c7df0-eb90-4670-9aa8-3e2007aefc2d/41c72b07-cf60-4ca9-96a7-6ae96aaa0c90"
-					(reference "#FLG09")
+					(reference "#FLG07")
 					(unit 1)
 				)
@@
 		(dnp no)
 		(fields_autoplaced yes)
-		(property "Reference" "#FLG06"
+		(property "Reference" "#FLG04"
 			(at 88.9 79.375 0)
 			(effects
@@
 			(project "PS-Buck"
 				(path "/ad6c7df0-eb90-4670-9aa8-3e2007aefc2d/41c72b07-cf60-4ca9-96a7-6ae96aaa0c90"
-					(reference "#FLG06")
+					(reference "#FLG04")
 					(unit 1)
 				)
@@
 		(on_board yes)
 		(dnp no)
-		(property "Reference" "#FLG08"
+		(property "Reference" "#FLG06"
 			(at 149.86 84.455 0)
 			(effects
@@
 			(project "PS-Buck"
 				(path "/ad6c7df0-eb90-4670-9aa8-3e2007aefc2d/41c72b07-cf60-4ca9-96a7-6ae96aaa0c90"
-					(reference "#FLG08")
+					(reference "#FLG06")
 					(unit 1)
 				)
@@
 		(dnp no)
 		(fields_autoplaced yes)
-		(property "Reference" "R18"
+		(property "Reference" "R16"
 			(at 227.33 85.0899 0)
 			(effects
@@
 			(project "PS-Buck"
 				(path "/ad6c7df0-eb90-4670-9aa8-3e2007aefc2d/41c72b07-cf60-4ca9-96a7-6ae96aaa0c90"
-					(reference "R18")
+					(reference "R16")
 					(unit 1)
 				)
@@
 		(dnp no)
 		(fields_autoplaced yes)
-		(property "Reference" "R19"
+		(property "Reference" "R17"
 			(at 227.33 92.7099 0)
 			(effects
@@
 			(project "PS-Buck"
 				(path "/ad6c7df0-eb90-4670-9aa8-3e2007aefc2d/41c72b07-cf60-4ca9-96a7-6ae96aaa0c90"
-					(reference "R19")
-					(unit 1)
-				)
+					(reference "R17")
+					(unit 1)
+				)

Commit message: updated with PP + gen gebers
Parts:
- renumbered R16 to R15, R17 to R16, TP7 to TP12, TP8 to TP13, TP9 to TP14, TP10 to TP15
Changed lines of the file:
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@@
 		(on_board yes)
 		(dnp no)
-		(property "Reference" "TP7"
+		(property "Reference" "TP12"
 			(at 229.87 123.6979 0)
 			(effects
@@
 			(project "PowerPath"
 				(path "/ad6c7df0-eb90-4670-9aa8-3e2007aefc2d/41c72b07-cf60-4ca9-96a7-6ae96aaa0c90"
-					(reference "TP7")
+					(reference "TP12")
 					(unit 1)
 				)
@@
 		(on_board yes)
 		(dnp no)
-		(property "Reference" "TP9"
+		(property "Reference" "TP14"
 			(at 242.57 123.6979 0)
 			(effects
@@
 			(project "PowerPath"
 				(path "/ad6c7df0-eb90-4670-9aa8-3e2007aefc2d/41c72b07-cf60-4ca9-96a7-6ae96aaa0c90"
-					(reference "TP9")
+					(reference "TP14")
 					(unit 1)
 				)
@@
 		(on_board yes)
 		(dnp no)
-		(property "Reference" "TP8"
+		(property "Reference" "TP13"
 			(at 229.87 136.3979 0)
 			(effects
@@
 			(project "PowerPath"
 				(path "/ad6c7df0-eb90-4670-9aa8-3e2007aefc2d/41c72b07-cf60-4ca9-96a7-6ae96aaa0c90"
-					(reference "TP8")
+					(reference "TP13")
 					(unit 1)
 				)
@@
 		(on_board yes)
 		(dnp no)
-		(property "Reference" "TP10"
+		(property "Reference" "TP15"
 			(at 242.57 136.3979 0)
 			(effects
@@
 			(project "PowerPath"
 				(path "/ad6c7df0-eb90-4670-9aa8-3e2007aefc2d/41c72b07-cf60-4ca9-96a7-6ae96aaa0c90"
-					(reference "TP10")
+					(reference "TP15")
 					(unit 1)
 				)
@@
 		(dnp no)
 		(fields_autoplaced yes)
-		(property "Reference" "R16"
+		(property "Reference" "R15"
 			(at 227.33 85.0899 0)
 			(effects
@@
 			(project "PS-Buck"
 				(path "/ad6c7df0-eb90-4670-9aa8-3e2007aefc2d/41c72b07-cf60-4ca9-96a7-6ae96aaa0c90"
-					(reference "R16")
+					(reference "R15")
 					(unit 1)
 				)
@@
 		(dnp no)
 		(fields_autoplaced yes)
-		(property "Reference" "R17"
+		(property "Reference" "R16"
 			(at 227.33 92.7099 0)
 			(effects
@@
 			(project "PS-Buck"
 				(path "/ad6c7df0-eb90-4670-9aa8-3e2007aefc2d/41c72b07-cf60-4ca9-96a7-6ae96aaa0c90"
-					(reference "R17")
-					(unit 1)
-				)
+					(reference "R16")
+					(unit 1)
+				)

Commit message: updated with new comments + new gen gebers
Parts:
- C9: footprint Capacitor_SMD:C_0603_1608Metric -> Capacitor_SMD:C_0603_1608Metric_Pad1.08x0.95mm_HandSolder
- R15, R16: footprint Resistor_SMD:R_0603_1608Metric -> Resistor_SMD:R_0603_1608Metric_Pad0.98x0.95mm_HandSolder
Changed lines of the file:
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@@
 			)
 		)
-		(property "Footprint" "Capacitor_SMD:C_0603_1608Metric"
+		(property "Footprint" "Capacitor_SMD:C_0603_1608Metric_Pad1.08x0.95mm_HandSolder"
 			(at 153.67 83.82 0)
 			(effects
@@
 			)
 		)
-		(property "Footprint" "Resistor_SMD:R_0603_1608Metric"
+		(property "Footprint" "Resistor_SMD:R_0603_1608Metric_Pad0.98x0.95mm_HandSolder"
 			(at 224.79 86.36 0)
 			(effects
@@
 			)
 		)
-		(property "Footprint" "Resistor_SMD:R_0603_1608Metric"
+		(property "Footprint" "Resistor_SMD:R_0603_1608Metric_Pad0.98x0.95mm_HandSolder"
 			(at 224.79 93.98 0)
 			(effects
