File: PowerPath_TestBoard/5VBuck.kicad_sch (KiCad schematic)
At the start: 12 parts, among them U1 LMR51635XDDCR

Commit message: addressed all reviews, starting layout
Parts:
- C13: renamed from C2; footprint Resistor_SMD:R_0201_0603Metric_Pad0.64x0.40mm_HandSolder -> Capacitor_SMD:C_0603_1608Metric
- TP13: renamed from TP5; footprint (none) -> TestPoint:TestPoint_THTPad_D3.0mm_Drill1.5mm
- TP14: renamed from TP7; footprint (none) -> TestPoint:TestPoint_THTPad_D3.0mm_Drill1.5mm
- TP15: renamed from TP6; footprint (none) -> TestPoint:TestPoint_THTPad_D3.0mm_Drill1.5mm
- TP16: renamed from TP8; footprint (none) -> TestPoint:TestPoint_THTPad_D3.0mm_Drill1.5mm
- renumbered C1 to C12, C3 to C14, C4 to C15, L1 to L2, R1 to R20, R2 to R21, U1 to U4
Changed lines of the file:
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@@
 		(on_board yes)
 		(dnp no)
-		(property "Reference" "L1"
+		(property "Reference" "L2"
 			(at 106.68 48.514 90)
 			(effects
@@
 			)
 			(project "5VBuck"
-				(path "/ad6c7df0-eb90-4670-9aa8-3e2007aefc2d/4ce3c563-64ba-4b6e-b334-e3956b5d5a33"
-					(reference "L1")
-					(unit 1)
-				)
-				(path "/ad6c7df0-eb90-4670-9aa8-3e2007aefc2d/c59a1097-f91e-4d56-b57d-869363ca5893"
-					(reference "L1")
+				(path "/ad6c7df0-eb90-4670-9aa8-3e2007aefc2d/ae63f0a9-78b8-4efb-b2ee-a2699a24d705"
+					(reference "L2")
 					(unit 1)
 				)
@@
 		(dnp no)
 		(fields_autoplaced yes)
-		(property "Reference" "R2"
+		(property "Reference" "R21"
 			(at 170.18 49.5299 0)
 			(effects
@@
 			)
 			(project "5VBuck"
-				(path "/ad6c7df0-eb90-4670-9aa8-3e2007aefc2d/4ce3c563-64ba-4b6e-b334-e3956b5d5a33"
-					(reference "R2")
-					(unit 1)
-				)
-				(path "/ad6c7df0-eb90-4670-9aa8-3e2007aefc2d/c59a1097-f91e-4d56-b57d-869363ca5893"
-					(reference "R2")
+				(path "/ad6c7df0-eb90-4670-9aa8-3e2007aefc2d/ae63f0a9-78b8-4efb-b2ee-a2699a24d705"
+					(reference "R21")
 					(unit 1)
 				)
@@
 		(dnp no)
 		(fields_autoplaced yes)
-		(property "Reference" "C1"
+		(property "Reference" "C12"
 			(at 40.64 45.7262 0)
 			(effects
@@
 			)
 			(project "5VBuck"
-				(path "/ad6c7df0-eb90-4670-9aa8-3e2007aefc2d/4ce3c563-64ba-4b6e-b334-e3956b5d5a33"
-					(reference "C1")
-					(unit 1)
-				)
-				(path "/ad6c7df0-eb90-4670-9aa8-3e2007aefc2d/c59a1097-f91e-4d56-b57d-869363ca5893"
-					(reference "C1")
+				(path "/ad6c7df0-eb90-4670-9aa8-3e2007aefc2d/ae63f0a9-78b8-4efb-b2ee-a2699a24d705"
+					(reference "C12")
 					(unit 1)
 				)
@@
 		(on_board yes)
 		(dnp no)
-		(property "Reference" "TP6"
+		(property "Reference" "TP15"
 			(at 184.15 80.5179 0)
 			(effects
@@
 			)
 		)
-		(property "Footprint" ""
+		(property "Footprint" "TestPoint:TestPoint_THTPad_D3.0mm_Drill1.5mm"
 			(at 186.69 85.09 0)
 			(effects
@@
 		(instances
 			(project "PowerPath"
-				(path "/ad6c7df0-eb90-4670-9aa8-3e2007aefc2d/4ce3c563-64ba-4b6e-b334-e3956b5d5a33"
-					(reference "TP6")
-					(unit 1)
-				)
-				(path "/ad6c7df0-eb90-4670-9aa8-3e2007aefc2d/c59a1097-f91e-4d56-b57d-869363ca5893"
-					(reference "TP6")
+				(path "/ad6c7df0-eb90-4670-9aa8-3e2007aefc2d/ae63f0a9-78b8-4efb-b2ee-a2699a24d705"
+					(reference "TP15")
 					(unit 1)
 				)
@@
 		(on_board yes)
 		(dnp no)
-		(property "Reference" "C2"
+		(property "Reference" "C13"
 			(at 100.838 40.64 0)
 			(effects
@@
 			)
 		)
-		(property "Footprint" "Resistor_SMD:R_0201_0603Metric_Pad0.64x0.40mm_HandSolder"
+		(property "Footprint" "Capacitor_SMD:C_0603_1608Metric"
 			(at 97.79 44.45 0)
 			(effects
@@
 			)
 			(project "5VBuck"
-				(path "/ad6c7df0-eb90-4670-9aa8-3e2007aefc2d/4ce3c563-64ba-4b6e-b334-e3956b5d5a33"
-					(reference "C2")
-					(unit 1)
-				)
-				(path "/ad6c7df0-eb90-4670-9aa8-3e2007aefc2d/c59a1097-f91e-4d56-b57d-869363ca5893"
-					(reference "C2")
+				(path "/ad6c7df0-eb90-4670-9aa8-3e2007aefc2d/ae63f0a9-78b8-4efb-b2ee-a2699a24d705"
+					(reference "C13")
 					(unit 1)
 				)
@@
 		(dnp no)
 		(fields_autoplaced yes)
-		(property "Reference" "U1"
+		(property "Reference" "U4"
 			(at 73.66 31.75 0)
 			(effects
@@
 			)
 			(project "5VBuck"
-				(path "/ad6c7df0-eb90-4670-9aa8-3e2007aefc2d/4ce3c563-64ba-4b6e-b334-e3956b5d5a33"
-					(reference "U1")
-					(unit 1)
-				)
-				(path "/ad6c7df0-eb90-4670-9aa8-3e2007aefc2d/c59a1097-f91e-4d56-b57d-869363ca5893"
-					(reference "U1")
+				(path "/ad6c7df0-eb90-4670-9aa8-3e2007aefc2d/ae63f0a9-78b8-4efb-b2ee-a2699a24d705"
+					(reference "U4")
 					(unit 1)
 				)
@@
 		(on_board yes)
 		(dnp no)
-		(property "Reference" "TP5"
+		(property "Reference" "TP13"
 			(at 171.45 80.5179 0)
 			(effects
@@
 			)
 		)
-		(property "Footprint" ""
+		(property "Footprint" "TestPoint:TestPoint_THTPad_D3.0mm_Drill1.5mm"
 			(at 173.99 85.09 0)
 			(effects
@@
 		(instances
 			(project ""
-				(path "/ad6c7df0-eb90-4670-9aa8-3e2007aefc2d/4ce3c563-64ba-4b6e-b334-e3956b5d5a33"
-					(reference "TP5")
-					(unit 1)
-				)
-				(path "/ad6c7df0-eb90-4670-9aa8-3e2007aefc2d/c59a1097-f91e-4d56-b57d-869363ca5893"
-					(reference "TP5")
+				(path "/ad6c7df0-eb90-4670-9aa8-3e2007aefc2d/ae63f0a9-78b8-4efb-b2ee-a2699a24d705"
+					(reference "TP13")
 					(unit 1)
 				)
@@
 		(dnp no)
 		(fields_autoplaced yes)
-		(property "Reference" "#FLG01"
+		(property "Reference" "#FLG010"
 			(at 93.98 40.005 0)
 			(effects
@@
 			)
 			(project "5VBuck"
-				(path "/ad6c7df0-eb90-4670-9aa8-3e2007aefc2d/4ce3c563-64ba-4b6e-b334-e3956b5d5a33"
-					(reference "#FLG01")
-					(unit 1)
-				)
-				(path "/ad6c7df0-eb90-4670-9aa8-3e2007aefc2d/c59a1097-f91e-4d56-b57d-869363ca5893"
-					(reference "#FLG01")
+				(path "/ad6c7df0-eb90-4670-9aa8-3e2007aefc2d/ae63f0a9-78b8-4efb-b2ee-a2699a24d705"
+					(reference "#FLG010")
 					(unit 1)
 				)
@@
 		(on_board yes)
 		(dnp no)
-		(property "Reference" "TP8"
+		(property "Reference" "TP16"
 			(at 184.15 93.2179 0)
 			(effects
@@
 			)
 		)
-		(property "Footprint" ""
+		(property "Footprint" "TestPoint:TestPoint_THTPad_D3.0mm_Drill1.5mm"
 			(at 186.69 97.79 0)
 			(effects
@@
 		(instances
 			(project "PowerPath"
-				(path "/ad6c7df0-eb90-4670-9aa8-3e2007aefc2d/4ce3c563-64ba-4b6e-b334-e3956b5d5a33"
-					(reference "TP8")
-					(unit 1)
-				)
-				(path "/ad6c7df0-eb90-4670-9aa8-3e2007aefc2d/c59a1097-f91e-4d56-b57d-869363ca5893"
-					(reference "TP8")
+				(path "/ad6c7df0-eb90-4670-9aa8-3e2007aefc2d/ae63f0a9-78b8-4efb-b2ee-a2699a24d705"
+					(reference "TP16")
 					(unit 1)
 				)
@@
 		(dnp no)
 		(fields_autoplaced yes)
-		(property "Reference" "C4"
+		(property "Reference" "C15"
 			(at 129.54 49.5362 0)
 			(effects
@@
 			)
 			(project "5VBuck"
-				(path "/ad6c7df0-eb90-4670-9aa8-3e2007aefc2d/4ce3c563-64ba-4b6e-b334-e3956b5d5a33"
-					(reference "C4")
-					(unit 1)
-				)
-				(path "/ad6c7df0-eb90-4670-9aa8-3e2007aefc2d/c59a1097-f91e-4d56-b57d-869363ca5893"
-					(reference "C4")
+				(path "/ad6c7df0-eb90-4670-9aa8-3e2007aefc2d/ae63f0a9-78b8-4efb-b2ee-a2699a24d705"
+					(reference "C15")
 					(unit 1)
 				)
@@
 		(on_board yes)
 		(dnp no)
-		(property "Reference" "#FLG02"
+		(property "Reference" "#FLG011"
 			(at 93.98 45.085 0)
 			(effects
@@
 			)
 			(project "5VBuck"
-				(path "/ad6c7df0-eb90-4670-9aa8-3e2007aefc2d/4ce3c563-64ba-4b6e-b334-e3956b5d5a33"
-					(reference "#FLG02")
-					(unit 1)
-				)
-				(path "/ad6c7df0-eb90-4670-9aa8-3e2007aefc2d/c59a1097-f91e-4d56-b57d-869363ca5893"
-					(reference "#FLG02")
+				(path "/ad6c7df0-eb90-4670-9aa8-3e2007aefc2d/ae63f0a9-78b8-4efb-b2ee-a2699a24d705"
+					(reference "#FLG011")
 					(unit 1)
 				)
@@
 		(dnp no)
 		(fields_autoplaced yes)
-		(property "Reference" "R1"
+		(property "Reference" "R20"
 			(at 170.18 41.9099 0)
 			(effects
@@
 			)
 			(project "5VBuck"
-				(path "/ad6c7df0-eb90-4670-9aa8-3e2007aefc2d/4ce3c563-64ba-4b6e-b334-e3956b5d5a33"
-					(reference "R1")
-					(unit 1)
-				)
-				(path "/ad6c7df0-eb90-4670-9aa8-3e2007aefc2d/c59a1097-f91e-4d56-b57d-869363ca5893"
-					(reference "R1")
+				(path "/ad6c7df0-eb90-4670-9aa8-3e2007aefc2d/ae63f0a9-78b8-4efb-b2ee-a2699a24d705"
+					(reference "R20")
 					(unit 1)
 				)
@@
 		(dnp no)
 		(fields_autoplaced yes)
-		(property "Reference" "C3"
+		(property "Reference" "C14"
 			(at 118.11 49.5362 0)
 			(effects
@@
 			)
 			(project "5VBuck"
-				(path "/ad6c7df0-eb90-4670-9aa8-3e2007aefc2d/4ce3c563-64ba-4b6e-b334-e3956b5d5a33"
-					(reference "C3")
-					(unit 1)
-				)
-				(path "/ad6c7df0-eb90-4670-9aa8-3e2007aefc2d/c59a1097-f91e-4d56-b57d-869363ca5893"
-					(reference "C3")
+				(path "/ad6c7df0-eb90-4670-9aa8-3e2007aefc2d/ae63f0a9-78b8-4efb-b2ee-a2699a24d705"
+					(reference "C14")
 					(unit 1)
 				)
@@
 		(on_board yes)
 		(dnp no)
-		(property "Reference" "TP7"
+		(property "Reference" "TP14"
 			(at 171.45 93.2179 0)
 			(effects
@@
 			)
 		)
-		(property "Footprint" ""
+		(property "Footprint" "TestPoint:TestPoint_THTPad_D3.0mm_Drill1.5mm"
 			(at 173.99 97.79 0)
 			(effects
@@
 		(instances
 			(project "PowerPath"
-				(path "/ad6c7df0-eb90-4670-9aa8-3e2007aefc2d/4ce3c563-64ba-4b6e-b334-e3956b5d5a33"
-					(reference "TP7")
-					(unit 1)
-				)
-				(path "/ad6c7df0-eb90-4670-9aa8-3e2007aefc2d/c59a1097-f91e-4d56-b57d-869363ca5893"
-					(reference "TP7")
-					(unit 1)
-				)
+				(path "/ad6c7df0-eb90-4670-9aa8-3e2007aefc2d/ae63f0a9-78b8-4efb-b2ee-a2699a24d705"
+					(reference "TP14")
+					(unit 1)
+				)

Commit message: addressed final rounds of schematic comments, inital layouting
Parts:
- U4: footprint utsvt_ics:DDC0006A-MFG -> UTSVT_ICs:DDC0006A-MFG
Changed lines of the file:
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@@
 			)
 		)
-		(property "Footprint" "utsvt_ics:DDC0006A-MFG"
+		(property "Footprint" "UTSVT_ICs:DDC0006A-MFG"
 			(at 58.42 41.91 0)
 			(effects

Commit message: addressed all final comments, review?
Parts:
- removed TP13: V_in_24V, TestPoint:TestPoint_THTPad_D3.0mm_Drill1.5mm, symbol Connector:TestPoint
- renumbered R20 to R18, R21 to R19, TP14 to TP11, TP15 to TP12, TP16 to TP13, U4 to U3
Changed lines of the file:
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@@
 	(wire
 		(pts
-			(xy 168.91 87.63) (xy 168.91 85.09)
-		)
-		(stroke
-			(width 0)
-			(type default)
-		)
-	)
-	(wire
-		(pts
 			(xy 91.44 57.15) (xy 88.9 57.15)
 		)
@@
 		)
 	)
-	(hierarchical_label "V_in_24V"
-		(shape input)
-		(at 168.91 87.63 180)
-		(effects
-			(font
-				(size 1.27 1.27)
-			)
-			(justify right)
-		)
-	)
 	(symbol
 		(lib_id "Device:L_Small")
@@
 		(dnp no)
 		(fields_autoplaced yes)
-		(property "Reference" "R21"
+		(property "Reference" "R19"
 			(at 170.18 49.5299 0)
 			(effects
@@
 			(project "5VBuck"
 				(path "/ad6c7df0-eb90-4670-9aa8-3e2007aefc2d/ae63f0a9-78b8-4efb-b2ee-a2699a24d705"
-					(reference "R21")
+					(reference "R19")
 					(unit 1)
 				)
@@
 		(on_board yes)
 		(dnp no)
-		(property "Reference" "TP15"
+		(property "Reference" "TP12"
 			(at 184.15 80.5179 0)
 			(effects
@@
 			(project "PowerPath"
 				(path "/ad6c7df0-eb90-4670-9aa8-3e2007aefc2d/ae63f0a9-78b8-4efb-b2ee-a2699a24d705"
-					(reference "TP15")
+					(reference "TP12")
 					(unit 1)
 				)
@@
 		(dnp no)
 		(fields_autoplaced yes)
-		(property "Reference" "U4"
+		(property "Reference" "U3"
 			(at 73.66 31.75 0)
 			(effects
@@
 			(project "5VBuck"
 				(path "/ad6c7df0-eb90-4670-9aa8-3e2007aefc2d/ae63f0a9-78b8-4efb-b2ee-a2699a24d705"
-					(reference "U4")
-					(unit 1)
-				)
-			)
-		)
-	)
-	(symbol
-		(lib_id "Connector:TestPoint")
-		(at 168.91 85.09 0)
-		(unit 1)
-		(exclude_from_sim no)
-		(in_bom yes)
-		(on_board yes)
-		(dnp no)
-		(property "Reference" "TP13"
-			(at 171.45 80.5179 0)
-			(effects
-				(font
-					(size 1.27 1.27)
-				)
-				(justify left)
-				(hide yes)
-			)
-		)
-		(property "Value" "V_in_24V"
-			(at 163.83 79.248 0)
-			(effects
-				(font
-					(size 1.27 1.27)
-				)
-				(justify left)
-			)
-		)
-		(property "Footprint" "TestPoint:TestPoint_THTPad_D3.0mm_Drill1.5mm"
-			(at 173.99 85.09 0)
-			(effects
-				(font
-					(size 1.27 1.27)
-				)
-				(hide yes)
-			)
-		)
-		(property "Datasheet" "~"
-			(at 173.99 85.09 0)
-			(effects
-				(font
-					(size 1.27 1.27)
-				)
-				(hide yes)
-			)
-		)
-		(property "Description" "test point"
-			(at 168.91 85.09 0)
-			(effects
-				(font
-					(size 1.27 1.27)
-				)
-				(hide yes)
-			)
-		)
-		(pin "1"
-		)
-		(instances
-			(project ""
-				(path "/ad6c7df0-eb90-4670-9aa8-3e2007aefc2d/ae63f0a9-78b8-4efb-b2ee-a2699a24d705"
-					(reference "TP13")
+					(reference "U3")
 					(unit 1)
 				)
@@
 		(dnp no)
 		(fields_autoplaced yes)
-		(property "Reference" "#FLG010"
+		(property "Reference" "#FLG08"
 			(at 93.98 40.005 0)
 			(effects
@@
 			(project "5VBuck"
 				(path "/ad6c7df0-eb90-4670-9aa8-3e2007aefc2d/ae63f0a9-78b8-4efb-b2ee-a2699a24d705"
-					(reference "#FLG010")
+					(reference "#FLG08")
 					(unit 1)
 				)
@@
 		(on_board yes)
 		(dnp no)
-		(property "Reference" "TP16"
+		(property "Reference" "TP13"
 			(at 184.15 93.2179 0)
 			(effects
@@
 			(project "PowerPath"
 				(path "/ad6c7df0-eb90-4670-9aa8-3e2007aefc2d/ae63f0a9-78b8-4efb-b2ee-a2699a24d705"
-					(reference "TP16")
+					(reference "TP13")
 					(unit 1)
 				)
@@
 		(on_board yes)
 		(dnp no)
-		(property "Reference" "#FLG011"
+		(property "Reference" "#FLG09"
 			(at 93.98 45.085 0)
 			(effects
@@
 			(project "5VBuck"
 				(path "/ad6c7df0-eb90-4670-9aa8-3e2007aefc2d/ae63f0a9-78b8-4efb-b2ee-a2699a24d705"
-					(reference "#FLG011")
+					(reference "#FLG09")
 					(unit 1)
 				)
@@
 		(dnp no)
 		(fields_autoplaced yes)
-		(property "Reference" "R20"
+		(property "Reference" "R18"
 			(at 170.18 41.9099 0)
 			(effects
@@
 			(project "5VBuck"
 				(path "/ad6c7df0-eb90-4670-9aa8-3e2007aefc2d/ae63f0a9-78b8-4efb-b2ee-a2699a24d705"
-					(reference "R20")
+					(reference "R18")
 					(unit 1)
 				)
@@
 		(on_board yes)
 		(dnp no)
-		(property "Reference" "TP14"
+		(property "Reference" "TP11"
 			(at 171.45 93.2179 0)
 			(effects
@@
 			(project "PowerPath"
 				(path "/ad6c7df0-eb90-4670-9aa8-3e2007aefc2d/ae63f0a9-78b8-4efb-b2ee-a2699a24d705"
-					(reference "TP14")
+					(reference "TP11")
 					(unit 1)
 				)

Commit message: updated with PP + gen gebers
Parts:
- renumbered R18 to R17, R19 to R18, TP11 to TP16, TP12 to TP17, TP13 to TP18
Changed lines of the file:
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@@
 		(dnp no)
 		(fields_autoplaced yes)
-		(property "Reference" "R19"
+		(property "Reference" "R18"
 			(at 170.18 49.5299 0)
 			(effects
@@
 			(project "5VBuck"
 				(path "/ad6c7df0-eb90-4670-9aa8-3e2007aefc2d/ae63f0a9-78b8-4efb-b2ee-a2699a24d705"
-					(reference "R19")
+					(reference "R18")
 					(unit 1)
 				)
@@
 		(on_board yes)
 		(dnp no)
-		(property "Reference" "TP12"
+		(property "Reference" "TP17"
 			(at 184.15 80.5179 0)
 			(effects
@@
 			(project "PowerPath"
 				(path "/ad6c7df0-eb90-4670-9aa8-3e2007aefc2d/ae63f0a9-78b8-4efb-b2ee-a2699a24d705"
-					(reference "TP12")
+					(reference "TP17")
 					(unit 1)
 				)
@@
 		(on_board yes)
 		(dnp no)
-		(property "Reference" "TP13"
+		(property "Reference" "TP18"
 			(at 184.15 93.2179 0)
 			(effects
@@
 			(project "PowerPath"
 				(path "/ad6c7df0-eb90-4670-9aa8-3e2007aefc2d/ae63f0a9-78b8-4efb-b2ee-a2699a24d705"
-					(reference "TP13")
+					(reference "TP18")
 					(unit 1)
 				)
@@
 		(dnp no)
 		(fields_autoplaced yes)
-		(property "Reference" "R18"
+		(property "Reference" "R17"
 			(at 170.18 41.9099 0)
 			(effects
@@
 			(project "5VBuck"
 				(path "/ad6c7df0-eb90-4670-9aa8-3e2007aefc2d/ae63f0a9-78b8-4efb-b2ee-a2699a24d705"
-					(reference "R18")
+					(reference "R17")
 					(unit 1)
 				)
@@
 		(on_board yes)
 		(dnp no)
-		(property "Reference" "TP11"
+		(property "Reference" "TP16"
 			(at 171.45 93.2179 0)
 			(effects
@@
 			(project "PowerPath"
 				(path "/ad6c7df0-eb90-4670-9aa8-3e2007aefc2d/ae63f0a9-78b8-4efb-b2ee-a2699a24d705"
-					(reference "TP11")
-					(unit 1)
-				)
+					(reference "TP16")
+					(unit 1)
+				)

Commit message: updated with new comments + new gen gebers
Parts:
- C13: footprint Capacitor_SMD:C_0603_1608Metric -> Capacitor_SMD:C_0603_1608Metric_Pad1.08x0.95mm_HandSolder
- R17, R18: footprint Resistor_SMD:R_0603_1608Metric -> Resistor_SMD:R_0603_1608Metric_Pad0.98x0.95mm_HandSolder
Changed lines of the file:
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@@
 			)
 		)
-		(property "Footprint" "Resistor_SMD:R_0603_1608Metric"
+		(property "Footprint" "Resistor_SMD:R_0603_1608Metric_Pad0.98x0.95mm_HandSolder"
 			(at 167.64 50.8 0)
 			(effects
@@
 			)
 		)
-		(property "Footprint" "Capacitor_SMD:C_0603_1608Metric"
+		(property "Footprint" "Capacitor_SMD:C_0603_1608Metric_Pad1.08x0.95mm_HandSolder"
 			(at 97.79 44.45 0)
 			(effects
@@
 			)
 		)
-		(property "Footprint" "Resistor_SMD:R_0603_1608Metric"
+		(property "Footprint" "Resistor_SMD:R_0603_1608Metric_Pad0.98x0.95mm_HandSolder"
 			(at 167.64 43.18 0)
 			(effects
