File: Bootloader_TestBoard/CAN1.kicad_sch (KiCad schematic)
At the start: 9 parts, among them IC1 TCAN3413DR

Commit message: boar
Parts:
- renumbered C3 to C32, C4 to C33, C5 to C34, C6 to C35, D2 to D7, JP1 to JP3, R1 to R10, R2 to R11
Changed lines of the file:
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@@
 		(in_pos_files yes)
 		(dnp no)
-		(property "Reference" "C4"
+		(property "Reference" "C33"
 			(at 95.25 92.71 0)
 			(show_name no)
@@
 			(project "Bootloader_TestBoard"
 				(path "/50e7fe4f-0bd9-43c3-9b2f-ed7a525f4a83/7be88f65-0fb9-43aa-8523-28f2b8a03d0d"
-					(reference "C4")
+					(reference "C33")
 					(unit 1)
 				)
@@
 		(in_pos_files yes)
 		(dnp no)
-		(property "Reference" "C6"
+		(property "Reference" "C35"
 			(at 213.614 107.696 0)
 			(show_name no)
@@
 			(project "Bootloader_TestBoard"
 				(path "/50e7fe4f-0bd9-43c3-9b2f-ed7a525f4a83/7be88f65-0fb9-43aa-8523-28f2b8a03d0d"
-					(reference "C6")
+					(reference "C35")
 					(unit 1)
 				)
@@
 		(dnp no)
 		(fields_autoplaced yes)
-		(property "Reference" "JP1"
+		(property "Reference" "JP3"
 			(at 234.95 97.79 0)
 			(show_name no)
@@
 			(project "Bootloader_TestBoard"
 				(path "/50e7fe4f-0bd9-43c3-9b2f-ed7a525f4a83/7be88f65-0fb9-43aa-8523-28f2b8a03d0d"
-					(reference "JP1")
+					(reference "JP3")
 					(unit 1)
 				)
@@
 		(in_pos_files yes)
 		(dnp no)
-		(property "Reference" "C5"
+		(property "Reference" "C34"
 			(at 107.188 92.71 0)
 			(show_name no)
@@
 			(project "Bootloader_TestBoard"
 				(path "/50e7fe4f-0bd9-43c3-9b2f-ed7a525f4a83/7be88f65-0fb9-43aa-8523-28f2b8a03d0d"
-					(reference "C5")
+					(reference "C34")
 					(unit 1)
 				)
@@
 		(in_pos_files yes)
 		(dnp no)
-		(property "Reference" "C3"
+		(property "Reference" "C32"
 			(at 84.328 92.71 0)
 			(show_name no)
@@
 			(project "Bootloader_TestBoard"
 				(path "/50e7fe4f-0bd9-43c3-9b2f-ed7a525f4a83/7be88f65-0fb9-43aa-8523-28f2b8a03d0d"
-					(reference "C3")
+					(reference "C32")
 					(unit 1)
 				)
@@
 		(in_pos_files yes)
 		(dnp no)
-		(property "Reference" "R2"
+		(property "Reference" "R11"
 			(at 220.98 99.06 90)
 			(show_name no)
@@
 			(project "Bootloader_TestBoard"
 				(path "/50e7fe4f-0bd9-43c3-9b2f-ed7a525f4a83/7be88f65-0fb9-43aa-8523-28f2b8a03d0d"
-					(reference "R2")
+					(reference "R11")
 					(unit 1)
 				)
@@
 		(dnp no)
 		(fields_autoplaced yes)
-		(property "Reference" "D2"
+		(property "Reference" "D7"
 			(at 215.9 66.04 0)
 			(show_name no)
@@
 			(project "Bootloader_TestBoard"
 				(path "/50e7fe4f-0bd9-43c3-9b2f-ed7a525f4a83/7be88f65-0fb9-43aa-8523-28f2b8a03d0d"
-					(reference "D2")
+					(reference "D7")
 					(unit 1)
 				)
@@
 		(in_pos_files yes)
 		(dnp no)
-		(property "Reference" "R1"
+		(property "Reference" "R10"
 			(at 195.58 99.06 90)
 			(show_name no)
@@
 			(project "Bootloader_TestBoard"
 				(path "/50e7fe4f-0bd9-43c3-9b2f-ed7a525f4a83/7be88f65-0fb9-43aa-8523-28f2b8a03d0d"
-					(reference "R1")
-					(unit 1)
-				)
+					(reference "R10")
+					(unit 1)
+				)
