File: Bootloader_TestBoard/CAN2.kicad_sch (KiCad schematic)
At the start: 9 parts, among them IC2 TCAN3413DR

Commit message: boar
Parts:
- renumbered C7 to C36, C8 to C37, C9 to C38, C10 to C39, D3 to D8, JP2 to JP4, R3 to R12, R4 to R13
Changed lines of the file:
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@@
 		(in_pos_files yes)
 		(dnp no)
-		(property "Reference" "C7"
+		(property "Reference" "C36"
 			(at 70.358 88.9 0)
 			(show_name no)
@@
 			(project "Bootloader_TestBoard"
 				(path "/50e7fe4f-0bd9-43c3-9b2f-ed7a525f4a83/0229a54e-8096-4c6c-b360-e75226f9ff5b"
-					(reference "C7")
+					(reference "C36")
 					(unit 1)
 				)
@@
 		(dnp no)
 		(fields_autoplaced yes)
-		(property "Reference" "JP2"
+		(property "Reference" "JP4"
 			(at 220.98 93.98 0)
 			(show_name no)
@@
 			(project "Bootloader_TestBoard"
 				(path "/50e7fe4f-0bd9-43c3-9b2f-ed7a525f4a83/0229a54e-8096-4c6c-b360-e75226f9ff5b"
-					(reference "JP2")
+					(reference "JP4")
 					(unit 1)
 				)
@@
 		(in_pos_files yes)
 		(dnp no)
-		(property "Reference" "R3"
+		(property "Reference" "R12"
 			(at 181.61 95.25 90)
 			(show_name no)
@@
 			(project "Bootloader_TestBoard"
 				(path "/50e7fe4f-0bd9-43c3-9b2f-ed7a525f4a83/0229a54e-8096-4c6c-b360-e75226f9ff5b"
-					(reference "R3")
+					(reference "R12")
 					(unit 1)
 				)
@@
 		(in_pos_files yes)
 		(dnp no)
-		(property "Reference" "C10"
+		(property "Reference" "C39"
 			(at 199.644 103.886 0)
 			(show_name no)
@@
 			(project "Bootloader_TestBoard"
 				(path "/50e7fe4f-0bd9-43c3-9b2f-ed7a525f4a83/0229a54e-8096-4c6c-b360-e75226f9ff5b"
-					(reference "C10")
+					(reference "C39")
 					(unit 1)
 				)
@@
 		(dnp no)
 		(fields_autoplaced yes)
-		(property "Reference" "D3"
+		(property "Reference" "D8"
 			(at 201.93 62.23 0)
 			(show_name no)
@@
 			(project "Bootloader_TestBoard"
 				(path "/50e7fe4f-0bd9-43c3-9b2f-ed7a525f4a83/0229a54e-8096-4c6c-b360-e75226f9ff5b"
-					(reference "D3")
+					(reference "D8")
 					(unit 1)
 				)
@@
 		(in_pos_files yes)
 		(dnp no)
-		(property "Reference" "C8"
+		(property "Reference" "C37"
 			(at 81.28 88.9 0)
 			(show_name no)
@@
 			(project "Bootloader_TestBoard"
 				(path "/50e7fe4f-0bd9-43c3-9b2f-ed7a525f4a83/0229a54e-8096-4c6c-b360-e75226f9ff5b"
-					(reference "C8")
+					(reference "C37")
 					(unit 1)
 				)
@@
 		(in_pos_files yes)
 		(dnp no)
-		(property "Reference" "C9"
+		(property "Reference" "C38"
 			(at 93.218 88.9 0)
 			(show_name no)
@@
 			(project "Bootloader_TestBoard"
 				(path "/50e7fe4f-0bd9-43c3-9b2f-ed7a525f4a83/0229a54e-8096-4c6c-b360-e75226f9ff5b"
-					(reference "C9")
+					(reference "C38")
 					(unit 1)
 				)
@@
 		(in_pos_files yes)
 		(dnp no)
-		(property "Reference" "R4"
+		(property "Reference" "R13"
 			(at 207.01 95.25 90)
 			(show_name no)
@@
 			(project "Bootloader_TestBoard"
 				(path "/50e7fe4f-0bd9-43c3-9b2f-ed7a525f4a83/0229a54e-8096-4c6c-b360-e75226f9ff5b"
-					(reference "R4")
-					(unit 1)
-				)
+					(reference "R13")
+					(unit 1)
+				)
