File: Bootloader_TestBoard/LDO.kicad_sch (KiCad schematic)
At the start: 5 parts, among them U1 MCP1826S

Commit message: boar
Parts:
- renumbered C1 to C30, C2 to C31, D1 to D6, U1 to U3
Changed lines of the file:
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@@
 		(dnp no)
 		(fields_autoplaced yes)
-		(property "Reference" "C2"
+		(property "Reference" "C31"
 			(at 104.775 80.0035 0)
 			(show_name no)
@@
 			(project "Bootloader_TestBoard"
 				(path "/50e7fe4f-0bd9-43c3-9b2f-ed7a525f4a83/1d22cda5-1944-4aa3-84c0-0b43a853088a"
-					(reference "C2")
+					(reference "C31")
 					(unit 1)
 				)
@@
 		(dnp no)
 		(fields_autoplaced yes)
-		(property "Reference" "U1"
+		(property "Reference" "U3"
 			(at 88.9 67.945 0)
 			(show_name no)
@@
 			(project "Bootloader_TestBoard"
 				(path "/50e7fe4f-0bd9-43c3-9b2f-ed7a525f4a83/1d22cda5-1944-4aa3-84c0-0b43a853088a"
-					(reference "U1")
+					(reference "U3")
 					(unit 1)
 				)
@@
 		(dnp no)
 		(fields_autoplaced yes)
-		(property "Reference" "C1"
+		(property "Reference" "C30"
 			(at 79.375 80.0035 0)
 			(show_name no)
@@
 			(project "Bootloader_TestBoard"
 				(path "/50e7fe4f-0bd9-43c3-9b2f-ed7a525f4a83/1d22cda5-1944-4aa3-84c0-0b43a853088a"
-					(reference "C1")
+					(reference "C30")
 					(unit 1)
 				)
@@
 		(dnp no)
 		(fields_autoplaced yes)
-		(property "Reference" "D1"
+		(property "Reference" "D6"
 			(at 70.104 68.58 0)
 			(show_name no)
@@
 			(project "Bootloader_TestBoard"
 				(path "/50e7fe4f-0bd9-43c3-9b2f-ed7a525f4a83/1d22cda5-1944-4aa3-84c0-0b43a853088a"
-					(reference "D1")
-					(unit 1)
-				)
+					(reference "D6")
+					(unit 1)
+				)
