File: Bootloader_TestBoard/100Pin.kicad_sch (KiCad schematic)
At the start: 23 parts, among them J2 SWD_Header, U2 STM32G473VET6, Y2 Crystal

Commit message: schem
Parts:
- U2: footprint LHRS_Special:100PinMCU -> Project:100PinMCU
Connections:
- net PA11 renamed USB_DM
- net PA12 renamed USB_DP
Changed lines of the file:
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@@
 	(wire
 		(pts
-			(xy 124.46 77.47) (xy 133.35 77.47)
+			(xy 0.0762 0.0762) (xy 2.6162 0.0762)
 		)
 		(stroke
@@
 	(wire
 		(pts
-			(xy 124.46 80.01) (xy 133.35 80.01)
-		)
-		(stroke
-			(width 0)
-			(type default)
-		)
-	)
-	(wire
-		(pts
 			(xy 105.41 29.21) (xy 107.95 29.21)
 		)
@@
 	)
 	(label "SWCLK"
-		(at 133.35 80.01 0)
-		(effects
-			(font
-				(size 1.27 1.27)
-			)
-			(justify left bottom)
-		)
-	)
-	(label "SWCLK"
 		(at 237.49 100.33 180)
 		(effects
@@
 	)
 	(label "SWDIO"
-		(at 133.35 77.47 0)
-		(effects
-			(font
-				(size 1.27 1.27)
-			)
-			(justify left bottom)
-		)
-	)
-	(label "SWDIO"
 		(at 237.49 102.87 180)
 		(effects
@@
 		)
 	)
+	(hierarchical_label "SWDIO"
+		(shape bidirectional)
+		(at 124.46 77.47 0)
+		(effects
+			(font
+				(size 1.27 1.27)
+			)
+			(justify left)
+		)
+	)
 	(hierarchical_label "GND"
 		(shape input)
@@
 		)
 	)
+	(hierarchical_label "SWCLK"
+		(shape bidirectional)
+		(at 124.46 80.01 0)
+		(effects
+			(font
+				(size 1.27 1.27)
+			)
+			(justify left)
+		)
+	)
 	(hierarchical_label "3V3"
 		(shape input)
@@
 		)
 	)
-	(hierarchical_label "PA12"
+	(hierarchical_label "USB_DP"
 		(shape bidirectional)
 		(at 124.46 74.93 0)
@@
 		)
 	)
-	(hierarchical_label "PA11"
+	(hierarchical_label "USB_DM"
 		(shape bidirectional)
 		(at 124.46 72.39 0)
@@
 			)
 		)
-		(property "Footprint" "LHRS_Special:100PinMCU"
+		(property "Footprint" "Project:100PinMCU"
 			(at 71.12 171.45 0)
 			(hide yes)

Commit message: schem g
Parts:
- removed J2: SWD_Header, LHRS_Connectors:SWD_Conn, symbol 100PinMCU:SWD_Header_02x02
- removed R12, R13: 22, Resistor_SMD:R_0603_1608Metric_Pad0.98x0.95mm_HandSolder, symbol Device:R
- Reset1: footprint LHRS_Special:TL3365AF180QG -> Project:TL3365AF180QG
Other:
- note removed: "Serial Wire Communication"

Commit message: boar
Parts:
- renumbered C26 to C16, C27 to C17, C28 to C18, C29 to C19, C30 to C20, C31 to C21, C32 to C22, C33 to C23, C34 to C24, C35 to C25, C36 to C26, C37 to C27, C38 to C28, C39 to C29, R11 to R9
Changed lines of the file:
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@@
 		(dnp no)
 		(fields_autoplaced yes)
-		(property "Reference" "C33"
+		(property "Reference" "C23"
 			(at 205.74 29.2099 0)
 			(show_name no)
@@
 			(project "Bootloader_TestBoard"
 				(path "/50e7fe4f-0bd9-43c3-9b2f-ed7a525f4a83/e4caf007-92bb-4b24-8786-7cda9bdbd753"
-					(reference "C33")
+					(reference "C23")
 					(unit 1)
 				)
@@
 		(dnp no)
 		(fields_autoplaced yes)
-		(property "Reference" "C30"
+		(property "Reference" "C20"
 			(at 193.04 29.2099 0)
 			(show_name no)
@@
 			(project "Bootloader_TestBoard"
 				(path "/50e7fe4f-0bd9-43c3-9b2f-ed7a525f4a83/e4caf007-92bb-4b24-8786-7cda9bdbd753"
-					(reference "C30")
+					(reference "C20")
 					(unit 1)
 				)
@@
 		(dnp no)
 		(fields_autoplaced yes)
-		(property "Reference" "C36"
+		(property "Reference" "C26"
 			(at 228.6 54.6099 0)
 			(show_name no)
@@
 			(project "Bootloader_TestBoard"
 				(path "/50e7fe4f-0bd9-43c3-9b2f-ed7a525f4a83/e4caf007-92bb-4b24-8786-7cda9bdbd753"
-					(reference "C36")
+					(reference "C26")
 					(unit 1)
 				)
@@
 		(dnp no)
 		(fields_autoplaced yes)
-		(property "Reference" "C29"
+		(property "Reference" "C19"
 			(at 182.88 54.6099 0)
 			(show_name no)
@@
 			(project "Bootloader_TestBoard"
 				(path "/50e7fe4f-0bd9-43c3-9b2f-ed7a525f4a83/e4caf007-92bb-4b24-8786-7cda9bdbd753"
-					(reference "C29")
+					(reference "C19")
 					(unit 1)
 				)
@@
 		(in_pos_files yes)
 		(dnp no)
-		(property "Reference" "C32"
+		(property "Reference" "C22"
 			(at 202.946 100.4316 0)
 			(show_name no)
@@
 			(project "Bootloader_TestBoard"
 				(path "/50e7fe4f-0bd9-43c3-9b2f-ed7a525f4a83/e4caf007-92bb-4b24-8786-7cda9bdbd753"
-					(reference "C32")
+					(reference "C22")
 					(unit 1)
 				)
@@
 		(dnp no)
 		(fields_autoplaced yes)
-		(property "Reference" "C35"
+		(property "Reference" "C25"
 			(at 218.44 29.2099 0)
 			(show_name no)
@@
 			(project "Bootloader_TestBoard"
 				(path "/50e7fe4f-0bd9-43c3-9b2f-ed7a525f4a83/e4caf007-92bb-4b24-8786-7cda9bdbd753"
-					(reference "C35")
+					(reference "C25")
 					(unit 1)
 				)
@@
 		(in_pos_files yes)
 		(dnp no)
-		(property "Reference" "C26"
+		(property "Reference" "C16"
 			(at 30.988 47.752 90)
 			(show_name no)
@@
 			(project "Bootloader_TestBoard"
 				(path "/50e7fe4f-0bd9-43c3-9b2f-ed7a525f4a83/e4caf007-92bb-4b24-8786-7cda9bdbd753"
-					(reference "C26")
+					(reference "C16")
 					(unit 1)
 				)
@@
 		(dnp no)
 		(fields_autoplaced yes)
-		(property "Reference" "C39"
+		(property "Reference" "C29"
 			(at 266.065 58.4199 0)
 			(show_name no)
@@
 			(project "Bootloader_TestBoard"
 				(path "/50e7fe4f-0bd9-43c3-9b2f-ed7a525f4a83/e4caf007-92bb-4b24-8786-7cda9bdbd753"
-					(reference "C39")
+					(reference "C29")
 					(unit 1)
 				)
@@
 		(dnp no)
 		(fields_autoplaced yes)
-		(property "Reference" "C28"
+		(property "Reference" "C18"
 			(at 182.245 29.2099 0)
 			(show_name no)
@@
 			(project "Bootloader_TestBoard"
 				(path "/50e7fe4f-0bd9-43c3-9b2f-ed7a525f4a83/e4caf007-92bb-4b24-8786-7cda9bdbd753"
-					(reference "C28")
+					(reference "C18")
 					(unit 1)
 				)
@@
 		(in_pos_files yes)
 		(dnp no)
-		(property "Reference" "C38"
+		(property "Reference" "C28"
 			(at 243.967 29.083 0)
 			(show_name no)
@@
 			(project "Bootloader_TestBoard"
 				(path "/50e7fe4f-0bd9-43c3-9b2f-ed7a525f4a83/e4caf007-92bb-4b24-8786-7cda9bdbd753"
-					(reference "C38")
+					(reference "C28")
 					(unit 1)
 				)
@@
 		(dnp no)
 		(fields_autoplaced yes)
-		(property "Reference" "C31"
+		(property "Reference" "C21"
 			(at 198.12 54.6099 0)
 			(show_name no)
@@
 			(project "Bootloader_TestBoard"
 				(path "/50e7fe4f-0bd9-43c3-9b2f-ed7a525f4a83/e4caf007-92bb-4b24-8786-7cda9bdbd753"
-					(reference "C31")
+					(reference "C21")
 					(unit 1)
 				)
@@
 		(in_pos_files yes)
 		(dnp no)
-		(property "Reference" "C27"
+		(property "Reference" "C17"
 			(at 30.734 69.342 90)
 			(show_name no)
@@
 			(project "Bootloader_TestBoard"
 				(path "/50e7fe4f-0bd9-43c3-9b2f-ed7a525f4a83/e4caf007-92bb-4b24-8786-7cda9bdbd753"
-					(reference "C27")
+					(reference "C17")
 					(unit 1)
 				)
@@
 		(dnp no)
 		(fields_autoplaced yes)
-		(property "Reference" "R11"
+		(property "Reference" "R9"
 			(at 201.93 88.8999 0)
 			(show_name no)
@@
 			(project "Bootloader_TestBoard"
 				(path "/50e7fe4f-0bd9-43c3-9b2f-ed7a525f4a83/e4caf007-92bb-4b24-8786-7cda9bdbd753"
-					(reference "R11")
+					(reference "R9")
 					(unit 1)
 				)
@@
 		(dnp no)
 		(fields_autoplaced yes)
-		(property "Reference" "C34"
+		(property "Reference" "C24"
 			(at 213.36 54.6099 0)
 			(show_name no)
@@
 			(project "Bootloader_TestBoard"
 				(path "/50e7fe4f-0bd9-43c3-9b2f-ed7a525f4a83/e4caf007-92bb-4b24-8786-7cda9bdbd753"
-					(reference "C34")
+					(reference "C24")
 					(unit 1)
 				)
@@
 		(dnp no)
 		(fields_autoplaced yes)
-		(property "Reference" "C37"
+		(property "Reference" "C27"
 			(at 231.14 29.2099 0)
 			(show_name no)
@@
 			(project "Bootloader_TestBoard"
 				(path "/50e7fe4f-0bd9-43c3-9b2f-ed7a525f4a83/e4caf007-92bb-4b24-8786-7cda9bdbd753"
-					(reference "C37")
+					(reference "C27")
 					(unit 1)
 				)

Commit message: changes
Parts:
- added D5: RGB_LED, LHRS_Special:RGB_LED, symbol lhrs_special:RGB_LED
- added R5, R6, R7: 1k, Resistor_SMD:R_0603_1608Metric_Pad0.98x0.95mm_HandSolder, symbol Device:R
- Reset1: footprint Project:TL3365AF180QG -> LHRS_Special:TL3365AF180QG
- U2: footprint Project:100PinMCU -> LHRS_Special:100PinMCU
Connections:
- net GND: now also R5.2, R6.2, R7.2
- net PA0: now also D5.5
- net PA1: now also D5.3
- net PA2: now also D5.1
- new net: D5.4, R6.1
- new net: D5.6, R7.1
- new net: D5.2, R5.1
Other:
- note added: "RGB LED"
