File: Bootloader_TestBoard/48Pin.kicad_sch (KiCad schematic)
At the start: 24 parts, among them J1 SWD_Header, SW1 Reset, Y1 Crystal

Commit message: schem
Parts:
- kicad-embed://stm32g473cb.pdf1: footprint LHRS_Special:48PinMCU -> Project:48PinMCU
Changed lines of the file:
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@@
 	(wire
 		(pts
-			(xy 124.46 69.85) (xy 133.35 69.85)
-		)
-		(stroke
-			(width 0)
-			(type default)
-		)
-	)
-	(wire
-		(pts
 			(xy 183.642 107.442) (xy 183.642 109.982)
 		)
@@
 	(wire
 		(pts
-			(xy 124.46 67.31) (xy 133.35 67.31)
-		)
-		(stroke
-			(width 0)
-			(type default)
-		)
-	)
-	(wire
-		(pts
 			(xy 234.95 107.95) (xy 245.11 107.95)
 		)
@@
 	)
 	(label "SWCLK"
-		(at 133.35 69.85 0)
-		(effects
-			(font
-				(size 1.27 1.27)
-			)
-			(justify left bottom)
-		)
-	)
-	(label "SWCLK"
 		(at 224.79 105.41 180)
 		(effects
@@
 		)
 	)
-	(label "SWDIO"
-		(at 133.35 67.31 0)
-		(effects
-			(font
-				(size 1.27 1.27)
-			)
-			(justify left bottom)
-		)
-	)
 	(hierarchical_label "PB14"
 		(shape bidirectional)
@@
 		)
 	)
+	(hierarchical_label "SWCLK"
+		(shape bidirectional)
+		(at 124.46 69.85 0)
+		(effects
+			(font
+				(size 1.27 1.27)
+			)
+			(justify left)
+		)
+	)
 	(hierarchical_label "PB1"
 		(shape bidirectional)
@@
 		)
 	)
+	(hierarchical_label "SWDIO"
+		(shape bidirectional)
+		(at 124.46 67.31 0)
+		(effects
+			(font
+				(size 1.27 1.27)
+			)
+			(justify left)
+		)
+	)
 	(hierarchical_label "PB12"
 		(shape bidirectional)
@@
 			)
 		)
-		(property "Footprint" "LHRS_Special:48PinMCU"
+		(property "Footprint" "Project:48PinMCU"
 			(at 76.2 102.87 0)
 			(hide yes)

Commit message: schem g
Parts:
- removed J1: SWD_Header, LHRS_Connectors:SWD_Conn, symbol lhrs_connectors:SWD_Header
- removed R10, R9: 22, Resistor_SMD:R_0603_1608Metric_Pad0.98x0.95mm_HandSolder, symbol Device:R
- SW1: footprint LHRS_Special:TL3365AF180QG -> Project:TL3365AF180QG
Other:
- note removed: "Serial Wire Communication"

Commit message: boar
Parts:
- renumbered C11 to C1, C20 to C10, C21 to C11, C22 to C12, C23 to C13, C24 to C14, C25 to C15, C12 to C2, C13 to C3, C14 to C4, C15 to C5, C16 to C6, C17 to C7, C18 to C8, C19 to C9, R5 to R8, kicad-embed://stm32g473cb.pdf1 to U1
Changed lines of the file:
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@@
 		(dnp no)
 		(fields_autoplaced yes)
-		(property "Reference" "C12"
+		(property "Reference" "C2"
 			(at 37.338 56.388 90)
 			(show_name no)
@@
 			(project "Bootloader_TestBoard"
 				(path "/50e7fe4f-0bd9-43c3-9b2f-ed7a525f4a83/72425528-8904-4950-9d54-72562d24669d"
-					(reference "C12")
+					(reference "C2")
 					(unit 1)
 				)
@@
 		(in_pos_files yes)
 		(dnp no)
-		(property "Reference" "C14"
+		(property "Reference" "C4"
 			(at 176.53 30.48 0)
 			(show_name no)
@@
 			(project "Bootloader_TestBoard"
 				(path "/50e7fe4f-0bd9-43c3-9b2f-ed7a525f4a83/72425528-8904-4950-9d54-72562d24669d"
-					(reference "C14")
+					(reference "C4")
 					(unit 1)
 				)
@@
 		(in_pos_files yes)
 		(dnp no)
-		(property "Reference" "C11"
+		(property "Reference" "C1"
 			(at 37.084 37.084 90)
 			(show_name no)
@@
 			(project "Bootloader_TestBoard"
 				(path "/50e7fe4f-0bd9-43c3-9b2f-ed7a525f4a83/72425528-8904-4950-9d54-72562d24669d"
-					(reference "C11")
+					(reference "C1")
 					(unit 1)
 				)
@@
 		(in_pos_files yes)
 		(dnp no)
-		(property "Reference" "C20"
+		(property "Reference" "C10"
 			(at 213.36 30.226 0)
 			(show_name no)
@@
 			(project "Bootloader_TestBoard"
 				(path "/50e7fe4f-0bd9-43c3-9b2f-ed7a525f4a83/72425528-8904-4950-9d54-72562d24669d"
-					(reference "C20")
+					(reference "C10")
 					(unit 1)
 				)
@@
 		(in_pos_files yes)
 		(dnp no)
-		(property "Reference" "C15"
+		(property "Reference" "C5"
 			(at 175.006 112.268 0)
 			(show_name no)
@@
 			(project "Bootloader_TestBoard"
 				(path "/50e7fe4f-0bd9-43c3-9b2f-ed7a525f4a83/72425528-8904-4950-9d54-72562d24669d"
-					(reference "C15")
+					(reference "C5")
 					(unit 1)
 				)
@@
 		(dnp no)
 		(fields_autoplaced yes)
-		(property "Reference" "C25"
+		(property "Reference" "C15"
 			(at 260.477 54.737 0)
 			(show_name no)
@@
 			(project "Bootloader_TestBoard"
 				(path "/50e7fe4f-0bd9-43c3-9b2f-ed7a525f4a83/72425528-8904-4950-9d54-72562d24669d"
-					(reference "C25")
+					(reference "C15")
 					(unit 1)
 				)
@@
 		(in_pos_files yes)
 		(dnp no)
-		(property "Reference" "C16"
+		(property "Reference" "C6"
 			(at 187.706 30.48 0)
 			(show_name no)
@@
 			(project "Bootloader_TestBoard"
 				(path "/50e7fe4f-0bd9-43c3-9b2f-ed7a525f4a83/72425528-8904-4950-9d54-72562d24669d"
-					(reference "C16")
+					(reference "C6")
 					(unit 1)
 				)
@@
 		(dnp no)
 		(fields_autoplaced yes)
-		(property "Reference" "C22"
+		(property "Reference" "C12"
 			(at 226.568 30.4799 0)
 			(show_name no)
@@
 			(project "Bootloader_TestBoard"
 				(path "/50e7fe4f-0bd9-43c3-9b2f-ed7a525f4a83/72425528-8904-4950-9d54-72562d24669d"
-					(reference "C22")
+					(reference "C12")
 					(unit 1)
 				)
@@
 		(in_pos_files yes)
 		(dnp no)
-		(property "Reference" "C24"
+		(property "Reference" "C14"
 			(at 249.682 29.718 0)
 			(show_name no)
@@
 			(project "Bootloader_TestBoard"
 				(path "/50e7fe4f-0bd9-43c3-9b2f-ed7a525f4a83/72425528-8904-4950-9d54-72562d24669d"
-					(reference "C24")
+					(reference "C14")
 					(unit 1)
 				)
@@
 		(dnp no)
 		(fields_autoplaced yes)
-		(property "Reference" "C19"
+		(property "Reference" "C9"
 			(at 207.137 54.8639 0)
 			(show_name no)
@@
 			(project "Bootloader_TestBoard"
 				(path "/50e7fe4f-0bd9-43c3-9b2f-ed7a525f4a83/72425528-8904-4950-9d54-72562d24669d"
-					(reference "C19")
+					(reference "C9")
 					(unit 1)
 				)
@@
 		(dnp no)
 		(fields_autoplaced yes)
-		(property "Reference" "C17"
+		(property "Reference" "C7"
 			(at 192.532 54.8639 0)
 			(show_name no)
@@
 			(project "Bootloader_TestBoard"
 				(path "/50e7fe4f-0bd9-43c3-9b2f-ed7a525f4a83/72425528-8904-4950-9d54-72562d24669d"
-					(reference "C17")
+					(reference "C7")
 					(unit 1)
 				)
@@
 		(dnp no)
 		(fields_autoplaced yes)
-		(property "Reference" "R5"
+		(property "Reference" "R8"
 			(at 186.182 101.3459 0)
 			(show_name no)
@@
 			(project "Bootloader_TestBoard"
 				(path "/50e7fe4f-0bd9-43c3-9b2f-ed7a525f4a83/72425528-8904-4950-9d54-72562d24669d"
-					(reference "R5")
+					(reference "R8")
 					(unit 1)
 				)
@@
 		(in_pos_files yes)
 		(dnp no)
-		(property "Reference" "kicad-embed://stm32g473cb.pdf1"
+		(property "Reference" "U1"
 			(at 90.932 71.12 0)
 			(hide yes)
@@
 			(project "Bootloader_TestBoard"
 				(path "/50e7fe4f-0bd9-43c3-9b2f-ed7a525f4a83/72425528-8904-4950-9d54-72562d24669d"
-					(reference "kicad-embed://stm32g473cb.pdf1")
+					(reference "U1")
 					(unit 1)
 				)
@@
 		(dnp no)
 		(fields_autoplaced yes)
-		(property "Reference" "C13"
+		(property "Reference" "C3"
 			(at 177.292 54.8639 0)
 			(show_name no)
@@
 			(project "Bootloader_TestBoard"
 				(path "/50e7fe4f-0bd9-43c3-9b2f-ed7a525f4a83/72425528-8904-4950-9d54-72562d24669d"
-					(reference "C13")
+					(reference "C3")
 					(unit 1)
 				)
@@
 		(in_pos_files yes)
 		(dnp no)
-		(property "Reference" "C18"
+		(property "Reference" "C8"
 			(at 199.898 30.48 0)
 			(show_name no)
@@
 			(project "Bootloader_TestBoard"
 				(path "/50e7fe4f-0bd9-43c3-9b2f-ed7a525f4a83/72425528-8904-4950-9d54-72562d24669d"
-					(reference "C18")
+					(reference "C8")
 					(unit 1)
 				)
@@
 		(in_pos_files yes)
 		(dnp no)
-		(property "Reference" "C21"
+		(property "Reference" "C11"
 			(at 219.71 54.102 0)
 			(show_name no)
@@
 			(project "Bootloader_TestBoard"
 				(path "/50e7fe4f-0bd9-43c3-9b2f-ed7a525f4a83/72425528-8904-4950-9d54-72562d24669d"
-					(reference "C21")
+					(reference "C11")
 					(unit 1)
 				)
@@
 		(in_pos_files yes)
 		(dnp no)
-		(property "Reference" "C23"
+		(property "Reference" "C13"
 			(at 235.712 29.464 0)
 			(show_name no)
@@
 			(project "Bootloader_TestBoard"
 				(path "/50e7fe4f-0bd9-43c3-9b2f-ed7a525f4a83/72425528-8904-4950-9d54-72562d24669d"
-					(reference "C23")
+					(reference "C13")
 					(unit 1)
 				)

Commit message: changes
Parts:
- added D9: RGB_LED, LHRS_Special:RGB_LED, symbol lhrs_special:RGB_LED
- added R14, R15, R16: 1k, Resistor_SMD:R_0603_1608Metric_Pad0.98x0.95mm_HandSolder, symbol Device:R
- SW1: footprint Project:TL3365AF180QG -> LHRS_Special:TL3365AF180QG
- U1: footprint Project:48PinMCU -> LHRS_Special:48PinMCU
Connections:
- net GND: now also R14.2, R15.2, R16.2
- net PA0: now also D9.5
- net PA1: now also D9.3
- net PA2: now also D9.1
- new net: D9.2, R14.1
- new net: D9.4, R15.1
- new net: D9.6, R16.1
Other:
- note added: "RGB LED"
- moved on the sheet: C5, R8, SW1
