File: Bootloader_TestBoard/Bootloader_TestBoard.kicad_sch (KiCad schematic)
At the start: 4 parts

Commit message: schem
Parts:
- added D5, D6: LED, LED_SMD:LED_0603_1608Metric, symbol Device:LED
- added D7: D, Diode_SMD:D_SOD-123, symbol Device:D_Schottky
- added D8: TPD2EUSB30DRTR, Project:DRT0003A, symbol UTSVT_ICs:TPD2EUSB30DRTR
- added J10, J9: SWD, Connector_PinHeader_2.54mm:PinHeader_1x04_P2.54mm_Vertical, symbol Connector_Generic:Conn_01x04
- added J3: Conn_01x05, Connector_PinHeader_2.54mm:PinHeader_1x05_P2.54mm_Vertical, symbol Connector_Generic:Conn_01x05
- added J6, J7: Conn_01x03, Connector_PinHeader_2.54mm:PinHeader_1x03_P2.54mm_Vertical, symbol Connector_Generic:Conn_01x03
- added J8: USB_C_Receptacle, Project:GCT_USB4105-GF-A, symbol utsvt_connectors:USB_C_Receptacle_USB2.0_16P
- added JP3, JP5: Jumper, Connector_PinHeader_2.54mm:PinHeader_1x02_P2.54mm_Vertical, symbol Jumper:Jumper_2_Open
- added R14, R15: 1k, Resistor_SMD:R_0603_1608Metric_Pad0.98x0.95mm_HandSolder, symbol Device:R
- added R16, R17: 5.1k, Resistor_SMD:R_0603_1608Metric_Pad0.98x0.95mm_HandSolder, symbol Device:R
- added TP1, TP2, TP3: TestPoint, Connector_PinHeader_2.54mm:PinHeader_1x01_P2.54mm_Horizontal, symbol Connector:TestPoint
- D4: footprint LHRS_Special:RGB_LED -> Project:RGB_LED; P/N (none) -> 19-337/R6GHBHC-A01/2T
Connections:
- net GND: now also D5.1 (K), D6.1 (K), D8.3 (GND), J10.4 (Pin_4), J3.5 (Pin_5), J8.A1 (GND), J8.A12 (GND), J8.B1 (GND), J8.B12 (GND), J8.S1 (SHIELD), J8.S2 (Shield), J8.S3 (Shield), J8.S4 (Shield), J9.4 (Pin_4), R16.2, R17.2, TP3.1
- net PA0 renamed GPIO_B
- net PA1 renamed GPIO_R
- net PA2 renamed GPIO_G
- new net: D7.2 (A), J8.A4 (VBUS), J8.A9 (VBUS), J8.B4 (VBUS), J8.B9 (VBUS)
- new net: J8.A5 (CC1), R16.1
- new net: D5.2 (A), R14.2
- new net: D6.2 (A), R15.2
- new net: J8.B5 (CC2), R17.1
- new net +3V3: JP3.1 (A), JP5.1 (A)
- new net +3V3_100P: J10.1 (Pin_1), JP3.2 (B)
- new net +3V3_48P: J9.1 (Pin_1), JP5.2 (B)
- new net +5V: D7.1 (K), TP1.1
- new net 100Pin/PA3: R15.1
- new net 3V3: TP2.1
- new net 48Pin/PA3: R14.1
- new net CAN_H: J3.4 (Pin_4)
- new net CAN_L: J3.3 (Pin_3)
- new net SWCLK_100P: J10.2 (Pin_2)
- new net SWCLK_48P: J9.2 (Pin_2)
- new net SWDIO_100P: J10.3 (Pin_3)
- new net SWDIO_48P: J9.3 (Pin_3)
- new net USB_DM: D8.1 (D+), J3.1 (Pin_1), J6.2 (Pin_2), J8.A7 (D-), J8.B7 (D-)
- new net USB_DM_100P: J6.3 (Pin_3)
- new net USB_DM_48P: J6.1 (Pin_1)
- new net USB_DP: D8.2 (D-), J3.2 (Pin_2), J7.2 (Pin_2), J8.A6 (D+), J8.B6 (D+)
- new net USB_DP_100P: J7.3 (Pin_3)
- new net USB_DP_48P: J7.1 (Pin_1)
- no-connect marks 0 -> 2
Other:
- sheet 100Pin ports: added 3V3, GND, PA0, PA1, PA2, PA3, PB12, PB13, SWCLK, SWDIO, USB_DM, USB_DP; removed none
- sheet 48Pin ports: added +3.3V, GND, PA0, PA1, PA2, PA3, PB12, PB13, SWCLK, SWDIO, USB_DM, USB_DP; removed none
- note added: "Debug Breakout"
- note added: "Debug LED"
- note added: "Integration"
- note added: "Jumper Select"
- note added: "LDO"
- note added: "RGB"
- note added: "SWD Headers"
- note added: "Select which MCU has USB"
- note added: "Select which MCU(s) to power"
- note added: "USB TVS Array"
- note removed: "Debug Pins"
- note removed: "JUMPERS"
- note removed: "RGB LED"
- note removed: "debug led"
- note removed: "rgb led (1) power (both) usb data lines (1)"
- note removed: "usb lines can lines"
- moved on the sheet: D4, R6, R7, R8

Commit message: schem g
Parts:
- removed TP2: TestPoint, Connector_PinHeader_2.54mm:PinHeader_1x01_P2.54mm_Horizontal, symbol Connector:TestPoint
- TP1, TP3: footprint Connector_PinHeader_2.54mm:PinHeader_1x01_P2.54mm_Horizontal -> TestPoint:TestPoint_Loop_D1.80mm_Drill1.0mm_Beaded
Other:
- note added: "3V3 testpoint on LDO scheet"
- moved on the sheet: TP3
Changed lines of the file:
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@@
 		)
 	)
+	(text "3V3 testpoint on LDO scheet"
+		(exclude_from_sim no)
+		(at 205.74 154.94 0)
+		(effects
+			(font
+				(size 1.27 1.27)
+			)
+		)
+	)
 	(text "Debug LED\n"
 		(exclude_from_sim no)
@@
 	(wire
 		(pts
-			(xy 194.31 149.86) (xy 194.31 152.4)
-		)
-		(stroke
-			(width 0)
-			(type default)
-		)
-	)
-	(wire
-		(pts
-			(xy 196.85 140.97) (xy 194.31 140.97)
+			(xy 194.31 139.7) (xy 194.31 142.24)
 		)
 		(stroke
@@
 	(wire
 		(pts
-			(xy 194.31 138.43) (xy 194.31 140.97)
-		)
-		(stroke
-			(width 0)
-			(type default)
-		)
-	)
-	(wire
-		(pts
 			(xy 76.2 38.1) (xy 80.01 38.1)
 		)
@@
 	(wire
 		(pts
-			(xy 196.85 149.86) (xy 194.31 149.86)
+			(xy 196.85 139.7) (xy 194.31 139.7)
 		)
 		(stroke
@@
 	)
 	(symbol
-		(lib_id "Connector:TestPoint")
-		(at 196.85 140.97 270)
-		(unit 1)
-		(body_style 1)
-		(exclude_from_sim no)
-		(in_bom yes)
-		(on_board yes)
-		(in_pos_files yes)
-		(dnp no)
-		(fields_autoplaced yes)
-		(property "Reference" "TP2"
-			(at 201.93 139.6999 90)
-			(show_name no)
-			(do_not_autoplace no)
-			(effects
-				(font
-					(size 1.27 1.27)
-				)
-				(justify left)
-			)
-		)
-		(property "Value" "TestPoint"
-			(at 201.93 142.2399 90)
-			(show_name no)
-			(do_not_autoplace no)
-			(effects
-				(font
-					(size 1.27 1.27)
-				)
-				(justify left)
-			)
-		)
-		(property "Footprint" "Connector_PinHeader_2.54mm:PinHeader_1x01_P2.54mm_Horizontal"
-			(at 196.85 146.05 0)
-			(hide yes)
-			(show_name no)
-			(do_not_autoplace no)
-			(effects
-				(font
-					(size 1.27 1.27)
-				)
-			)
-		)
-		(property "Datasheet" ""
-			(at 196.85 146.05 0)
-			(hide yes)
-			(show_name no)
-			(do_not_autoplace no)
-			(effects
-				(font
-					(size 1.27 1.27)
-				)
-			)
-		)
-		(property "Description" "test point"
-			(at 196.85 140.97 0)
-			(hide yes)
-			(show_name no)
-			(do_not_autoplace no)
-			(effects
-				(font
-					(size 1.27 1.27)
-				)
-			)
-		)
-		(pin "1"
-		)
-		(instances
-			(project "Bootloader_TestBoard"
-				(path "/50e7fe4f-0bd9-43c3-9b2f-ed7a525f4a83"
-					(reference "TP2")
-					(unit 1)
-				)
-			)
-		)
-	)
-	(symbol
 		(lib_id "power:+3V3")
 		(at 243.84 107.95 0)
@@
 	)
 	(symbol
-		(lib_id "power:+5V")
-		(at 194.31 138.43 0)
-		(unit 1)
-		(body_style 1)
-		(exclude_from_sim no)
-		(in_bom yes)
-		(on_board yes)
-		(in_pos_files yes)
-		(dnp no)
-		(fields_autoplaced yes)
-		(property "Reference" "#PWR020"
-			(at 194.31 142.24 0)
-			(hide yes)
-			(show_name no)
-			(do_not_autoplace no)
-			(effects
-				(font
-					(size 1.27 1.27)
-				)
-			)
-		)
-		(property "Value" "3V3"
-			(at 194.31 133.35 0)
-			(show_name no)
-			(do_not_autoplace no)
-			(effects
-				(font
-					(size 1.27 1.27)
-				)
-			)
-		)
-		(property "Footprint" ""
-			(at 194.31 138.43 0)
-			(hide yes)
-			(show_name no)
-			(do_not_autoplace no)
-			(effects
-				(font
-					(size 1.27 1.27)
-				)
-			)
-		)
-		(property "Datasheet" ""
-			(at 194.31 138.43 0)
-			(hide yes)
-			(show_name no)
-			(do_not_autoplace no)
-			(effects
-				(font
-					(size 1.27 1.27)
-				)
-			)
-		)
-		(property "Description" "Power symbol creates a global label with name \"+5V\""
-			(at 194.31 138.43 0)
-			(hide yes)
-			(show_name no)
-			(do_not_autoplace no)
-			(effects
-				(font
-					(size 1.27 1.27)
-				)
-			)
-		)
-		(pin "1"
-		)
-		(instances
-			(project "Bootloader_TestBoard"
-				(path "/50e7fe4f-0bd9-43c3-9b2f-ed7a525f4a83"
-					(reference "#PWR020")
-					(unit 1)
-				)
-			)
-		)
-	)
-	(symbol
 		(lib_id "power:GND")
 		(at 57.15 72.39 0)
@@
 	(symbol
 		(lib_id "power:GND")
-		(at 194.31 152.4 0)
+		(at 194.31 142.24 0)
 		(unit 1)
 		(body_style 1)
@@
 		(fields_autoplaced yes)
 		(property "Reference" "#PWR021"
-			(at 194.31 158.75 0)
+			(at 194.31 148.59 0)
 			(hide yes)
 			(show_name no)
@@
 		)
 		(property "Value" "GND"
-			(at 194.31 157.48 0)
+			(at 194.31 147.32 0)
 			(show_name no)
 			(do_not_autoplace no)
@@
 		)
 		(property "Footprint" ""
-			(at 194.31 152.4 0)
+			(at 194.31 142.24 0)
 			(hide yes)
 			(show_name no)
@@
 		)
 		(property "Datasheet" ""
-			(at 194.31 152.4 0)
+			(at 194.31 142.24 0)
 			(hide yes)
 			(show_name no)
@@
 		)
 		(property "Description" "Power symbol creates a global label with name \"GND\" , ground"
-			(at 194.31 152.4 0)
+			(at 194.31 142.24 0)
 			(hide yes)
 			(show_name no)
@@
 	(symbol
 		(lib_id "Connector:TestPoint")
-		(at 196.85 149.86 270)
+		(at 196.85 139.7 270)
 		(unit 1)
 		(body_style 1)
@@
 		(fields_autoplaced yes)
 		(property "Reference" "TP3"
-			(at 201.93 148.5899 90)
+			(at 201.93 138.4299 90)
 			(show_name no)
 			(do_not_autoplace no)
@@
 		)
 		(property "Value" "TestPoint"
-			(at 201.93 151.1299 90)
+			(at 201.93 140.9699 90)
 			(show_name no)
 			(do_not_autoplace no)
@@
 			)
 		)
-		(property "Footprint" "Connector_PinHeader_2.54mm:PinHeader_1x01_P2.54mm_Horizontal"
-			(at 196.85 154.94 0)
+		(property "Footprint" "TestPoint:TestPoint_Loop_D1.80mm_Drill1.0mm_Beaded"
+			(at 196.85 144.78 0)
 			(hide yes)
 			(show_name no)
@@
 		)
 		(property "Datasheet" ""
-			(at 196.85 154.94 0)
+			(at 196.85 144.78 0)
 			(hide yes)
 			(show_name no)
@@
 		)
 		(property "Description" "test point"
-			(at 196.85 149.86 0)
+			(at 196.85 139.7 0)
 			(hide yes)
 			(show_name no)
@@
 			)
 		)
-		(property "Footprint" "Connector_PinHeader_2.54mm:PinHeader_1x01_P2.54mm_Horizontal"
+		(property "Footprint" "TestPoint:TestPoint_Loop_D1.80mm_Drill1.0mm_Beaded"
 			(at 196.85 135.89 0)
 			(hide yes)

Commit message: boar
Parts:
- removed D6: LED, LED_SMD:LED_0603_1608Metric, symbol Device:LED
- added D4: LED, LED_SMD:LED_0603_1608Metric, symbol Device:LED
- added LOGO1: Dr. Hallock, symbol lhrs_misc:Logo_Placeholder
- D1: renamed from D5; LCSC P/N (none) -> C125103; P/N (none) -> LTST-C193TBKT-5A
- renumbered D7 to D2, D8 to D3, D4 to D5, J8 to J1, J9 to J2, J10 to J3, J3 to J4, J6 to J5, J7 to J6, JP3 to JP1, JP5 to JP2, R14 to R1, R16 to R2, R17 to R3, R15 to R4, R6 to R5, R7 to R6, R8 to R7, TP3 to TP2
Connections:
- net GND: now also D4.1 (K)
- net at R4.2: now also D4.2 (A)
Other:
- note added: "Silk"

Commit message: changes
Parts:
- removed D5: RGB_LED, Project:RGB_LED, symbol lhrs_special:RGB_LED
- removed J4: Conn_01x05, Connector_PinHeader_2.54mm:PinHeader_1x05_P2.54mm_Vertical, symbol Connector_Generic:Conn_01x05
- removed J5, J6: Conn_01x03, Connector_PinHeader_2.54mm:PinHeader_1x03_P2.54mm_Vertical, symbol Connector_Generic:Conn_01x03
- removed JP1, JP2: Jumper, Connector_PinHeader_2.54mm:PinHeader_1x02_P2.54mm_Vertical, symbol Jumper:Jumper_2_Open
- removed LOGO1: Dr. Hallock, symbol lhrs_misc:Logo_Placeholder
- removed R5, R6, R7: 1k, Resistor_SMD:R_0603_1608Metric_Pad0.98x0.95mm_HandSolder, symbol Device:R
- removed TP1: TestPoint, TestPoint:TestPoint_Loop_D1.80mm_Drill1.0mm_Beaded, symbol Connector:TestPoint
- added D10: D, Diode_SMD:D_SOD-123, symbol Device:D_Schottky
- added D11: TPD2EUSB30DRTR, Project:USB_TVS, symbol UTSVT_ICs:TPD2EUSB30DRTR
- added J7: USB_C_Receptacle, Project:USB_Conn, symbol utsvt_connectors:USB_C_Receptacle_USB2.0_16P
- added J8: Conn_01x03, Connector_PinHeader_2.54mm:PinHeader_1x03_P2.54mm_Vertical, symbol Connector_Generic:Conn_01x03
- added R17, R18: 5.1k, Resistor_SMD:R_0603_1608Metric_Pad0.98x0.95mm_HandSolder, symbol Device:R
- D3: footprint Project:DRT0003A -> Project:USB_TVS
- J1: footprint Project:GCT_USB4105-GF-A -> Project:USB_Conn
Connections:
- net USB_DM is gone; now on net USB_DM_48P: D3.1 (D+), J1.A7 (D-), J1.B7 (D-)
- net USB_DP is gone; now on net USB_DP_48P: D3.2 (D-), J1.A6 (D+), J1.B6 (D+)
- net CAN_H: now also J8.1 (Pin_1)
- net CAN_L: now also J8.2 (Pin_2)
- net GND: now also D11.3 (GND), J7.A1 (GND), J7.A12 (GND), J7.B1 (GND), J7.B12 (GND), J7.S1 (SHIELD), J7.S2 (Shield), J7.S3 (Shield), J7.S4 (Shield), J8.3 (Pin_3), R17.2, R18.2
- net USB_DM_100P: now also D11.1 (D+), J7.A7 (D-), J7.B7 (D-)
- net USB_DP_100P: now also D11.2 (D-), J7.A6 (D+), J7.B6 (D+)
- net +5V renamed +5V_48P
- new net: J7.B5 (CC2), R18.1
- new net: D10.2 (A), J7.A4 (VBUS), J7.A9 (VBUS), J7.B4 (VBUS), J7.B9 (VBUS)
- new net: J7.A5 (CC1), R17.1
- new net +5V_100P: D10.1 (K)
- no-connect marks 2 -> 4
Other:
- sheet LDO renamed LDO_48P
- added sheet LDO_100P (LDO_100P.kicad_sch)
- sheet 100Pin ports: added none; removed PA0, PA1, PA2
- sheet 48Pin ports: added none; removed PA0, PA1, PA2
- sheet LDO_48P: file LDO.kicad_sch -> LDO_48P.kicad_sch
- note added: "3V3 testpoints on LDO sheet"
- note added: "LDO - 100P"
- note added: "LDO - 48P"
- note added: "USB - 100P"
- note added: "USB - 48P"
- note removed: "3V3 testpoint on LDO scheet"
- note removed: "Jumper Select"
- note removed: "LDO"
- note removed: "RGB"
- note removed: "Select which MCU has USB"
- note removed: "Select which MCU(s) to power"
- note removed: "Silk"
- note removed: "USB"
- moved on the sheet: D1, D2, D3, D4, J1, J2, J3, R1, R2, R3, R4, TP2
